File: tsar_SensorFrontEnd/tsar_SensorFrontEnd.brd (EAGLE design)
At the start: 278.1 x 210.5 mm, 99 parts, among them X1 057-040-1, X2 057-040-1

Commit message: some changes from Andrew during design review (now with supplies).
Parts:
- C7: value (none) -> 100n
- moved C11 24.3 mm to (61.0, 122.4)
- moved C12 5.86 mm to (48.3, 131.8), turned to 0 degrees
Connections:
- net 12V renamed +12V
- net 5V renamed +5V
Routing:
- net +5V: track 197.5 -> 190.6 mm
- net GND: track 87.1 -> 86.0 mm

Commit message: Resized Schematic Frame Added connectors for Thrust Plate Input Amp Added 3v3 Regulator (missing resistor values set to TBD)
Parts:
- removed D1, D2, D3: 1N4004, diode:DO41-10
- removed SV1: (no value), con-dil:16PL
- added 123132: DFLS160, diode:DO214AA
- added C24, C27: 0.1uF, rcl:C0805
- added C25: 10uF, rcl:C0805
- added C26: 4.7uF, rcl:C0805
- added CR2: 1N4148W-7-F, TSAR_Controller (2):SOD123
- added R35, R36, R38: TBD, rcl:R0603
- added R37: 500k, rcl:R0603
- added TP: 22-23-2041, con-molex:22-23-2041
- added U$4: MP2456GJ-P, TSAR_Controller (2):SOT6
- added U$5: 10uH, TSAR_Controller (2):0.209"LX0.197"W(5.30MMX5.00MM)
- R34: value 0 -> TBD
- renumbered X1 to SER, X2 to AN
Connections:
- removed net N$20: C13.1, C14.1, D1.C, U$3.11
- removed net N$30: U$3.15
- removed net N$31: SV1.9
- removed net N$32: SV1.11
- removed net N$33: D2.C, D3.A
- removed net N$39: U$3.17
- removed net N$47: U$3.19
- new net +3V3: C13.1, C14.1, C25.1, CR2.2, R35.2, U$3.11, U$5.2
- new net GND2: 123132.C, C24.2, U$4.P$6, U$5.1
- new net N$12: AN.15, TP.4
- new net N$14: AN.19, TP.2
- new net N$15: AN.21, TP.1
- new net N$16: AN.17, TP.3
- new net N$5: R35.1, R36.2, U$4.P$3
- new net N$8: R37.1, R38.2
- net +12V: now also C26.1, C27.1, POE_IN.1, R37.2, U$4.P$5; no longer POE_IN.2
- net +5V: no longer D2.A
- net 1: now also AN.16; no longer SV1.1
- net 2: now also AN.18; no longer SV1.3
- net 3: now also AN.20; no longer SV1.5
- net 4: now also AN.22; no longer SV1.7
- net 5: now also AN.24
- net 6: now also AN.26
- net 7: now also AN.28; no longer SV1.13
- net GND: now also 123132.A, C25.2, C26.2, C27.2, POE_IN.2, R36.1, R38.1, U$4.P$2; no longer POE_IN.1, SV1.15, SV1.16
- net N$34: now also AN.27; no longer SV1.14
- net N$35: now also AN.25; no longer SV1.12
- net N$36: now also AN.23; no longer SV1.10
- net N$4: now also C24.1, CR2.1, U$4.P$1; no longer D1.A, D3.C
Routing:
- net N$20: track 55.0 -> 0.00 mm
- net +12V: track 292.4 -> 261.9 mm
- net +3V3: track 0.00 -> 9.22 mm
- net GND: track 86.0 -> 82.7 mm, vias 56 -> 52
- net N$4: track 3.05 -> 0.00 mm
- net N$33: track 3.05 -> 0.00 mm
- net +5V: track 190.6 -> 188.5 mm

Commit message: Reduced board size
fixed missing TVS cap values
modified board layout to reduce size
Parts:
- removed SER: 057-040-1, con-panduit:057-040-1
- added X1: 057-040-1, con-panduit:057-040-1
- C1, C10, C16, C17, C18, C2, C21, C3, C4, C5, C6, C8, C9: value (none) -> 120pF
- C20: value (none) -> 120pf
- C7: value 100n -> 120pF
- moved TP 182.0 mm to (83.2, 18.2), turned to 180 degrees
- moved POE_IN 130.5 mm to (102.2, 81.8)
- moved C19 110.2 mm to (75.3, 70.7)
- moved R26 110.2 mm to (70.0, 70.7)
- moved C15 110.2 mm to (83.7, 66.4)
- moved C23 110.2 mm to (92.6, 55.0)
- moved R30 110.2 mm to (70.0, 67.2)
- moved R33 110.2 mm to (88.0, 50.4)
- moved R34 110.2 mm to (92.6, 49.6)
- moved U$1 110.2 mm to (81.7, 61.8)
- moved U$2 110.2 mm to (81.2, 75.0)
- moved C22 110.2 mm to (92.6, 60.6)
- moved CR1 110.2 mm to (78.1, 65.1)
- moved DFLS160 110.2 mm to (96.4, 65.9)
- moved R21 107.1 mm to (52.5, 74.7)
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Connections:
- removed net N$34: AN.27
- removed net N$35: AN.25
- removed net N$36: AN.23
- net 10: now also AN.23
- net 8: now also AN.27
- net 9: now also AN.25
- net N$10: now also U$1.P$4
- net N$8: now also U$4.P$4
Routing:
- net N$14: track 0.00 -> 83.1 mm
- net N$15: track 0.00 -> 82.2 mm
- net 10: track 4.62 -> 83.2 mm
- net N$16: track 0.00 -> 77.0 mm
- net N$12: track 0.00 -> 75.2 mm
- net +3V3: track 9.22 -> 69.0 mm, vias 0 -> 3
- net 9: track 4.62 -> 64.1 mm
- net 5: track 4.63 -> 62.8 mm
- net 4: track 4.78 -> 56.1 mm
- net 3: track 4.71 -> 54.0 mm
- net 2: track 4.87 -> 49.5 mm
- net 8: track 4.78 -> 44.9 mm
- net 1: track 4.63 -> 43.2 mm
- net GND2: track 0.00 -> 29.8 mm
- net 7: track 4.63 -> 30.9 mm
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- added copper zone on layer 16, net GND
Other:
- board size 278.1 x 210.5 mm -> 195.1 x 91 mm

Commit message: Shrunk Board Layout
Reduced size of board
Replaced 20x2 connectors with marionette library part.
Missing digital pin connections
Parts:
- removed AN, X1: 057-040-1, con-panduit:057-040-1
- added J1, SERIAL_TO_DAQ: IDC_RECEPTACLE_2X20-S9175-ND, marionette:IDC_RECEPTACLES
- moved TP 61.2 mm to (144.4, 17.7), turned to 270 degrees
- moved C10 54.1 mm to (130.0, 60.3)
- moved R10 54.1 mm to (132.5, 69.2)
- moved R19 54.1 mm to (122.4, 56.5)
- moved R20 54.1 mm to (130.0, 65.4)
- moved TVS10 54.1 mm to (130.0, 62.9)
- moved TVS9 54.1 mm to (122.4, 54.0)
- moved R9 54.1 mm to (124.9, 60.3)
- moved C9 53.6 mm to (122.9, 52.5)
- moved C5 41.4 mm to (101.5, 60.8)
- moved R5 41.4 mm to (100.8, 69.7)
- moved C4 41.4 mm to (93.9, 51.9)
- moved R14 41.4 mm to (93.9, 57.0)
- moved R15 41.4 mm to (100.3, 65.9)
- moved R4 41.4 mm to (94.9, 60.8)
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Connections:
- net 1: now also J1.16; no longer AN.16
- net 10: now also J1.23; no longer AN.23
- net 2: now also J1.18; no longer AN.18
- net 3: now also J1.20; no longer AN.20
- net 4: now also J1.22; no longer AN.22
- net 5: now also J1.24; no longer AN.24
- net 6: now also J1.26; no longer AN.26
- net 7: now also J1.28; no longer AN.28
- net 8: now also J1.27; no longer AN.27
- net 9: now also J1.25; no longer AN.25
- net N$12: now also J1.15; no longer AN.15
- net N$14: now also J1.19; no longer AN.19
- net N$15: now also J1.21; no longer AN.21
- net N$16: now also J1.17; no longer AN.17
Routing:
- net N$15: track 82.2 -> 46.9 mm
- net N$14: track 83.1 -> 49.7 mm
- net +5V: track 179.2 -> 153.6 mm, vias 0 -> 2
- net N$16: track 77.0 -> 52.0 mm
- net +3V3: track 69.0 -> 47.4 mm, vias 3 -> 2
- net N$12: track 75.2 -> 54.4 mm
- net N$7: track 28.0 -> 7.64 mm
- net N$46: track 35.5 -> 15.2 mm
- net N$29: track 35.0 -> 14.8 mm
- net 1: track 43.2 -> 23.3 mm
- net N$1: track 28.7 -> 8.80 mm
- net 2: track 49.5 -> 30.8 mm
- net 3: track 54.0 -> 37.7 mm
- net 19: track 33.1 -> 22.8 mm
- net CRYO4: track 20.5 -> 12.3 mm
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Other:
- board size 195.1 x 91 mm -> 150.1 x 82.7 mm

Commit message: Labeled pressure/temp sensor limits Moved ADS pins in schematic Missing digital pin connections
Parts:
- moved C12 4.23 mm to (8.79, 45.7), turned to 90 degrees
Routing:
- net GND: track 90.0 -> 87.0 mm, vias 63 -> 64
- net +5V: track 153.6 -> 152.3 mm
Changed lines of the file:
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@@
 <attribute name="VALUE" x="131.8768" y="64.77" size="1.27" layer="27" rot="R90"/>
 </element>
-<element name="C12" library="rcl" library_urn="urn:adsk.eagle:library:334" package="C0805K" package3d_urn="urn:adsk.eagle:package:23681/2" value="0.1u" x="10.9474" y="49.3776" smashed="yes">
-<attribute name="NAME" x="9.9474" y="50.2526" size="1.016" layer="25"/>
-<attribute name="POPULARITY" value="52" x="10.9474" y="49.3776" size="1.778" layer="27" display="off"/>
-<attribute name="SPICEPREFIX" value="C" x="10.9474" y="49.3776" size="1.778" layer="27" display="off"/>
-<attribute name="VALUE" x="9.9474" y="47.4776" size="1.016" layer="27"/>
+<element name="C12" library="rcl" library_urn="urn:adsk.eagle:library:334" package="C0805K" package3d_urn="urn:adsk.eagle:package:23681/2" value="0.1u" x="8.7884" y="45.7454" smashed="yes" rot="R90">
+<attribute name="NAME" x="7.9134" y="44.7454" size="1.016" layer="25" rot="R90"/>
+<attribute name="POPULARITY" value="52" x="8.7884" y="45.7454" size="1.778" layer="27" rot="R90" display="off"/>
+<attribute name="SPICEPREFIX" value="C" x="8.7884" y="45.7454" size="1.778" layer="27" rot="R90" display="off"/>
+<attribute name="VALUE" x="10.6884" y="44.7454" size="1.016" layer="27" rot="R90"/>
 </element>
 <element name="C14" library="rcl" library_urn="urn:adsk.eagle:library:334" package="C0805K" package3d_urn="urn:adsk.eagle:package:23681/2" value="1u" x="7.7216" y="38.5064" smashed="yes" rot="R90">
@@
 <via x="13.9954" y="35.9156" extent="1-16" drill="0.35"/>
 <via x="12.7254" y="35.9156" extent="1-16" drill="0.35"/>
-<via x="13.7414" y="49.6316" extent="1-16" drill="0.35"/>
-<wire x1="13.7414" y1="49.6316" x2="13.712021875" y2="49.3776" width="0.1524" layer="1"/>
-<wire x1="13.712021875" y1="49.3776" x2="11.9634" y2="49.3776" width="0.1524" layer="1"/>
-<wire x1="11.9634" y1="49.3776" x2="11.9474" y2="49.3776" width="0.1524" layer="1"/>
+<via x="8.5344" y="48.5394" extent="1-16" drill="0.35"/>
+<wire x1="8.5344" y1="48.5394" x2="8.7884" y2="48.510021875" width="0.1524" layer="1"/>
+<wire x1="8.7884" y1="48.510021875" x2="8.7884" y2="46.7614" width="0.1524" layer="1"/>
+<wire x1="8.7884" y1="46.7614" x2="8.7884" y2="46.7454" width="0.1524" layer="1"/>
 <wire x1="12.7254" y1="35.9156" x2="12.7254" y2="37.3846" width="0.1524" layer="1"/>
 <wire x1="12.7254" y1="37.3846" x2="12.8524" y2="37.5116" width="0.1524" layer="1"/>
@@
 <contactref element="POE_IN" pad="2"/>
 <via x="23.6474" y="42.2656" extent="1-16" drill="0.35"/>
-<wire x1="11.5824" y1="46.4866" x2="11.5824" y2="48.2346" width="0.1524" layer="1"/>
-<wire x1="11.5824" y1="48.2346" x2="11.9634" y2="48.6156" width="0.1524" layer="1"/>
-<wire x1="11.9634" y1="48.6156" x2="11.9634" y2="49.3776" width="0.1524" layer="1"/>
 <contactref element="C25" pad="2"/>
 <contactref element="123132" pad="A"/>
@@
 <wire x1="51.2064" y1="69.7636" x2="51.308" y2="69.662" width="0.1524" layer="1"/>
 <wire x1="51.308" y1="69.662" x2="51.308" y2="68.326" width="0.1524" layer="1"/>
+<via x="11.559540625" y="48.01361875" extent="1-16" drill="0.35"/>
 </signal>
 <signal name="1">
@@
 <wire x1="135.3718" y1="21.5544" x2="127.5334" y2="13.716" width="0.1524" layer="1"/>
 <wire x1="127.5334" y1="13.716" x2="120.65" y2="13.716" width="0.1524" layer="1"/>
-<wire x1="120.65" y1="13.716" x2="117.856" y2="10.922" width="0.1524" layer="1"/>
-<wire x1="117.856" y1="10.922" x2="117.856" y2="8.0772" width="0.1524" layer="1"/>
+<wire x1="120.65" y1="13.716" x2="117.764559375" y2="10.830559375" width="0.1524" layer="1"/>
+<wire x1="117.764559375" y1="10.830559375" x2="117.764559375" y2="7.985759375" width="0.1524" layer="1"/>
 <contactref element="J1" pad="27"/>
-<wire x1="117.856" y1="8.0772" x2="116.9088" y2="7.13" width="0.1524" layer="1"/>
+<wire x1="117.764559375" y1="7.985759375" x2="116.9088" y2="7.13" width="0.1524" layer="1"/>
 <wire x1="116.9088" y1="7.13" x2="116.49" y2="7.13" width="0.1524" layer="1"/>
 </signal>
@@
 <contactref element="C11" pad="1"/>
 <contactref element="U$3" pad="12"/>
-<contactref element="U$3" pad="10"/>
 <contactref element="U$3" pad="20"/>
 <contactref element="R21" pad="2"/>
@@
 <wire x1="21.8694" y1="35.6616" x2="21.8694" y2="37.5116" width="0.1524" layer="1"/>
 <wire x1="11.5824" y1="35.2806" x2="11.9634" y2="34.8996" width="0.1524" layer="1"/>
-<wire x1="9.9474" y1="49.3776" x2="10.1994" y2="46.5996" width="0.1524" layer="1"/>
-<wire x1="10.1994" y1="46.5996" x2="10.3124" y2="46.4866" width="0.1524" layer="1"/>
 <wire x1="11.5824" y1="37.5116" x2="11.5824" y2="43.6626" width="0.1524" layer="1"/>
-<wire x1="10.3124" y1="44.9326" x2="10.3124" y2="46.4866" width="0.1524" layer="1"/>
-<wire x1="11.5824" y1="43.6626" x2="10.3124" y2="44.9326" width="0.1524" layer="1"/>
+<wire x1="11.5824" y1="43.6626" x2="10.3505" y2="44.8945" width="0.1524" layer="1"/>
 <wire x1="23.6474" y1="38.9796" x2="23.6474" y2="37.5116" width="0.1524" layer="1"/>
 <wire x1="45.8724" y1="71.5636" x2="41.9354" y2="75.5006" width="0.1524" layer="1"/>
@@
 <wire x1="23.6474" y1="38.9796" x2="23.765" y2="38.862" width="0.1524" layer="1"/>
 <wire x1="23.765" y1="38.862" x2="25.146" y2="38.862" width="0.1524" layer="1"/>
+<contactref element="U$3" pad="10"/>
+<wire x1="10.3124" y1="46.4866" x2="10.3505" y2="46.4485" width="0.1524" layer="1"/>
+<wire x1="10.3505" y1="46.4485" x2="10.3505" y2="44.958" width="0.1524" layer="1"/>
+<wire x1="10.3505" y1="44.958" x2="10.3505" y2="44.8945" width="0.1524" layer="1"/>
+<wire x1="10.3505" y1="44.958" x2="10.1379" y2="44.7454" width="0.1524" layer="1"/>
+<wire x1="10.1379" y1="44.7454" x2="8.7884" y2="44.7454" width="0.1524" layer="1"/>
 </signal>
 <signal name="+3V3">

Commit message: changed wire size
replaced 0603 resistors with 0805
replaced thrust plate 4 pin connector with 6 pin
missing digital connections
missing mounting holes
tvs diodes need to be replaced
Parts:
- removed POE_IN: 22-23-2021, con-molex:22-23-2021
- added POE: 22-23-2021, con-molex:22-23-2021
- R1, R10, R11, R12, R13, R14, R15, R16, R17, R18, R19, R2, R20, R21, R22, R23, R24, R25, R26, R27, R28, R29, R3, R30, R31, R32, R33, R34, R35, R36, R37, R38, R4, R5, R6, R7, R8, R9: device rcl:R0603 -> marionette:.0805-B
- TP: value 22-23-2041 -> (none); device con-molex:22-23-2041 -> con-molex:KK-156-6
- moved TP 9.24 mm to (143.8, 26.9)
- moved R34 8.88 mm to (59.6, 50.0), turned to 0 degrees
- moved DFLS160 7.84 mm to (75.6, 58.8)
- moved CR1 7.84 mm to (57.3, 58.0)
- moved U$1 7.84 mm to (60.9, 54.7)
- moved C17 7.84 mm to (35.0, 52.1)
- moved CRYO2 7.84 mm to (35.0, 59.7)
- moved R28 7.84 mm to (35.0, 54.6)
- moved TVS13 7.84 mm to (35.0, 49.6)
- moved AMBIENT 7.84 mm to (9.04, 59.7)
- moved C13 7.84 mm to (28.3, 38.5)
- moved C15 7.84 mm to (62.9, 59.3)
- moved C16 7.84 mm to (43.6, 52.1)
- moved C18 7.84 mm to (26.3, 52.1)
- moved C19 7.84 mm to (54.5, 63.6)
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Connections:
- net +12V: now also POE.1; no longer POE_IN.1
- net GND: now also POE.2, TP.1, TP.6; no longer POE_IN.2
- net N$12: now also TP.5; no longer TP.4
- net N$14: now also TP.3; no longer TP.2
- net N$15: now also TP.2; no longer TP.1
- net N$16: now also TP.4; no longer TP.3
Routing:
- net +12V: track 264.0 -> 242.1 mm
- net N$15: track 46.9 -> 59.2 mm
- net N$10: track 18.2 -> 6.69 mm
- net N$14: track 49.7 -> 59.2 mm
- net N$16: track 52.0 -> 59.7 mm
- net N$12: track 54.4 -> 59.7 mm
- net N$4: track 12.5 -> 9.44 mm
- net GND2: track 29.8 -> 32.5 mm
- net 18: track 19.1 -> 17.8 mm
- net +3V3: track 47.4 -> 48.5 mm
- net +5V: track 152.3 -> 153.3 mm
- net GND: track 87.0 -> 87.8 mm, vias 64 -> 67
- net N$19: track 8.22 -> 9.08 mm
- net N$29: track 14.8 -> 15.6 mm
- net N$22: track 21.4 -> 22.2 mm
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
Commit message: ADS connected
Parts:
- added H1, H2, H3, H4: MOUNT-HOLE4.5, holes:4,5
- added POE_BYPASS: 100u, capacitor-wima:C2.5-4
- R33, R37: value 500k -> 10k
- R34, R38: value TBD -> NP
- TP: value (none) -> 22-27-2061-06; device con-molex:KK-156-6 -> con-molex:6410-06
- moved SERIAL_TO_DAQ 9.66 mm to (45.8, 8.52)
- moved TP 8.93 mm to (152.4, 29.2), turned to 90 degrees
- moved C8 7.37 mm to (143.7, 42.8)
- moved R16 7.37 mm to (129.7, 30.1)
- moved R17 7.37 mm to (136.1, 39.0)
- moved R18 7.37 mm to (142.4, 47.9)
- moved R19 7.37 mm to (129.7, 56.8)
- moved TVS6 7.37 mm to (129.7, 27.6)
- moved TVS7 7.37 mm to (136.1, 36.4)
- moved TVS8 7.37 mm to (142.4, 45.3)
- moved TVS9 7.37 mm to (129.7, 54.2)
- moved R10 7.37 mm to (139.9, 69.5)
- moved CR1 7.37 mm to (64.7, 58.3)
- moved R34 7.37 mm to (67.0, 50.2)
- moved C13 7.37 mm to (35.6, 38.8)
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Connections:
- new net N$11: SERIAL_TO_DAQ.7, U$3.19
- new net N$13: SERIAL_TO_DAQ.10, U$3.17
- new net N$17: SERIAL_TO_DAQ.9, U$3.15
- new net N$18: SERIAL_TO_DAQ.8, U$3.18
- new net N$20: SERIAL_TO_DAQ.11, U$3.16
- net +12V: now also POE_BYPASS.1
- net GND: now also POE_BYPASS.2
Routing:
- net N$17: track 0.00 -> 32.5 mm, vias 0 -> 1
- net N$20: track 0.00 -> 27.5 mm, vias 0 -> 2
- net N$11: track 0.00 -> 24.4 mm, vias 0 -> 1
- net N$13: track 0.00 -> 23.2 mm, vias 0 -> 2
- net N$18: track 0.00 -> 21.3 mm, vias 0 -> 1
- net N$12: track 59.7 -> 65.1 mm
- net GND: track 87.8 -> 83.0 mm, vias 67 -> 65
- net +12V: track 242.1 -> 246.8 mm
- net N$16: track 59.7 -> 63.2 mm
- net N$14: track 59.2 -> 61.1 mm
- net N$15: track 59.2 -> 60.4 mm
Other:
- board size 150.1 x 82.7 mm -> 165.4 x 87.6 mm

Commit message: I broke everything
Parts:
- removed TP: 22-27-2061-06, con-molex:6410-06
- removed TVS12, TVS13, TVS14, TVS16, TVS17: DF2B5M4CT,L3F, TSAR_Controller:SOD-882(SOT2)
- added C28, C29, C30: 120pF, rcl:C0805
- added OPEN1, OPEN2, OPEN3: 22-23-2021, con-molex:22-23-2021
- added R39, R40, R41, R42, R43, R44: 1k, marionette:.0805-B
- added R45, R46, R47, R48, R49, R50: NP, Resistor_Capacitor:RES_0805
- added R51, R52, R53: 150, marionette:.0805-B
- added THRUST: Thrust Plate Connector, con-molex:6410-05
- R25: value 150 -> 22k
- R35: value TBD -> 73.2k
- R36: value TBD -> 23.7k
- moved R38 28.4 mm to (73.2, 32.8), turned to 90 degrees
- moved R37 26.7 mm to (73.9, 35.8)
- moved R35 26.3 mm to (65.6, 40.0)
- moved R36 26.3 mm to (65.6, 35.6)
- moved CR2 26.0 mm to (71.9, 47.6)
- moved C25 24.7 mm to (67.5, 46.2), turned to 90 degrees
- moved C24 24.6 mm to (77.4, 45.1), turned to 270 degrees
- moved C26 23.0 mm to (77.5, 35.5)
- moved C11 22.9 mm to (56.9, 29.3)
- moved C14 22.9 mm to (41.0, 27.8)
- moved U$3 22.9 mm to (49.3, 31.3)
- moved C12 22.9 mm to (42.1, 35.1)
- moved C13 22.9 mm to (58.2, 35.0)
- moved U$4 21.0 mm to (70.2, 37.4)
- moved U$5 20.7 mm to (72.2, 42.7)
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- renumbered J1 to ANALOG_TO_DAQ
Connections:
- removed net 14: C16.1, R27.1, TVS12.P$1, U$3.1
- removed net 15: C17.1, R28.1, TVS13.P$1, U$3.2
- removed net 16: C18.1, R29.1, TVS14.P$1, U$3.3
- removed net 18: C20.1, R31.1, TVS16.P$1, U$3.4
- new net 11: C28.1, R39.1, U$3.6
- new net 12: C29.1, R40.1, U$3.7
- new net 13: C30.1, R41.1, U$3.8
- new net N$21: C16.1, R27.1, U$3.1
- new net N$23: C17.1, R28.1, U$3.2
- new net N$24: C18.1, R29.1, U$3.3
- new net N$25: C20.1, R31.1, U$3.4
- new net N$26: OPEN1.2, R42.2, R46.2
- new net N$27: OPEN2.2, R43.2, R47.2
- new net N$28: OPEN3.2, R44.2, R50.2
- new net N$30: R40.2, R47.1, R48.1
- new net N$31: R41.2, R49.1, R50.1
- new net N$32: R39.2, R45.1, R46.1
- new net N$33: OPEN3.1, R49.2, R53.1
- new net N$34: OPEN2.1, R48.2, R52.1
- new net N$35: OPEN1.1, R45.2, R51.1
- net +5V: now also R51.2, R52.2, R53.2
- net 19: no longer TVS17.P$1
- net GND: now also C28.2, C29.2, C30.2, R42.1, R43.1, R44.1, THRUST.5; no longer TP.1, TP.6, TVS12.P$2, TVS13.P$2, TVS14.P$2, TVS16.P$2, TVS17.P$2
- net N$12: now also THRUST.4; no longer TP.5
- net N$14: now also THRUST.2; no longer TP.3
- net N$15: now also THRUST.1; no longer TP.2
- net N$16: now also THRUST.3; no longer TP.4
Routing:
- net +5V: track 153.3 -> 77.9 mm, vias 2 -> 1
- net +12V: track 246.8 -> 179.2 mm
- net 14: track 39.2 -> 0.00 mm
- net GND: track 83.0 -> 45.5 mm, vias 65 -> 35
- net N$17: track 32.5 -> 0.00 mm, vias 1 -> 0
- net GND2: track 32.5 -> 0.00 mm
- net 15: track 30.7 -> 0.00 mm
- net N$20: track 27.5 -> 0.14 mm, vias 2 -> 0
- net GND1: track 26.1 -> 0.00 mm
- net N$11: track 24.4 -> 0.00 mm, vias 1 -> 0
- net N$13: track 23.2 -> 0.00 mm, vias 2 -> 0
- net 16: track 22.3 -> 0.00 mm
- net N$18: track 21.3 -> 0.00 mm, vias 1 -> 0
- net 8: track 52.1 -> 31.1 mm
- net 19: track 22.9 -> 3.67 mm
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- added copper zone on layer 1, net +12V
- added copper zone on layer 1, net +3V3
- added copper zone on layer 1, net +5V
- added copper zone on layer 1, net GND1
- added copper zone on layer 1, net GND2
- added copper zone on layer 1, net N$10
- added copper zone on layer 1, net N$3
- added copper zone on layer 1, net N$4
- added copper zone on layer 1, net N$5
- added copper zone on layer 1, net N$8
- added copper zone on layer 1, net N$9
