File: tsar_SensorFrontEnd/tsar_SensorFrontEnd.brd (EAGLE design)
At the start: 128.5 x 85.1 mm, 239 parts

Commit message: sfe edits, added part library
Parts:
- removed U$3: ADS8344, TSAR_Controller:SSOP-20
- added U1, U2: ADS8344N, ADS8344N:DB20
Connections:
- new net GND_2: U2.13
- new net VCC+: U2.20
- new net VCC+_2: U2.12
- net +3V3: now also U1.11; no longer U$3.11
- net +5V: now also U1.10, U1.12, U1.20; no longer U$3.10, U$3.12, U$3.20
- net 11: now also U1.6; no longer U$3.6
- net 12: now also U1.7; no longer U$3.7
- net 13: now also U1.8; no longer U$3.8
- net 19: now also U1.5; no longer U$3.5
- net DIO32/SPI0-SCK: now also U1.19; no longer U$3.19
- net DIO33/SPI0-NSS: now also U1.18; no longer U$3.18
- net DIO34/SPI0-MISO: now also U1.15; no longer U$3.15
- net DIO35/SPI0-MOSI: now also U1.17; no longer U$3.17
- net DIO36: now also U1.16; no longer U$3.16
- net GND: now also U1.13, U1.14, U1.9, U2.14; no longer U$3.13, U$3.14, U$3.9
- net N$21: now also U1.1; no longer U$3.1
- net N$23: now also U1.2; no longer U$3.2
- net N$24: now also U1.3; no longer U$3.3
- net N$25: now also U1.4; no longer U$3.4
Routing:
- net +5V: track 296.9 -> 290.2 mm
- net N$21: track 13.9 -> 9.51 mm
- net N$23: track 21.8 -> 18.7 mm
- net N$24: track 28.9 -> 26.0 mm
- net N$25: track 38.0 -> 35.4 mm
- net DIO35/SPI0-MOSI: track 10.9 -> 8.57 mm
- net 19: track 15.0 -> 12.8 mm
- net 12: track 16.9 -> 15.0 mm
- net 11: track 34.2 -> 32.3 mm
- net DIO36: track 16.0 -> 14.2 mm
- net 13: track 42.2 -> 40.5 mm
- net DIO34/SPI0-MISO: track 21.5 -> 20.0 mm

Commit message: replaced ssop20 with correct package
Parts:
- removed U$8: ADS8344, TSAR_Controller:SSOP-20
- moved U2 29.2 mm to (83.8, 24.4), turned to 180 degrees
- moved U1 26.8 mm to (22.9, 22.1), turned to 270 degrees
Connections:
- removed net GND_2: U2.13
- removed net VCC+: U2.20
- removed net VCC+_2: U2.12
- net +3V3: now also U2.11; no longer U$8.11
- net +5V: now also U2.10, U2.12, U2.20; no longer U$8.10, U$8.12, U$8.20
- net 14: now also U2.4; no longer U$8.4
- net 15: now also U2.6; no longer U$8.6
- net 16: now also U2.7; no longer U$8.7
- net 17: now also U2.8; no longer U$8.8
- net 18: now also U2.3; no longer U$8.3
- net 20: now also U2.2; no longer U$8.2
- net 21: now also U2.1; no longer U$8.1
- net 22: now also U2.5; no longer U$8.5
- net DIO37: now also U2.16; no longer U$8.16
- net DIO39/SPI1-NSS: now also U2.18; no longer U$8.18
- net DIO40/SPI1-MISO: now also U2.15; no longer U$8.15
- net DIO40/SPI1-SCK: now also U2.19; no longer U$8.19
- net DIO41/SPI1-MOSI: now also U2.17; no longer U$8.17
- net GND: now also U2.13, U2.9; no longer U$8.13, U$8.14, U$8.9
Routing:
- net +5V: track 290.2 -> 297.0 mm
- net N$21: track 9.51 -> 15.6 mm
- net N$23: track 18.7 -> 23.2 mm
- net +3V3: track 118.2 -> 122.5 mm
- net N$24: track 26.0 -> 29.9 mm
- net 13: track 40.5 -> 44.3 mm
- net 12: track 15.0 -> 18.8 mm
- net N$25: track 35.4 -> 39.0 mm
- net 11: track 32.3 -> 35.9 mm
- net 19: track 12.8 -> 16.4 mm
- net DIO40/SPI1-SCK: track 65.3 -> 68.5 mm
- net DIO39/SPI1-NSS: track 66.3 -> 69.2 mm
- net DIO41/SPI1-MOSI: track 58.5 -> 61.2 mm
- net DIO32/SPI0-SCK: track 19.6 -> 22.1 mm
- net DIO37: track 63.4 -> 65.9 mm
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
Commit message: poe/ac/sfe changes, libraries
POE low risk input board created; will manage POE+ power distribution to subsystems. added 24-> 5v regulator for SFE and BB-AI
added libraries for SFE and POE.
SFE: removed 24->5V regulator from SFE, replaced D27&D31 with correct package, replaced ADC to correct SSOP20 package.
AC: replaced all passives with oresat rcl parts
Parts:
- removed C15: 100nF, rcl:C0603
- removed C19: 10uF, rcl:R1206
- removed C22: 4.7uF, rcl:C0805
- removed C23: 0.1uF, rcl:C0603
- removed C48: 47pF, rcl:C0603
- removed D28: DFLS160, diode:DO214AA
- removed D29: 1N4148W-7-F, TSAR_Controller:SOD123
- removed JP1, JP2, JP4, JP5: (no value), adafruit:1X03
- removed L2: 10uH, TSAR_Controller (2):0.209"LX0.197"W(5.30MMX5.00MM)
- removed OPEN1, OPEN2: 22-23-2021, con-molex:22-23-2021
- removed R33: 500k, rcl:R1206
- removed R34, R42, R43, R51, R52: NP, rcl:R0603
- removed R78, R79: 0, rcl:R0603
- removed U$1: MP2456GJ-P, TSAR_Controller (2):SOT6
- added AMBIENT2, CRYO5: 22-23-2021, con-molex:22-23-2021
- added POE_IB_5V: (no value), pinhead:1X02
- D27, D31: device diode:DO214AA -> DFLS160-7:POWERDI-123
- R26: value 124k -> 150
- R30: value 23.7k -> 22k
- moved D27 93.8 mm to (141.0, 48.0)
- moved 3V3. 91.0 mm to (151.4, 36.3)
- moved 5V. 91.0 mm to (147.7, 36.3)
- moved C10 91.0 mm to (210.7, 81.7)
- moved C12 91.0 mm to (106.1, 34.1)
- moved C32 91.0 mm to (170.2, 39.1)
- moved C33 91.0 mm to (167.1, 38.6)
- moved C39 91.0 mm to (159.3, 47.5)
- moved C40 91.0 mm to (159.3, 59.4)
- moved C41 91.0 mm to (159.3, 70.9)
- moved C42 91.0 mm to (160.0, 81.3)
- moved C43 91.0 mm to (129.0, 81.5)
- moved C47 91.0 mm to (129.0, 75.4)
- moved C49 91.0 mm to (130.6, 47.5)
- moved C6 91.0 mm to (210.7, 47.4)
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Connections:
- removed net FLY2: C15.2, D28.C, L2.1, U$1.P$6
- removed net N$10: R33.1, R34.2, U$1.P$4
- removed net N$17: C15.1, R78.1
- removed net N$26: JP4.3, OPEN1.2, R42.2
- removed net N$27: JP5.3, OPEN2.2, R43.2
- removed net N$3: D29.1, R78.2, U$1.P$1
- removed net N$35: JP4.1, OPEN1.1, R51.1
- removed net N$37: JP1.2, R51.2
- removed net N$39: JP2.2, R52.2
- removed net N$41: JP5.2, R40.2
- removed net N$9: C48.2, R26.1, R30.2, U$1.P$3
- new net CAN0_H: SERIAL_TO_DAQ.38
- new net CAN0_L: SERIAL_TO_DAQ.37
- new net DAC0: ANALOG_TO_DAQ.7
- new net DAC1: ANALOG_TO_DAQ.8
- new net DAC2: ANALOG_TO_DAQ.9
- new net DAC3: ANALOG_TO_DAQ.10
- new net DIO42: SERIAL_TO_DAQ.17
- new net DIO43: SERIAL_TO_DAQ.18
- new net DIO44/I2C0-SDA: SERIAL_TO_DAQ.19
- new net DIO45/I2C0-SCL: SERIAL_TO_DAQ.20
- new net DIO46: SERIAL_TO_DAQ.21
- new net DIO47: SERIAL_TO_DAQ.22
- new net DIO48/UART0-TX: SERIAL_TO_DAQ.23
- new net DIO49/UART0-RX: SERIAL_TO_DAQ.24
- new net DIO50: SERIAL_TO_DAQ.25
- new net DIO51: SERIAL_TO_DAQ.26
- new net DIO52/UART1-TX: SERIAL_TO_DAQ.27
- new net DIO53/UART1-RX: SERIAL_TO_DAQ.28
- new net DIO54/UART1-CTS: SERIAL_TO_DAQ.29
- new net DIO55/UART1-RTS: SERIAL_TO_DAQ.30
- new net DIO56/UART2-TX: SERIAL_TO_DAQ.31
- new net DIO57/UART2-RX: SERIAL_TO_DAQ.32
- new net DIO58/UART2-CTS: SERIAL_TO_DAQ.33
- new net DIO59/UART2-RTS: SERIAL_TO_DAQ.34
- new net DIO60: SERIAL_TO_DAQ.35
- new net DIO61: SERIAL_TO_DAQ.36
- new net DIO62: ANALOG_TO_DAQ.31
- new net DIO63: ANALOG_TO_DAQ.32
- new net DIO64: ANALOG_TO_DAQ.33
- new net DIO65: ANALOG_TO_DAQ.34
- new net DIO66: ANALOG_TO_DAQ.35
- new net DIO67: ANALOG_TO_DAQ.36
- new net DIO68: ANALOG_TO_DAQ.37
- new net DIO69: ANALOG_TO_DAQ.38
- new net MBUS-SCL: ANALOG_TO_DAQ.4
- new net MBUS-SCL-1: SERIAL_TO_DAQ.4
- new net MBUS-SDA: ANALOG_TO_DAQ.3
- new net MBUS-SDA-1: SERIAL_TO_DAQ.3
- new net V5D: SERIAL_TO_DAQ.5, SERIAL_TO_DAQ.6
- net +12V: no longer JP1.1, JP2.1
- net +24V: no longer C22.1, C23.1, R33.2, U$1.P$5
- net +5V: now also ANALOG_TO_DAQ.5, ANALOG_TO_DAQ.6, POE_IB_5V.1, R30.2; no longer C19.1, D29.2, JP1.3, JP2.3, L2.2, R79.2
- net GND: now also AMBIENT2.2, CRYO5.2, POE_IB_5V.2; no longer C19.2, C22.2, C23.2, D28.A, R30.1, R34.1, R42.1, R43.1, U$1.P$2
- net N$16: now also ANALOG_TO_DAQ.11; no longer C48.1, R79.1
- net N$32: now also CRYO5.1, R26.1; no longer JP4.2
- net N$34: now also AMBIENT2.1, R30.1, R40.2; no longer JP5.1, OPEN2.1, R52.1
Routing:
- net +5V: track 297.0 -> 383.0 mm, vias 2 -> 3
- net N$34: track 36.9 -> 10.2 mm
- net N$9: track 19.8 -> 0.00 mm
- net N$35: track 17.5 -> 0.00 mm
- net +24V: track 89.9 -> 76.3 mm, vias 2 -> 1
- net +12V: track 308.6 -> 321.5 mm
- net N$37: track 12.0 -> 0.00 mm
- net N$39: track 11.8 -> 0.00 mm
- net N$26: track 10.6 -> 0.00 mm
- net N$27: track 10.5 -> 0.00 mm
- net N$3: track 8.97 -> 0.00 mm
- net N$32: track 5.41 -> 11.6 mm
- net N$16: track 3.56 -> 0.00 mm
- net N$41: track 3.32 -> 0.00 mm
- net N$17: track 3.17 -> 0.00 mm
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- removed copper zone on layer 1, net +5V
- removed copper zone on layer 1, net FLY2
- removed copper zone on layer 1, net N$10

Commit message: SFE/AC changes
AC: began replacing nucleo with bare metal stm
SFE: replaced all passives with oresal parts
Parts:
- C1, C10, C11, C12, C13, C14, C16, C17, C18, C2, C20, C21, C24, C27, C28, C29, C3, C30, C31, C32, C33, C34, C35, C36, C37, C38, C39, C4, C40, C41, C42, C43, C46, C47, C49, C5, C50, C51, C6, C7, C8, C9: device rcl:C0603 -> oresat-rcl:C0603K
- C25, C52, C53: device rcl:R1206 -> oresat-rcl:C1206K
- C26, C45: device rcl:C0805 -> oresat-rcl:C0805K
- R1, R10, R11, R12, R13, R14, R15, R16, R17, R18, R19, R2, R20, R27, R28, R29, R3, R31, R32, R39, R4, R40, R41, R44, R45, R46, R47, R48, R49, R5, R50, R54, R55, R56, R57, R58, R59, R6, R60, R61, R62, R63, R64, R65, R66, R67, R68, R7, R70, R71, R72, R73, R74, R8, R80, R81, R82, R83, R84, R85, R9: device rcl:R0603 -> oresat-rcl:.0603-A-NOSILK
- R21, R22, R23, R24, R25, R26, R30, R35, R36, R69, R75: device marionette:.0805-B -> oresat-rcl:.0805-A-NOSILK
- R53, R77: device rcl:R0603 -> oresat-rcl:.0805-A-NOSILK
- R76: device rcl:R1206 -> oresat-rcl:1206-A

Commit message: board corrections following test case.
issue #6 closed.
Parts:
- removed JP6: (no value), adafruit:1X03
- removed R44: NP, oresat-rcl:.0603-A-NOSILK
- R1, R10, R2, R3, R4, R5, R6, R7, R8, R9: device oresat-rcl:.0603-A-NOSILK -> oresat-rcl:.0805-A-NOSILK
Connections:
- removed net N$28: JP6.3, OPEN3.2, R44.2
- removed net N$42: JP6.2, R41.2
- net GND: now also OPEN3.2; no longer R44.1
- net N$33: now also R41.2; no longer JP6.1
Routing:
- net N$28: track 9.11 -> 0.00 mm
- net GND: track 0.00 -> 5.84 mm
- net N$42: track 4.98 -> 0.00 mm
- net N$33: track 15.0 -> 13.2 mm

Commit message: POE, SFE changes
POE: added gnd vias and text info
SFE: moved to mar dxf outline. removed unallocated lines and added valve position sensor pinout. updated attributes. the board is currently unrouted.
Parts:
- removed AMBIENT, AMBIENT2, CRYO1, CRYO2, CRYO3, CRYO4, CRYO5, OPEN10, OPEN3, OPEN7, OPEN8, OPEN9, OPENHS1, OPENHS2, PIT2, PIT5, PIT6, PT1, PT2, PT3, PT4, PT5: 22-23-2021, con-molex:22-23-2021
- removed JP3, UA_10_S, UA_10_V, UA_11_S, UA_11_V, UA_4_S, UA_4_V, UA_5_S, UA_5_V, UA_6_S, UA_6_V, UA_7_S, UA_7_V, UA_8_S, UA_8_V, UA_9_S, UA_9_V: (no value), adafruit:1X03
- removed OPEN11, OPEN4, OPEN5, OPEN6: (no value), con-molex:22-23-2021
- removed R48, R50, R55, R57, R59, R63, R64, R65, R66, R67, R68, R70, R71, R72, R73, R74: NP, oresat-rcl:.0603-A-NOSILK
- removed R53: NP, oresat-rcl:.0805-A-NOSILK
- added PT-F01, PT-F02, PT-F03, PT-F04, PT-L01, PT-L02, PT-L03, PT-L04, PT-M01, PT-M02, TT-F01, TT-F02, TT-L01, TT-L02, TT-L03, TT-L04, TT-L05: 22-23-2021, con-molex:22-23-2021
- added TO_VI: (no value), pinhead:1X12
- moved THRUSTPOWER 198.4 mm to (18.3, 80.2), turned to 270 degrees
- moved D21 177.3 mm to (17.0, 31.2), turned to 90 degrees
- moved C35 177.3 mm to (14.3, 31.5), turned to 270 degrees
- moved R47 177.0 mm to (12.1, 31.4), turned to 270 degrees
- moved C36 173.8 mm to (14.3, 35.0), turned to 270 degrees
- moved D22 173.7 mm to (17.0, 34.7), turned to 90 degrees
- moved R49 173.7 mm to (12.1, 35.0), turned to 270 degrees
- moved C37 170.8 mm to (14.3, 38.6), turned to 270 degrees
- moved D23 170.7 mm to (17.0, 38.3), turned to 90 degrees
- moved R54 170.5 mm to (12.1, 38.6), turned to 270 degrees
- moved C38 169.7 mm to (14.3, 42.2), turned to 270 degrees
- moved D24 169.6 mm to (17.0, 41.8), turned to 90 degrees
- moved R56 169.4 mm to (12.1, 42.2), turned to 270 degrees
- moved R62 159.2 mm to (12.1, 17.1)
- moved C42 159.2 mm to (14.3, 17.2), turned to 270 degrees
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Connections:
- removed net N$33: OPEN3.1, R41.2, R53.1
- removed net N$36: JP3.2, R53.2
- removed net N$55: R68.2, UA_6_V.2
- removed net N$57: R67.2, UA_5_V.2
- removed net N$58: R66.2, UA_4_V.2
- removed net N$59: OPEN4.2, R63.2, UA_4_S.3
- removed net N$60: OPEN5.2, R64.2, UA_5_S.3
- removed net N$61: OPEN6.2, R65.2, UA_6_S.3
- removed net N$62: OPEN6.1, R68.1, UA_6_S.1
- removed net N$63: OPEN5.1, R67.1, UA_5_S.1
- removed net N$64: OPEN4.1, R66.1, UA_4_S.1
- removed net N$65: OPEN7.2, R48.2, UA_7_S.3
- removed net N$66: OPEN7.1, R73.1, UA_7_S.1
- removed net N$67: R47.2, UA_7_S.2
- removed net N$68: R60.2, UA_4_S.2
- removed net N$69: R61.2, UA_5_S.2
- removed net N$70: R62.2, UA_6_S.2
- removed net N$71: OPEN8.2, R50.2, UA_8_S.3
- removed net N$72: OPEN8.1, R72.1, UA_8_S.1
- removed net N$73: R49.2, UA_8_S.2
- removed net N$74: OPEN9.2, R55.2, UA_9_S.3
- removed net N$75: OPEN9.1, R71.1, UA_9_S.1
- removed net N$76: R54.2, UA_9_S.2
- removed net N$77: OPEN10.2, R57.2, UA_10_S.3
- removed net N$78: OPEN10.1, R70.1, UA_10_S.1
- removed net N$79: R56.2, UA_10_S.2
- removed net N$80: OPEN11.2, R59.2, UA_11_S.3
- removed net N$81: OPEN11.1, R74.1, UA_11_S.1
- removed net N$82: R58.2, UA_11_S.2
- removed net N$87: R71.2, UA_9_V.2
- removed net N$88: R70.2, UA_10_V.2
- removed net N$93: R74.2, UA_11_V.2
- removed net N$94: R73.2, UA_7_V.2
- removed net N$95: R72.2, UA_8_V.2
- new net HES1: R56.2, TO_VI.1
- new net HES2: R54.2, TO_VI.2
- new net HES3: R49.2, TO_VI.3
- new net HES4: R47.2, TO_VI.4
- new net HES5: R58.2, TO_VI.5
- new net HES6: R60.2, TO_VI.6
- new net HES7: R61.2, TO_VI.7
- new net HES8: R62.2, TO_VI.8
- new net HES9: R41.2, TO_VI.9
- net +12V: now also PT-F01.1, PT-F02.1, PT-F03.1, PT-F04.1, PT-L01.1, PT-L02.1, PT-L03.1, PT-L04.1, PT-M01.1, PT-M02.1; no longer JP3.1, OPENHS1.1, OPENHS2.1, PIT2.1, PIT5.1, PIT6.1, PT1.1, PT2.1, PT3.1, PT4.1, PT5.1, UA_10_V.3, UA_11_V.3, UA_4_V.3, UA_5_V.3, UA_6_V.3, UA_7_V.3, UA_8_V.3, UA_9_V.3
- net +5V: no longer JP3.3, UA_10_V.1, UA_11_V.1, UA_4_V.1, UA_5_V.1, UA_6_V.1, UA_7_V.1, UA_8_V.1, UA_9_V.1
- net AMBIENT: now also R26.1, TT-L01.1; no longer AMBIENT.1, R25.1
- net CRYO1: now also TT-L05.1; no longer CRYO1.1
- net CRYO2: now also TT-L04.1; no longer CRYO2.1
- net CRYO3: now also TT-L03.1; no longer CRYO3.1
- net CRYO4: now also TT-L02.1; no longer CRYO4.1
- net GND: now also TT-F01.2, TT-F02.2, TT-L01.2, TT-L02.2, TT-L03.2, TT-L04.2, TT-L05.2; no longer AMBIENT.2, AMBIENT2.2, CRYO1.2, CRYO2.2, CRYO3.2, CRYO4.2, CRYO5.2, OPEN3.2, R48.1, R50.1, R55.1, R57.1, R59.1, R63.1, R64.1, R65.1
- net N$1: now also PT-L02.2; no longer PT2.2
- net N$19: now also PT-F01.2; no longer OPENHS2.2
- net N$2: now also PT-F02.2; no longer OPENHS1.2
- net N$22: now also PT-L01.2; no longer PT1.2
- net N$29: now also PT-L03.2; no longer PT3.2
- net N$32: now also R25.1, TT-F02.1; no longer CRYO5.1, R26.1
- net N$34: now also TT-F01.1; no longer AMBIENT2.1
- net N$38: now also PT-L04.2; no longer PT4.2
- net N$40: now also PT-M01.2; no longer PT5.2
- net N$46: now also PT-F04.2; no longer PIT6.2
- net N$6: now also PT-M02.2; no longer PIT2.2
- net N$7: now also PT-F03.2; no longer PIT5.2
Routing:
- net +5V: track 382.6 -> 0.00 mm, vias 3 -> 0
- net +12V: track 321.5 -> 0.00 mm, vias 1 -> 0
- net +3V3: track 122.4 -> 0.00 mm, vias 2 -> 0
- net ADC0.4: track 110.0 -> 0.00 mm
- net ADC0.5: track 93.1 -> 0.00 mm
- net ADC1.4: track 77.8 -> 0.00 mm, vias 1 -> 0
- net +24V: track 76.1 -> 0.00 mm, vias 1 -> 0
- net ADC0.6: track 69.8 -> 0.00 mm
- net DIO39/SPI1-NSS: track 69.2 -> 0.00 mm
- net DIO40/SPI1-MISO: track 68.8 -> 0.00 mm, vias 1 -> 0
- net DIO40/SPI1-SCK: track 68.5 -> 0.00 mm
- net 17: track 68.1 -> 0.00 mm, vias 2 -> 0
- net ADC1.3: track 67.7 -> 0.00 mm, vias 1 -> 0
- net DIO37: track 65.9 -> 0.00 mm
- net ADC0.0: track 63.2 -> 0.00 mm
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- removed copper zone on layer 1, net +3V3
- removed copper zone on layer 1, net FLY1
- removed copper zone on layer 1, net FLY3
- removed copper zone on layer 1, net GND
- removed copper zone on layer 16, net GND
- removed copper zone on layer 1, net N$8
Other:
- board size 128.5 x 85.1 mm -> 93.3 x 94.9 mm
- board text added: "Jennifer Jordan, jejor2@pdx.edu"
- board text added: "TSAR capstone 2020-2021 Sensor Front End Board REV 2.0 2021/2/21"
- board text removed: "12V"
- board text removed: "Conrad Clemans, cclemans@pdx.edu Jennifer Jordan, jejor2@pdx.edu"
- board text removed: "O1"
- board text removed: "O2"
- board text removed: "O3"
- board text removed: "OPEN1_IN"
- board text removed: "OPEN2_IN"
- board text removed: "OPEN3_IN"
- board text removed: "TSAR capstone 2019-2020 Sensor Front End Board REV 1.1 2020-12-29"
- board text removed: "V"
- board text removed: "i"

Commit message: SFE routes completed
Parts:
- moved C13 62.1 mm to (46.6, 18.3)
- moved U$5 52.1 mm to (46.1, 47.8)
- moved C33 15.0 mm to (33.3, 19.8), turned to 180 degrees
- moved C32 14.2 mm to (33.3, 18.4), turned to 180 degrees
- moved POE_BYPASS 9.51 mm to (25.9, 43.9), turned to 0 degrees
- moved C46 9.43 mm to (22.4, 44.8)
- moved R24 9.02 mm to (44.6, 72.1)
- moved R23 8.23 mm to (44.6, 57.6), turned to 0 degrees
- moved R26 5.84 mm to (44.6, 66.1)
- moved C34 5.55 mm to (36.1, 29.8)
- moved R22 5.31 mm to (44.6, 63.3)
- moved C31 4.93 mm to (28.1, 20.1)
- moved 12V. 3.96 mm to (16.2, 90.6), turned to 0 degrees
- moved 5V. 3.96 mm to (19.9, 90.6), turned to 0 degrees
- moved POE. 3.96 mm to (12.6, 90.6), turned to 0 degrees
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Connections:
- new net N$3: ANALOG_TO_DAQ.5, ANALOG_TO_DAQ.6
- net +5V: no longer ANALOG_TO_DAQ.5, ANALOG_TO_DAQ.6
Routing:
- net +5V: track 0.00 -> 211.4 mm, vias 0 -> 5
- net +12V: track 0.00 -> 204.0 mm
- net +24V: track 0.00 -> 170.7 mm, vias 0 -> 1
- net +3V3: track 0.00 -> 139.9 mm, vias 0 -> 3
- net N$25: track 0.00 -> 84.5 mm, vias 0 -> 2
- net 13: track 0.00 -> 83.4 mm
- net 19: track 0.00 -> 77.1 mm, vias 0 -> 2
- net N$21: track 0.00 -> 75.4 mm
- net N$23: track 0.00 -> 70.7 mm
- net 11: track 0.00 -> 70.0 mm, vias 0 -> 2
- net N$24: track 0.00 -> 64.7 mm
- net 12: track 0.00 -> 62.0 mm, vias 0 -> 2
- net ADC0.3: track 0.00 -> 49.2 mm, vias 0 -> 1
- net DIO32/SPI0-SCK: track 0.00 -> 49.1 mm, vias 0 -> 1
- net ADC0.6: track 0.00 -> 46.9 mm
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- added copper zone on layer 1, net GND
- added copper zone on layer 16, net GND
Other:
- board text added: "+ -"
- board text removed: "- +"

Commit message: SFE changes
Replaced ADC's with two 16 channel SPI
Parts:
- removed C12, C31: 0.1u, oresat-rcl:C0603K
- removed C34: 1u, oresat-rcl:C0603K
- removed U1, U2: ADS8344N, ADS8344N:DB20
- added C15: 1u, oresat-rcl:C0603K
- added JP1: (no value), pinhead:1X02
- added U3, U4: ADS7953QDBTRQ1DBT38_TEX-M, ADS7953QDBTRQ1:DBT38_TEX-M
- moved C11 83.8 mm to (-19.3, -15.2), turned to 0 degrees
Connections:
- removed net 11: C28.1, D2.P$2, R39.1, U1.6
- removed net 12: C29.1, D18.P$2, R40.1, U1.7
- removed net 13: C30.1, D1.P$2, R41.1, U1.8
- removed net 14: C35.1, D21.P$2, R47.1, U2.4
- removed net 15: C40.1, D20.P$2, R60.1, U2.6
- removed net 16: C41.1, D26.P$2, R61.1, U2.7
- removed net 17: C42.1, D19.P$2, R62.1, U2.8
- removed net 18: C36.1, D22.P$2, R49.1, U2.3
- removed net 19: C21.1, D3.P$2, R32.1, U1.5
- removed net 20: C37.1, D23.P$2, R54.1, U2.2
- removed net 21: C38.1, D24.P$2, R56.1, U2.1
- removed net 22: C39.1, D25.P$2, R58.1, U2.5
- removed net N$23: C17.1, D6.P$2, R28.1, U1.2
- removed net N$24: C18.1, D5.P$2, R29.1, U1.3
- removed net N$25: C20.1, D4.P$2, R31.1, U1.4
- new net HES1_SIGNAL: C38.1, D24.P$2, R56.1, U3.18
- new net HES2_SIGNAL: C37.1, D23.P$2, R54.1, U3.17
- new net HES3_SIGNAL: C36.1, D22.P$2, R49.1, U3.16
- new net HES4_SIGNAL: C35.1, D21.P$2, R47.1, U3.15
- new net HES5_SIGNAL: C39.1, D25.P$2, R58.1, U3.14
- new net HES6_SIGNAL: C40.1, D20.P$2, R60.1, U3.13
- new net HES7_SIGNAL: C41.1, D26.P$2, R61.1, U3.12
- new net HES8_SIGNAL: C42.1, D19.P$2, R62.1, U3.11
- new net HES9_SIGNAL: C30.1, D1.P$2, R41.1, U3.21
- new net N$10: U3.7, U3.8
- new net N$17: U3.10, U3.19, U3.20, U3.30, U3.35, U3.6, U3.9
- new net N$9: U4.10, U4.19, U4.20, U4.30, U4.35, U4.6
- new net SEN_TBD0: U4.28
- new net SEN_TBD1: U4.27
- new net SEN_TBD10: U4.16
- new net SEN_TBD11: U4.15
- new net SEN_TBD12: U4.14
- new net SEN_TBD13: U4.13
- new net SEN_TBD14: U4.12
- new net SEN_TBD15: U4.11
- new net SEN_TBD2: U4.26
- new net SEN_TBD3: U4.25
- new net SEN_TBD4: U4.24
- new net SEN_TBD5: U4.23
- new net SEN_TBD6: U4.22
- new net SEN_TBD7: U4.21
- new net SEN_TBD8: U4.18
- new net SEN_TBD9: U4.17
- new net TT-F01_SIGNAL: C29.1, D18.P$2, R40.1, U3.28
- new net TT-F02_SIGNAL: C28.1, D2.P$2, R39.1, U3.27
- new net TT-L01_SIGNAL: C21.1, D3.P$2, R32.1, U3.26
- new net TT-L03_SIGNAL: C18.1, D5.P$2, R29.1, U3.24
- new net TT-L04_SIGNAL: C17.1, D6.P$2, R28.1, U3.22, U3.23
- new net TT-L05_SIGNAL: C16.1, D7.P$2, R27.1
- new net TT-LO2_SIGNAL: C20.1, D4.P$2, R31.1, U3.25
- net +3V3: now also C11.1, C15.1, U3.29, U3.36, U3.5, U4.29, U4.36, U4.5; no longer U1.11, U2.11
- net +5V: no longer C11.1, C12.1, C31.1, C34.1, U1.10, U1.12, U1.20, U2.10, U2.12, U2.20
- net DIO32/SPI0-SCK: now also U3.32; no longer U1.19
- net DIO33/SPI0-NSS: now also U3.31; no longer U1.18
- net DIO34/SPI0-MISO: now also U3.34; no longer U1.15
- net DIO35/SPI0-MOSI: now also U3.33; no longer U1.17
- net DIO36: no longer U1.16
- net DIO37: no longer U2.16
- net DIO39/SPI1-NSS: now also U4.31; no longer U2.18
- net DIO40/SPI1-MISO: now also U4.34; no longer U2.15
- net DIO40/SPI1-SCK: now also U4.32; no longer U2.19
- net DIO41/SPI1-MOSI: now also U4.33; no longer U2.17
- net GND: now also C15.2; no longer C12.2, C31.2, C34.2, U1.13, U1.14, U1.9, U2.13, U2.14, U2.9
- net N$21: now also U4.7, U4.8; no longer C16.1, D7.P$2, R27.1, U1.1
Routing:
- net N$25: track 84.5 -> 0.00 mm, vias 2 -> 0
- net 13: track 83.4 -> 0.00 mm
- net HES9_SIGNAL: track 0.00 -> 82.0 mm
- net TT-LO2_SIGNAL: track 0.00 -> 80.7 mm, vias 0 -> 2
- net 19: track 77.1 -> 0.00 mm, vias 2 -> 0
- net N$21: track 75.4 -> 0.00 mm
- net TT-L01_SIGNAL: track 0.00 -> 74.0 mm, vias 0 -> 2
- net N$23: track 70.7 -> 0.00 mm
- net 11: track 70.0 -> 0.00 mm, vias 2 -> 0
- net TT-F02_SIGNAL: track 0.00 -> 67.9 mm, vias 0 -> 2
- net TT-L04_SIGNAL: track 0.00 -> 65.2 mm
- net N$24: track 64.7 -> 0.00 mm
- net 12: track 62.0 -> 0.00 mm, vias 2 -> 0
- net TT-F01_SIGNAL: track 0.00 -> 61.9 mm, vias 0 -> 2
- net TT-L03_SIGNAL: track 0.00 -> 60.0 mm
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