File: tsar_SensorFrontEnd/tsar_SensorFrontEnd.sch (EAGLE design)
At the start: 99 parts, among them X1 057-040-1, X2 057-040-1

Commit message: some changes from Andrew during design review (now with supplies).
Parts:
- C7: value (none) -> 100n
Connections:
- net 12V renamed +12V
- net 5V renamed +5V
Other:
- note added: "Power in from POE 12V @ < 500 mA"
- note added: "Pressure"
- note added: "Temperature via RTD"
- moved on the sheet: POE_IN-1, POE_IN-2

Commit message: Resized Schematic Frame Added connectors for Thrust Plate Input Amp Added 3v3 Regulator (missing resistor values set to TBD)
Parts:
- removed D1, D2, D3: 1N4004, diode:1N4004
- removed SV1: (no value), con-dil:16PL
- removed X1, X2: 057-040-1, con-panduit:057-040-1
- added 123132: DFLS160, diode:DIODE-DO214AA
- added AN, SER: 057-040-1, con-panduit:057-040-1
- added C24, C27: 0.1uF, rcl:C-EUC0805
- added C25: 10uF, rcl:C-EUC0805
- added C26: 4.7uF, rcl:C-EUC0805
- added CR2: 1N4148W-7-F, TSAR_Controller (2):1N4148W-7-F
- added R35, R36, R38: TBD, rcl:R-US_R0603
- added R37: 500k, rcl:R-US_R0603
- added TP: 22-23-2041, con-molex:22-23-2041
- added U$4: MP2456GJ-P, TSAR_Controller (2):MP2456GJ-P
- added U$5: 10uH, TSAR_Controller (2):CLF5030NIT-100M-D
- R34: value 0 -> TBD
Connections:
- removed net N$20: C13.1, C14.1, D1.C, U$3.VREF
- removed net N$30: U$3.D_OUT
- removed net N$31: SV1.9
- removed net N$32: SV1.11
- removed net N$33: D2.C, D3.A
- removed net N$39: U$3.D_IN
- removed net N$47: U$3.DCLK
- new net +3V3: C13.1, C14.1, C25.1, CR2.2, R35.2, U$3.VREF, U$5.2
- new net GND2: 123132.C, C24.2, U$4.SW, U$5.1
- new net N$12: AN-15.S, TP-4.S
- new net N$14: AN-19.S, TP-2.S
- new net N$15: AN-21.S, TP-1.S
- new net N$16: AN-17.S, TP-3.S
- new net N$5: R35.1, R36.2, U$4.FB
- new net N$8: R37.1, R38.2
- net +12V: now also C26.1, C27.1, POE_IN-1.S, R37.2, U$4.IN; no longer POE_IN-2.S
- net +5V: no longer D2.A
- net 1: now also AN-16.S; no longer SV1.1
- net 2: now also AN-18.S; no longer SV1.3
- net 3: now also AN-20.S; no longer SV1.5
- net 4: now also AN-22.S; no longer SV1.7
- net 5: now also AN-24.S
- net 6: now also AN-26.S
- net 7: now also AN-28.S; no longer SV1.13
- net GND: now also 123132.A, C25.2, C26.2, C27.2, POE_IN-2.S, R36.1, R38.1, U$4.GND; no longer POE_IN-1.S, SV1.15, SV1.16
- net N$34: now also AN-27.S; no longer SV1.14
- net N$35: now also AN-25.S; no longer SV1.12
- net N$36: now also AN-23.S; no longer SV1.10
- net N$4: now also C24.1, CR2.1, U$4.BST; no longer D1.A, D3.C
Other:
- note added: "12V input, 3V3 output voltage regulator (for ADS8344 output logic level)"
- note added: "12V input, 5V output voltage regulator (for ADS8344 and RTD Sensors)"
- note added: "Thrust Plate Amplifier Signal Input"
- moved on the sheet: AMBIENT-1, AMBIENT-2, C1, C10, C11, C12, C13, C14, C15, C16, C17, C18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

Commit message: Reduced board size
fixed missing TVS cap values
modified board layout to reduce size
Parts:
- removed SER: 057-040-1, con-panduit:057-040-1
- added X1: 057-040-1, con-panduit:057-040-1
- C1, C10, C16, C17, C18, C2, C21, C3, C4, C5, C6, C8, C9: value (none) -> 120pF
- C20: value (none) -> 120pf
- C7: value 100n -> 120pF
Connections:
- removed net N$34: AN-27.S
- removed net N$35: AN-25.S
- removed net N$36: AN-23.S
- net 10: now also AN-23.S
- net 8: now also AN-27.S
- net 9: now also AN-25.S
- net N$10: now also U$1.EN
- net N$8: now also U$4.EN
Other:
- moved on the sheet: R34, R38

Commit message: Shrunk Board Layout
Reduced size of board
Replaced 20x2 connectors with marionette library part.
Missing digital pin connections
Parts:
- removed AN, X1: 057-040-1, con-panduit:057-040-1
- added J1, SERIAL_TO_DAQ: IDC_RECEPTACLE_2X20-S9175-ND, marionette:IDC_RECEPTACLE_2X20-S9175-ND
Connections:
- net 1: now also J1.16; no longer AN-16.S
- net 10: now also J1.23; no longer AN-23.S
- net 2: now also J1.18; no longer AN-18.S
- net 3: now also J1.20; no longer AN-20.S
- net 4: now also J1.22; no longer AN-22.S
- net 5: now also J1.24; no longer AN-24.S
- net 6: now also J1.26; no longer AN-26.S
- net 7: now also J1.28; no longer AN-28.S
- net 8: now also J1.27; no longer AN-27.S
- net 9: now also J1.25; no longer AN-25.S
- net N$12: now also J1.15; no longer AN-15.S
- net N$14: now also J1.19; no longer AN-19.S
- net N$15: now also J1.21; no longer AN-21.S
- net N$16: now also J1.17; no longer AN-17.S

Commit message: Labeled pressure/temp sensor limits Moved ADS pins in schematic Missing digital pin connections
Other:
- note added: "-220 C"
- note added: "-40-25 C"
- note added: "1k psi"
- note added: "3k psi"
- note added: "Power in from POE 12V @ < 1000 mA"
- note added: "Pressure Sensors"
- note removed: "Power in from POE 12V @ < 500 mA"
- note removed: "Pressure"
- moved on the sheet: C11, C12, C13, C14

Commit message: changed wire size
replaced 0603 resistors with 0805
replaced thrust plate 4 pin connector with 6 pin
missing digital connections
missing mounting holes
tvs diodes need to be replaced
Parts:
- removed POE_IN: 22-23-2021, con-molex:22-23-2021
- added POE: 22-23-2021, con-molex:22-23-2021
- LP1: SPICEPREFIX (none) -> X
- R1, R10, R11, R12, R13, R14, R15, R16, R17, R18, R19, R2, R20, R21, R22, R23, R24, R25, R26, R27, R28, R29, R3, R30, R31, R32, R33, R34, R35, R36, R37, R38, R4, R5, R6, R7, R8, R9: device rcl:R-US_R0603 -> marionette:R-US_0805-B
- TP: value 22-23-2041 -> (none); device con-molex:22-23-2041 -> con-molex:KK-156-6; MPN Thrust Plate Connector -> (none)
Connections:
- net +12V: now also POE-1.S; no longer POE_IN-1.S
- net GND: now also POE-2.S, TP-1.S, TP-6.S; no longer POE_IN-2.S
- net N$12: now also TP-5.S; no longer TP-4.S
- net N$14: now also TP-3.S; no longer TP-2.S
- net N$15: now also TP-2.S; no longer TP-1.S
- net N$16: now also TP-4.S; no longer TP-3.S
Other:
- note added: "+12V input from POE 12V @ < 1000mA"
- note added: "ALL CAPACITORS ARE 0805 10% X5R WITH WORKING VOLTAGE > ??? v UNLESS OTHERWISE MARKED"
- note added: "ALL RESISTORS ARE 0805 1% UNLESS OTHERWISE MARKED"
- note removed: "Power in from POE 12V @ < 1000 mA"
- note removed: "Thrust Plate Amplifier Signal Input"
- moved on the sheet: AMBIENT-1, AMBIENT-2, C15, C16, C17, C18, C19, C20, C21, C22, C23, C24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

Commit message: ADS connected
Parts:
- added H1, H2, H3, H4: MOUNT-HOLE4.5, holes:MOUNT-HOLE4.5
- added POE_BYPASS: 100u, capacitor-wima:C2.5/4
- R33, R37: value 500k -> 10k
- R34, R38: value TBD -> NP
- TP: value (none) -> 22-27-2061-06; device con-molex:KK-156-6 -> con-molex:22-27-2061-06
Connections:
- new net N$11: SERIAL_TO_DAQ.7, U$3.DCLK
- new net N$13: SERIAL_TO_DAQ.10, U$3.D_IN
- new net N$17: SERIAL_TO_DAQ.9, U$3.D_OUT
- new net N$18: SERIAL_TO_DAQ.8, U$3.!CS
- new net N$20: SERIAL_TO_DAQ.11, U$3.BUSY
- net +12V: now also POE_BYPASS.1
- net GND: now also POE_BYPASS.2
Other:
- note added: "Electrolytic Cap"
- moved on the sheet: AMBIENT-1, AMBIENT-2, C1, C10, C11, C12, C13, C14, C15, C16, C17, C18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

Commit message: I broke everything
Parts:
- removed J1: IDC_RECEPTACLE_2X20-S9175-ND, marionette:IDC_RECEPTACLE_2X20-S9175-ND
- removed TP: 22-27-2061-06, con-molex:22-27-2061-06
- removed TVS12, TVS13, TVS14, TVS16, TVS17: DF2B5M4CT,L3F, TSAR_Controller:DF2B5M4CT,L3F
- added ANALOG_TO_DAQ: IDC_RECEPTACLE_2X20-S9175-ND, marionette:IDC_RECEPTACLE_2X20-S9175-ND
- added C28, C29, C30: 120pF, rcl:C-EUC0805
- added OPEN1, OPEN2, OPEN3: 22-23-2021, con-molex:22-23-2021
- added R39, R40, R41, R42, R43, R44: 1k, marionette:R-US_0805-B
- added R45, R46, R47, R48, R49, R50: NP, Resistor_Capacitor:CRCW08050000Z0EA
- added R51, R52, R53: 150, marionette:R-US_0805-B
- added THRUST: Thrust Plate Connector, con-molex:22-27-2051-05
- R25: value 150 -> 22k
- R35: value TBD -> 73.2k
- R36: value TBD -> 23.7k
Connections:
- removed net 14: C16.1, R27.1, TVS12.P$1, U$3.CH0
- removed net 15: C17.1, R28.1, TVS13.P$1, U$3.CH1
- removed net 16: C18.1, R29.1, TVS14.P$1, U$3.CH2
- removed net 18: C20.1, R31.1, TVS16.P$1, U$3.CH3
- new net 11: C28.1, R39.1, U$3.CH5
- new net 12: C29.1, R40.1, U$3.CH6
- new net 13: C30.1, R41.1, U$3.CH7
- new net N$21: C16.1, R27.1, U$3.CH0
- new net N$23: C17.1, R28.1, U$3.CH1
- new net N$24: C18.1, R29.1, U$3.CH2
- new net N$25: C20.1, R31.1, U$3.CH3
- new net N$26: OPEN1-2.S, R42.2, R46.2
- new net N$27: OPEN2-2.S, R43.2, R47.2
- new net N$28: OPEN3-2.S, R44.2, R50.2
- new net N$30: R40.2, R47.1, R48.1
- new net N$31: R41.2, R49.1, R50.1
- new net N$32: R39.2, R45.1, R46.1
- new net N$33: OPEN3-1.S, R49.2, R53.1
- new net N$34: OPEN2-1.S, R48.2, R52.1
- new net N$35: OPEN1-1.S, R45.2, R51.1
- net +5V: now also R51.2, R52.2, R53.2
- net 1: now also ANALOG_TO_DAQ.16; no longer J1.16
- net 10: now also ANALOG_TO_DAQ.23; no longer J1.23
- net 19: no longer TVS17.P$1
- net 2: now also ANALOG_TO_DAQ.18; no longer J1.18
- net 3: now also ANALOG_TO_DAQ.20; no longer J1.20
- net 4: now also ANALOG_TO_DAQ.22; no longer J1.22
- net 5: now also ANALOG_TO_DAQ.24; no longer J1.24
- net 6: now also ANALOG_TO_DAQ.26; no longer J1.26
- net 7: now also ANALOG_TO_DAQ.28; no longer J1.28
- net 8: now also ANALOG_TO_DAQ.27; no longer J1.27
- net 9: now also ANALOG_TO_DAQ.25; no longer J1.25
- net GND: now also C28.2, C29.2, C30.2, R42.1, R43.1, R44.1, THRUST-5.S; no longer TP-1.S, TP-6.S, TVS12.P$2, TVS13.P$2, TVS14.P$2, TVS16.P$2, TVS17.P$2
- net N$12: now also ANALOG_TO_DAQ.15, THRUST-4.S; no longer J1.15, TP-5.S
- net N$14: now also ANALOG_TO_DAQ.19, THRUST-2.S; no longer J1.19, TP-3.S
- net N$15: now also ANALOG_TO_DAQ.21, THRUST-1.S; no longer J1.21, TP-2.S
- net N$16: now also ANALOG_TO_DAQ.17, THRUST-3.S; no longer J1.17, TP-4.S
Other:
- moved on the sheet: AMBIENT-1, AMBIENT-2, C1, C10, C11, C12, C13, C14, C15, C16, C17, C18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
