File: tsar_SensorFrontEnd/tsar_SensorFrontEnd.sch (EAGLE design)
At the start: 238 parts

Commit message: final changes to bom, tr to ct.
Parts:
- C12, C15, C23, C24, C27, C31, C43, C46: DPN 1276-CL10B104KB8NNNLTR-ND -> 1276-CL10B104KB8NNNLCT-ND
- C19, C25, C52, C53: DPN 490-18664-2-ND -> 1276-6736-1-ND; MFR Murata Electronics -> Samsung Electro-Mechanics; MPN GRM21BR61H106ME43L -> CL31A106MBHNNNE
- C22, C26, C45: DPN 1276-1248-2-ND -> 1276-1248-1-ND
- C50, C51: DPN 1276-1860-2-ND -> 1276-1860-1-ND
- L3: DPN 240-3161-2-ND -> 553-PM4340.333NLTCT-ND; MFR Laird-Signal Integrity Products -> Pulse Electronics Power; MPN MGV0503330M-10 -> PM4340.333NLT
- R26: DPN 2019-RK73H2ATTD1243FTR-ND -> 2019-RK73H2ATTD1243FCT-ND
- R30, R36: DPN 2019-RK73H2ATTD2372FTR-ND -> 2019-RK73H2ATTD2372FCT-ND
- R33, R76: DPN BC4966TR-ND -> BC4966CT-ND
- R35: DPN 2019-RK73H2ATTD7322FTR-ND -> 2019-RK73H2ATTD7322FCT-ND
- R37: DPN RHM10KADTR-ND -> RHM10KADCT-ND
- R78, R79, R80, R81, R82, R83: DPN 541-2779-2-ND -> 541-2779-1-ND
Changed lines of the file:
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@@
 </spice>
 <attribute name="DIS" value="Digi-Key"/>
-<attribute name="DPN" value="1276-CL10B104KB8NNNLTR-ND"/>
+<attribute name="DPN" value="1276-CL10B104KB8NNNLCT-ND"/>
 <attribute name="MFR" value="Murata Electronics"/>
 <attribute name="MPN" value="CL10B104KB8NNNL"/>
@@
 </spice>
 <attribute name="DIS" value="Digi-Key"/>
-<attribute name="DPN" value="1276-CL10B104KB8NNNLTR-ND"/>
+<attribute name="DPN" value="1276-CL10B104KB8NNNLCT-ND"/>
 <attribute name="MFR" value="Samsung Electro-Mechanics"/>
 <attribute name="MPN" value="CL10B104KB8NNNL"/>
@@
 </spice>
 <attribute name="DIS" value="Digi-Key"/>
-<attribute name="DPN" value="490-18664-2-ND"/>
-<attribute name="MFR" value="Murata Electronics"/>
-<attribute name="MPN" value="GRM21BR61H106ME43L"/>
+<attribute name="DPN" value="1276-6736-1-ND"/>
+<attribute name="MFR" value="Samsung Electro-Mechanics"/>
+<attribute name="MPN" value="CL31A106MBHNNNE"/>
 </part>
 <part name="R26" library="marionette" deviceset="R-US_" device="0805-B" value="124k">
 <attribute name="DIS" value="Digi-Key"/>
-<attribute name="DPN" value="2019-RK73H2ATTD1243FTR-ND"/>
+<attribute name="DPN" value="2019-RK73H2ATTD1243FCT-ND"/>
 <attribute name="MFR" value="KOA Speer Electronics, Inc."/>
 <attribute name="MPN" value="RK73H2ATTD1243F"/>
@@
 <part name="R30" library="marionette" deviceset="R-US_" device="0805-B" value="23.7k">
 <attribute name="DIS" value="Digi-Key"/>
-<attribute name="DPN" value="2019-RK73H2ATTD2372FTR-ND"/>
+<attribute name="DPN" value="2019-RK73H2ATTD2372FCT-ND"/>
 <attribute name="MFR" value="KOA Speer Electronics, Inc."/>
 <attribute name="MPN" value="RK73H2ATTD2372F"/>
@@
 </spice>
 <attribute name="DIS" value="Digi-Key"/>
-<attribute name="DPN" value="1276-1248-2-ND"/>
+<attribute name="DPN" value="1276-1248-1-ND"/>
 <attribute name="MFR" value="Samsung Electro-Mechanics"/>
 <attribute name="MPN" value="CL21A475KBQNNNE"/>
@@
 </spice>
 <attribute name="DIS" value="Digi-Key"/>
-<attribute name="DPN" value="1276-CL10B104KB8NNNLTR-ND"/>
+<attribute name="DPN" value="1276-CL10B104KB8NNNLCT-ND"/>
 <attribute name="MFR" value="Samsung Electro-Mechanics"/>
 <attribute name="MPN" value="CL10B104KB8NNNL"/>
@@
 </spice>
 <attribute name="DIS" value="Digi-Key"/>
-<attribute name="DPN" value="BC4966TR-ND"/>
+<attribute name="DPN" value="BC4966CT-ND"/>
 <attribute name="MFR" value="Vishay Dale"/>
 <attribute name="MPN" value="CRMA1206AF500KFKEF"/>
@@
 </spice>
 <attribute name="DIS" value="Digi-Key"/>
-<attribute name="DPN" value="1276-CL10B104KB8NNNLTR-ND"/>
+<attribute name="DPN" value="1276-CL10B104KB8NNNLCT-ND"/>
 <attribute name="MFR" value="Samsung Electro-Mechanics"/>
 <attribute name="MPN" value="CL10B104KB8NNNL"/>
@@
 </spice>
 <attribute name="DIS" value="Digi-Key"/>
-<attribute name="DPN" value="490-18664-2-ND"/>
-<attribute name="MFR" value="Murata Electronics"/>
-<attribute name="MPN" value="GRM21BR61H106ME43L"/>
+<attribute name="DPN" value="1276-6736-1-ND"/>
+<attribute name="MFR" value="Samsung Electro-Mechanics"/>
+<attribute name="MPN" value="CL31A106MBHNNNE"/>
 </part>
 <part name="R35" library="marionette" deviceset="R-US_" device="0805-B" value="73.2k">
 <attribute name="DIS" value="Digi-Key"/>
-<attribute name="DPN" value="2019-RK73H2ATTD7322FTR-ND"/>
+<attribute name="DPN" value="2019-RK73H2ATTD7322FCT-ND"/>
 <attribute name="MFR" value="KOA Speer Electronics, Inc."/>
 <attribute name="MPN" value="RK73H2ATTD7322F"/>
@@
 <part name="R36" library="marionette" deviceset="R-US_" device="0805-B" value="23.7k">
 <attribute name="DIS" value="Digi-Key"/>
-<attribute name="DPN" value="2019-RK73H2ATTD2372FTR-ND"/>
+<attribute name="DPN" value="2019-RK73H2ATTD2372FCT-ND"/>
 <attribute name="MFR" value="KOA Speer Electronics, Inc."/>
 <attribute name="MPN" value="RK73H2ATTD2372F"/>
@@
 </spice>
 <attribute name="DIS" value="Digi-Key"/>
-<attribute name="DPN" value="1276-1248-2-ND"/>
+<attribute name="DPN" value="1276-1248-1-ND"/>
 <attribute name="MFR" value="Samsung Electro-Mechanics"/>
 <attribute name="MPN" value="CL21A475KBQNNNE"/>
@@
 </spice>
 <attribute name="DIS" value="Digi-Key"/>
-<attribute name="DPN" value="1276-CL10B104KB8NNNLTR-ND"/>
+<attribute name="DPN" value="1276-CL10B104KB8NNNLCT-ND"/>
 <attribute name="MFR" value="Samsung Electro-Mechanics"/>
 <attribute name="MPN" value="CL10B104KB8NNNL"/>
@@
 <part name="R37" library="marionette" deviceset="R-US_" device="0805-B" value="10k">
 <attribute name="DIS" value="Digi-Key"/>
-<attribute name="DPN" value="RHM10KADTR-ND"/>
+<attribute name="DPN" value="RHM10KADCT-ND"/>
 <attribute name="MFR" value="Rohm Semiconductor"/>
 <attribute name="MPN" value="ESR03EZPF1002"/>
@@
 </spice>
 <attribute name="DIS" value="Digi-Key"/>
-<attribute name="DPN" value="1276-CL10B104KB8NNNLTR-ND"/>
+<attribute name="DPN" value="1276-CL10B104KB8NNNLCT-ND"/>
 <attribute name="MFR" value="Murata Electronics"/>
 <attribute name="MPN" value="CL10B104KB8NNNL"/>
@@
 <part name="L3" library="TSAR_Controller (2)" deviceset="CLF5030NIT-100M-D" device="" value="33uH">
 <attribute name="DIS" value="Digi-Key"/>
-<attribute name="DPN" value="240-3161-2-ND"/>
-<attribute name="MFR" value="Laird-Signal Integrity Products"/>
-<attribute name="MPN" value="MGV0503330M-10"/>
+<attribute name="DPN" value="553-PM4340.333NLTCT-ND"/>
+<attribute name="MFR" value="Pulse Electronics Power"/>
+<attribute name="MPN" value="PM4340.333NLT"/>
 </part>
 <part name="C43" library="rcl" library_urn="urn:adsk.eagle:library:334" deviceset="C-US" device="C0603" package3d_urn="urn:adsk.eagle:package:23616/2" value="100nF">
@@
 </spice>
 <attribute name="DIS" value="Digi-Key"/>
-<attribute name="DPN" value="1276-CL10B104KB8NNNLTR-ND"/>
+<attribute name="DPN" value="1276-CL10B104KB8NNNLCT-ND"/>
 <attribute name="MFR" value="Samsung Electro-Mechanics"/>
 <attribute name="MPN" value="CL10B104KB8NNNL"/>
@@
 </spice>
 <attribute name="DIS" value="Digi-Key"/>
-<attribute name="DPN" value="1276-1248-2-ND"/>
+<attribute name="DPN" value="1276-1248-1-ND"/>
 <attribute name="MFR" value="Samsung Electro-Mechanics"/>
 <attribute name="MPN" value="CL21A475KBQNNNE"/>
@@
 </spice>
 <attribute name="DIS" value="Digi-Key"/>
-<attribute name="DPN" value="1276-CL10B104KB8NNNLTR-ND"/>
+<attribute name="DPN" value="1276-CL10B104KB8NNNLCT-ND"/>
 <attribute name="MFR" value="Samsung Electro-Mechanics"/>
 <attribute name="MPN" value="CL10B104KB8NNNL"/>
@@
 </spice>
 <attribute name="DIS" value="Digi-Key"/>
-<attribute name="DPN" value="BC4966TR-ND"/>
+<attribute name="DPN" value="BC4966CT-ND"/>
 <attribute name="MFR" value="Vishay Dale"/>
 <attribute name="MPN" value="CRMA1206AF500KFKEF"/>
@@
 </spice>
 <attribute name="DIS" value="Digi-Key"/>
-<attribute name="DPN" value="541-2779-2-ND"/>
+<attribute name="DPN" value="541-2779-1-ND"/>
 <attribute name="MFR" value="Vishay Dale"/>
 <attribute name="MPN" value="RCS06030000Z0EA"/>
@@
 </spice>
 <attribute name="DIS" value="Digi-Key"/>
-<attribute name="DPN" value="541-2779-2-ND"/>
+<attribute name="DPN" value="541-2779-1-ND"/>
 <attribute name="MFR" value="Vishay Dale"/>
 <attribute name="MPN" value="RCS06030000Z0EA"/>
@@
 </spice>
 <attribute name="DIS" value="Digi-Key"/>
-<attribute name="DPN" value="541-2779-2-ND"/>
+<attribute name="DPN" value="541-2779-1-ND"/>
 <attribute name="MFR" value="Vishay Dale"/>
 <attribute name="MPN" value="RCS06030000Z0EA"/>
@@
 </spice>
 <attribute name="DIS" value="Digi-Key"/>
-<attribute name="DPN" value="541-2779-2-ND"/>
+<attribute name="DPN" value="541-2779-1-ND"/>
 <attribute name="MFR" value="Vishay Dale"/>
 <attribute name="MPN" value="RCS06030000Z0EA"/>
@@
 </spice>
 <attribute name="DIS" value="Digi-Key"/>
-<attribute name="DPN" value="541-2779-2-ND"/>
+<attribute name="DPN" value="541-2779-1-ND"/>
 <attribute name="MFR" value="Vishay Dale"/>
 <attribute name="MPN" value="RCS06030000Z0EA"/>
@@
 </spice>
 <attribute name="DIS" value="Digi-Key"/>
-<attribute name="DPN" value="541-2779-2-ND"/>
+<attribute name="DPN" value="541-2779-1-ND"/>
 <attribute name="MFR" value="Vishay Dale"/>
 <attribute name="MPN" value="RCS06030000Z0EA"/>
@@
 </spice>
 <attribute name="DIS" value="Digi-Key"/>
-<attribute name="DPN" value="1276-1860-2-ND"/>
+<attribute name="DPN" value="1276-1860-1-ND"/>
 <attribute name="MFR" value="Samsung Electro-Mechanics"/>
 <attribute name="MPN" value="CL10A105KB8NNNC"/>
@@
 </spice>
 <attribute name="DIS" value="Digi-Key"/>
-<attribute name="DPN" value="1276-1860-2-ND"/>
+<attribute name="DPN" value="1276-1860-1-ND"/>
 <attribute name="MFR" value="Samsung Electro-Mechanics"/>
 <attribute name="MPN" value="CL10A105KB8NNNC"/>
@@
 </spice>
 <attribute name="DIS" value="Digi-Key"/>
-<attribute name="DPN" value="490-18664-2-ND"/>
-<attribute name="MFR" value="Murata Electronics"/>
-<attribute name="MPN" value="GRM21BR61H106ME43L"/>
+<attribute name="DPN" value="1276-6736-1-ND"/>
+<attribute name="MFR" value="Samsung Electro-Mechanics"/>
+<attribute name="MPN" value="CL31A106MBHNNNE"/>
 </part>
 <part name="C53" library="rcl" library_urn="urn:adsk.eagle:library:334" deviceset="R-US_" device="R1206" package3d_urn="urn:adsk.eagle:package:23540/2" value="10uF">
@@
 </spice>
 <attribute name="DIS" value="Digi-Key"/>
-<attribute name="DPN" value="490-18664-2-ND"/>
-<attribute name="MFR" value="Murata Electronics"/>
-<attribute name="MPN" value="GRM21BR61H106ME43L"/>
+<attribute name="DPN" value="1276-6736-1-ND"/>
+<attribute name="MFR" value="Samsung Electro-Mechanics"/>
+<attribute name="MPN" value="CL31A106MBHNNNE"/>
 </part>
 <part name="P+15" library="supply1" library_urn="urn:adsk.eagle:library:371" deviceset="+12V" device="" value="+12V"/>

Commit message: sfe edits, added part library
Parts:
- removed U$3: ADS8344, TSAR_Controller:ADS8344
- added U1, U2: ADS8344N, ADS8344N:ADS8344N
Connections:
- net +3V3: now also U1.VREF; no longer U$3.VREF
- net +5V: now also U1.!SHDN, U1.VCC+, U1.VCC+_2; no longer U$3.!SHDN, U$3.+VCC, U$3.+VCC2
- net 11: now also U1.CH5; no longer U$3.CH5
- net 12: now also U1.CH6; no longer U$3.CH6
- net 13: now also U1.CH7; no longer U$3.CH7
- net 19: now also U1.CH4; no longer U$3.CH4
- net DIO32/SPI0-SCK: now also U1.DCLK; no longer U$3.DCLK
- net DIO33/SPI0-NSS: now also U1.!CS; no longer U$3.!CS
- net DIO34/SPI0-MISO: now also U1.DOUT; no longer U$3.D_OUT
- net DIO35/SPI0-MOSI: now also U1.DIN; no longer U$3.D_IN
- net DIO36: now also U1.BUSY; no longer U$3.BUSY
- net GND: now also U1.COM, U1.GND, U1.GND_2; no longer U$3.COM, U$3.GND, U$3.GND2
- net N$21: now also U1.CH0; no longer U$3.CH0
- net N$23: now also U1.CH1; no longer U$3.CH1
- net N$24: now also U1.CH2; no longer U$3.CH2
- net N$25: now also U1.CH3; no longer U$3.CH3
Other:
- moved on the sheet: C13, C14

Commit message: replaced ssop20 with correct package
Parts:
- removed U$8: ADS8344, TSAR_Controller:ADS8344
Connections:
- net +3V3: now also U2.VREF; no longer U$8.VREF
- net +5V: now also U2.!SHDN, U2.VCC+, U2.VCC+_2; no longer U$8.!SHDN, U$8.+VCC, U$8.+VCC2
- net 14: now also U2.CH3; no longer U$8.CH3
- net 15: now also U2.CH5; no longer U$8.CH5
- net 16: now also U2.CH6; no longer U$8.CH6
- net 17: now also U2.CH7; no longer U$8.CH7
- net 18: now also U2.CH2; no longer U$8.CH2
- net 20: now also U2.CH1; no longer U$8.CH1
- net 21: now also U2.CH0; no longer U$8.CH0
- net 22: now also U2.CH4; no longer U$8.CH4
- net DIO37: now also U2.BUSY; no longer U$8.BUSY
- net DIO39/SPI1-NSS: now also U2.!CS; no longer U$8.!CS
- net DIO40/SPI1-MISO: now also U2.DOUT; no longer U$8.D_OUT
- net DIO40/SPI1-SCK: now also U2.DCLK; no longer U$8.DCLK
- net DIO41/SPI1-MOSI: now also U2.DIN; no longer U$8.D_IN
- net GND: now also U2.COM, U2.GND, U2.GND_2; no longer U$8.COM, U$8.GND, U$8.GND2
Other:
- moved on the sheet: C11, C12, C13, C14, C16, C29, C31, C32, C33, C34, D18, D7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
