File: tsar_SensorFrontEnd/tsar_SensorFrontEnd.sch (EAGLE design)
At the start: 174 parts, among them U1 ADS8344N, U2 ADS8344N

Commit message: SFE changes
Replaced ADC's with two 16 channel SPI
Parts:
- removed C12, C31: 0.1u, oresat-rcl:C-USC0603K
- removed C34: 1u, oresat-rcl:C-USC0603K
- removed U1, U2: ADS8344N, ADS8344N:ADS8344N
- added C15: 1u, oresat-rcl:C-USC0603K
- added JP1: (no value), pinhead:PINHD-1X2
- added U3, U4: ADS7953QDBTRQ1DBT38_TEX-M, ADS7953QDBTRQ1:ADS7953QDBTRQ1DBT38_TEX-M
Connections:
- removed net 11: C28.1, D2.P$2, R39.1, U1.CH5
- removed net 12: C29.1, D18.P$2, R40.1, U1.CH6
- removed net 13: C30.1, D1.P$2, R41.1, U1.CH7
- removed net 14: C35.1, D21.P$2, R47.1, U2.CH3
- removed net 15: C40.1, D20.P$2, R60.1, U2.CH5
- removed net 16: C41.1, D26.P$2, R61.1, U2.CH6
- removed net 17: C42.1, D19.P$2, R62.1, U2.CH7
- removed net 18: C36.1, D22.P$2, R49.1, U2.CH2
- removed net 19: C21.1, D3.P$2, R32.1, U1.CH4
- removed net 20: C37.1, D23.P$2, R54.1, U2.CH1
- removed net 21: C38.1, D24.P$2, R56.1, U2.CH0
- removed net 22: C39.1, D25.P$2, R58.1, U2.CH4
- removed net N$23: C17.1, D6.P$2, R28.1, U1.CH1
- removed net N$24: C18.1, D5.P$2, R29.1, U1.CH2
- removed net N$25: C20.1, D4.P$2, R31.1, U1.CH3
- new net HES1_SIGNAL: C38.1, D24.P$2, R56.1, U3.CH8
- new net HES2_SIGNAL: C37.1, D23.P$2, R54.1, U3.CH9
- new net HES3_SIGNAL: C36.1, D22.P$2, R49.1, U3.CH10
- new net HES4_SIGNAL: C35.1, D21.P$2, R47.1, U3.CH11
- new net HES5_SIGNAL: C39.1, D25.P$2, R58.1, U3.CH12
- new net HES6_SIGNAL: C40.1, D20.P$2, R60.1, U3.CH13
- new net HES7_SIGNAL: C41.1, D26.P$2, R61.1, U3.CH14
- new net HES8_SIGNAL: C42.1, D19.P$2, R62.1, U3.CH15
- new net HES9_SIGNAL: C30.1, D1.P$2, R41.1, U3.CH7
- new net N$10: U3.AINP, U3.MXO
- new net N$17: U3.AGND, U3.AGND_2, U3.AGND_3, U3.AGND_4, U3.AGND_5, U3.AINM, U3.BDGND
- new net N$9: U4.AGND, U4.AGND_2, U4.AGND_3, U4.AGND_4, U4.AGND_5, U4.BDGND
- new net SEN_TBD0: U4.CH0
- new net SEN_TBD1: U4.CH1
- new net SEN_TBD10: U4.CH10
- new net SEN_TBD11: U4.CH11
- new net SEN_TBD12: U4.CH12
- new net SEN_TBD13: U4.CH13
- new net SEN_TBD14: U4.CH14
- new net SEN_TBD15: U4.CH15
- new net SEN_TBD2: U4.CH2
- new net SEN_TBD3: U4.CH3
- new net SEN_TBD4: U4.CH4
- new net SEN_TBD5: U4.CH5
- new net SEN_TBD6: U4.CH6
- new net SEN_TBD7: U4.CH7
- new net SEN_TBD8: U4.CH8
- new net SEN_TBD9: U4.CH9
- new net TT-F01_SIGNAL: C29.1, D18.P$2, R40.1, U3.CH0
- new net TT-F02_SIGNAL: C28.1, D2.P$2, R39.1, U3.CH1
- new net TT-L01_SIGNAL: C21.1, D3.P$2, R32.1, U3.CH2
- new net TT-L03_SIGNAL: C18.1, D5.P$2, R29.1, U3.CH4
- new net TT-L04_SIGNAL: C17.1, D6.P$2, R28.1, U3.CH5, U3.CH6
- new net TT-L05_SIGNAL: C16.1, D7.P$2, R27.1
- new net TT-LO2_SIGNAL: C20.1, D4.P$2, R31.1, U3.CH3
- net +3V3: now also C11.1, C15.1, U3.VA+, U3.VA+_2, U3.VBD+, U4.VA+, U4.VA+_2, U4.VBD+; no longer U1.VREF, U2.VREF
- net +5V: no longer C11.1, C12.1, C31.1, C34.1, U1.!SHDN, U1.VCC+, U1.VCC+_2, U2.!SHDN, U2.VCC+, U2.VCC+_2
- net DIO32/SPI0-SCK: now also U3.SCLK; no longer U1.DCLK
- net DIO33/SPI0-NSS: now also U3.!CS; no longer U1.!CS
- net DIO34/SPI0-MISO: now also U3.SDO; no longer U1.DOUT
- net DIO35/SPI0-MOSI: now also U3.SDI; no longer U1.DIN
- net DIO36: no longer U1.BUSY
- net DIO37: no longer U2.BUSY
- net DIO39/SPI1-NSS: now also U4.!CS; no longer U2.!CS
- net DIO40/SPI1-MISO: now also U4.SDO; no longer U2.DOUT
- net DIO40/SPI1-SCK: now also U4.SCLK; no longer U2.DCLK
- net DIO41/SPI1-MOSI: now also U4.SDI; no longer U2.DIN
- net GND: now also C15.2; no longer C12.2, C31.2, C34.2, U1.COM, U1.GND, U1.GND_2, U2.COM, U2.GND, U2.GND_2
- net N$21: now also U4.AINP, U4.MXO; no longer C16.1, D7.P$2, R27.1, U1.CH0
Other:
- note added: "To Thrust Plate Amp Board"
- moved on the sheet: C11, C13, C14, C16, C17, C18, C20, C21, C28, C29, C30, C32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

Commit message: AC, SFE, Library Changes
AC: Reverted to headers for Nucleo. Removed sensors (data coming over usb cable to nucleo), removed power regulator (power coming from usb cable). Replaced leds with correct size and attributes.
SFE: Removed RTD/TVS circuits. Added thermocouple inputs and thermocouple amplifier circuit. Finished ADC wiring. Added schematic info annotations. Cleaned up schematic. TODO: change labels to consistent font/size. layout new components, complete attributes for new components.
Library: Added oresat-rcl library.
Parts:
- removed D18: D5V0H1U2LP1610-7, D5V0H1U2LP1610-7:D5V0H1U2LP1610-7
- removed JP1: (no value), pinhead:PINHD-1X2
- added C12, C22, C31, C48, C54, C57, C58, C61, C62, C65, C66: 0.1uF, oresat-rcl:C-USC0805K
- added C19, C23, C34, C44, C55, C56, C59, C60, C63, C64: 0.01uF, oresat-rcl:C-USC0805K
- added D28: TLVH431, microbuilder:SHUNT-VREF
- added R33, R34, R50, R51, R55, R57: 100, oresat-rcl:R-US_0805-C-NOSILK
- added R42, R44, R52, R59: 1M, oresat-rcl:R-US_0805-C-NOSILK
- added R43, R48, R53, R63: 1K, oresat-rcl:R-US_0805-C-NOSILK
- added U1, U2, U5, U6, U7, U8, U9: AD8495ARMZ, microbuilder:AD849X
- 12V.: value blue -> Green; DIS (none) -> Digi-Key; DPN (none) -> 350-2035-1-ND; MFR (none) -> Dialight; MPN (none) -> 5988070107F
- 3V3., 5V., POE+.: value red -> Green; DIS (none) -> Digi-Key; DPN (none) -> 350-2035-1-ND; MFR (none) -> Dialight; MPN (none) -> 5988070107F
- C16, C17, C21, C28: value 120pF -> 0.01uF; device oresat-rcl:C-USC0603K -> oresat-rcl:C-USC0805K; DIS Digi-Key -> (none); DPN 1276-1160-1-ND -> (none); MFR Samsung Electro-Mechanics -> (none); MPN CL10C121JB8NNNC -> (none)
- C18, C29: value 120pF -> 0.1uF; device oresat-rcl:C-USC0603K -> oresat-rcl:C-USC0805K; DIS Digi-Key -> (none); DPN 1276-1160-1-ND -> (none); MFR Samsung Electro-Mechanics -> (none); MPN CL10C121JB8NNNC -> (none)
- C20: value 120pf -> 0.1uF; device oresat-rcl:C-USC0603K -> oresat-rcl:C-USC0805K; DIS Digi-Key -> (none); DPN 1276-1160-1-ND -> (none); MFR Samsung Electro-Mechanics -> (none); MPN CL10C121JB8NNNC -> (none)
- D2, D3, D4, D5, D6, D7: value D5V0H1U2LP1610-7 -> TLVH431; device D5V0H1U2LP1610-7:D5V0H1U2LP1610-7 -> microbuilder:SHUNT-VREF; DIS Digi-Key -> (none); DPN D5V0H1U2LP1610-7DICT-ND -> (none); MFR Diodes Incorporated -> (none); MPN D5V0H1U2LP1610-7 -> (none)
- R21, R22, R26: value 150 -> 100; device oresat-rcl:R-US_0805-A-NOSILK -> oresat-rcl:R-US_0805-C-NOSILK; DIS Digi-Key -> (none); DPN RNCP0805FTD150RCT-ND -> (none); MFR Stackpole Electronics Inc -> (none); MPN RNCP0805FTD150R -> (none)
- R23: value 150 -> 1M; device oresat-rcl:R-US_0805-A-NOSILK -> oresat-rcl:R-US_0805-C-NOSILK; DIS Digi-Key -> (none); DPN RNCP0805FTD150RCT-ND -> (none); MFR Stackpole Electronics Inc -> (none); MPN RNCP0805FTD150R -> (none)
- R24: value 150 -> 1K; device oresat-rcl:R-US_0805-A-NOSILK -> oresat-rcl:R-US_0805-C-NOSILK; DIS Digi-Key -> (none); DPN RNCP0805FTD150RCT-ND -> (none); MFR Stackpole Electronics Inc -> (none); MPN RNCP0805FTD150R -> (none)
- R25, R30: value 22k -> 100; device oresat-rcl:R-US_0805-A-NOSILK -> oresat-rcl:R-US_0805-C-NOSILK; DIS Digi-Key -> (none); DPN 311-22.0KCRCT-ND -> (none); MFR Yageo -> (none); MPN RC0805FR-0722KL -> (none)
- R27, R31: value 1k -> 1M; device oresat-rcl:R-US_0603-A-NOSILK -> oresat-rcl:R-US_0805-C-NOSILK; DIS Digi-Key -> (none); DPN P1.0KBYCT-ND -> (none); MFR Panasonic Electronic Components -> (none); MPN ERJ-PA3F1001V -> (none)
- R28, R32: value 1k -> 1K; device oresat-rcl:R-US_0603-A-NOSILK -> oresat-rcl:R-US_0805-C-NOSILK; DIS Digi-Key -> (none); DPN P1.0KBYCT-ND -> (none); MFR Panasonic Electronic Components -> (none); MPN ERJ-PA3F1001V -> (none)
- R29, R39, R40: value 1k -> 100; device oresat-rcl:R-US_0603-A-NOSILK -> oresat-rcl:R-US_0805-C-NOSILK; DIS Digi-Key -> (none); DPN P1.0KBYCT-ND -> (none); MFR Panasonic Electronic Components -> (none); MPN ERJ-PA3F1001V -> (none)
- renumbered POE. to POE+.
Connections:
- removed net AMBIENT: R26.1, R32.2, TT-L01-1.S
- removed net CRYO1: R21.1, R27.2, TT-L05-1.S
- removed net CRYO2: R22.1, R28.2, TT-L04-1.S
- removed net CRYO3: R23.1, R29.2, TT-L03-1.S
- removed net CRYO4: R24.1, R31.2, TT-L02-1.S
- removed net N$17: U3.AGND, U3.AGND_2, U3.AGND_3, U3.AGND_4, U3.AGND_5, U3.AINM, U3.BDGND
- removed net N$32: R25.1, R39.2, TT-F02-1.S
- removed net N$34: R30.1, R40.2, TT-F01-1.S
- removed net N$9: U4.AGND, U4.AGND_2, U4.AGND_3, U4.AGND_4, U4.AGND_5, U4.BDGND
- new net IN-: R34.1, R42.2, TT-L05-2.S
- new net IN-1: R22.1, R23.2, TT-L04-2.S
- new net IN-2: R26.1, R27.2, TT-L03-2.S
- new net IN-3: R30.1, R31.2, TT-L02-2.S
- new net IN-4: R40.1, R44.2, TT-L01-2.S
- new net IN-5: R51.1, R52.2, TT-F02-2.S
- new net IN-6: R57.1, R59.2, TT-F01-2.S
- new net N$23: C12.1, C23.2, R33.2, U1.IN+
- new net N$24: C12.2, C19.1, R34.2, U1.IN-
- new net N$25: D28.C, D28.VREF, R43.2, U1.REF
- new net N$26: C17.2, C18.1, R21.2, U2.IN+
- new net N$27: C16.1, C18.2, R22.2, U2.IN-
- new net N$28: D2.C, D2.VREF, R24.2, U2.REF
- new net N$31: C28.2, C29.1, R25.2, U5.IN+
- new net N$33: C21.1, C29.2, R26.2, U5.IN-
- new net N$35: D3.C, D3.VREF, R28.2, U5.REF
- new net N$36: C44.2, C48.1, R29.2, U6.IN+
- new net N$37: C34.1, C48.2, R30.2, U6.IN-
- new net N$39: D4.C, D4.VREF, R32.2, U6.REF
- new net N$41: C56.2, C57.1, R39.2, U7.IN+
- new net N$42: C55.1, C57.2, R40.2, U7.IN-
- new net N$47: D5.C, D5.VREF, R48.2, U7.REF
- new net N$48: C60.2, C61.1, R50.2, U8.IN+
- new net N$49: C59.1, C61.2, R51.2, U8.IN-
- new net N$50: D6.C, D6.VREF, R53.2, U8.REF
- new net N$51: C64.2, C65.1, R55.2, U9.IN+
- new net N$52: C63.1, C65.2, R57.2, U9.IN-
- new net N$53: D7.C, D7.VREF, R63.2, U9.REF
- new net TT-F01: R55.1, TT-F01-1.S
- new net TT-F02: R50.1, TT-F02-1.S
- new net TT-L01: R39.1, TT-L01-1.S
- new net TT-L02: R29.1, TT-L02-1.S
- new net TT-L03: R25.1, TT-L03-1.S
- new net TT-L04: R21.1, TT-L04-1.S
- new net TT-L05: R33.1, TT-L05-1.S
- net +5V: now also C20.1, C22.1, C31.1, C54.1, C58.1, C62.1, C66.1, R24.1, R28.1, R32.1, R43.1, R48.1, R53.1, R63.1, U1.VS+, U2.VS+, U5.VS+, U6.VS+, U7.VS+, U8.VS+, U9.VS+; no longer R21.2, R22.2, R23.2, R24.2, R25.2, R26.2, R30.2
- net GND: now also C17.1, C19.2, C22.2, C23.1, C28.1, C31.2, C34.2, C44.1, C54.2, C55.2, C56.1, C58.2, C59.2, C60.1, C62.2, C63.2, C64.1, C66.2, D2.A, D28.A, D3.A, D4.A, D5.A, D6.A, D7.A, R23.1, R27.1, R31.1, R42.1, R44.1, R52.1, R59.1, U1.VS-, U2.VS-, U3.AGND, U3.AGND_2, U3.AGND_3, U3.AGND_4, U3.AGND_5, U3.AINM, U3.BDGND, U3.REFM, U4.AGND, U4.AGND_2, U4.AGND_3, U4.AGND_4, U4.AGND_5, U4.AINM, U4.BDGND, U4.REFM, U5.VS-, U6.VS-, U7.VS-, U8.VS-, U9.VS-; no longer C17.2, C18.2, C28.2, C29.2, D18.P$1, D2.P$1, D3.P$1, D4.P$1, D5.P$1, D6.P$1, D7.P$1, TT-F01-2.S, TT-F02-2.S, TT-L01-2.S, TT-L02-2.S, TT-L03-2.S, TT-L04-2.S, TT-L05-2.S
- net TT-F01_SIGNAL: now also U9.OUT, U9.SENSE; no longer C29.1, D18.P$2, R40.1
- net TT-F02_SIGNAL: now also U8.OUT, U8.SENSE; no longer C28.1, D2.P$2, R39.1
- net TT-L01_SIGNAL: now also U7.OUT, U7.SENSE; no longer C21.1, D3.P$2, R32.1
- net TT-L03_SIGNAL: now also U5.OUT, U5.SENSE; no longer C18.1, D5.P$2, R29.1
- net TT-L04_SIGNAL: now also U2.OUT, U2.SENSE; no longer C17.1, D6.P$2, R28.1
- net TT-L05_SIGNAL: now also U1.OUT, U1.SENSE; no longer C16.1, D7.P$2, R27.1
- net TT-LO2_SIGNAL: now also U6.OUT, U6.SENSE; no longer C20.1, D4.P$2, R31.1
Other:
- note added: "0.9V REF = -180°C to 820°C"
- note added: "0V REF = 0°C to 1000°C"
- note added: "0V signal indicates the valves default position. 3.3V signal indicates the valves non-default position."
- note added: "1.24V REF = -248°C to 752°C"
- note added: "1k Sensors are 824-M305100000501KPG 3k Sensors are M3051-000005-05KPG (Confirm). 4-20mA output signal."
- note added: "24V input, 12V output voltage regulator (for Pressure Sensors)"
- note added: "5V input from POE+ Input Board; up to 3A (for AD58344 & Thermocouple Sensors)"
- note added: "ADCs to DAQ"
- note added: "All analog sensors go into the ADCs then are sent using SPI to the marionette data bus."
- note added: "K-Type Range = -180°C to 1200°C"
- note added: "Temperature = (Vout - 1.25) / 0.005 V. So, for example, if the voltage is 1.5VDC, the temperature is (1.5 - 1.25) / 0.005 = 50°C"
- note added: "Temperature via Thermocouple"
- note added: "Thrust Plate Amp Connector"
- note added: "Thrust Plate Signals come from the Thrust Plate Amplifier Board. Sensors going into amp board are FC23 load cells."
- note added: "With a Single 5V Supply:"
- note removed: "24V input, 12V output voltage regulator (for Pressure and Unallocated Sensors)"
- note removed: "5V input from POE+ Input Board; up to 3A (for AD58344 & RTD Sensors)"
- note removed: "Temperature via RTD"
- note removed: "Thrust Plate Amplifier Connector"
- moved on the sheet: ANALOG_TO_DAQ, C11, C13, C14, C15, C16, C17, C18, C20, C21, C28, C29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

Commit message: SFE Changes
Added amplifier circuit for thermocouples. Added reference voltage for ADCs.
Parts:
- added C67: 1u, oresat-rcl:C-USC0603K
- added C68: 22u, oresat-rcl:C-USC0603K
- added U10: REF5025AIDR, REF5025AIDR:REF5025AIDR
- C12, C18, C20, C22, C29, C31, C48, C54, C57, C58, C61, C62, C65, C66: device oresat-rcl:C-USC0805K -> oresat-rcl:C-USC0603K; DIS (none) -> Digi-Key; DPN (none) -> 1276-CL10B104KB8NNNLCT-ND; MFR (none) -> Samsung Electro-Mechanics; MPN (none) -> CL10B104KB8NNNL
- C16, C17, C19, C21, C23, C28, C34, C44, C55, C56, C59, C60, C63, C64: device oresat-rcl:C-USC0805K -> oresat-rcl:C-USC0603K; DIS (none) -> Digi-Key; DPN (none) -> 1276-1009-1-ND; MFR (none) -> Samsung Electro-Mechanics; MPN (none) -> CL10B103KB8NNNC
- D2, D28, D3, D4, D5, D6, D7: DIS (none) -> Digi-Key; DPN (none) -> 497-13181-1-ND; MFR (none) -> STMicroelectronics; MPN (none) -> TLVH431AIL3T
- R21, R25, R29, R33, R39, R50, R55: device oresat-rcl:R-US_0805-C-NOSILK -> oresat-rcl:R-US_0603-C-NOSILK; DIS (none) -> Digi-Key; DPN (none) -> 2019-SG73P1JTTD1000FCT-ND; MFR (none) -> KOA Speer Electronics, Inc.; MPN (none) -> SG73P1JTTD1000F
- R22, R26, R30, R34, R40, R51, R57: device oresat-rcl:R-US_0805-C-NOSILK -> oresat-rcl:R-US_0603-C-NOSILK; DIS (none) -> Digi-Key; DPN (none) -> 2019-SG73P1JTTD1000FCT-ND; MFR (none) -> Stackpole Electronics Inc; MPN (none) -> SG73P1JTTD1000F
- R23, R27, R31, R42, R44, R52, R59: device oresat-rcl:R-US_0805-C-NOSILK -> oresat-rcl:R-US_0603-C-NOSILK; DIS (none) -> Digi-Key; DPN (none) -> 118-CMP0603-FX-1004ELFCT-ND; MFR (none) -> Bourns Inc.; MPN (none) -> CMP0603-FX-1004ELF
- R24, R28, R32, R43, R48, R53, R63: device oresat-rcl:R-US_0805-C-NOSILK -> oresat-rcl:R-US_0603-C-NOSILK; DIS (none) -> Digi-Key; DPN (none) -> 511-1732-1-ND; MFR (none) -> Stackpole Electronics Inc; MPN (none) -> SDR03EZPJ102
- U1, U2, U5, U6, U7, U8, U9: DIS (none) -> Digi-Key; DPN (none) -> AD8495ARMZ-ND; MFR (none) -> Analog Devices Inc.; MPN (none) -> AD8495ARMZ
Connections:
- new net V+: C68.1, U10.VOUT, U3.REFP, U4.REFP
- net +5V: now also C67.1, U10.VIN
- net GND: now also C67.2, C68.2, U10.GND, U3.GPIO0, U3.GPIO1, U3.GPIO2, U3.GPIO3, U4.GPIO0, U4.GPIO1, U4.GPIO2, U4.GPIO3
Other:
- moved on the sheet: C11, C13, C14, C15, C32, C33, SERIAL_TO_DAQ, U3, U4

Commit message: AC, SFE, VI changes
AC: Added 5 pin header for sending UART status updates to the valve indicator board. Will only send the current test stand state status, so recieving data from the Vi. Routed header and added labels. Updated attributes and BOM.
SFE: Routed thermocouple amps and ADCs. Made all labels consistent. Updated attributes and BOM.
VI: Updated attributes and BOM.
Parts:
- added C70, C71, C73, C74, C75, C76, C77, C78, C79, C80, C83, C84, C85, C86: 120pF, oresat-rcl:C-USC0603K
- added D32, D33, D34, D35, D36, D37, D38, D39, D41, D42, D44, D45, D46, D47: D5V0H1U2LP1610-7, D5V0H1U2LP1610-7:D5V0H1U2LP1610-7
- added JP1: (no value), pinhead:PINHD-2X12
- added R65, R66, R68, R70, R71, R72, R73, R74, R78, R79, R88, R89, R90, R91: 1k, oresat-rcl:R-US_0603-A-NOSILK
- POE, THRUSTPOWER: DIS (none) -> Digi-Key; DPN (none) -> 900-0022232021-ND; MFR (none) -> Molex
- U3, U4: DPN (none) -> 296-50898-1-ND; MFR (none) -> Texas Instruments; MPN (none) -> ADS7953QDBTRQ1
- renumbered POE_IB_5V to POE_IN_5V
Connections:
- removed net SEN_TBD15: U4.CH15
- removed net SEN_TBD7: U4.CH7
- new net SEN0: JP1.1, R90.2
- new net SEN1: JP1.2, R89.2
- new net SEN10: JP1.19, R73.2
- new net SEN11: JP1.21, R68.2
- new net SEN12: JP1.22, R70.2
- new net SEN13: JP1.23, R71.2
- new net SEN14: JP1.24, R72.2
- new net SEN2: JP1.3, R88.2
- new net SEN3: JP1.5, R91.2
- new net SEN4: JP1.9, R78.2
- new net SEN5: JP1.11, R79.2
- new net SEN7: JP1.15, R74.2
- new net SEN8: JP1.18, R66.2
- new net SEN9: JP1.17, R65.2
- net GND: now also C70.2, C71.2, C73.2, C74.2, C75.2, C76.2, C77.2, C78.2, C79.2, C80.2, C83.2, C84.2, C85.2, C86.2, D32.P$1, D33.P$1, D34.P$1, D35.P$1, D36.P$1, D37.P$1, D38.P$1, D39.P$1, D41.P$1, D42.P$1, D44.P$1, D45.P$1, D46.P$1, D47.P$1, TO_VI.5, TO_VI.6, TO_VI.9
- net HES5: now also TO_VI.7; no longer TO_VI.5
- net HES6: now also TO_VI.8; no longer TO_VI.6
- net HES7: now also TO_VI.10; no longer TO_VI.7
- net HES8: now also TO_VI.11; no longer TO_VI.8
- net HES9: now also TO_VI.12; no longer TO_VI.9
- net SEN_TBD0: now also C85.1, D46.P$2, R90.1
- net SEN_TBD1: now also C84.1, D45.P$2, R89.1
- net SEN_TBD10: now also C77.1, D38.P$2, R73.1
- net SEN_TBD11: now also C73.1, D34.P$2, R68.1
- net SEN_TBD12: now also C74.1, D35.P$2, R70.1
- net SEN_TBD13: now also C75.1, D36.P$2, R71.1
- net SEN_TBD14: now also C76.1, D37.P$2, R72.1
- net SEN_TBD2: now also C83.1, D44.P$2, R88.1
- net SEN_TBD3: now also C86.1, D47.P$2, R91.1
- net SEN_TBD4: now also C79.1, D41.P$2, R78.1
- net SEN_TBD5: now also C80.1, D42.P$2, R79.1
- net SEN_TBD6: now also C78.1, D39.P$2, R74.1
- net SEN_TBD8: now also C71.1, D33.P$2, R66.1
- net SEN_TBD9: now also C70.1, D32.P$2, R65.1
- net TT-L04_SIGNAL: no longer U3.CH6
- net TT-L05_SIGNAL: now also U3.CH6
