File: Thrust Plate Amplifier/ThrustAmpV1.brd (EAGLE design)
At the start: 130.8 x 78.7 mm, 54 parts, among them U1 INA126PA, U2 INA126PA, U3 INA126PA, U4 INA126PA, U5 LP2985AIM5-3.3, U6 LP2985AIM5-5.0/NOPB

Commit message: Major layout changes, per design review
Parts:
- removed J3: (no value), SparkFun-Connectors:1X10
- added J4, J5, J6, J7: (no value), SparkFun-Connectors:1X04
- C13, C6: value 2,2 uF -> 2.2 uF
- R1, R2, R3, R4: value (none) -> TBD
- moved R5 87.1 mm to (10.8, 18.1)
- moved R6 87.1 mm to (21.0, 21.9)
- moved R7 86.4 mm to (10.8, 30.2)
- moved R8 86.4 mm to (21.0, 34.0)
- moved R10 85.4 mm to (21.0, 48.3)
- moved R9 85.4 mm to (10.8, 44.5)
- moved R11 84.8 mm to (10.8, 58.1)
- moved R12 84.8 mm to (21.0, 61.9)
- moved D4 84.3 mm to (82.2, 25.1)
- moved D6 83.5 mm to (81.6, 41.9), turned to 0 degrees
- moved J2 83.0 mm to (89.5, 35.9)
- moved C14 82.1 mm to (79.4, 42.9)
- moved C16 81.5 mm to (80.3, 26.0)
- moved D3 81.3 mm to (81.6, 36.2)
- moved R19 79.1 mm to (76.2, 43.8)
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Connections:
- removed net N$14: J3.2, R5.2, U1.3
- removed net N$15: J3.5, R8.2, U2.2
- removed net N$16: J3.4, R7.2, U2.3
- removed net N$29: J3.3, R6.2, U1.2
- removed net N$32: J3.6, R9.2, U3.3
- removed net N$33: J3.7, R10.2, U3.2
- removed net N$34: J3.8, R11.2, U4.3
- removed net N$35: J3.9, R12.2, U4.2
- new net 0: J1.1
- new net N$100: J7.3, R12.2, U4.2
- new net N$93: J4.2, R5.2, U1.3
- new net N$94: J4.3, R6.2, U1.2
- new net N$95: J5.2, R7.2, U2.3
- new net N$96: J5.3, R8.2, U2.2
- new net N$97: J6.2, R9.2, U3.3
- new net N$98: J6.3, R10.2, U3.2
- new net N$99: J7.2, R11.2, U4.3
- net 5V: now also J4.1, J5.1, J6.1, J7.1; no longer J3.1
- net GND: now also J4.4, J5.4, J6.4, J7.4; no longer J1.1, J3.10
Routing:
- net 5V: track 132.2 -> 272.9 mm
- net N$97: track 0.00 -> 62.5 mm
- net N$93: track 0.00 -> 58.2 mm
- net N$95: track 0.00 -> 48.0 mm
- net N$14: track 47.9 -> 0.00 mm
- net N$99: track 0.00 -> 46.6 mm
- net N$98: track 0.00 -> 45.6 mm
- net N$94: track 0.00 -> 45.4 mm
- net N$32: track 45.3 -> 0.00 mm
- net N$29: track 38.3 -> 0.00 mm
- net N$33: track 35.7 -> 0.00 mm
- net N$96: track 0.00 -> 31.8 mm
- net N$100: track 0.00 -> 31.6 mm
- net N$34: track 29.6 -> 0.00 mm
- net N$16: track 28.0 -> 0.00 mm
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Other:
- board size 130.8 x 78.7 mm -> 97.1 x 77.5 mm
- board text removed: "+5V"
- board text removed: "1+"
- board text removed: "1-"
- board text removed: "2+"
- board text removed: "2-"
- board text removed: "3+"
- board text removed: "3-"
- board text removed: "4+"
- board text removed: "4-"

Commit message: Minor Plate Amp Tweaks- improved grounding
Parts:
- added H1, H2, H3, H4: MOUNT-HOLE2.8, holes:2,8
Connections:
- removed net 0: J1.1
- net GND: now also J1.1
Routing:
- net 5V: track 272.9 -> 273.9 mm
- net 6V: track 28.6 -> 29.5 mm
Other:
- board text added: "Designed by Mike Hall 2019-2020 ECE Capstone"
- board text added: "THRUST PLATE AMPLIFIER v 1.0"

Commit message: THE PENULTIMATE AMPLIFIER
ALMOST ready for OSHpark. Just a few minor chores left.
Parts:
- added C18, C23, C24, C25, C26, C27, C28, C29: 100 pF, rcl:C0805K
- added C19, C22: 100 nF, rcl:C0805K
- added D10, D11, D12, D13, D14, D15, D2, D7, D8, D9: (no value), D5V0H1U2LP1610-7:0603DIODE
- D1: value (none) -> 10BQ060TR
- moved C1 9.02 mm to (75.1, 8.47)
- moved C12 8.02 mm to (75.1, 64.7), turned to 90 degrees
- moved R4 7.57 mm to (63.4, 64.4)
- moved R2 7.53 mm to (63.7, 45.9)
- moved C11 7.51 mm to (81.5, 59.6)
- moved C10 7.49 mm to (83.4, 30.4)
- moved C15 7.49 mm to (87.2, 37.4)
- moved C8 7.49 mm to (83.4, 47.2)
- moved CR1 7.49 mm to (65.3, 8.15)
- moved D3 7.49 mm to (89.1, 36.1)
- moved D6 7.49 mm to (89.1, 41.8)
- moved H1 7.49 mm to (97.0, 6.88)
- moved J2 7.49 mm to (97.0, 35.8)
- moved C3 7.49 mm to (57.0, 12.9)
- moved C7 7.49 mm to (69.7, 59.9)
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Connections:
- net 12V: now also C22.1, D9.P$2
- net 5V: now also C19.1, D15.P$2
- net GND: now also C18.2, C19.2, C22.2, C23.2, C24.2, C25.2, C26.2, C27.2, C28.2, C29.2, D10.P$1, D11.P$1, D12.P$1, D13.P$1, D14.P$1, D15.P$1, D2.P$1, D7.P$1, D8.P$1, D9.P$1
- net N$100: now also C29.1, D2.P$2
- net N$93: now also C18.1, D11.P$2
- net N$94: now also C26.1, D10.P$2
- net N$95: now also C23.1, D12.P$2
- net N$96: now also C27.1, D8.P$2
- net N$97: now also C24.1, D13.P$2
- net N$98: now also C28.1, D7.P$2
- net N$99: now also C25.1, D14.P$2
Routing:
- net N$95: track 48.0 -> 59.0 mm
- net N$98: track 45.6 -> 55.8 mm
- net N$93: track 58.2 -> 67.0 mm
- net N$100: track 31.6 -> 40.5 mm
- net N$96: track 31.8 -> 40.3 mm
- net N$94: track 45.4 -> 53.7 mm
- net 5V: track 273.9 -> 281.5 mm
- net 6V: track 29.5 -> 37.1 mm
- net N$99: track 46.6 -> 53.4 mm
- net 3.3V: track 87.0 -> 93.5 mm
- net N$97: track 62.5 -> 69.0 mm
- net N$28: track 4.77 -> 6.04 mm
- net 12V: track 31.7 -> 30.7 mm
- net N$7: track 5.93 -> 5.30 mm
- net N$25: track 3.01 -> 2.39 mm
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Other:
- board size 97.1 x 77.5 mm -> 104.9 x 77.5 mm

Commit message: THE ACTUAL PENULTIMATE AMPLIFIER
SIKE
Parts:
- D3, D4, D5, D6: value DF2B5M4CT,L3F -> (none); device TSAR_Controller:SOD-882(SOT2) -> D5V0H1U2LP1610-7:0603DIODE
- moved D4 31.2 mm to (88.9, 56.1), turned to 270 degrees
- moved D5 31.0 mm to (89.9, 25.4), turned to 90 degrees
- moved D3 6.33 mm to (88.9, 42.4), turned to 90 degrees
- moved D6 4.98 mm to (89.2, 36.8), turned to 90 degrees
- moved R20 0.25 mm to (83.4, 54.5)
Connections:
- net GND: now also D3.P$1, D4.P$1, D5.P$1, D6.P$1; no longer D3.P$2, D4.P$2, D5.P$2, D6.P$2
- net N$19: now also D5.P$2; no longer D4.P$1
- net N$20: now also D6.P$2; no longer D3.P$1
- net N$23: now also D3.P$2; no longer D6.P$1
- net N$24: now also D4.P$2; no longer D5.P$1
Routing:
- net N$20: track 14.0 -> 13.0 mm
- net N$23: track 15.1 -> 14.3 mm
- net N$19: track 18.6 -> 18.0 mm
Other:
- board text removed: "D3"
- board text removed: "D4"
- board text removed: "D5"
- board text removed: "D6"

Commit message: THE ULTIMATE AMPLIFIER
Routing:
- net N$21: track 10.9 -> 0.48 mm
- added copper zone on layer 1, net N$21
Changed lines of the file:
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@@
 <element name="D3" library="D5V0H1U2LP1610-7" package="0603DIODE" value="" x="88.9" y="42.418" smashed="yes" rot="R90"/>
 <element name="D4" library="D5V0H1U2LP1610-7" package="0603DIODE" value="" x="88.9" y="56.134" smashed="yes" rot="R270"/>
-<element name="D5" library="D5V0H1U2LP1610-7" package="0603DIODE" value="" x="89.916" y="25.4" smashed="yes" rot="R90"/>
+<element name="D5" library="D5V0H1U2LP1610-7" package="0603DIODE" value="" x="89.916" y="25.4" smashed="yes" rot="R90">
+<attribute name="D5" value="" x="92.964" y="23.876" size="1.778" layer="27" rot="R90" display="name"/>
+</element>
 <element name="D6" library="D5V0H1U2LP1610-7" package="0603DIODE" value="" x="89.154" y="36.83" smashed="yes" rot="R90"/>
 </elements>
@@
 <contactref element="D9" pad="P$1"/>
 <contactref element="R15" pad="2"/>
-<polygon width="0" layer="1">
+<polygon width="0" layer="1" rank="2">
 <vertex x="0" y="0"/>
 <vertex x="0" y="77.47"/>
@@
 <contactref element="D1" pad="C"/>
 <contactref element="U$2" pad="1"/>
-<wire x1="72.6567" y1="8.468359375" x2="72.578" y2="8.547059375" width="0.635" layer="1"/>
-<wire x1="72.578" y1="10.6934" x2="72.578" y2="8.547059375" width="0.635" layer="1"/>
-<wire x1="72.578" y1="10.6934" x2="72.578" y2="14.2059" width="0.635" layer="1"/>
 <wire x1="72.578" y1="14.2059" x2="72.5805" y2="14.2084" width="0.635" layer="1"/>
 <wire x1="72.5805" y1="14.2084" x2="72.2405" y2="13.8684" width="0.635" layer="1"/>
-<wire x1="72.2405" y1="13.8684" x2="67.5955" y2="13.8684" width="0.635" layer="1"/>
+<polygon width="0.1524" layer="1" thermals="no">
+<vertex x="73.406" y="8.128"/>
+<vertex x="71.882" y="8.128"/>
+<vertex x="71.882" y="11.684"/>
+<vertex x="71.374" y="12.192"/>
+<vertex x="66.04" y="12.192"/>
+<vertex x="66.04" y="15.24"/>
+<vertex x="67.056" y="16.256"/>
+<vertex x="73.406" y="16.256"/>
+<vertex x="74.93" y="14.732"/>
+<vertex x="74.93" y="12.954"/>
+<vertex x="73.66" y="11.684"/>
+<vertex x="73.66" y="8.382"/>
+</polygon>
 </signal>
 <signal name="N$28">

Commit message: THE ACTUAL ULTIMATE AMPLIFIER
Made all changes from the last design review. Added test points. Fixed isolation. Fixed TVS diode placement. Added proper mounting holes. Also adjusted all names on top silkscreen so they're legible and don't overlap. Suspect board is ready for fab.
Parts:
- added C20: 100 nF, rcl:C0805K
- added D16: (no value), D5V0H1U2LP1610-7:0603DIODE
- added TP1, TP2, TP3, TP4: TEST-POINTTP_15TH_THRU, SparkFun-Connectors:TP_15TH
- H1, H2, H3, H4: value MOUNT-HOLE2.8 -> STAND-OFF; device holes:2,8 -> SparkFun-Hardware:STAND-OFF
- moved H4 114.8 mm to (99.1, 5.08)
- moved H3 114.3 mm to (99.1, 73.7)
- moved H2 114.0 mm to (5.08, 5.08)
- moved H1 113.6 mm to (5.08, 73.7)
- moved D12 1.21 mm to (53.3, 37.6)
- moved D7 1.19 mm to (53.1, 52.6)
- moved D2 1.15 mm to (53.3, 59.7)
- moved D8 1.07 mm to (53.6, 41.7)
- moved D14 1.00 mm to (53.1, 56.1)
- moved D13 0.96 mm to (53.1, 47.2)
- moved D11 0.95 mm to (53.1, 23.9)
- moved D5 0.92 mm to (89.4, 26.2)
- moved D9 0.91 mm to (87.1, 14.2)
- moved D10 0.90 mm to (53.3, 28.7)
- moved D15 0.82 mm to (13.0, 13.0)
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Connections:
- net 12V: now also TP1.P$1
- net 3.3V: now also TP4.P$1
- net 5V: now also C20.1, D16.P$2, TP3.P$1
- net 6V: now also TP2.P$1
- net GND: now also C20.2, D16.P$1
Routing:
- net N$95: track 59.0 -> 55.9 mm
- net 3.3V: track 93.5 -> 95.7 mm
- net N$100: track 40.5 -> 39.8 mm
- net N$93: track 67.0 -> 66.4 mm
- net N$99: track 53.4 -> 52.7 mm
- net N$97: track 69.0 -> 68.3 mm
- net N$96: track 40.3 -> 39.7 mm
- net 6V: track 37.1 -> 37.6 mm
- net N$98: track 55.8 -> 55.2 mm
Other:
- board text added: "TP 12V"
- board text added: "TP 3.3V"
- board text added: "TP 5V"
- board text added: "TP 6V"
