File: Thrust Plate Amplifier/ThrustAmpV1.brd (EAGLE design)
At the start: 104.9 x 77.5 mm, 87 parts, among them U1 INA126PA, U2 INA126PA, U3 INA126PA, U4 INA126PA, U5 LP2985AIM5-3.3, U6 LP2985AIM5-5.0/NOPB

Commit message: Minor Plate Amp changes
Un-derping
Parts:
- R17: value 500 k -> 499 k
- moved H3 5.39 mm to (95.2, 69.8)
- moved H1 4.02 mm to (6.35, 69.8)
- moved H4 4.02 mm to (95.2, 6.35)
- moved H2 1.80 mm to (6.35, 6.35)
- moved D16 0.51 mm to (4.83, 59.7)
- moved D3 0.51 mm to (89.2, 42.9)
- moved D5 0.51 mm to (89.9, 26.2)
- moved R20 0.51 mm to (82.9, 54.5)
- moved D9 0.36 mm to (86.9, 14.5)
- moved C13 0.25 mm to (82.0, 64.7)
- moved C15 0.25 mm to (86.9, 37.4)
- moved C17 0.25 mm to (86.4, 55.5)
- moved C24 0.25 mm to (55.3, 46.9)
- moved C29 0.25 mm to (55.2, 60.2)
- moved D15 0.25 mm to (13.2, 13.0)
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Routing:
- net 12V: track 30.8 -> 30.2 mm
- net N$17: track 16.0 -> 15.5 mm
- net N$23: track 14.3 -> 13.8 mm
- net N$24: track 21.5 -> 22.1 mm
- net N$19: track 17.9 -> 17.4 mm
Other:
- board size 104.9 x 77.5 mm -> 101.6 x 76.2 mm

Commit message: Overthinking Tweaks
Routing:
- net 3.3V: track 95.7 -> 94.5 mm
Other:
- board text added: "Designed by Mike Hall mjhall85@gmail.com 2019-2020 ECE Capstone"
- board text added: "KILROY WAS HERE"
- board text removed: "Designed by Mike Hall 2019-2020 ECE Capstone"
Changed lines of the file:
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@@
 <text x="17.4625" y="66.3575" size="0.762" layer="21" font="vector">TO
 INVERTING</text>
-<text x="6.6675" y="66.3575" size="0.762" layer="21" font="vector">TO NON
+<text x="7.1755" y="66.3575" size="0.762" layer="21" font="vector">TO NON
 INVERTING</text>
 <text x="94.1705" y="12.5984" size="1.27" layer="22" font="vector" rot="MR180">+12 V</text>
@@
 <wire x1="43.815" y1="15.875" x2="43.815" y2="27.6225" width="0.1524" layer="21"/>
 <text x="12.3825" y="6.985" size="1.27" layer="21" font="vector">THRUST PLATE AMPLIFIER v 1.0</text>
-<text x="12.7" y="3.4925" size="1.016" layer="21" font="vector">Designed by Mike Hall
+<text x="12.7" y="2.2225" size="1.016" layer="21" font="vector">Designed by Mike Hall
+mjhall85@gmail.com
 2019-2020 ECE Capstone</text>
 <wire x1="0" y1="76.2" x2="101.6" y2="76.2" width="0" layer="20"/>
@@
 <dimension x1="-6.35" y1="0" x2="-6.35" y2="76.2" x3="-19.05" y3="38.1" textsize="1.778" layer="47" unit="inch" visible="yes"/>
 <dimension x1="0" y1="-6.35" x2="101.6" y2="-6.35" x3="50.8" y3="-19.05" textsize="1.778" layer="47" unit="inch" visible="yes"/>
+<text x="2.54" y="48.514" size="1.778" layer="22" font="vector" rot="MR270">KILROY WAS HERE</text>
 </plain>
 <attributes>
@@
 <wire x1="83.693" y1="63.7159" x2="78.9813" y2="59.0042" width="0.635" layer="16"/>
 <wire x1="78.9813" y1="59.0042" x2="67.2592" y2="59.0042" width="0.635" layer="16"/>
-<wire x1="78.9813" y1="59.0042" x2="76.6064" y2="56.6293" width="0.635" layer="16"/>
-<wire x1="76.6064" y1="50.4317" x2="80.7847" y2="46.2534" width="0.635" layer="16"/>
-<wire x1="76.6064" y1="56.6293" x2="76.6064" y2="50.4317" width="0.635" layer="16"/>
-<wire x1="76.6064" y1="50.4317" x2="76.6064" y2="33.6296" width="0.635" layer="16"/>
-<wire x1="76.6064" y1="33.6296" x2="80.8355" y2="29.4005" width="0.635" layer="16"/>
+<wire x1="78.9813" y1="59.0042" x2="77.1144" y2="57.1373" width="0.635" layer="16"/>
+<wire x1="77.1144" y1="49.9237" x2="80.7847" y2="46.2534" width="0.635" layer="16"/>
+<wire x1="77.1144" y1="57.1373" x2="77.1144" y2="49.9237" width="0.635" layer="16"/>
+<wire x1="77.1144" y1="49.9237" x2="77.1144" y2="33.1216" width="0.635" layer="16"/>
+<wire x1="77.1144" y1="33.1216" x2="80.8355" y2="29.4005" width="0.635" layer="16"/>
 <wire x1="67.2592" y1="59.0042" x2="65.405" y2="59.0042" width="0.635" layer="16"/>
 <wire x1="65.405" y1="59.0042" x2="63.5762" y2="57.1754" width="0.635" layer="16"/>

Commit message: Stole Conrad's stand-offs for plate amp
Parts:
- removed H1, H2, H3, H4: STAND-OFF, SparkFun-Hardware:STAND-OFF
- added H5, H6, H7, H8: #4-BARE_MOUNTING_HOLE/.300, mount:#4/.300-BARE+STD_NUT_OR_STAR_WASHER
Changed lines of the file:
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@@
 <layer number="56" name="wert" color="7" fill="1" visible="no" active="no"/>
 <layer number="57" name="tCAD" color="7" fill="1" visible="no" active="no"/>
+<layer number="58" name="tCAD" color="7" fill="1" visible="no" active="no"/>
 <layer number="59" name="tCarbon" color="7" fill="1" visible="no" active="no"/>
 <layer number="60" name="bCarbon" color="7" fill="1" visible="no" active="no"/>
+<layer number="61" name="stand" color="7" fill="1" visible="no" active="no"/>
 <layer number="88" name="SimResults" color="9" fill="1" visible="no" active="no"/>
 <layer number="89" name="SimProbes" color="9" fill="1" visible="no" active="no"/>
@@
 <layer number="115" name="ReferenceISLANDS" color="7" fill="1" visible="no" active="yes"/>
 <layer number="116" name="Patch_BOT" color="9" fill="4" visible="no" active="yes"/>
+<layer number="117" name="BACKMAAT1" color="7" fill="1" visible="no" active="yes"/>
 <layer number="118" name="Rect_Pads" color="7" fill="1" visible="no" active="yes"/>
+<layer number="119" name="KAP_TEKEN" color="7" fill="1" visible="no" active="yes"/>
+<layer number="120" name="KAP_MAAT1" color="7" fill="1" visible="no" active="yes"/>
 <layer number="121" name="_tsilk" color="7" fill="1" visible="no" active="yes"/>
 <layer number="122" name="_bsilk" color="7" fill="1" visible="no" active="yes"/>
@@
 <layer number="128" name="_bValues" color="7" fill="1" visible="no" active="yes"/>
 <layer number="129" name="Mask" color="7" fill="1" visible="no" active="yes"/>
+<layer number="130" name="SMDSTROOK" color="7" fill="1" visible="no" active="yes"/>
 <layer number="131" name="tAdjust" color="7" fill="1" visible="no" active="yes"/>
 <layer number="132" name="bAdjust" color="7" fill="1" visible="no" active="yes"/>
+<layer number="133" name="bottom_silk" color="7" fill="1" visible="no" active="yes"/>
+<layer number="134" name="silk_top" color="7" fill="1" visible="no" active="no"/>
+<layer number="135" name="silk_bottom" color="7" fill="1" visible="no" active="no"/>
+<layer number="136" name="silktop" color="7" fill="1" visible="no" active="yes"/>
+<layer number="137" name="silkbottom" color="7" fill="1" visible="no" active="yes"/>
+<layer number="140" name="Testjig_Mill" color="26" fill="1" visible="no" active="yes"/>
+<layer number="141" name="TestjigBotDepthMill" color="49" fill="1" visible="no" active="yes"/>
+<layer number="142" name="top_plate_holes" color="42" fill="1" visible="no" active="yes"/>
+<layer number="143" name="bottom_plate_holes" color="50" fill="1" visible="no" active="yes"/>
 <layer number="144" name="Drill_legend" color="7" fill="1" visible="no" active="yes"/>
+<layer number="145" name="DrillLegend_01-16" color="2" fill="9" visible="no" active="yes"/>
+<layer number="146" name="DrillLegend_01-20" color="7" fill="1" visible="no" active="yes"/>
 <layer number="150" name="Notes" color="7" fill="1" visible="no" active="yes"/>
 <layer number="151" name="HeatSink" color="7" fill="1" visible="no" active="yes"/>
@@
 <layer number="250" name="Descript" color="3" fill="1" visible="no" active="no"/>
 <layer number="251" name="SMDround" color="12" fill="11" visible="no" active="no"/>
+<layer number="252" name="coverlay15" color="13" fill="7" visible="no" active="yes"/>
 <layer number="254" name="cooling" color="7" fill="1" visible="no" active="yes"/>
 <layer number="255" name="routoute" color="7" fill="1" visible="no" active="yes"/>
@@
 <text x="92.964" y="37.0459" size="1.778" layer="22" font="vector" rot="MR0">3</text>
 <text x="92.964" y="34.5059" size="1.778" layer="22" font="vector" rot="MR0">4</text>
-<text x="17.4625" y="66.3575" size="0.762" layer="21" font="vector">TO
+<text x="18.4785" y="66.1035" size="0.762" layer="21" font="vector">TO
 INVERTING</text>
-<text x="7.1755" y="66.3575" size="0.762" layer="21" font="vector">TO NON
+<text x="9.9695" y="66.1035" size="0.762" layer="21" font="vector">TO NON
 INVERTING</text>
 <text x="94.1705" y="12.5984" size="1.27" layer="22" font="vector" rot="MR180">+12 V</text>
@@
 <attribute name="VALUE" x="5.572" y="63.622" size="1.016" layer="27" rot="R180"/>
 </element>
-<element name="H1" library="SparkFun-Hardware" library_urn="urn:adsk.eagle:library:519" package="STAND-OFF" package3d_urn="urn:adsk.eagle:package:38630/1" value="STAND-OFF" x="6.35" y="69.85" smashed="yes">
-<attribute name="NAME" x="6.35" y="71.882" size="0.6096" layer="25" font="vector" ratio="20" align="bottom-center"/>
-<attribute name="VALUE" x="6.35" y="67.818" size="0.6096" layer="27" font="vector" ratio="20" align="top-center"/>
-</element>
-<element name="H2" library="SparkFun-Hardware" library_urn="urn:adsk.eagle:library:519" package="STAND-OFF" package3d_urn="urn:adsk.eagle:package:38630/1" value="STAND-OFF" x="6.35" y="6.35" smashed="yes">
-<attribute name="NAME" x="6.35" y="8.382" size="0.6096" layer="25" font="vector" ratio="20" align="bottom-center"/>
-<attribute name="VALUE" x="6.35" y="4.318" size="0.6096" layer="27" font="vector" ratio="20" align="top-center"/>
-</element>
-<element name="H3" library="SparkFun-Hardware" library_urn="urn:adsk.eagle:library:519" package="STAND-OFF" package3d_urn="urn:adsk.eagle:package:38630/1" value="STAND-OFF" x="95.25" y="69.85" smashed="yes">
-<attribute name="NAME" x="95.25" y="71.882" size="0.6096" layer="25" font="vector" ratio="20" align="bottom-center"/>
-<attribute name="VALUE" x="95.25" y="67.818" size="0.6096" layer="27" font="vector" ratio="20" align="top-center"/>
-</element>
-<element name="H4" library="SparkFun-Hardware" library_urn="urn:adsk.eagle:library:519" package="STAND-OFF" package3d_urn="urn:adsk.eagle:package:38630/1" value="STAND-OFF" x="95.25" y="6.35" smashed="yes">
-<attribute name="NAME" x="95.25" y="8.382" size="0.6096" layer="25" font="vector" ratio="20" align="bottom-center"/>
-<attribute name="VALUE" x="95.25" y="4.318" size="0.6096" layer="27" font="vector" ratio="20" align="top-center"/>
-</element>
 <element name="TP1" library="SparkFun-Connectors" library_urn="urn:adsk.eagle:library:513" package="TP_15TH" package3d_urn="urn:adsk.eagle:package:38288/1" value="TEST-POINTTP_15TH_THRU" x="91.948" y="15.24" smashed="yes"/>
 <element name="TP2" library="SparkFun-Connectors" library_urn="urn:adsk.eagle:library:513" package="TP_15TH" package3d_urn="urn:adsk.eagle:package:38288/1" value="TEST-POINTTP_15TH_THRU" x="44.704" y="13.97" smashed="yes"/>
@@
 <element name="D9" library="D5V0H1U2LP1610-7" package="0603DIODE" value="" x="86.868" y="14.478" smashed="yes" rot="R90">
 <attribute name="NAME" x="85.598" y="11.938" size="1.016" layer="25" rot="R90"/>
+</element>
+<element name="H5" library="mount" package="#4/.300-BARE+STD_NUT_OR_STAR_WASHER" value="#4-BARE_MOUNTING_HOLE/.300" x="6.35" y="69.85" smashed="yes">
+<attribute name="NAME" x="9.2075" y="72.7075" size="1.27" layer="25" font="vector"/>
+<attribute name="NAME" x="5.35" y="73.35" size="0.5" layer="33" font="vector" ratio="15"/>
+<attribute name="VALUE" x="9.525" y="66.675" size="1.27" layer="27" font="vector"/>
+</element>
+<element name="H6" library="mount" package="#4/.300-BARE+STD_NUT_OR_STAR_WASHER" value="#4-BARE_MOUNTING_HOLE/.300" x="95.25" y="69.85" smashed="yes">
+<attribute name="NAME" x="98.1075" y="72.7075" size="1.27" layer="25" font="vector"/>
+<attribute name="NAME" x="94.25" y="73.35" size="0.5" layer="33" font="vector" ratio="15"/>
+<attribute name="VALUE" x="98.425" y="66.675" size="1.27" layer="27" font="vector"/>
+</element>
+<element name="H7" library="mount" package="#4/.300-BARE+STD_NUT_OR_STAR_WASHER" value="#4-BARE_MOUNTING_HOLE/.300" x="6.35" y="6.35" smashed="yes">
+<attribute name="NAME" x="9.2075" y="9.2075" size="1.27" layer="25" font="vector"/>
+<attribute name="NAME" x="5.35" y="9.85" size="0.5" layer="33" font="vector" ratio="15"/>
+<attribute name="VALUE" x="9.525" y="3.175" size="1.27" layer="27" font="vector"/>
+</element>
+<element name="H8" library="mount" package="#4/.300-BARE+STD_NUT_OR_STAR_WASHER" value="#4-BARE_MOUNTING_HOLE/.300" x="95.25" y="6.35" smashed="yes">
+<attribute name="NAME" x="98.1075" y="9.2075" size="1.27" layer="25" font="vector"/>
+<attribute name="NAME" x="94.25" y="9.85" size="0.5" layer="33" font="vector" ratio="15"/>
+<attribute name="VALUE" x="98.425" y="3.175" size="1.27" layer="27" font="vector"/>
 </element>
 </elements>
@@
 <wire x1="5.715" y1="27.6225" x2="5.715" y2="41.91" width="1.27" layer="1"/>
 <wire x1="5.715" y1="41.91" x2="5.715" y2="55.5625" width="1.27" layer="1"/>
-<wire x1="5.715" y1="61.722" x2="5.715" y2="63.1825" width="1.27" layer="1"/>
-<wire x1="5.715" y1="63.1825" x2="9.7409" y2="67.2084" width="1.27" layer="1"/>
-<wire x1="9.7409" y1="67.2084" x2="68.453" y2="67.2084" width="1.27" layer="1"/>
+<wire x1="5.715" y1="61.722" x2="5.715" y2="62.6745" width="1.27" layer="1"/>
+<wire x1="5.715" y1="62.6745" x2="10.2489" y2="67.2084" width="1.27" layer="1"/>
+<wire x1="10.2489" y1="67.2084" x2="68.453" y2="67.2084" width="1.27" layer="1"/>
 <wire x1="68.453" y1="67.2084" x2="71.9455" y2="63.7159" width="1.27" layer="1"/>
 <wire x1="71.9455" y1="63.7159" x2="75.118" y2="63.7159" width="1.27" layer="1"/>
