File: Thrust Plate Amplifier/ThrustAmpV1.sch (EAGLE design)
At the start: 54 parts, among them U1 INA126PA, U2 INA126PA, U3 INA126PA, U4 INA126PA, U5 LP2985AIM5-3.3, U6 LP2985AIM5-5.0/NOPB

Commit message: Adjusting annotations
Other:
- note added: "Data Out"
- note removed: "Marionette Connector"
Changed lines of the file:
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@@
 <text x="-139.7" y="40.64" size="2.54" layer="97">Amplifier Power Supply: 3.3 V</text>
 <text x="-193.04" y="-101.6" size="2.54" layer="97">Thrust Plate Connector and Bridge Biasing Resistors</text>
-<text x="200.66" y="-20.32" size="2.54" layer="97">Marionette Connector</text>
+<text x="200.66" y="-20.32" size="2.54" layer="97">Data Out</text>
 <text x="-284.48" y="182.88" size="6.4516" layer="97">Thrust Plate Amplifier and Power Supply Board</text>
 <text x="-284.48" y="175.26" size="2.54" layer="97">Designed by Mike Hall for 2019-2020 TSAR ECE Capstone</text>

Commit message: Major layout changes, per design review
Parts:
- removed J3: (no value), SparkFun-Connectors:CONN_10"
- added J4, J5, J6, J7: (no value), SparkFun-Connectors:CONN_04
- C11, C12, C14, C15, C16, C17, C4, C5: device rcl:C-USC0805 -> rcl:C-EUC0805
- C13, C6: value 2,2 uF -> 2.2 uF; device rcl:C-USC0805 -> rcl:C-EUC0805
- R1, R2, R3, R4: value (none) -> TBD
Connections:
- removed net N$14: J3.2, R5.2, U1.V+IN
- removed net N$15: J3.5, R8.2, U2.V-IN
- removed net N$16: J3.4, R7.2, U2.V+IN
- removed net N$29: J3.3, R6.2, U1.V-IN
- removed net N$32: J3.6, R9.2, U3.V+IN
- removed net N$33: J3.7, R10.2, U3.V-IN
- removed net N$34: J3.8, R11.2, U4.V+IN
- removed net N$35: J3.9, R12.2, U4.V-IN
- new net 0: J1.1
- new net N$100: J7.3, R12.2, U4.V-IN
- new net N$93: J4.2, R5.2, U1.V+IN
- new net N$94: J4.3, R6.2, U1.V-IN
- new net N$95: J5.2, R7.2, U2.V+IN
- new net N$96: J5.3, R8.2, U2.V-IN
- new net N$97: J6.2, R9.2, U3.V+IN
- new net N$98: J6.3, R10.2, U3.V-IN
- new net N$99: J7.2, R11.2, U4.V+IN
- net 5V: now also J4.1, J5.1, J6.1, J7.1; no longer J3.1
- net GND: now also J4.4, J5.4, J6.4, J7.4; no longer J1.1, J3.10
Other:
- note added: "Power In (12 V)"
- moved on the sheet: C1, C10, C11, C12, C13, C14, C15, C16, C17, C2, C3, C4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

Commit message: Minor Plate Amp Tweaks- improved grounding
Parts:
- added H1, H2, H3, H4: MOUNT-HOLE2.8, holes:MOUNT-HOLE2.8
Connections:
- removed net 0: J1.1
- net GND: now also J1.1
Changed lines of the file:
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@@
 <part name="X_25" library="ngspice-simulation" library_urn="urn:adsk.eagle:library:527439" deviceset="GND" device=""/>
 <part name="X_26" library="ngspice-simulation" library_urn="urn:adsk.eagle:library:527439" deviceset="GND" device=""/>
+<part name="H1" library="holes" library_urn="urn:adsk.eagle:library:237" deviceset="MOUNT-HOLE" device="2.8" package3d_urn="urn:adsk.eagle:package:14271/1"/>
+<part name="H2" library="holes" library_urn="urn:adsk.eagle:library:237" deviceset="MOUNT-HOLE" device="2.8" package3d_urn="urn:adsk.eagle:package:14271/1"/>
+<part name="H3" library="holes" library_urn="urn:adsk.eagle:library:237" deviceset="MOUNT-HOLE" device="2.8" package3d_urn="urn:adsk.eagle:package:14271/1"/>
+<part name="H4" library="holes" library_urn="urn:adsk.eagle:library:237" deviceset="MOUNT-HOLE" device="2.8" package3d_urn="urn:adsk.eagle:package:14271/1"/>
 </parts>
 <sheets>
@@
 <instance part="X_25" gate="G$1" x="208.28" y="78.74" smashed="yes"/>
 <instance part="X_26" gate="G$1" x="208.28" y="48.26" smashed="yes"/>
+<instance part="H1" gate="G$1" x="35.56" y="121.92" smashed="yes">
+<attribute name="NAME" x="37.592" y="122.5042" size="1.778" layer="95"/>
+<attribute name="VALUE" x="37.592" y="119.4562" size="1.778" layer="96"/>
+</instance>
+<instance part="H2" gate="G$1" x="35.56" y="114.3" smashed="yes">
+<attribute name="NAME" x="37.592" y="114.8842" size="1.778" layer="95"/>
+<attribute name="VALUE" x="37.592" y="111.8362" size="1.778" layer="96"/>
+</instance>
+<instance part="H3" gate="G$1" x="35.56" y="106.68" smashed="yes">
+<attribute name="NAME" x="37.592" y="107.2642" size="1.778" layer="95"/>
+<attribute name="VALUE" x="37.592" y="104.2162" size="1.778" layer="96"/>
+</instance>
+<instance part="H4" gate="G$1" x="35.56" y="99.06" smashed="yes">
+<attribute name="NAME" x="37.592" y="99.6442" size="1.778" layer="95"/>
+<attribute name="VALUE" x="37.592" y="96.5962" size="1.778" layer="96"/>
+</instance>
 </instances>
 <busses>
@@
 <pinref part="X_23" gate="G$1" pin="0"/>
 <wire x1="208.28" y1="137.16" x2="208.28" y2="132.08" width="0.1524" layer="91"/>
+</segment>
+<segment>
+<pinref part="J1" gate="G$1" pin="1"/>
+<pinref part="X_13" gate="G$1" pin="0"/>
+<wire x1="66.04" y1="332.74" x2="73.66" y2="332.74" width="0.1524" layer="91"/>
+<wire x1="73.66" y1="332.74" x2="73.66" y2="327.66" width="0.1524" layer="91"/>
 </segment>
 </net>
@@
 </segment>
 </net>
-<net name="0" class="0">
-<segment>
-<pinref part="J1" gate="G$1" pin="1"/>
-<pinref part="X_13" gate="G$1" pin="0"/>
-<wire x1="66.04" y1="332.74" x2="73.66" y2="332.74" width="0.1524" layer="91"/>
-<wire x1="73.66" y1="332.74" x2="73.66" y2="327.66" width="0.1524" layer="91"/>
-</segment>
-</net>

Commit message: THE PENULTIMATE AMPLIFIER
ALMOST ready for OSHpark. Just a few minor chores left.
Parts:
- added C18, C23, C24, C25, C26, C27, C28, C29: 100 pF, rcl:C-EUC0805K
- added C19, C22: 100 nF, rcl:C-EUC0805K
- added D10, D11, D12, D13, D14, D15, D2, D7, D8: (no value), D5V0H1U2LP1610-7:D5V0H1U2LP1610-7
- added D9: (no value), D5V0H1U2LP1610-7:D12V0H1U2LP1610-70603DIODE12V
- D1: value (none) -> 10BQ060TR
Connections:
- net 12V: now also C22.1, D9.P$2
- net 5V: now also C19.1, D15.P$2
- net GND: now also C18.2, C19.2, C22.2, C23.2, C24.2, C25.2, C26.2, C27.2, C28.2, C29.2, D10.P$1, D11.P$1, D12.P$1, D13.P$1, D14.P$1, D15.P$1, D2.P$1, D7.P$1, D8.P$1, D9.P$1
- net N$100: now also C29.1, D2.P$2
- net N$93: now also C18.1, D11.P$2
- net N$94: now also C26.1, D10.P$2
- net N$95: now also C23.1, D12.P$2
- net N$96: now also C27.1, D8.P$2
- net N$97: now also C24.1, D13.P$2
- net N$98: now also C28.1, D7.P$2
- net N$99: now also C25.1, D14.P$2
Other:
- note added: "All resistors are 0805 1% unless otherwise specified. All capacitors are 0805 10% X5R with working voltage 25 V unless otherwise specified."
- note added: "To Do: -Values for gain setting resistors"
- note removed: "To Do: -Values for gain setting resistors -TVS on input"

Commit message: THE ACTUAL PENULTIMATE AMPLIFIER
SIKE
Parts:
- D3, D4, D5, D6: value DF2B5M4CT,L3F -> (none); device TSAR_Controller:DF2B5M4CT,L3F -> D5V0H1U2LP1610-7:D5V0H1U2LP1610-7
Connections:
- net GND: now also D3.P$1, D4.P$1, D5.P$1, D6.P$1; no longer D3.P$2, D4.P$2, D5.P$2, D6.P$2
- net N$19: now also D5.P$2; no longer D4.P$1
- net N$20: now also D6.P$2; no longer D3.P$1
- net N$23: now also D3.P$2; no longer D6.P$1
- net N$24: now also D4.P$2; no longer D5.P$1
Changed lines of the file:
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@@
 <part name="R16" library="rcl" library_urn="urn:adsk.eagle:library:334" deviceset="R-US_" device="R0805" package3d_urn="urn:adsk.eagle:package:23553/2" value="124k"/>
 <part name="R14" library="rcl" library_urn="urn:adsk.eagle:library:334" deviceset="R-US_" device="R0805" package3d_urn="urn:adsk.eagle:package:23553/2" value="19.1 k"/>
-<part name="D6" library="TSAR_Controller" deviceset="DF2B5M4CT,L3F" device=""/>
-<part name="D5" library="TSAR_Controller" deviceset="DF2B5M4CT,L3F" device=""/>
-<part name="D3" library="TSAR_Controller" deviceset="DF2B5M4CT,L3F" device=""/>
-<part name="D4" library="TSAR_Controller" deviceset="DF2B5M4CT,L3F" device=""/>
 <part name="C14" library="rcl" library_urn="urn:adsk.eagle:library:334" deviceset="C-EU" device="C0805" package3d_urn="urn:adsk.eagle:package:23617/2" value="120 pF"/>
 <part name="C15" library="rcl" library_urn="urn:adsk.eagle:library:334" deviceset="C-EU" device="C0805" package3d_urn="urn:adsk.eagle:package:23617/2" value="120 pF"/>
@@
 <part name="SUPPLY46" library="supply2" library_urn="urn:adsk.eagle:library:372" deviceset="GND" device=""/>
 <part name="SUPPLY47" library="supply2" library_urn="urn:adsk.eagle:library:372" deviceset="GND" device=""/>
+<part name="D3" library="D5V0H1U2LP1610-7" deviceset="D5V0H1U2LP1610-7" device=""/>
+<part name="D4" library="D5V0H1U2LP1610-7" deviceset="D5V0H1U2LP1610-7" device=""/>
+<part name="D5" library="D5V0H1U2LP1610-7" deviceset="D5V0H1U2LP1610-7" device=""/>
+<part name="D6" library="D5V0H1U2LP1610-7" deviceset="D5V0H1U2LP1610-7" device=""/>
 </parts>
 <sheets>
@@
 <attribute name="VALUE" x="234.442" y="300.99" size="1.778" layer="96" rot="R90"/>
 </instance>
-<instance part="D6" gate="G$1" x="477.52" y="165.1" smashed="yes">
-<attribute name="NAME" x="480.06" y="167.64" size="1.27" layer="95"/>
-<attribute name="VALUE" x="480.06" y="162.56" size="1.27" layer="96"/>
-</instance>
-<instance part="D5" gate="G$1" x="439.42" y="165.1" smashed="yes">
-<attribute name="NAME" x="431.8" y="167.64" size="1.27" layer="95"/>
-<attribute name="VALUE" x="424.18" y="160.02" size="1.27" layer="96"/>
-</instance>
-<instance part="D3" gate="G$1" x="477.52" y="195.58" smashed="yes" rot="R180">
-<attribute name="NAME" x="474.98" y="193.04" size="1.27" layer="95" rot="R180"/>
-<attribute name="VALUE" x="474.98" y="198.12" size="1.27" layer="96" rot="R180"/>
-</instance>
-<instance part="D4" gate="G$1" x="439.42" y="195.58" smashed="yes" rot="R180">
-<attribute name="NAME" x="436.88" y="193.04" size="1.27" layer="95" rot="R180"/>
-<attribute name="VALUE" x="436.88" y="198.12" size="1.27" layer="96" rot="R180"/>
-</instance>
 <instance part="C14" gate="G$1" x="495.3" y="165.1" smashed="yes">
 <attribute name="NAME" x="496.316" y="165.735" size="1.778" layer="95"/>
@@
 <instance part="SUPPLY47" gate="GND" x="520.7" y="167.64" smashed="yes">
 <attribute name="VALUE" x="518.795" y="164.465" size="1.778" layer="96"/>
+</instance>
+<instance part="D3" gate="G$1" x="477.52" y="165.1" smashed="yes" rot="R180">
+<attribute name="NAME" x="474.98" y="162.56" size="1.778" layer="95" rot="R180"/>
+</instance>
+<instance part="D4" gate="G$1" x="439.42" y="165.1" smashed="yes" rot="R180">
+<attribute name="NAME" x="436.88" y="162.56" size="1.778" layer="95" rot="R180"/>
+</instance>
+<instance part="D5" gate="G$1" x="439.42" y="195.58" smashed="yes">
+<attribute name="NAME" x="441.96" y="198.12" size="1.778" layer="95"/>
+</instance>
+<instance part="D6" gate="G$1" x="477.52" y="195.58" smashed="yes">
+<attribute name="NAME" x="480.06" y="198.12" size="1.778" layer="95"/>
 </instance>
 </instances>
@@
 </segment>
 <segment>
-<pinref part="D4" gate="G$1" pin="P$2"/>
-<wire x1="439.42" y1="200.66" x2="439.42" y2="203.2" width="0.1524" layer="91"/>
+<wire x1="439.42" y1="199.39" x2="439.42" y2="203.2" width="0.1524" layer="91"/>
 <wire x1="439.42" y1="203.2" x2="447.04" y2="203.2" width="0.1524" layer="91"/>
 <wire x1="447.04" y1="203.2" x2="447.04" y2="200.66" width="0.1524" layer="91"/>
@@
 <junction x="447.04" y="203.2"/>
 <pinref part="SUPPLY42" gate="GND" pin="GND"/>
-</segment>
-<segment>
-<pinref part="D3" gate="G$1" pin="P$2"/>
-<wire x1="477.52" y1="200.66" x2="477.52" y2="203.2" width="0.1524" layer="91"/>
+<pinref part="D5" gate="G$1" pin="P$1"/>
+</segment>
+<segment>
+<wire x1="477.52" y1="199.39" x2="477.52" y2="203.2" width="0.1524" layer="91"/>
 <wire x1="477.52" y1="203.2" x2="485.14" y2="203.2" width="0.1524" layer="91"/>
 <wire x1="485.14" y1="203.2" x2="485.14" y2="200.66" width="0.1524" layer="91"/>
@@
 <junction x="485.14" y="203.2"/>
 <pinref part="SUPPLY41" gate="GND" pin="GND"/>
+<pinref part="D6" gate="G$1" pin="P$1"/>
 </segment>
 <segment>
@@
 <wire x1="452.12" y1="160.02" x2="439.42" y2="160.02" width="0.1524" layer="91"/>
 <wire x1="439.42" y1="160.02" x2="439.42" y2="154.94" width="0.1524" layer="91"/>
-<pinref part="D5" gate="G$1" pin="P$2"/>
+<pinref part="SUPPLY39" gate="GND" pin="GND"/>
+<pinref part="D4" gate="G$1" pin="P$1"/>
+<wire x1="439.42" y1="161.29" x2="439.42" y2="160.02" width="0.1524" layer="91"/>
 <junction x="439.42" y="160.02"/>
-<pinref part="SUPPLY39" gate="GND" pin="GND"/>
-</segment>
-<segment>
-<pinref part="D6" gate="G$1" pin="P$2"/>
+</segment>
+<segment>
 <pinref part="C14" gate="G$1" pin="2"/>
 <wire x1="477.52" y1="160.02" x2="495.3" y2="160.02" width="0.1524" layer="91"/>
 <wire x1="477.52" y1="160.02" x2="477.52" y2="154.94" width="0.1524" layer="91"/>
+<pinref part="SUPPLY40" gate="GND" pin="GND"/>
+<pinref part="D3" gate="G$1" pin="P$1"/>
+<wire x1="477.52" y1="160.02" x2="477.52" y2="161.29" width="0.1524" layer="91"/>
 <junction x="477.52" y="160.02"/>
-<pinref part="SUPPLY40" gate="GND" pin="GND"/>
 </segment>
 <segment>
@@
 <wire x1="520.7" y1="182.88" x2="452.12" y2="182.88" width="0.1524" layer="91"/>
 <pinref part="J2" gate="G$1" pin="1"/>
-<pinref part="D4" gate="G$1" pin="P$1"/>
 <wire x1="452.12" y1="182.88" x2="439.42" y2="182.88" width="0.1524" layer="91"/>
 <wire x1="439.42" y1="182.88" x2="419.1" y2="182.88" width="0.1524" layer="91"/>
@@
 <wire x1="419.1" y1="182.88" x2="419.1" y2="238.76" width="0.1524" layer="91"/>
 <pinref part="R13" gate="G$1" pin="1"/>
+<pinref part="D5" gate="G$1" pin="P$2"/>
 </segment>
 </net>
@@
 <wire x1="520.7" y1="180.34" x2="495.3" y2="180.34" width="0.1524" layer="91"/>
 <pinref part="J2" gate="G$1" pin="2"/>
-<pinref part="D3" gate="G$1" pin="P$1"/>
 <wire x1="495.3" y1="180.34" x2="477.52" y2="180.34" width="0.1524" layer="91"/>
 <wire x1="477.52" y1="180.34" x2="416.56" y2="180.34" width="0.1524" layer="91"/>
@@
 <pinref part="R18" gate="G$1" pin="1"/>
 <wire x1="416.56" y1="193.04" x2="416.56" y2="180.34" width="0.1524" layer="91"/>
+<pinref part="D6" gate="G$1" pin="P$2"/>
 </segment>
 </net>
@@
 <wire x1="477.52" y1="177.8" x2="416.56" y2="177.8" width="0.1524" layer="91"/>
 <pinref part="J2" gate="G$1" pin="3"/>
-<pinref part="D6" gate="G$1" pin="P$1"/>
 <wire x1="477.52" y1="177.8" x2="477.52" y2="170.18" width="0.1524" layer="91"/>
 <junction x="477.52" y="177.8"/>
@@
 <pinref part="R19" gate="G$1" pin="2"/>
 <wire x1="416.56" y1="177.8" x2="416.56" y2="160.02" width="0.1524" layer="91"/>
+<pinref part="D3" gate="G$1" pin="P$2"/>
 </segment>
 </net>
@@
 <wire x1="439.42" y1="175.26" x2="419.1" y2="175.26" width="0.1524" layer="91"/>
 <pinref part="J2" gate="G$1" pin="4"/>
-<pinref part="D5" gate="G$1" pin="P$1"/>
 <wire x1="439.42" y1="175.26" x2="439.42" y2="170.18" width="0.1524" layer="91"/>
 <junction x="439.42" y="175.26"/>
@@
 <pinref part="R20" gate="G$1" pin="2"/>
 <wire x1="419.1" y1="175.26" x2="419.1" y2="116.84" width="0.1524" layer="91"/>
-</segment>
-</net>
+<pinref part="D4" gate="G$1" pin="P$2"/>
+</segment>
+</net>

Commit message: THE ACTUAL ULTIMATE AMPLIFIER
Made all changes from the last design review. Added test points. Fixed isolation. Fixed TVS diode placement. Added proper mounting holes. Also adjusted all names on top silkscreen so they're legible and don't overlap. Suspect board is ready for fab.
Parts:
- added C20: 100 nF, rcl:C-EUC0805K
- added D16: (no value), D5V0H1U2LP1610-7:D5V0H1U2LP1610-7
- added TP1, TP2, TP3, TP4: TEST-POINTTP_15TH_THRU, SparkFun-Connectors:TEST-POINTTP_15TH_THRU
- D9: device D5V0H1U2LP1610-7:D12V0H1U2LP1610-70603DIODE12V -> D5V0H1U2LP1610-7:D5V0H1U2LP1610-7
- H1, H2, H3, H4: value MOUNT-HOLE2.8 -> STAND-OFF; device holes:MOUNT-HOLE2.8 -> SparkFun-Hardware:STAND-OFF
Connections:
- net 12V: now also TP1.1
- net 3.3V: now also TP4.1
- net 5V: now also C20.1, D16.P$2, TP3.1
- net 6V: now also TP2.1
- net GND: now also C20.2, D16.P$1
Other:
- note removed: "To Do: -Values for gain setting resistors"
- moved on the sheet: C19

Commit message: Minor Plate Amp changes
Un-derping
Parts:
- D9: device D5V0H1U2LP1610-7:D5V0H1U2LP1610-7 -> D5V0H1U2LP1610-7:D12V0H1U2LP1610-70603DIODE12V
- R17: value 500 k -> 499 k
Changed lines of the file:
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@@
 <part name="C3" library="rcl" library_urn="urn:adsk.eagle:library:334" deviceset="C-EU" device="C0805" package3d_urn="urn:adsk.eagle:package:23617/2" value="22 uF"/>
 <part name="FRAME1" library="frames" library_urn="urn:adsk.eagle:library:229" deviceset="FRAME_C_L" device=""/>
-<part name="R17" library="rcl" library_urn="urn:adsk.eagle:library:334" deviceset="R-US_" device="R0805" package3d_urn="urn:adsk.eagle:package:23553/2" value="500 k"/>
+<part name="R17" library="rcl" library_urn="urn:adsk.eagle:library:334" deviceset="R-US_" device="R0805" package3d_urn="urn:adsk.eagle:package:23553/2" value="499 k"/>
 <part name="SUPPLY2" library="SparkFun-PowerSymbols" library_urn="urn:adsk.eagle:library:530" deviceset="3.3V" device=""/>
 <part name="SUPPLY4" library="SparkFun-PowerSymbols" library_urn="urn:adsk.eagle:library:530" deviceset="3.3V" device=""/>
@@
 <part name="D15" library="D5V0H1U2LP1610-7" deviceset="D5V0H1U2LP1610-7" device=""/>
 <part name="D16" library="D5V0H1U2LP1610-7" deviceset="D5V0H1U2LP1610-7" device=""/>
-<part name="D9" library="D5V0H1U2LP1610-7" deviceset="D5V0H1U2LP1610-7" device=""/>
+<part name="D9" library="D5V0H1U2LP1610-7" deviceset="D12V0H1U2LP1610-7" device="0603DIODE12V"/>
 </parts>
 <sheets>
@@
 <instance part="D9" gate="G$1" x="81.28" y="340.36" smashed="yes" rot="R270">
 <attribute name="NAME" x="83.82" y="337.82" size="1.778" layer="95" rot="R270"/>
+<attribute name="VALUE" x="78.74" y="337.82" size="1.778" layer="96" rot="R270"/>
 </instance>
 </instances>
@@
 </sheet>
 </sheets>
+<errors>
+</errors>
 </schematic>
 </drawing>
