File: Thrust Plate Amplifier/ThrustAmpV1.sch (EAGLE design)
At the start: 87 parts, among them U1 INA126PA, U2 INA126PA, U3 INA126PA, U4 INA126PA, U5 LP2985AIM5-3.3, U6 LP2985AIM5-5.0/NOPB

Commit message: Stole Conrad's stand-offs for plate amp
Parts:
- removed H1, H2, H3, H4: STAND-OFF, SparkFun-Hardware:STAND-OFF
- added H5, H6, H7, H8: #4-BARE_MOUNTING_HOLE/.300, mount:#4-BARE_MOUNTING_HOLE/.300
Changed lines of the file:
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@@
 <layer number="56" name="wert" color="7" fill="1" visible="no" active="no"/>
 <layer number="57" name="tCAD" color="7" fill="1" visible="no" active="no"/>
+<layer number="58" name="tCAD" color="7" fill="1" visible="no" active="no"/>
 <layer number="59" name="tCarbon" color="7" fill="1" visible="no" active="no"/>
 <layer number="60" name="bCarbon" color="7" fill="1" visible="no" active="no"/>
+<layer number="61" name="stand" color="7" fill="1" visible="no" active="no"/>
 <layer number="88" name="SimResults" color="9" fill="1" visible="yes" active="yes"/>
 <layer number="89" name="SimProbes" color="9" fill="1" visible="yes" active="yes"/>
@@
 <layer number="115" name="ReferenceISLANDS" color="7" fill="1" visible="no" active="yes"/>
 <layer number="116" name="Patch_BOT" color="9" fill="4" visible="yes" active="yes"/>
+<layer number="117" name="BACKMAAT1" color="7" fill="1" visible="no" active="yes"/>
 <layer number="118" name="Rect_Pads" color="7" fill="1" visible="no" active="yes"/>
+<layer number="119" name="KAP_TEKEN" color="7" fill="1" visible="no" active="yes"/>
+<layer number="120" name="KAP_MAAT1" color="7" fill="1" visible="no" active="yes"/>
 <layer number="121" name="_tsilk" color="7" fill="1" visible="yes" active="yes"/>
 <layer number="122" name="_bsilk" color="7" fill="1" visible="yes" active="yes"/>
@@
 <layer number="128" name="_bValues" color="7" fill="1" visible="yes" active="yes"/>
 <layer number="129" name="Mask" color="7" fill="1" visible="yes" active="yes"/>
+<layer number="130" name="SMDSTROOK" color="7" fill="1" visible="no" active="yes"/>
 <layer number="131" name="tAdjust" color="7" fill="1" visible="yes" active="yes"/>
 <layer number="132" name="bAdjust" color="7" fill="1" visible="yes" active="yes"/>
+<layer number="133" name="bottom_silk" color="7" fill="1" visible="no" active="yes"/>
+<layer number="134" name="silk_top" color="7" fill="1" visible="no" active="no"/>
+<layer number="135" name="silk_bottom" color="7" fill="1" visible="no" active="no"/>
+<layer number="136" name="silktop" color="7" fill="1" visible="no" active="yes"/>
+<layer number="137" name="silkbottom" color="7" fill="1" visible="no" active="yes"/>
+<layer number="140" name="Testjig_Mill" color="26" fill="1" visible="no" active="yes"/>
+<layer number="141" name="TestjigBotDepthMill" color="49" fill="1" visible="no" active="yes"/>
+<layer number="142" name="top_plate_holes" color="42" fill="1" visible="no" active="yes"/>
+<layer number="143" name="bottom_plate_holes" color="50" fill="1" visible="no" active="yes"/>
 <layer number="144" name="Drill_legend" color="7" fill="1" visible="yes" active="yes"/>
+<layer number="145" name="DrillLegend_01-16" color="2" fill="9" visible="no" active="yes"/>
+<layer number="146" name="DrillLegend_01-20" color="7" fill="1" visible="no" active="yes"/>
 <layer number="150" name="Notes" color="7" fill="1" visible="yes" active="yes"/>
 <layer number="151" name="HeatSink" color="7" fill="1" visible="yes" active="yes"/>
@@
 <layer number="250" name="Descript" color="3" fill="1" visible="no" active="no"/>
 <layer number="251" name="SMDround" color="12" fill="11" visible="no" active="no"/>
+<layer number="252" name="coverlay15" color="13" fill="7" visible="no" active="yes"/>
 <layer number="254" name="cooling" color="7" fill="1" visible="yes" active="yes"/>
 <layer number="255" name="routoute" color="7" fill="1" visible="yes" active="yes"/>
@@
 <part name="C20" library="rcl" library_urn="urn:adsk.eagle:library:334" deviceset="C-EU" device="C0805K" package3d_urn="urn:adsk.eagle:package:23681/2" value="100 nF"/>
 <part name="SUPPLY48" library="supply2" library_urn="urn:adsk.eagle:library:372" deviceset="GND" device=""/>
-<part name="H1" library="SparkFun-Hardware" library_urn="urn:adsk.eagle:library:519" deviceset="STAND-OFF" device="" package3d_urn="urn:adsk.eagle:package:38630/1"/>
-<part name="H2" library="SparkFun-Hardware" library_urn="urn:adsk.eagle:library:519" deviceset="STAND-OFF" device="" package3d_urn="urn:adsk.eagle:package:38630/1"/>
-<part name="H3" library="SparkFun-Hardware" library_urn="urn:adsk.eagle:library:519" deviceset="STAND-OFF" device="" package3d_urn="urn:adsk.eagle:package:38630/1"/>
-<part name="H4" library="SparkFun-Hardware" library_urn="urn:adsk.eagle:library:519" deviceset="STAND-OFF" device="" package3d_urn="urn:adsk.eagle:package:38630/1"/>
 <part name="TP1" library="SparkFun-Connectors" library_urn="urn:adsk.eagle:library:513" deviceset="TEST-POINT" device="TP_15TH_THRU" package3d_urn="urn:adsk.eagle:package:38288/1"/>
 <part name="TP2" library="SparkFun-Connectors" library_urn="urn:adsk.eagle:library:513" deviceset="TEST-POINT" device="TP_15TH_THRU" package3d_urn="urn:adsk.eagle:package:38288/1"/>
@@
 <part name="D16" library="D5V0H1U2LP1610-7" deviceset="D5V0H1U2LP1610-7" device=""/>
 <part name="D9" library="D5V0H1U2LP1610-7" deviceset="D12V0H1U2LP1610-7" device="0603DIODE12V"/>
+<part name="H5" library="mount" deviceset="#4-BARE_MOUNTING_HOLE" device="/.300"/>
+<part name="H6" library="mount" deviceset="#4-BARE_MOUNTING_HOLE" device="/.300"/>
+<part name="H7" library="mount" deviceset="#4-BARE_MOUNTING_HOLE" device="/.300"/>
+<part name="H8" library="mount" deviceset="#4-BARE_MOUNTING_HOLE" device="/.300"/>
 </parts>
 <sheets>
@@
 <attribute name="VALUE" x="158.115" y="42.545" size="1.778" layer="96"/>
 </instance>
-<instance part="H1" gate="G$1" x="20.32" y="22.86" smashed="yes"/>
-<instance part="H2" gate="G$1" x="30.48" y="22.86" smashed="yes"/>
-<instance part="H3" gate="G$1" x="20.32" y="17.78" smashed="yes"/>
-<instance part="H4" gate="G$1" x="30.48" y="17.78" smashed="yes"/>
 <instance part="TP1" gate="G$1" x="68.58" y="335.28" smashed="yes" rot="R90">
 <attribute name="NAME" x="66.04" y="332.74" size="1.778" layer="95" font="vector" rot="R90"/>
@@
 <attribute name="VALUE" x="78.74" y="337.82" size="1.778" layer="96" rot="R270"/>
 </instance>
+<instance part="H5" gate="MT" x="50.038" y="17.018" smashed="yes">
+<attribute name="NAME" x="51.308" y="19.558" size="1.27" layer="95"/>
+<attribute name="VALUE" x="52.578" y="14.478" size="1.27" layer="96" display="off"/>
+</instance>
+<instance part="H6" gate="MT" x="50.038" y="24.638" smashed="yes">
+<attribute name="NAME" x="51.308" y="27.178" size="1.27" layer="95"/>
+<attribute name="VALUE" x="52.578" y="22.098" size="1.27" layer="96" display="off"/>
+</instance>
+<instance part="H7" gate="MT" x="62.738" y="24.638" smashed="yes">
+<attribute name="NAME" x="64.008" y="27.178" size="1.27" layer="95"/>
+<attribute name="VALUE" x="65.278" y="22.098" size="1.27" layer="96" display="off"/>
+</instance>
+<instance part="H8" gate="MT" x="62.738" y="17.018" smashed="yes">
+<attribute name="NAME" x="64.008" y="19.558" size="1.27" layer="95"/>
+<attribute name="VALUE" x="65.278" y="14.478" size="1.27" layer="96" display="off"/>
+</instance>
 </instances>

Commit message: Added Attributes to TP-board
Parts:
- C1: DIS (none) -> Digi-Key; DPN (none) -> 1276-1244-1-ND; MFR (none) -> Samsung Electro-Mechanics; MPN (none) -> CL21A475KAQNNNE
- C10, C19, C2, C20, C22, C7, C8, C9: DIS (none) -> Digi-Key; DPN (none) -> 478-12790-1-ND; MFR (none) -> AVX Corporation; MPN (none) -> 08055D104KAT2A
- C11, C4: DIS (none) -> Digi-Key; DPN (none) -> 445-14445-1-ND; MFR (none) -> TDK Corporation; MPN (none) -> C2012X5R2E103K125AA
- C12, C5: DIS (none) -> Digi-Key; DPN (none) -> 1276-2395-1-ND; MFR (none) -> Samsung Electro-Mechanics; MPN (none) -> CL21A105KACLNNC
- C13, C6: DIS (none) -> Digi-Key; DPN (none) -> 1276-6458-1-ND; MFR (none) -> Samsung Electro-Mechanics; MPN (none) -> CL21A225KAFNNNG
- C14, C15, C16, C17: DIS (none) -> Digi-Key; DPN (none) -> 399-7139-1-ND; MFR (none) -> KEMET; MPN (none) -> C0805C121KDRACTU
- C18, C23, C24, C25, C26, C27, C28, C29: DIS (none) -> Digi-Key; DPN (none) -> 732-8046-1-ND; MFR (none) -> Würth Elektronik; MPN (none) -> 885012207054
- C3: DIS (none) -> Digi-Key; DPN (none) -> 1276-6786-1-ND; MFR (none) -> Samsung Electro-Mechanics; MPN (none) -> CL21A226KPCLRNC
- CR1: DIS (none) -> Digi-Key; DPN (none) -> 1N4148W-FDICT-ND; MFR (none) -> Diodes Incorporated; MPN (none) -> 1N4148W-7-F
- D1: DIS (none) -> Digi-Key; DPN (none) -> 1655-1342-1-ND; MFR (none) -> SMC Diode Solutions; MPN (none) -> 10BQ060TR
- D10, D11, D12, D13, D14, D15, D16, D2, D3, D4, D5, D6, D7, D8: DIS (none) -> Digi-Key; DPN (none) -> D5V0H1U2LP1610-7DICT-ND; MFR (none) -> Diodes Incorporated; MPN (none) -> D5V0H1U2LP1610-7
- D9: DIS (none) -> Digi-Key; DPN (none) -> D12V0H1U2LP1610-7DICT-ND; MFR (none) -> Diodes Incorporated; MPN (none) -> D12V0H1U2LP1610-7
- J1: DIS (none) -> Digi-Key; DPN (none) -> 900-0022232021-ND; MFR (none) -> Molex; MPN (none) -> 22232021
- J2: DIS (none) -> Digi-Key; DPN (none) -> WM4203-ND; MFR (none) -> Molex; MPN (none) -> 0022232051
- J4, J5, J6, J7: DIS (none) -> Digi-Key; DPN (none) -> WM4202-ND; MFR (none) -> Molex; MPN (none) -> 0022232041
- R13, R18, R19, R20: DIS (none) -> Digi-Key; DPN (none) -> 311-1.00KCRCT-ND; MFR (none) -> Yageo; MPN (none) -> RC0805FR-071KL
- R14: DIS (none) -> Digi-Key; DPN (none) -> RNCP0805FTD19K1CT-ND; MFR (none) -> Stackpole Electronics Inc; MPN (none) -> RNCP0805FTD19K1
- R16: DIS (none) -> Digi-Key; DPN (none) -> 2019-RK73H2ATTD1243FCT-ND; MFR (none) -> KOA Speer Electronics, Inc.; MPN (none) -> RK73H2ATTD1243F
- R17: DIS (none) -> Digi-Key; DPN (none) -> 2019-RK73H2ATTD4993FCT-ND; MFR (none) -> KOA Speer Electronics, Inc.; MPN (none) -> RK73H2ATTD4993F
- U$1: DIS (none) -> Digi-Key; DPN (none) -> 1589-1120-1-ND; MFR (none) -> Monolithic Power Systems Inc.; MPN (none) -> MP2456GJ-P
- U$2: DIS (none) -> Digi-Key; DPN (none) -> 445-174699-1-ND; MFR (none) -> TDK Corporation; MPN (none) -> CLF5030NIT-100M-D
- U1, U2, U3, U4: DIS (none) -> Digi-Key; DPN (none) -> INA126PA-ND; MFR (none) -> Texas Instruments; MPN (none) -> INA126PA
- U5: DIS (none) -> Digi-Key; DPN (none) -> LP2985AIM5-3.3/NOPBCT-ND; MFR (none) -> Texas Instruments; MPN (none) -> LP2985AIM5-3.3/NOPB
- U6: DIS (none) -> Digi-Key; DPN (none) -> LP2985AIM5-5.0/NOPBCT-ND; MFR (none) -> Texas Instruments; MPN (none) -> LP2985AIM5-5.0/NOPB
