File: TSAR_Actuator_Controller.brd (EAGLE design)
At the start: 152.5 x 158.8 mm, 143 parts, among them Q1 220mA/50V/3.5Ω, Q10 220mA/50V/3.5Ω, Q11 IRF9530, Q12 220mA/50V/3.5Ω, Q13 IRF9530, Q14 220mA/50V/3.5Ω, Q15 IRF9530, Q16 220mA/50V/3.5Ω, Q17 IRF9530, Q18 220mA/50V/3.5Ω, Q19 IRF9530, Q2 IRF9530, Q20 220mA/50V/3.5Ω, Q3 IRF9530, Q4 220mA/50V/3.5Ω, Q5 IRF9530, Q6 220mA/50V/3.5Ω, Q7 IRF9530, Q8 220mA/50V/3.5Ω, Q9 IRF9530

Commit message: Corrected Morpho Connector Position Again.
Parts:
- moved CN7 1.27 mm to (39.4, 88.9)
- moved CN10 1.27 mm to (100.3, 88.9)
Routing:
- net SOL_GPIO_5: track 21.3 -> 20.0 mm
- net TBD_SENSOR_6: track 101.8 -> 103.0 mm
- net TBD_SENSOR_1: track 79.3 -> 78.0 mm
- net TBD_SENSOR_4: track 39.2 -> 37.9 mm
- net +5V: track 66.2 -> 67.5 mm
- net TBD_SENSOR_8: track 119.4 -> 120.7 mm
- net TBD_SENSOR_7: track 107.5 -> 108.8 mm
- net TBD_SENSOR_5: track 98.7 -> 100.0 mm
- net TBD_SENSOR_2: track 125.6 -> 126.8 mm
- net TBD_SENSOR_0: track 90.7 -> 89.4 mm
- net SOL_GPIO_4: track 24.1 -> 23.0 mm
- net TBD_SENSOR_3: track 91.4 -> 92.4 mm
- net TBD_SENSOR_9: track 72.4 -> 73.4 mm
- net EVAL-3V3: track 6.50 -> 7.34 mm
- net SOL_GPIO_2: track 63.9 -> 63.3 mm
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