File: actuator-controller/TSAR_Actuator_Controller.brd (EAGLE design)
At the start: 160 x 100 mm, 140 parts, among them J1 282834-2, J10 282834-2, J11 282834-2, J12 282834-2, J13 282834-2, J14 282834-2, J15 282834-2, J16 282834-2, J17 282834-2, J18 282834-2, J19 282834-2, J2 282834-2, J20 282834-2, J21 282834-2, J3 282834-2, J4 282834-2, J5 282834-2, J6 282834-2, J7 282834-2, J8 282834-2, J9 282834-2, Q1 BUZ11BV, Q10 BUZ11BV, Q2 BUZ11BV, Q3 BUZ11BV, Q4 BUZ11BV, Q5 BUZ11BV, Q6 BUZ11BV, Q7 BUZ11BV, Q8 BUZ11BV, Q9 BUZ11BV

Commit message: Updated Schematic after last design review.
Updated according to Andrews input.
Parts:
- removed C10, C25, C26, C27, C28, C29, C30, C31, C32, C33, C34, C35, C36, C37, C38, C39, C8, C9: 120pF, rcl:C0805
- removed D10, D11, D12, D6, D7, D8, D9: BAS40, diode:SOT23
- removed J10, J11, J12, J13, J14, J15, J16, J17, J18, J19, J5, J6, J7, J8, J9: 282834-2, TSAR_Controller:CONN_282834-2
- removed Q10, Q9: BUZ11BV, transistor-power:TO220BV
- removed R32, R33, R34, R35, R36, R37, R44, R49: 28K, rcl:R0603
- removed R38, R39, R40, R41, R42, R43, R45, R46, R47, R48: 1K, rcl:R0603
- removed TVSD_12, TVSD_13, TVSD_14, TVSD_15, TVSD_16, TVSD_17, TVSD_18, TVSD_19, TVSD_20, TVSD_21, TVSD_22, TVSD_23, TVSD_24, TVSD_25, TVSD_26, TVSD_27, TVSD_28, TVSD_29, TVSD_30: DF2B5M4CT,L3F, TSAR_Controller:SOD-882(SOT2)
- added C1, C11, C12, C13, C14, C15, C17, C18, C19, C40, C41: 120pF, rcl:C0805
- added D13: BAS40, diode:SOT23
- added J23, J24, J25, J26, J27, J29, J30, J31, J32, J33: 282834-2, TSAR_Controller:CONN_282834-2
- added R1, R10, R11, R12, R13, R14, R15, R50, R51, R52, R8, R9: 1K, rcl:R0603
- added R7: 28K, rcl:R0603
- added TVSD_1, TVSD_2, TVSD_3, TVSD_31, TVSD_32, TVSD_33, TVSD_4, TVSD_5, TVSD_6, TVSD_7, TVSD_8, TVSD_9: DF2B5M4CT,L3F, TSAR_Controller:SOD-882(SOT2)
- Q1, Q3, Q5, Q7: value BUZ11BV -> MMBT3904-TP; device transistor-power:TO220BV -> TSAR_Controller:SOT-23_MCC
- Q2, Q4, Q6, Q8: value BUZ11BV -> IRF9530
- R16, R5: value 500k -> 10K
- R2, R22, R26: value 1K -> 3K
- R21, R25, R29: value 1K -> 28K
- R23, R27, R3: value 1K -> 4.7K
- R30: value 28K -> 3K
- R31: value 28K -> 4.7K
- R4, R6: value 0 -> NP
- moved Q8 382.3 mm to (-47.0, -495.3)
- moved Q6 359.4 mm to (-47.0, -467.4)
- moved Q7 332.7 mm to (-48.3, -519.4)
- moved Q3 330.2 mm to (-48.3, -463.6)
- moved D5 308.8 mm to (-38.1, -497.8)
- moved J3 301.0 mm to (-47.0, -480.1)
- moved Q4 262.9 mm to (-47.0, -439.4)
- moved Q5 236.2 mm to (-48.3, -491.5)
- moved J1 228.6 mm to (-47.0, -410.2)
- moved J21 222.3 mm to (-47.0, 443.2)
- moved J20 222.2 mm to (-47.0, 435.6)
- moved Q2 222.2 mm to (-47.0, -429.3)
- moved J2 219.7 mm to (-47.0, -452.1)
- moved J4 214.6 mm to (-47.0, -508.0)
- moved D3 204.8 mm to (-38.1, -442.0)
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Connections:
- net 5V renamed +5V
- removed net 12V: D10.3, D11.3, D12.3, D3.3, D4.3, D5.3, D6.3, D7.3, D8.3, D9.3, J1.1, J10.1, J11.1, J17.1, J18.1, J2.1, J4.1, J5.1, J7.1, J9.1
- removed net 24V: C21.1, C4.1, C5.1, C6.1, R16.1, R5.1, U$3.P$5, U$4.P$5
- removed net 3V3: C24.1, CR2.2, U$5.2
- removed net N$20: D6.1, R33.2
- removed net N$21: Q5.G, R28.2
- removed net N$22: J5.2, Q5.D
- removed net N$23: D7.1, R34.2
- removed net N$24: D5.1, R32.2
- removed net N$25: Q3.G, R27.2
- removed net N$26: J8.1, R29.2
- removed net N$27: J9.2, Q6.D
- removed net N$28: D8.1, R35.2
- removed net N$29: Q6.G, R23.2
- removed net N$30: J10.2, Q7.D
- removed net N$31: D9.1, R36.2
- removed net N$32: Q7.G, R24.2
- removed net N$33: J11.2, Q8.D
- removed net N$34: D10.1, R37.2
- removed net N$35: Q8.G, R25.2
- removed net N$36: J12.1, R38.2
- removed net N$37: J13.1, R39.2
- removed net N$38: J14.1, R40.2
- removed net N$39: J15.1, R41.2
- removed net N$40: J16.1, R42.2
- removed net N$41: J18.2, Q9.D
- removed net N$42: D11.1, R44.2
- removed net N$43: Q9.G, R43.2
- removed net N$44: R45.2
- removed net N$45: R46.2
- removed net N$46: R47.2
- removed net N$47: Q10.G, R48.2
- removed net N$48: J17.2, Q10.D
- removed net N$49: D12.1, R49.2
- removed net N$50: J19.1
- removed net N$51: J20.1
- removed net N$52: J21.1
- removed net VLV_FB_0: C38.1, CN7.28, R47.1, TVSD_29.P$1
- removed net VLV_FB_1: C37.1, CN7.30, R46.1, TVSD_28.P$1
- removed net VLV_FB_10: C34.1, CN10.19, R42.1, TVSD_25.P$1
- removed net VLV_FB_2: C3.1, CN10.34, R3.1, TVSD_11.P$1
- removed net VLV_FB_3: C26.1, CN10.6, R26.1, TVSD_17.P$1
- removed net VLV_FB_4: C36.1, CN7.32, R45.1, TVSD_27.P$1
- removed net VLV_FB_5: C29.1, CN10.11, R38.1, TVSD_21.P$1
- removed net VLV_FB_6: C30.1, CN10.13, R39.1, TVSD_22.P$1
- removed net VLV_FB_7: C31.1, CN10.15, R40.1, TVSD_23.P$1
- removed net VLV_FB_8: C33.1, CN10.17, R41.1, TVSD_24.P$1
- new net +12V: C21.1, C4.1, C5.1, C6.1, J20.2, J21.1, Q2.S, Q4.S, Q6.S, Q8.S, R16.1, R23.2, R27.2, R3.2, R31.2, R5.1, U$3.P$5, U$4.P$5
- new net N$54: D13.1, R7.2
- new net N$56: R8.2
- new net N$57: J23.1
- new net N$58: R9.2
- new net N$59: J24.1
- new net N$60: R10.2
- new net N$61: R11.2
- new net N$62: J25.1
- new net N$63: J26.1
- new net N$64: R12.2
- new net N$65: J27.1
- new net N$68: R14.2
- new net N$69: J29.1
- new net N$70: R15.2
- new net N$71: J30.1
- new net N$72: R50.2
- new net N$73: J31.1
- new net N$74: R51.2
- new net N$75: J32.1
- new net N$76: R52.2
- new net N$77: J33.1
- new net SOL_GPIO_03: CN10.19
- new net SOL_GPIO_10: D13.3, J1.1, Q2.D
- new net SOL_GPIO_14: D4.3, J3.1, Q6.D
- new net SOL_GPIO_15: C7.1, R28.1, TVSD_11.P$1
- new net SOL_GPIO_16: D5.3, J4.1, Q8.D
- new net SOL_GPIO_4: CN10.4
- new net TBD_SENSOR_0: C1.1, C12.1, C13.1, C14.1, C15.1, C17.1, C18.1, C19.1, C40.1, C41.1, CN7.28, R10.1, R11.1, R12.1, R14.1, R15.1, R50.1, R51.1, R52.1, R8.1, R9.1, TVSD_1.P$1, TVSD_3.P$1, TVSD_31.P$1, TVSD_32.P$1, TVSD_33.P$1, TVSD_4.P$1, TVSD_5.P$1, TVSD_6.P$1, TVSD_8.P$1, TVSD_9.P$1
- new net TBD_SENSOR_1: CN7.30
- new net TBD_SENSOR_2: CN10.34
- new net TBD_SENSOR_3: CN10.6
- new net TBD_SENSOR_4: CN7.32
- new net TBD_SENSOR_5: CN10.11
- new net TBD_SENSOR_6: CN10.13
- new net TBD_SENSOR_7: CN10.15
- new net TBD_SENSOR_8: CN10.17
- new net TBD_SENSOR_9: CN7.34
- net 48V1: now also C24.1, CR2.2, U$5.2
- net GND: now also C1.2, C11.2, C12.2, C13.2, C14.2, C15.2, C17.2, C18.2, C19.2, C40.2, C41.2, J1.2, J2.2, J20.1, J23.2, J24.2, J25.2, J26.2, J27.2, J29.2, J30.2, J31.2, J32.2, J33.2, J4.2, Q1.2, Q3.2, Q5.2, Q7.2, R2.1, R21.1, R22.1, R25.1, R26.1, R29.1, R7.1, TVSD_1.P$2, TVSD_2.P$2, TVSD_3.P$2, TVSD_31.P$2, TVSD_32.P$2, TVSD_33.P$2, TVSD_4.P$2, TVSD_5.P$2, TVSD_6.P$2, TVSD_7.P$2, TVSD_8.P$2, TVSD_9.P$2; no longer C10.2, C25.2, C26.2, C27.2, C28.2, C29.2, C30.2, C31.2, C32.2, C33.2, C34.2, C35.2, C36.2, C37.2, C38.2, C39.2, C8.2, C9.2, J12.2, J13.2, J14.2, J15.2, J16.2, J19.2, J20.2, J6.2, J8.2, Q1.S, Q10.S, Q2.S, Q3.S, Q4.S, Q5.S, Q6.S, Q7.S, Q8.S, Q9.S, R31.1, R32.1, R33.1, R34.1, R35.1, R36.1, R37.1, R44.1, R49.1, TVSD_12.P$2, TVSD_13.P$2, TVSD_14.P$2, TVSD_15.P$2, TVSD_16.P$2, TVSD_17.P$2, TVSD_18.P$2, TVSD_19.P$2, TVSD_20.P$2, TVSD_21.P$2, TVSD_22.P$2, TVSD_23.P$2, TVSD_24.P$2, TVSD_25.P$2, TVSD_26.P$2, TVSD_27.P$2, TVSD_28.P$2, TVSD_29.P$2, TVSD_30.P$2
- net N$1: now also Q1.3, Q2.G, R3.1; no longer Q1.G, R22.2
- net N$10: now also Q3.1, R13.2, R22.2; no longer Q4.G, R2.2
- net N$11: now also Q3.3, Q4.G, R23.1; no longer Q2.G, R21.2
- net N$12: now also D4.1, R25.2; no longer J2.2, Q2.D
- net N$13: now also Q5.1, R24.2, R26.2; no longer D4.1, R31.2
- net N$14: now also Q5.3, Q6.G, R27.1; no longer J3.1, R3.2
- net N$15: now also D5.1, R29.2; no longer J6.1, R26.2
- net N$16: now also Q7.1, R28.2, R30.2; no longer J7.2, Q3.D
- net N$18: now also Q7.3, Q8.G, R31.1; no longer J4.2, Q4.D
- net N$2: now also Q1.1, R1.2, R2.2; no longer J1.2, Q1.D
- net N$9: now also R21.2; no longer R30.2
- net SOL_GPIO_0: no longer C9.1, R23.1, TVSD_14.P$1
- net SOL_GPIO_1: no longer C7.1, R21.1, TVSD_12.P$1
- net SOL_GPIO_11: now also C2.1, R13.1, TVSD_7.P$1; no longer C27.1, CN10.4, R27.1, TVSD_18.P$1
- net SOL_GPIO_12: now also D3.3, J2.1, Q4.D; no longer C28.1, R29.1, TVSD_20.P$1
- net SOL_GPIO_13: now also C3.1, R24.1, TVSD_10.P$1; no longer C39.1, CN7.34, R48.1, TVSD_30.P$1
- net SOL_GPIO_2: now also C11.1, R1.1, TVSD_2.P$1; no longer C8.1, R22.1, TVSD_13.P$1
- net SOL_GPIO_5: no longer C35.1, R43.1, TVSD_26.P$1
- net SOL_GPIO_6: no longer C25.1, R25.1, TVSD_16.P$1
- net SOL_GPIO_7: no longer C32.1, R28.1, TVSD_19.P$1
- net SOL_GPIO_8: no longer C10.1, R24.1, TVSD_15.P$1
- net SOL_GPIO_9: no longer C2.1, R2.1, TVSD_10.P$1

Commit message: Replaced Resistors and 5V TVS Diodes.
Changed resistors to 0805 to be the same size as the caps.
Changed to a standard sized TVS Diode footprint.
Began Board layouts.
Parts:
- removed C11, C2, C3, C7: 120pF, rcl:C0805
- removed J1, J2, J23, J24, J25, J26, J27, J29, J3, J30, J31, J32, J33, J4: 282834-2, TSAR_Controller:CONN_282834-2
- removed R50, R51, R52: 1K, rcl:R0603
- removed TVSD_1, TVSD_10, TVSD_11, TVSD_2, TVSD_3, TVSD_31, TVSD_32, TVSD_33, TVSD_4, TVSD_5, TVSD_6, TVSD_7, TVSD_8, TVSD_9: DF2B5M4CT,L3F, TSAR_Controller:SOD-882(SOT2)
- added D10, D11, D6, D7, D8, D9: BAS40, diode:SOT23
- added D12, D14, D15, D16, D17, D18, D19, D20, D21, D22: 5V, SparkFun-DiscreteSemi:0603
- added Q10, Q12, Q14, Q16, Q18, Q20: 220mA/50V/3.5Ω, SparkFun-DiscreteSemi:SOT23-3
- added Q11, Q13, Q15, Q17, Q19, Q9: IRF9530, transistor-power:TO220BV
- added R32, R35, R38, R41, R44: 10k, rcl:R0805
- added R33, R36, R39, R42, R45: 28k, rcl:R0805
- added R34, R37, R40, R43: 4.7K, rcl:R0805
- added R46, R47, R48: 1k, rcl:R0805
- added SENSOR_0, SENSOR_1, SENSOR_2, SENSOR_3, SENSOR_4, SENSOR_5, SENSOR_6, SENSOR_7, SENSOR_8, SENSOR_9, SOLENOID_0, SOLENOID_1, SOLENOID_2, SOLENOID_3, SOLENOID_4, SOLENOID_5, SOLENOID_6, SOLENOID_7, SOLENOID_8, SOLENOID_9: 282834-2, TSAR_Controller:CONN_282834-2
- Q1: value MMBT3904-TP -> 220mA/50V/3.5Ω; device TSAR_Controller:SOT-23_MCC -> SparkFun-DiscreteSemi:SOT23-3
- Q3, Q5, Q7: value MMBT3904-TP -> IRF9530; device TSAR_Controller:SOT-23_MCC -> transistor-power:TO220BV
- Q4, Q6, Q8: value IRF9530 -> 220mA/50V/3.5Ω; device transistor-power:TO220BV -> SparkFun-DiscreteSemi:SOT23-3
- R1: value 1K -> 10K; device rcl:R0603 -> rcl:R0805
- R10, R11, R12, R14, R15, R8, R9: value 1K -> 1k; device rcl:R0603 -> rcl:R0805
- R13: value 1K -> NP; device rcl:R0603 -> rcl:R0805
- R16: value 10K -> 10k; device rcl:R0603 -> rcl:R0805
- R17: value (none) -> 10K; device rcl:R0603 -> rcl:R0805
- R18: value (none) -> NP; device rcl:R0603 -> rcl:R0805
- R19: value 23.7K -> 10k; device rcl:R0603 -> rcl:R0805
- R2, R22: value 3K -> 4.7K; device rcl:R0603 -> rcl:R0805
- R20: value 124K -> 33k; device rcl:R0603 -> rcl:R0805
- R21, R7: value 28K -> 28k; device rcl:R0603 -> rcl:R0805
- R23, R3: value 4.7K -> 10k; device rcl:R0603 -> rcl:R0805
- R24: value 1K -> 28k; device rcl:R0603 -> rcl:R0805
- R25: value 28K -> 4.7K; device rcl:R0603 -> rcl:R0805
- R26: value 3K -> 10k; device rcl:R0603 -> rcl:R0805
- R27: value 4.7K -> 28k; device rcl:R0603 -> rcl:R0805
- R28: value 1K -> 4.7K; device rcl:R0603 -> rcl:R0805
- R29: value 28K -> 10k; device rcl:R0603 -> rcl:R0805
- R30: value 3K -> 28k; device rcl:R0603 -> rcl:R0805
- R31: device rcl:R0603 -> rcl:R0805
- R4: value NP -> 124k; device rcl:R0603 -> rcl:R0805
- R5: value 10K -> 23.7k; device rcl:R0603 -> rcl:R0805
- R6: value NP -> 4.7K; device rcl:R0603 -> rcl:R0805
- moved Q7 560.5 mm to (-91.4, 39.4)
- moved R28 560.3 mm to (-101.6, 43.2)
- moved Q5 557.9 mm to (-91.4, 64.8)
- moved R31 556.3 mm to (-134.6, 35.6)
- moved R29 555.0 mm to (-115.6, 35.6)
- moved R30 554.8 mm to (-109.2, 35.6)
- moved R13 534.8 mm to (-58.4, 76.2)
- moved Q8 533.3 mm to (-82.5, 36.8)
- moved R24 532.0 mm to (-81.3, 44.5)
- moved Q6 530.8 mm to (-82.5, 62.2)
- moved D5 527.5 mm to (-94.0, 26.7)
- moved D4 525.0 mm to (-94.0, 52.1)
- moved Q4 520.8 mm to (-8.89, 80.0)
- moved R25 508.3 mm to (-94.0, 19.1)
- moved R26 508.1 mm to (-87.6, 19.1)
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Connections:
- removed net 48V1: C24.1, CR2.2, R18.1, U$5.2
- removed net 48V2: R20.1
- removed net EVAL-5V: CN7.18
- removed net N$56: R8.2
- removed net N$57: J23.1
- removed net N$58: R9.2
- removed net N$59: J24.1
- removed net N$60: R10.2
- removed net N$61: R11.2
- removed net N$62: J25.1
- removed net N$63: J26.1
- removed net N$64: R12.2
- removed net N$65: J27.1
- removed net N$68: R14.2
- removed net N$69: J29.1
- removed net N$70: R15.2
- removed net N$71: J30.1
- removed net N$72: R50.2
- removed net N$73: J31.1
- removed net N$74: R51.2
- removed net N$75: J32.1
- removed net N$76: R52.2
- removed net N$77: J33.1
- new net +3V3: C24.1, CR2.2, R19.2, U$5.2
- new net N$20: R48.2, SENSOR_9.1
- new net N$21: C40.1, D22.2, R15.1
- new net N$22: C1.1, D17.2, R11.1
- new net N$23: C12.1, D16.2, R8.1
- new net N$24: C14.1, D15.2, R10.1
- new net N$25: C15.1, D12.2, R12.1
- new net N$26: C17.1, D19.2, R47.1
- new net N$27: C18.1, D20.2, R14.1
- new net N$28: C19.1, D21.2, R9.1
- new net N$29: D3.1, R7.2
- new net N$30: Q3.G, Q4.3, R2.1
- new net N$31: D4.1, R24.2
- new net N$32: Q5.G, Q6.3, R22.1
- new net N$33: D5.1, R27.2
- new net N$34: Q7.G, Q8.3, R25.1
- new net N$35: Q1.1, R16.2
- new net N$36: D6.1, R30.2
- new net N$37: Q10.3, Q9.G, R28.1
- new net N$38: D7.1, R33.2
- new net N$39: Q11.G, Q12.3, R31.1
- new net N$40: D8.1, R36.2
- new net N$41: Q13.G, Q14.3, R34.1
- new net N$42: D9.1, R39.2
- new net N$43: Q15.G, Q16.3, R37.1
- new net N$44: D10.1, R42.2
- new net N$45: Q17.G, Q18.3, R40.1
- new net N$46: D11.1, R45.2
- new net N$47: Q19.G, Q20.3, R43.1
- new net SOL_GPIO_17: D9.3, Q15.D, SOLENOID_7.1
- new net SOL_GPIO_18: D10.3, Q17.D, SOLENOID_8.1
- new net SOL_GPIO_19: D11.3, Q19.D, SOLENOID_9.1
- new net SOL_GPIO_3: CN10.19
- new net V+: J21.1, Q11.S, Q13.S, Q15.S, Q17.S, Q19.S, Q2.S, Q3.S, Q5.S, Q7.S, Q9.S, R2.2, R22.2, R25.2, R28.2, R31.2, R34.2, R37.2, R40.2, R43.2, R6.2
- net +12V: now also R1.2, R17.2; no longer J21.1, Q2.S, Q4.S, Q6.S, Q8.S, R16.1, R23.2, R27.2, R3.2, R31.2, R5.1
- net +5V: now also CN7.18, R4.2
- net GND: now also D12.1, D14.1, D15.1, D16.1, D17.1, D18.1, D19.1, D20.1, D21.1, D22.1, Q10.2, Q12.2, Q14.2, Q16.2, Q18.2, Q20.2, Q4.2, Q6.2, Q8.2, R13.1, R16.1, R18.1, R20.1, R23.1, R24.1, R27.1, R3.1, R32.1, R33.1, R35.1, R36.1, R38.1, R39.1, R41.1, R42.1, R44.1, R45.1, R5.1, SENSOR_0.2, SENSOR_1.2, SENSOR_2.2, SENSOR_3.2, SENSOR_4.2, SENSOR_5.2, SENSOR_6.2, SENSOR_7.2, SENSOR_8.2, SENSOR_9.2, SOLENOID_0.2, SOLENOID_1.2, SOLENOID_2.2, SOLENOID_3.2, SOLENOID_4.2, SOLENOID_5.2, SOLENOID_6.2, SOLENOID_7.2, SOLENOID_8.2, SOLENOID_9.2; no longer C11.2, C2.2, C3.2, C7.2, J1.2, J2.2, J23.2, J24.2, J25.2, J26.2, J27.2, J29.2, J3.2, J30.2, J31.2, J32.2, J33.2, J4.2, Q3.2, Q5.2, Q7.2, R17.2, R19.2, R2.1, R22.1, R25.1, R4.2, R6.2, TVSD_1.P$2, TVSD_10.P$2, TVSD_11.P$2, TVSD_2.P$2, TVSD_3.P$2, TVSD_31.P$2, TVSD_32.P$2, TVSD_33.P$2, TVSD_4.P$2, TVSD_5.P$2, TVSD_6.P$2, TVSD_7.P$2, TVSD_8.P$2, TVSD_9.P$2
- net N$1: now also R6.1; no longer R3.1
- net N$10: now also R11.2, SENSOR_1.1; no longer Q3.1, R13.2, R22.2
- net N$11: now also R8.2, SENSOR_2.1; no longer Q3.3, Q4.G, R23.1
- net N$12: now also R10.2, SENSOR_3.1; no longer D4.1, R25.2
- net N$13: now also R12.2, SENSOR_4.1; no longer Q5.1, R24.2, R26.2
- net N$14: now also R47.2, SENSOR_5.1; no longer Q5.3, Q6.G, R27.1
- net N$15: now also R14.2, SENSOR_6.1; no longer D5.1, R29.2
- net N$16: now also R9.2, SENSOR_7.1; no longer Q7.1, R28.2, R30.2
- net N$17: now also R19.1, R20.2; no longer R17.1, R18.2
- net N$18: now also R15.2, SENSOR_8.1; no longer Q7.3, Q8.G, R31.1
- net N$19: now also R4.1, R5.2; no longer R19.1, R20.2
- net N$2: now also C41.1, D14.2, R48.1; no longer Q1.1, R1.2, R2.2
- net N$3: now also R1.1, R13.2; no longer R4.1, R5.2
- net N$5: now also R17.1, R18.2; no longer R16.2, R6.1
- net N$54: now also R21.2; no longer R7.2
- net N$9: now also R46.2, SENSOR_0.1; no longer D3.1, R21.2
- net SOL_GPIO_03: now also Q8.1, R26.2; no longer CN10.19
- net SOL_GPIO_1: now also Q4.1, R3.2
- net SOL_GPIO_10: now also SOLENOID_0.1; no longer J1.1
- net SOL_GPIO_11: now also D3.3, Q3.D, SOLENOID_1.1; no longer C2.1, R13.1, TVSD_7.P$1
- net SOL_GPIO_12: now also D4.3, Q5.D, SOLENOID_2.1; no longer D3.3, J2.1, Q4.D
- net SOL_GPIO_13: now also D5.3, Q7.D, SOLENOID_3.1; no longer C3.1, R24.1, TVSD_10.P$1
- net SOL_GPIO_14: now also D6.3, Q9.D, SOLENOID_4.1; no longer D4.3, J3.1, Q6.D
- net SOL_GPIO_15: now also D7.3, Q11.D, SOLENOID_5.1; no longer C7.1, R28.1, TVSD_11.P$1
- net SOL_GPIO_16: now also D8.3, Q13.D, SOLENOID_6.1; no longer D5.3, J4.1, Q8.D
- net SOL_GPIO_2: now also Q6.1, R23.2; no longer C11.1, R1.1, TVSD_2.P$1
- net SOL_GPIO_4: now also Q10.1, R29.2
- net SOL_GPIO_5: now also Q12.1, R32.2
- net SOL_GPIO_6: now also Q14.1, R35.2
- net SOL_GPIO_7: now also Q16.1, R38.2
- net SOL_GPIO_8: now also Q18.1, R41.2
- net SOL_GPIO_9: now also Q20.1, R44.2
- net TBD_SENSOR_0: now also D18.2, R46.1; no longer C1.1, C12.1, C14.1, C15.1, C17.1, C18.1, C19.1, C40.1, C41.1, R10.1, R11.1, R12.1, R14.1, R15.1, R50.1, R51.1, R52.1, R8.1, R9.1, TVSD_1.P$1, TVSD_3.P$1, TVSD_31.P$1, TVSD_32.P$1, TVSD_33.P$1, TVSD_4.P$1, TVSD_5.P$1, TVSD_6.P$1, TVSD_8.P$1, TVSD_9.P$1

Commit message: Adjusted Board Layout
Parts:
- added H1, H2, H3, H4: STAND-OFF, SparkFun-Hardware:STAND-OFF
- moved SOLENOID_5 285.8 mm to (153.7, 36.8), turned to 270 degrees
- moved SOLENOID_8 285.8 mm to (153.7, 0.00), turned to 270 degrees
- moved SOLENOID_6 275.0 mm to (153.7, 24.1), turned to 270 degrees
- moved SOLENOID_9 274.7 mm to (153.7, -11.4), turned to 270 degrees
- moved SOLENOID_7 264.7 mm to (153.7, 12.7), turned to 270 degrees
- moved SOLENOID_4 262.9 mm to (153.7, 47.0), turned to 270 degrees
- moved SOLENOID_3 239.4 mm to (153.7, 57.1), turned to 270 degrees
- moved SOLENOID_2 238.1 mm to (153.7, 68.6), turned to 270 degrees
- moved SOLENOID_1 216.7 mm to (153.7, 80.0), turned to 270 degrees
- moved J21 167.5 mm to (15.2, -10.2), turned to 180 degrees
- moved J20 153.3 mm to (15.2, -2.54), turned to 180 degrees
- moved C23 131.6 mm to (-95.2, -14.0)
- moved C24 131.6 mm to (-95.2, -19.1)
- moved D1 131.6 mm to (-94.0, -25.4)
- moved D2 131.6 mm to (-94.0, -30.5)
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Other:
- board size 160 x 100 mm -> 160 x 119 mm

Commit message: Completed initial board layout.
Parts:
- removed J20, J21: 282834-2, TSAR_Controller:CONN_282834-2
- removed U$3, U$4: MP2456GJ-P, TSAR_Controller:SOT6
- removed U$5, U$6: 10uH, TSAR_Controller:0.209"LX0.197"W(5.30MMX5.00MM)
- added 12V: 282834-2, TSAR_Controller:CONN_282834-2
- added 3V3_REG, 5V_REG: MP2456GJ-P, TSAR_Controller:SOT6
- added J1: (no value), SparkFun-Connectors:1X02_XTRA_BIG
- added L1, L2: 10uH, TSAR_Controller:0.209"LX0.197"W(5.30MMX5.00MM)
- moved SOLENOID_0 284.5 mm to (153.7, 104.1), turned to 270 degrees
- moved Q2 283.3 mm to (138.4, 106.7), turned to 270 degrees
- moved D7 282.2 mm to (147.4, 41.2)
- moved R33 277.6 mm to (142.8, 40.0)
- moved D10 276.9 mm to (147.3, 2.65)
- moved D8 275.3 mm to (147.4, 28.4)
- moved Q17 271.2 mm to (138.4, 3.81), turned to 270 degrees
- moved D11 270.6 mm to (147.8, -10.2)
- moved D9 268.8 mm to (147.1, 15.5)
- moved R31 265.2 mm to (130.6, 40.8), turned to 270 degrees
- moved R42 265.2 mm to (143.2, 1.48)
- moved R36 264.8 mm to (142.9, 27.2)
- moved R43 264.7 mm to (130.0, -10.4), turned to 270 degrees
- moved Q20 261.7 mm to (126.5, -6.41), turned to 270 degrees
- moved Q19 261.1 mm to (138.4, -8.89), turned to 270 degrees
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Connections:
- removed net N$2: C41.1, D14.2, R48.1
- removed net N$21: C40.1, D22.2, R15.1
- removed net N$22: C1.1, D17.2, R11.1
- removed net N$23: C12.1, D16.2, R8.1
- removed net N$24: C14.1, D15.2, R10.1
- removed net N$25: C15.1, D12.2, R12.1
- removed net N$26: C17.1, D19.2, R47.1
- removed net N$27: C18.1, D20.2, R14.1
- removed net N$28: C19.1, D21.2, R9.1
- removed net N$35: Q1.1, R16.2
- removed net SOL_GPIO_03: Q8.1, R26.2
- removed net V+: J21.1, Q11.S, Q13.S, Q15.S, Q17.S, Q19.S, Q2.S, Q3.S, Q5.S, Q7.S, Q9.S, R2.2, R22.2, R25.2, R28.2, R31.2, R34.2, R37.2, R40.2, R43.2, R6.2
- new net VBATT: J1.1, Q11.S, Q13.S, Q15.S, Q17.S, Q19.S, Q2.S, Q3.S, Q5.S, Q7.S, Q9.S, R2.2, R22.2, R25.2, R28.2, R31.2, R34.2, R37.2, R40.2, R43.2, R6.2
- net +12V: now also 12V.2, 3V3_REG.P$5, 5V_REG.P$5; no longer J20.2, U$3.P$5, U$4.P$5
- net +3V3: now also L2.2; no longer U$5.2
- net +5V: now also L1.2; no longer U$6.2
- net GND: now also 12V.1, 3V3_REG.P$2, 5V_REG.P$2, J1.2; no longer J20.1, J21.2, U$3.P$2, U$4.P$2
- net N$17: now also 3V3_REG.P$3; no longer U$4.P$3
- net N$19: now also 5V_REG.P$3; no longer U$3.P$3
- net N$3: now also 5V_REG.P$4; no longer U$3.P$4
- net N$4: now also 5V_REG.P$1; no longer U$3.P$1
- net N$5: now also 3V3_REG.P$4; no longer U$4.P$4
- net N$6: now also 3V3_REG.P$1; no longer U$4.P$1
- net N$7: now also 3V3_REG.P$6, L2.1; no longer U$4.P$6, U$5.1
- net N$8: now also 5V_REG.P$6, L1.1; no longer U$3.P$6, U$6.1
- net SOL_GPIO_0: now also Q1.1, R16.2
- net SOL_GPIO_3: now also Q8.1, R26.2
- net TBD_SENSOR_1: now also C1.1, D17.2, R11.1
- net TBD_SENSOR_2: now also C12.1, D16.2, R8.1
- net TBD_SENSOR_3: now also C14.1, D15.2, R10.1
- net TBD_SENSOR_4: now also C15.1, D12.2, R12.1
- net TBD_SENSOR_5: now also C17.1, D19.2, R47.1
- net TBD_SENSOR_6: now also C18.1, D20.2, R14.1
- net TBD_SENSOR_7: now also C19.1, D21.2, R9.1
- net TBD_SENSOR_8: now also C40.1, D22.2, R15.1
- net TBD_SENSOR_9: now also C41.1, D14.2, R48.1
Routing:
- net VBATT: track 0.00 -> 234.7 mm
- net +12V: track 0.00 -> 35.0 mm
- net +5V: track 0.00 -> 22.0 mm
- net SOL_GPIO_11: track 0.00 -> 18.1 mm
- net SOL_GPIO_15: track 0.00 -> 18.1 mm
- net SOL_GPIO_16: track 0.00 -> 18.0 mm
- net SOL_GPIO_12: track 0.00 -> 18.0 mm
- net SOL_GPIO_19: track 0.00 -> 17.8 mm
- net SOL_GPIO_18: track 0.00 -> 17.8 mm
- net SOL_GPIO_13: track 0.00 -> 17.8 mm
- net SOL_GPIO_14: track 0.00 -> 17.8 mm
- net SOL_GPIO_10: track 0.00 -> 17.8 mm
- net SOL_GPIO_17: track 0.00 -> 17.5 mm
- net +3V3: track 0.00 -> 15.6 mm
- net N$7: track 0.00 -> 14.3 mm
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- added copper zone on layer 1, net +12V
- added copper zone on layer 1, net GND
- added copper zone on layer 16, net GND
- added copper zone on layer 1, net N$8
- added copper zone on layer 1, net VBATT
Other:
- board size 160 x 119 mm -> 170.2 x 154.9 mm
