File: actuator-controller/TSAR_Actuator_Controller.brd (EAGLE design)
At the start: 147.6 x 77.7 mm, 168 parts, among them Q1 220mA/50V/3.5Ω, Q10 220mA/50V/3.5Ω, Q11 IRF9530, Q12 220mA/50V/3.5Ω, Q13 IRF9530, Q14 220mA/50V/3.5Ω, Q15 IRF9530, Q16 220mA/50V/3.5Ω, Q17 IRF9530, Q18 220mA/50V/3.5Ω, Q19 IRF9530, Q2 IRF9530, Q20 220mA/50V/3.5Ω, Q3 IRF9530, Q4 220mA/50V/3.5Ω, Q5 IRF9530, Q6 220mA/50V/3.5Ω, Q7 IRF9530, Q8 220mA/50V/3.5Ω, Q9 IRF9530

Commit message: thick routes on AC board. protections on SFE
Parts:
- moved Q17 114.2 mm to (126.3, 9.18)
- moved Q13 102.5 mm to (126.3, 21.6)
- moved Q19 98.3 mm to (114.7, 9.18)
- moved Q9 91.6 mm to (126.3, 34.1)
- moved Q15 87.4 mm to (114.7, 21.7)
- moved Q5 81.8 mm to (126.3, 46.6)
- moved Q11 77.7 mm to (114.7, 34.2)
- moved Q3 75.2 mm to (126.3, 59.1)
- moved Q7 69.7 mm to (114.7, 46.7)
- moved 5V 64.2 mm to (6.48, 55.8), turned to 0 degrees
- moved Q2 62.2 mm to (114.7, 59.2)
- moved IGN. 59.9 mm to (131.6, 61.9)
- moved SOV_9. 59.6 mm to (131.6, 7.21)
- moved POE+ 55.9 mm to (6.48, 49.1), turned to 180 degrees
- moved SOV_1. 55.3 mm to (131.6, 55.8)
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Routing:
- net SOL_GPIO_18: track 372.7 -> 24.7 mm, vias 2 -> 0
- net SOL_GPIO_19: track 374.3 -> 33.8 mm, vias 3 -> 0
- net SOL_GPIO_17: track 332.2 -> 33.7 mm, vias 1 -> 0
- net SOL_GPIO_16: track 320.9 -> 24.3 mm, vias 1 -> 0
- net SOL_GPIO_11: track 264.6 -> 24.3 mm, vias 6 -> 0
- net SOL_GPIO_15: track 268.6 -> 32.9 mm, vias 2 -> 0
- net SOL_GPIO_14: track 232.9 -> 30.2 mm, vias 2 -> 0
- net N$39: track 225.9 -> 34.8 mm, vias 2 -> 0
- net SOL_GPIO_13: track 215.8 -> 33.3 mm, vias 3 -> 0
- net SOL_GPIO_12: track 194.5 -> 29.5 mm, vias 3 -> 0
- net N$41: track 207.8 -> 47.4 mm, vias 1 -> 0
- net N$43: track 193.3 -> 44.7 mm, vias 1 -> 0
- net N$45: track 184.8 -> 48.1 mm, vias 1 -> 0
- net SOL_GPIO_10: track 158.7 -> 31.1 mm, vias 3 -> 0
- net N$47: track 153.9 -> 32.0 mm
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Other:
- board size 147.6 x 77.7 mm -> 144.9 x 68.1 mm
- board text removed: "IGN"
- board text removed: "SOV_1"
- board text removed: "SOV_2"
- board text removed: "SOV_3"
- board text removed: "SOV_4"
- board text removed: "SOV_5"
- board text removed: "SOV_6"
- board text removed: "SOV_7"
- board text removed: "SOV_8"
- board text removed: "SOV_9"

Commit message: Minor cleanup around the SPS, minor polish on ground and on vbatt distribution.
Parts:
- moved R68 22.1 mm to (12.6, 59.6), turned to 0 degrees
- moved CR1 3.09 mm to (28.8, 56.5), turned to 0 degrees
- moved C23 2.89 mm to (30.6, 47.6), turned to 270 degrees
- moved C20 1.81 mm to (21.1, 53.8)
- moved R65 1.78 mm to (24.3, 56.5)
- moved D1 0.13 mm to (21.1, 48.0)
- moved L1 0.13 mm to (26.2, 50.6)
- moved Q3 0.13 mm to (126.3, 59.2)
- moved Q7 0.11 mm to (114.7, 46.6)
- moved C2 0.09 mm to (18.3, 43.6)
- moved Q9 0.09 mm to (126.2, 34.2)
- moved Q11 0.05 mm to (114.7, 34.2)
- moved Q19 0.05 mm to (114.7, 9.14)
- moved Q2 0.05 mm to (114.7, 59.2)
Routing:
- net N$35: track 44.2 -> 6.61 mm
- net +5V: track 77.0 -> 69.1 mm
- net N$4: track 19.4 -> 13.8 mm
- net VBATT: track 290.9 -> 293.2 mm, vias 1 -> 0
- net N$8: track 10.8 -> 8.97 mm
- net +12V: track 43.8 -> 44.8 mm
- net N$26: track 4.25 -> 3.53 mm
Other:
- board size 144.9 x 68.1 mm -> 144.8 x 67.6 mm
- board text added: "TSAR Actuator Controller, 2020-12-24, v2.0"
- board text removed: "TSAR Actuator Controller, 2020 Dec 24, Version: 2.0"

Commit message: layout, attributes, bom.
Parts:
- moved U$1 7.80 mm to (66.8, 43.1)
Other:
- board size 144.8 x 67.6 mm -> 143.9 x 69 mm
- board text added: "components between CN7 and CN10 must be below 8.5mm in height"
Changed lines of the file:
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@@
 <?xml version="1.0" encoding="utf-8"?>
 <!DOCTYPE eagle SYSTEM "eagle.dtd">
-<eagle version="9.6.1">
+<eagle version="9.6.2">
 <drawing>
 <settings>
@@
 <layer number="14" name="Route14" color="22" fill="1" visible="no" active="no"/>
 <layer number="15" name="Route15" color="23" fill="1" visible="no" active="no"/>
-<layer number="16" name="Bottom" color="1" fill="1" visible="no" active="yes"/>
+<layer number="16" name="Bottom" color="1" fill="1" visible="yes" active="yes"/>
 <layer number="17" name="Pads" color="2" fill="1" visible="yes" active="yes"/>
 <layer number="18" name="Vias" color="2" fill="1" visible="yes" active="yes"/>
@@
 <board>
 <plain>
-<wire x1="0" y1="0" x2="144.78" y2="0" width="0" layer="20"/>
-<wire x1="144.78" y1="0" x2="144.78" y2="67.564" width="0" layer="20"/>
-<wire x1="144.78" y1="67.564" x2="0" y2="67.564" width="0" layer="20"/>
-<wire x1="0" y1="67.564" x2="0" y2="0" width="0" layer="20"/>
 <text x="23.05" y="11.8363125" size="1.016" layer="25">GND</text>
 <text x="14.16" y="12.0609375" size="1.016" layer="25">GND</text>
@@
             2020-12-24, v2.0</text>
 <text x="11.557" y="1.524" size="1.016" layer="21" font="vector">Jennifer Jordan: jejor2@pdx.edu, Jake Pratt: jakepratt42@gmail.com</text>
+<text x="60.198" y="53.213" size="1.016" layer="21" font="vector">components between CN7 and CN10
+must be below 8.5mm in height</text>
+<wire x1="0.127" y1="-0.127" x2="0.127" y2="68.834" width="0.1524" layer="20"/>
+<wire x1="0.127" y1="68.834" x2="144.018" y2="68.834" width="0.1524" layer="20"/>
+<wire x1="144.018" y1="68.834" x2="144.018" y2="-0.127" width="0.1524" layer="20"/>
+<wire x1="144.018" y1="-0.127" x2="0.127" y2="-0.127" width="0.1524" layer="20"/>
 </plain>
 <attributes>
@@
 <attribute name="SPICEPREFIX" value="C" x="18.288" y="43.561" size="1.778" layer="27" rot="R270" display="off"/>
 </element>
-<element name="U$1" library="psas-logo" package="PSAS_LOGO_10X10" value="" x="59.182" y="44.704" smashed="yes"/>
+<element name="U$1" library="psas-logo" package="PSAS_LOGO_10X10" value="" x="66.802" y="43.053" smashed="yes"/>
 <element name="SENSOR0" library="pinhead" library_urn="urn:adsk.eagle:library:325" package="1X02" package3d_urn="urn:adsk.eagle:package:22435/2" value="" x="32.568165625" y="16.44315625" smashed="yes" rot="R270">
 <attribute name="DIS" value="Digi-Key" x="32.568165625" y="16.44315625" size="1.778" layer="27" rot="R270" display="off"/>
@@
 <contactref element="POE+" pad="C"/>
 <contactref element="5V" pad="C"/>
-<polygon width="0.0762" layer="1">
-<vertex x="0" y="67.564"/>
-<vertex x="144.78" y="67.564"/>
-<vertex x="144.78" y="0"/>
-<vertex x="0" y="0"/>
-</polygon>
-<polygon width="0.0762" layer="16">
-<vertex x="0" y="67.564"/>
-<vertex x="144.78" y="67.564"/>
-<vertex x="144.78" y="0"/>
-<vertex x="0" y="0"/>
-</polygon>
 <via x="12.446" y="64.008" extent="1-16" drill="0.35"/>
 <via x="36.068" y="61.595" extent="1-16" drill="0.35"/>
@@
 <via x="80.518" y="49.403" extent="1-16" drill="0.35"/>
 <via x="51.054" y="38.989" extent="1-16" drill="0.35"/>
-<via x="65.913" y="38.608" extent="1-16" drill="0.35"/>
+<via x="65.913" y="38.862" extent="1-16" drill="0.35"/>
 <via x="80.391" y="36.703" extent="1-16" drill="0.35"/>
 <via x="79.756" y="22.606" extent="1-16" drill="0.35"/>
@@
 <via x="21.844" y="44.069" extent="1-16" drill="0.35"/>
 <via x="18.288" y="40.894" extent="1-16" drill="0.35"/>
+<polygon width="0.1524" layer="1">
+<vertex x="0.127" y="-0.127"/>
+<vertex x="0.127" y="68.834"/>
+<vertex x="144.018" y="68.834"/>
+<vertex x="144.018" y="-0.127"/>
+</polygon>
+<polygon width="0.1524" layer="16">
+<vertex x="0.127" y="-0.127"/>
+<vertex x="0.127" y="68.834"/>
+<vertex x="144.018" y="68.834"/>
+<vertex x="144.018" y="67.945"/>
+<vertex x="144.018" y="-0.127"/>
+<vertex x="141.986" y="-0.127"/>
+</polygon>
 </signal>
 <signal name="N$3">

Commit message: pin map to Nucleo L476RG
Parts:
- R13: value NP -> 2.2k; device rcl:R0805 -> oresat-rcl:.0603-C-NOSILK
Connections:
- net 5V_USB_CHG renamed U5V
- net EVAL-VIN renamed VIN
- net NRST renamed RESET
- net PA11 renamed PA_11
- net PA12 renamed PA_12
- net PA14 renamed BOOT0
- net PB10 renamed PB_14
- net PB11 renamed PC_1
- net PB12 renamed PC_0
- net PB2 renamed PB_2
- net PB3 renamed PB_3
- net PB4 renamed PB_4
- net PB5 renamed PB_5
- net PB6 renamed PB_1
- net PB7 renamed PB_7
- net PB8 renamed PB_8
- net PB9 renamed PB_9
- net PC0 renamed PB_11
- net PC1 renamed PB_12
- net PC10 renamed PC_10
- net PC11 renamed PC_11
- net PC12 renamed PC_12
- net PC13 renamed PC_13
- net PC14 renamed PC_14
- net PC15 renamed PC_15
- net PC2 renamed PC_2
- net PC3 renamed PC_3
- net PC4 renamed PA_2
- net PC5 renamed PA_3
- net PC8 renamed PC_8
- net PC9 renamed PC_9
- net PD0 renamed NC1
- net PD1 renamed NC3
- net PD13 renamed PA_13
- net PD15 renamed PA_15
- net PD2 renamed PD_2
- net PD3 renamed NC2
- net PD4 renamed PA_14
- net PD5 renamed NC4
- net PD6 renamed NC5
- net PF0 renamed PH_0
- net PF1 renamed PH_1
- removed net EVAL-3V3: CN7.12, CN7.16
- new net 3V3: CN7.16
- new net IOREF: CN7.12
- net AGND: now also CN10.32; no longer CN10.9
- net GND: now also CN10.9
Routing:
- net EVAL-3V3: track 7.55 -> 0.00 mm
- net IOREF: track 0.00 -> 6.79 mm

Commit message: poe/ac/sfe changes, libraries
POE low risk input board created; will manage POE+ power distribution to subsystems. added 24-> 5v regulator for SFE and BB-AI
added libraries for SFE and POE.
SFE: removed 24->5V regulator from SFE, replaced D27&D31 with correct package, replaced ADC to correct SSOP20 package.
AC: replaced all passives with oresat rcl parts
Parts:
- C1, C12, C13, C14, C15, C17, C18, C19, C20, C23, C3, C40, C41, C6: device rcl:C0805 -> oresat-rcl:C0805K
- C2: device rcl:C1206 -> oresat-rcl:C1206K
- R1, R10, R11, R12, R14, R15, R16, R2, R21, R22, R23, R24, R25, R26, R27, R28, R29, R3, R30, R31, R32, R33, R34, R35, R36, R37, R38, R39, R4, R40, R41, R42, R43, R44, R45, R46, R47, R48, R49, R5, R50, R51, R52, R53, R54, R55, R56, R57, R58, R6, R65, R66, R7, R8, R9: device rcl:R0805 -> oresat-rcl:.0805-A-NOSILK
- R17, R18, R19, R20, R59, R60, R61, R62, R63, R64, R67, R68: device rcl:R0603 -> oresat-rcl:.0603-A-NOSILK

Commit message: SFE/AC changes
AC: began replacing nucleo with bare metal stm
SFE: replaced all passives with oresal parts
Parts:
- removed 5V, POE+: LG_T679-F1G2-1, led:PLCC2
- removed H1, H2, H3, H4: STAND-OFF, SparkFun-Hardware:STAND-OFF
- added 5V., POE.: (no value), led:CHIPLED_0603
- added H5, H6, H7, H8: #4-BARE_MOUNTING_HOLE/.300, mount:#4/.300-BARE+STD_NUT_OR_STAR_WASHER
- IGN., SOV_1., SOV_2., SOV_3., SOV_4., SOV_5., SOV_6., SOV_7., SOV_8., SOV_9.: value LG_T679-F1G2-1 -> (none); device led:PLCC2 -> led:CHIPLED_0603
- moved BATTERY 81.0 mm to (75.5, 4.00)
- moved L1 45.1 mm to (71.3, 52.6)
- moved R4 45.1 mm to (62.1, 58.7)
- moved R67 45.1 mm to (68.2, 44.2)
- moved C20 45.1 mm to (66.2, 55.9)
- moved C3 45.1 mm to (57.7, 49.7)
- moved C6 45.1 mm to (71.0, 46.8)
- moved CR1 45.1 mm to (73.9, 58.5)
- moved D1 45.1 mm to (66.2, 50.0)
- moved R1 45.1 mm to (57.7, 44.5)
- moved R13 45.1 mm to (57.7, 47.2)
- moved R5 45.1 mm to (57.7, 58.7)
- moved R66 45.1 mm to (56.7, 53.8)
- moved R68 45.1 mm to (57.7, 61.6)
- moved 5V_REG 45.1 mm to (61.7, 53.9)
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Connections:
- net GND: now also 5V..C, POE..C; no longer 5V.C, POE+.C
- net N$28: now also POE..A; no longer POE+.A
- net N$35: now also 5V..A; no longer 5V.A
Routing:
- net +12V: track 44.6 -> 109.1 mm
- net VBATT: track 293.2 -> 231.8 mm
- net +5V: track 69.0 -> 91.0 mm
- net IOREF: track 6.79 -> 0.00 mm
- net N$28: track 22.9 -> 25.0 mm
- net N$2: track 3.03 -> 3.63 mm
- net N$21: track 3.03 -> 3.63 mm
- net N$22: track 3.03 -> 3.62 mm
- net N$25: track 3.03 -> 3.62 mm
- net N$16: track 3.03 -> 3.62 mm
- net N$20: track 3.03 -> 3.61 mm
- net N$23: track 3.03 -> 3.61 mm
- net N$24: track 3.03 -> 3.61 mm
- net N$17: track 3.03 -> 3.60 mm
- net N$18: track 3.03 -> 3.60 mm
