File: actuator-controller/TSAR_Actuator_Controller.brd (EAGLE design)
At the start: 119.1 x 95 mm, 118 parts, among them Q1 220mA/50V/3.5Ω, Q10 220mA/50V/3.5Ω, Q11 IRF9530, Q12 220mA/50V/3.5Ω, Q13 IRF9530, Q14 220mA/50V/3.5Ω, Q15 IRF9530, Q16 220mA/50V/3.5Ω, Q17 IRF9530, Q18 220mA/50V/3.5Ω, Q19 IRF9530, Q2 IRF9530, Q20 220mA/50V/3.5Ω, Q3 IRF9530, Q4 220mA/50V/3.5Ω, Q5 IRF9530, Q6 220mA/50V/3.5Ω, Q7 IRF9530, Q8 220mA/50V/3.5Ω, Q9 IRF9530

Commit message: AC Error Check
Routing:
- net +12V: track 99.3 -> 189.4 mm
- net VBATT: track 288.6 -> 305.7 mm
Changed lines of the file:
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@@
 <contactref element="Q16" pad="1"/>
 <contactref element="R38" pad="2"/>
-<wire x1="67.438" y1="23.9828625" x2="69.7028625" y2="23.9828625" width="0.4064" layer="1"/>
-<wire x1="69.7028625" y1="23.9828625" x2="71.755" y2="26.035" width="0.4064" layer="1"/>
-<via x="71.755" y="26.035" extent="1-16" drill="0.35"/>
+<wire x1="67.438" y1="23.9828625" x2="69.8298625" y2="23.9828625" width="0.4064" layer="1"/>
+<wire x1="69.8298625" y1="23.9828625" x2="72.771" y2="26.924" width="0.4064" layer="1"/>
+<via x="72.771" y="26.924" extent="1-16" drill="0.35"/>
 <wire x1="77.343" y1="29.845" x2="78.613" y2="31.115" width="0.4064" layer="16"/>
-<wire x1="71.755" y1="26.035" x2="75.565" y2="29.845" width="0.4064" layer="16"/>
-<wire x1="75.565" y1="29.845" x2="77.343" y2="29.845" width="0.4064" layer="16"/>
+<wire x1="72.771" y1="26.924" x2="75.692" y2="29.845" width="0.4064" layer="16"/>
+<wire x1="75.692" y1="29.845" x2="77.343" y2="29.845" width="0.4064" layer="16"/>
 <wire x1="64.907" y1="24.0216625" x2="67.4268" y2="23.9716625" width="0.4064" layer="1"/>
 <wire x1="67.4268" y1="23.9716625" x2="67.438" y2="23.9828625" width="0.4064" layer="1"/>
@@
 <wire x1="87.122" y1="24.638" x2="98.5455" y2="24.638" width="1.27" layer="16"/>
 <wire x1="98.5455" y1="24.638" x2="98.696" y2="24.4875" width="1.27" layer="16"/>
-<wire x1="98.679" y1="49.53" x2="87.122" y2="49.53" width="1.27" layer="16"/>
+<wire x1="98.679" y1="49.53" x2="93.726" y2="49.53" width="1.27" layer="16"/>
+<wire x1="93.726" y1="49.53" x2="87.122" y2="49.53" width="1.27" layer="16"/>
 <wire x1="98.696" y1="62.143" x2="87.162" y2="62.143" width="1.27" layer="16"/>
 <wire x1="87.122" y1="62.103" x2="87.162" y2="62.143" width="1.27" layer="16"/>
@@
 <wire x1="28.524" y1="79.832" x2="36.576" y2="79.832" width="1.27" layer="1"/>
 <wire x1="25.908" y1="77.216" x2="28.524" y2="79.832" width="1.27" layer="1"/>
-<wire x1="87.122" y1="49.53" x2="87.122" y2="37.084" width="0" layer="19" extent="1-1"/>
+<wire x1="87.122" y1="37.084" x2="90.424" y2="37.084" width="1.27" layer="16"/>
+<wire x1="90.424" y1="37.084" x2="93.726" y2="40.386" width="1.27" layer="16"/>
+<wire x1="93.726" y1="40.386" x2="93.726" y2="49.53" width="1.27" layer="16"/>
 </signal>
 <signal name="PA_1">
@@
 <via x="49.657" y="69.342" extent="1-16" drill="0.35"/>
 <wire x1="49.657" y1="69.342" x2="46.852" y2="69.342" width="0.508" layer="1"/>
-<wire x1="60.833" y1="34.798" x2="98.679" y2="37.084" width="0" layer="19" extent="1-1"/>
+<wire x1="98.679" y1="37.084" x2="90.043" y2="28.448" width="0.6096" layer="16"/>
+<wire x1="90.043" y1="28.448" x2="85.09" y2="28.448" width="0.6096" layer="16"/>
+<wire x1="85.09" y1="28.448" x2="81.407" y2="24.765" width="0.6096" layer="16"/>
+<wire x1="65.659" y1="32.512" x2="65.659" y2="66.675" width="0.6096" layer="16"/>
+<wire x1="65.659" y1="66.675" x2="64.135" y2="68.199" width="0.6096" layer="16"/>
+<wire x1="64.135" y1="68.199" x2="51.689" y2="68.199" width="0.6096" layer="16"/>
+<wire x1="81.407" y1="24.765" x2="73.406" y2="24.765" width="0.6096" layer="16"/>
+<wire x1="73.406" y1="24.765" x2="65.659" y2="32.512" width="0.6096" layer="16"/>
 </signal>
 <signal name="FLY3">

Commit message: AC, SFE, VI changes
Updated rev number and dates.
Parts:
- moved Q1 0.13 mm to (68.6, 54.5)
Routing:
- net CTS_VI: track 67.0 -> 65.8 mm
- net TX_VI: track 91.6 -> 92.5 mm
- net SOL_GPIO_0: track 59.2 -> 58.4 mm
- net RTS_VI: track 84.3 -> 83.8 mm
Other:
- board text added: "TSAR Actuator Controller 2021/4/6, V2.2"
- board text removed: "TSAR Actuator Controller 2021-03-24, V2.1"
