File: actuator-controller/TSAR_Actuator_Controller.sch (EAGLE design)
At the start: 140 parts, among them J1 282834-2, J10 282834-2, J11 282834-2, J12 282834-2, J13 282834-2, J14 282834-2, J15 282834-2, J16 282834-2, J17 282834-2, J18 282834-2, J19 282834-2, J2 282834-2, J20 282834-2, J21 282834-2, J3 282834-2, J4 282834-2, J5 282834-2, J6 282834-2, J7 282834-2, J8 282834-2, J9 282834-2, Q1 BUZ11BV, Q10 BUZ11BV, Q2 BUZ11BV, Q3 BUZ11BV, Q4 BUZ11BV, Q5 BUZ11BV, Q6 BUZ11BV, Q7 BUZ11BV, Q8 BUZ11BV, Q9 BUZ11BV

Commit message: Updated Schematic after last design review.
Updated according to Andrews input.
Parts:
- removed C10, C25, C26, C27, C28, C29, C30, C31, C32, C33, C34, C35, C36, C37, C38, C39, C8, C9: 120pF, rcl:C-EUC0805
- removed D10, D11, D12, D6, D7, D8, D9: BAS40, diode:BAS40
- removed J10, J11, J12, J13, J14, J15, J16, J17, J18, J19, J5, J6, J7, J8, J9: 282834-2, TSAR_Controller:282834-2
- removed Q10, Q9: BUZ11BV, transistor-power:BUZ11BV
- removed R32, R33, R34, R35, R36, R37, R44, R49: 28K, rcl:R-US_R0603
- removed R38, R39, R40, R41, R42, R43, R45, R46, R47, R48: 1K, rcl:R-EU_R0603
- removed TVSD_12, TVSD_13, TVSD_14, TVSD_15, TVSD_16, TVSD_17, TVSD_18, TVSD_19, TVSD_20, TVSD_21, TVSD_22, TVSD_23, TVSD_24, TVSD_25, TVSD_26, TVSD_27, TVSD_28, TVSD_29, TVSD_30: DF2B5M4CT,L3F, TSAR_Controller:DF2B5M4CT,L3F
- added C1, C11, C12, C13, C14, C15, C17, C18, C19, C40, C41: 120pF, rcl:C-EUC0805
- added D13: BAS40, diode:BAS40
- added J23, J24, J25, J26, J27, J29, J30, J31, J32, J33: 282834-2, TSAR_Controller:282834-2
- added R1, R10, R11, R12, R13, R14, R15, R50, R51, R52, R8, R9: 1K, rcl:R-EU_R0603
- added R7: 28K, rcl:R-US_R0603
- added TVSD_1, TVSD_2, TVSD_3, TVSD_31, TVSD_32, TVSD_33, TVSD_4, TVSD_5, TVSD_6, TVSD_7, TVSD_8, TVSD_9: DF2B5M4CT,L3F, TSAR_Controller:DF2B5M4CT,L3F
- Q1, Q3, Q5, Q7: value BUZ11BV -> MMBT3904-TP; device transistor-power:BUZ11BV -> TSAR_Controller:MMBT3904-TP
- Q2, Q4, Q6, Q8: value BUZ11BV -> IRF9530; device transistor-power:BUZ11BV -> transistor-power:IRF9530
- R16, R5: value 500k -> 10K
- R2, R22, R26: value 1K -> 3K
- R21, R25, R29: value 1K -> 28K; device rcl:R-EU_R0603 -> rcl:R-US_R0603
- R23, R27, R3: value 1K -> 4.7K
- R30: value 28K -> 3K; device rcl:R-US_R0603 -> rcl:R-EU_R0603
- R31: value 28K -> 4.7K; device rcl:R-US_R0603 -> rcl:R-EU_R0603
- R4, R6: value 0 -> NP
Connections:
- net 5V renamed +5V
- removed net 12V: D10.C, D11.C, D12.C, D3.C, D4.C, D5.C, D6.C, D7.C, D8.C, D9.C, J1.1, J10.1, J11.1, J17.1, J18.1, J2.1, J4.1, J5.1, J7.1, J9.1
- removed net 24V: C21.1, C4.1, C5.1, C6.1, R16.1, R5.1, U$3.IN, U$4.IN
- removed net 3V3: C24.1, CR2.2, U$5.2
- removed net N$20: D6.A, R33.2
- removed net N$21: Q5.G, R28.2
- removed net N$22: J5.2, Q5.D
- removed net N$23: D7.A, R34.2
- removed net N$24: D5.A, R32.2
- removed net N$25: Q3.G, R27.2
- removed net N$26: J8.1, R29.2
- removed net N$27: J9.2, Q6.D
- removed net N$28: D8.A, R35.2
- removed net N$29: Q6.G, R23.2
- removed net N$30: J10.2, Q7.D
- removed net N$31: D9.A, R36.2
- removed net N$32: Q7.G, R24.2
- removed net N$33: J11.2, Q8.D
- removed net N$34: D10.A, R37.2
- removed net N$35: Q8.G, R25.2
- removed net N$36: J12.1, R38.2
- removed net N$37: J13.1, R39.2
- removed net N$38: J14.1, R40.2
- removed net N$39: J15.1, R41.2
- removed net N$40: J16.1, R42.2
- removed net N$41: J18.2, Q9.D
- removed net N$42: D11.A, R44.2
- removed net N$43: Q9.G, R43.2
- removed net N$44: R45.2
- removed net N$45: R46.2
- removed net N$46: R47.2
- removed net N$47: Q10.G, R48.2
- removed net N$48: J17.2, Q10.D
- removed net N$49: D12.A, R49.2
- removed net N$50: J19.1
- removed net N$51: J20.1
- removed net N$52: J21.1
- removed net VLV_FB_0: C38.1, CN7.28, R47.1, TVSD_29.P$1
- removed net VLV_FB_1: C37.1, CN7.30, R46.1, TVSD_28.P$1
- removed net VLV_FB_10: C34.1, CN10.19, R42.1, TVSD_25.P$1
- removed net VLV_FB_2: C3.1, CN10.34, R3.1, TVSD_11.P$1
- removed net VLV_FB_3: C26.1, CN10.6, R26.1, TVSD_17.P$1
- removed net VLV_FB_4: C36.1, CN7.32, R45.1, TVSD_27.P$1
- removed net VLV_FB_5: C29.1, CN10.11, R38.1, TVSD_21.P$1
- removed net VLV_FB_6: C30.1, CN10.13, R39.1, TVSD_22.P$1
- removed net VLV_FB_7: C31.1, CN10.15, R40.1, TVSD_23.P$1
- removed net VLV_FB_8: C33.1, CN10.17, R41.1, TVSD_24.P$1
- new net +12V: C21.1, C4.1, C5.1, C6.1, J20.2, J21.1, Q2.S, Q4.S, Q6.S, Q8.S, R16.1, R23.2, R27.2, R3.2, R31.2, R5.1, U$3.IN, U$4.IN
- new net N$54: D13.A, R7.2
- new net N$56: R8.2
- new net N$57: J23.1
- new net N$58: R9.2
- new net N$59: J24.1
- new net N$60: R10.2
- new net N$61: R11.2
- new net N$62: J25.1
- new net N$63: J26.1
- new net N$64: R12.2
- new net N$65: J27.1
- new net N$68: R14.2
- new net N$69: J29.1
- new net N$70: R15.2
- new net N$71: J30.1
- new net N$72: R50.2
- new net N$73: J31.1
- new net N$74: R51.2
- new net N$75: J32.1
- new net N$76: R52.2
- new net N$77: J33.1
- new net SOL_GPIO_03: CN10.19
- new net SOL_GPIO_10: D13.C, J1.1, Q2.D
- new net SOL_GPIO_14: D4.C, J3.1, Q6.D
- new net SOL_GPIO_15: C7.1, R28.1, TVSD_11.P$1
- new net SOL_GPIO_16: D5.C, J4.1, Q8.D
- new net SOL_GPIO_4: CN10.4
- new net TBD_SENSOR_0: C1.1, C12.1, C13.1, C14.1, C15.1, C17.1, C18.1, C19.1, C40.1, C41.1, CN7.28, R10.1, R11.1, R12.1, R14.1, R15.1, R50.1, R51.1, R52.1, R8.1, R9.1, TVSD_1.P$1, TVSD_3.P$1, TVSD_31.P$1, TVSD_32.P$1, TVSD_33.P$1, TVSD_4.P$1, TVSD_5.P$1, TVSD_6.P$1, TVSD_8.P$1, TVSD_9.P$1
- new net TBD_SENSOR_1: CN7.30
- new net TBD_SENSOR_2: CN10.34
- new net TBD_SENSOR_3: CN10.6
- new net TBD_SENSOR_4: CN7.32
- new net TBD_SENSOR_5: CN10.11
- new net TBD_SENSOR_6: CN10.13
- new net TBD_SENSOR_7: CN10.15
- new net TBD_SENSOR_8: CN10.17
- new net TBD_SENSOR_9: CN7.34
- net 48V1: now also C24.1, CR2.2, U$5.2
- net GND: now also C1.2, C11.2, C12.2, C13.2, C14.2, C15.2, C17.2, C18.2, C19.2, C40.2, C41.2, J1.2, J2.2, J20.1, J23.2, J24.2, J25.2, J26.2, J27.2, J29.2, J30.2, J31.2, J32.2, J33.2, J4.2, Q1.2, Q3.2, Q5.2, Q7.2, R2.1, R21.1, R22.1, R25.1, R26.1, R29.1, R7.1, TVSD_1.P$2, TVSD_2.P$2, TVSD_3.P$2, TVSD_31.P$2, TVSD_32.P$2, TVSD_33.P$2, TVSD_4.P$2, TVSD_5.P$2, TVSD_6.P$2, TVSD_7.P$2, TVSD_8.P$2, TVSD_9.P$2; no longer C10.2, C25.2, C26.2, C27.2, C28.2, C29.2, C30.2, C31.2, C32.2, C33.2, C34.2, C35.2, C36.2, C37.2, C38.2, C39.2, C8.2, C9.2, J12.2, J13.2, J14.2, J15.2, J16.2, J19.2, J20.2, J6.2, J8.2, Q1.S, Q10.S, Q2.S, Q3.S, Q4.S, Q5.S, Q6.S, Q7.S, Q8.S, Q9.S, R31.1, R32.1, R33.1, R34.1, R35.1, R36.1, R37.1, R44.1, R49.1, TVSD_12.P$2, TVSD_13.P$2, TVSD_14.P$2, TVSD_15.P$2, TVSD_16.P$2, TVSD_17.P$2, TVSD_18.P$2, TVSD_19.P$2, TVSD_20.P$2, TVSD_21.P$2, TVSD_22.P$2, TVSD_23.P$2, TVSD_24.P$2, TVSD_25.P$2, TVSD_26.P$2, TVSD_27.P$2, TVSD_28.P$2, TVSD_29.P$2, TVSD_30.P$2
- net N$1: now also Q1.3, Q2.G, R3.1; no longer Q1.G, R22.2
- net N$10: now also Q3.1, R13.2, R22.2; no longer Q4.G, R2.2
- net N$11: now also Q3.3, Q4.G, R23.1; no longer Q2.G, R21.2
- net N$12: now also D4.A, R25.2; no longer J2.2, Q2.D
- net N$13: now also Q5.1, R24.2, R26.2; no longer D4.A, R31.2
- net N$14: now also Q5.3, Q6.G, R27.1; no longer J3.1, R3.2
- net N$15: now also D5.A, R29.2; no longer J6.1, R26.2
- net N$16: now also Q7.1, R28.2, R30.2; no longer J7.2, Q3.D
- net N$18: now also Q7.3, Q8.G, R31.1; no longer J4.2, Q4.D
- net N$2: now also Q1.1, R1.2, R2.2; no longer J1.2, Q1.D
- net N$9: now also R21.2; no longer R30.2
- net SOL_GPIO_0: no longer C9.1, R23.1, TVSD_14.P$1
- net SOL_GPIO_1: no longer C7.1, R21.1, TVSD_12.P$1
- net SOL_GPIO_11: now also C2.1, R13.1, TVSD_7.P$1; no longer C27.1, CN10.4, R27.1, TVSD_18.P$1
- net SOL_GPIO_12: now also D3.C, J2.1, Q4.D; no longer C28.1, R29.1, TVSD_20.P$1
- net SOL_GPIO_13: now also C3.1, R24.1, TVSD_10.P$1; no longer C39.1, CN7.34, R48.1, TVSD_30.P$1
- net SOL_GPIO_2: now also C11.1, R1.1, TVSD_2.P$1; no longer C8.1, R22.1, TVSD_13.P$1
- net SOL_GPIO_5: no longer C35.1, R43.1, TVSD_26.P$1
- net SOL_GPIO_6: no longer C25.1, R25.1, TVSD_16.P$1
- net SOL_GPIO_7: no longer C32.1, R28.1, TVSD_19.P$1
- net SOL_GPIO_8: no longer C10.1, R24.1, TVSD_15.P$1
- net SOL_GPIO_9: no longer C2.1, R2.1, TVSD_10.P$1
Other:
- note added: "12V Connector from PoE"
- note added: "12V From the Test Stand Battery."
- note added: "12V to 3V3 Regulator"
- note added: "12V to 5V Regulator"
- note added: "STM Nucleo G071RB Morpho Connectorsfor the MCU Eval Board."
- note added: "Screw Terminal are 0.1" Pitch."
- note added: "Valve Position Sensor Inputs."
- note removed: "24V to 3V3 Regulator"
- note removed: "24V to 5V Regulator"
- note removed: "Morpho Connectors coming from the MCU Eval Board."

Commit message: Replaced Resistors and 5V TVS Diodes.
Changed resistors to 0805 to be the same size as the caps.
Changed to a standard sized TVS Diode footprint.
Began Board layouts.
Parts:
- removed C11, C2, C3, C7: 120pF, rcl:C-EUC0805
- removed J1, J2, J23, J24, J25, J26, J27, J29, J3, J30, J31, J32, J33, J4: 282834-2, TSAR_Controller:282834-2
- removed R50, R51, R52: 1K, rcl:R-EU_R0603
- removed TVSD_1, TVSD_10, TVSD_11, TVSD_2, TVSD_3, TVSD_31, TVSD_32, TVSD_33, TVSD_4, TVSD_5, TVSD_6, TVSD_7, TVSD_8, TVSD_9: DF2B5M4CT,L3F, TSAR_Controller:DF2B5M4CT,L3F
- added D10, D11, D6, D7, D8, D9: BAS40, diode:BAS40
- added D12, D14, D15, D16, D17, D18, D19, D20, D21, D22: 5V, SparkFun-DiscreteSemi:DIODE_TVS
- added Q10, Q12, Q14, Q16, Q18, Q20: 220mA/50V/3.5Ω, SparkFun-DiscreteSemi:MOSFET-NCH-BSS138
- added Q11, Q13, Q15, Q17, Q19, Q9: IRF9530, transistor-power:IRF9530
- added R32, R35, R38, R41, R44: 10k, rcl:R-US_R0805
- added R33, R36, R39, R42, R45: 28k, rcl:R-US_R0805
- added R34, R37, R40, R43: 4.7K, rcl:R-US_R0805
- added R46, R47, R48: 1k, rcl:R-US_R0805
- added SENSOR_0, SENSOR_1, SENSOR_2, SENSOR_3, SENSOR_4, SENSOR_5, SENSOR_6, SENSOR_7, SENSOR_8, SENSOR_9, SOLENOID_0, SOLENOID_1, SOLENOID_2, SOLENOID_3, SOLENOID_4, SOLENOID_5, SOLENOID_6, SOLENOID_7, SOLENOID_8, SOLENOID_9: 282834-2, TSAR_Controller:282834-2
- Q1: value MMBT3904-TP -> 220mA/50V/3.5Ω; device TSAR_Controller:MMBT3904-TP -> SparkFun-DiscreteSemi:MOSFET-NCH-BSS138
- Q3, Q5, Q7: value MMBT3904-TP -> IRF9530; device TSAR_Controller:MMBT3904-TP -> transistor-power:IRF9530
- Q4, Q6, Q8: value IRF9530 -> 220mA/50V/3.5Ω; device transistor-power:IRF9530 -> SparkFun-DiscreteSemi:MOSFET-NCH-BSS138
- R1: value 1K -> 10K; device rcl:R-EU_R0603 -> rcl:R-US_R0805
- R10, R11, R12, R14, R15, R8, R9: value 1K -> 1k; device rcl:R-EU_R0603 -> rcl:R-US_R0805
- R13: value 1K -> NP; device rcl:R-EU_R0603 -> rcl:R-US_R0805
- R16: value 10K -> 10k; device rcl:R-US_R0603 -> rcl:R-US_R0805
- R17: value (none) -> 10K; device rcl:R-US_R0603 -> rcl:R-US_R0805
- R18: value (none) -> NP; device rcl:R-US_R0603 -> rcl:R-US_R0805
- R19: value 23.7K -> 10k; device rcl:R-US_R0603 -> rcl:R-US_R0805
- R2, R22: value 3K -> 4.7K; device rcl:R-EU_R0603 -> rcl:R-US_R0805
- R20: value 124K -> 33k; device rcl:R-US_R0603 -> rcl:R-US_R0805
- R21, R7: value 28K -> 28k; device rcl:R-US_R0603 -> rcl:R-US_R0805
- R23, R3: value 4.7K -> 10k; device rcl:R-EU_R0603 -> rcl:R-US_R0805
- R24: value 1K -> 28k; device rcl:R-EU_R0603 -> rcl:R-US_R0805
- R25: value 28K -> 4.7K; device rcl:R-US_R0603 -> rcl:R-US_R0805
- R26: value 3K -> 10k; device rcl:R-EU_R0603 -> rcl:R-US_R0805
- R27: value 4.7K -> 28k; device rcl:R-EU_R0603 -> rcl:R-US_R0805
- R28: value 1K -> 4.7K; device rcl:R-EU_R0603 -> rcl:R-US_R0805
- R29: value 28K -> 10k; device rcl:R-US_R0603 -> rcl:R-US_R0805
- R30: value 3K -> 28k; device rcl:R-EU_R0603 -> rcl:R-US_R0805
- R31: device rcl:R-EU_R0603 -> rcl:R-US_R0805
- R4: value NP -> 124k; device rcl:R-US_R0603 -> rcl:R-US_R0805
- R5: value 10K -> 23.7k; device rcl:R-US_R0603 -> rcl:R-US_R0805
- R6: value NP -> 4.7K; device rcl:R-US_R0603 -> rcl:R-US_R0805
Connections:
- removed net 48V1: C24.1, CR2.2, R18.1, U$5.2
- removed net 48V2: R20.1
- removed net EVAL-5V: CN7.18
- removed net N$56: R8.2
- removed net N$57: J23.1
- removed net N$58: R9.2
- removed net N$59: J24.1
- removed net N$60: R10.2
- removed net N$61: R11.2
- removed net N$62: J25.1
- removed net N$63: J26.1
- removed net N$64: R12.2
- removed net N$65: J27.1
- removed net N$68: R14.2
- removed net N$69: J29.1
- removed net N$70: R15.2
- removed net N$71: J30.1
- removed net N$72: R50.2
- removed net N$73: J31.1
- removed net N$74: R51.2
- removed net N$75: J32.1
- removed net N$76: R52.2
- removed net N$77: J33.1
- new net +3V3: C24.1, CR2.2, R19.2, U$5.2
- new net N$20: R48.2, SENSOR_9.1
- new net N$21: C40.1, D22.C, R15.1
- new net N$22: C1.1, D17.C, R11.1
- new net N$23: C12.1, D16.C, R8.1
- new net N$24: C14.1, D15.C, R10.1
- new net N$25: C15.1, D12.C, R12.1
- new net N$26: C17.1, D19.C, R47.1
- new net N$27: C18.1, D20.C, R14.1
- new net N$28: C19.1, D21.C, R9.1
- new net N$29: D3.A, R7.2
- new net N$30: Q3.G, Q4.D, R2.1
- new net N$31: D4.A, R24.2
- new net N$32: Q5.G, Q6.D, R22.1
- new net N$33: D5.A, R27.2
- new net N$34: Q7.G, Q8.D, R25.1
- new net N$35: Q1.G, R16.2
- new net N$36: D6.A, R30.2
- new net N$37: Q10.D, Q9.G, R28.1
- new net N$38: D7.A, R33.2
- new net N$39: Q11.G, Q12.D, R31.1
- new net N$40: D8.A, R36.2
- new net N$41: Q13.G, Q14.D, R34.1
- new net N$42: D9.A, R39.2
- new net N$43: Q15.G, Q16.D, R37.1
- new net N$44: D10.A, R42.2
- new net N$45: Q17.G, Q18.D, R40.1
- new net N$46: D11.A, R45.2
- new net N$47: Q19.G, Q20.D, R43.1
- new net SOL_GPIO_17: D9.C, Q15.D, SOLENOID_7.1
- new net SOL_GPIO_18: D10.C, Q17.D, SOLENOID_8.1
- new net SOL_GPIO_19: D11.C, Q19.D, SOLENOID_9.1
- new net SOL_GPIO_3: CN10.19
- new net V+: J21.1, Q11.S, Q13.S, Q15.S, Q17.S, Q19.S, Q2.S, Q3.S, Q5.S, Q7.S, Q9.S, R2.2, R22.2, R25.2, R28.2, R31.2, R34.2, R37.2, R40.2, R43.2, R6.2
- net +12V: now also R1.2, R17.2; no longer J21.1, Q2.S, Q4.S, Q6.S, Q8.S, R16.1, R23.2, R27.2, R3.2, R31.2, R5.1
- net +5V: now also CN7.18, R4.2
- net GND: now also D12.A, D14.A, D15.A, D16.A, D17.A, D18.A, D19.A, D20.A, D21.A, D22.A, Q1.S, Q10.S, Q12.S, Q14.S, Q16.S, Q18.S, Q20.S, Q4.S, Q6.S, Q8.S, R13.1, R16.1, R18.1, R20.1, R23.1, R24.1, R27.1, R3.1, R32.1, R33.1, R35.1, R36.1, R38.1, R39.1, R41.1, R42.1, R44.1, R45.1, R5.1, SENSOR_0.2, SENSOR_1.2, SENSOR_2.2, SENSOR_3.2, SENSOR_4.2, SENSOR_5.2, SENSOR_6.2, SENSOR_7.2, SENSOR_8.2, SENSOR_9.2, SOLENOID_0.2, SOLENOID_1.2, SOLENOID_2.2, SOLENOID_3.2, SOLENOID_4.2, SOLENOID_5.2, SOLENOID_6.2, SOLENOID_7.2, SOLENOID_8.2, SOLENOID_9.2; no longer C11.2, C2.2, C3.2, C7.2, J1.2, J2.2, J23.2, J24.2, J25.2, J26.2, J27.2, J29.2, J3.2, J30.2, J31.2, J32.2, J33.2, J4.2, Q1.2, Q3.2, Q5.2, Q7.2, R17.2, R19.2, R2.1, R22.1, R25.1, R4.2, R6.2, TVSD_1.P$2, TVSD_10.P$2, TVSD_11.P$2, TVSD_2.P$2, TVSD_3.P$2, TVSD_31.P$2, TVSD_32.P$2, TVSD_33.P$2, TVSD_4.P$2, TVSD_5.P$2, TVSD_6.P$2, TVSD_7.P$2, TVSD_8.P$2, TVSD_9.P$2
- net N$1: now also Q1.D, R6.1; no longer Q1.3, R3.1
- net N$10: now also R11.2, SENSOR_1.1; no longer Q3.1, R13.2, R22.2
- net N$11: now also R8.2, SENSOR_2.1; no longer Q3.3, Q4.G, R23.1
- net N$12: now also R10.2, SENSOR_3.1; no longer D4.A, R25.2
- net N$13: now also R12.2, SENSOR_4.1; no longer Q5.1, R24.2, R26.2
- net N$14: now also R47.2, SENSOR_5.1; no longer Q5.3, Q6.G, R27.1
- net N$15: now also R14.2, SENSOR_6.1; no longer D5.A, R29.2
- net N$16: now also R9.2, SENSOR_7.1; no longer Q7.1, R28.2, R30.2
- net N$17: now also R19.1, R20.2; no longer R17.1, R18.2
- net N$18: now also R15.2, SENSOR_8.1; no longer Q7.3, Q8.G, R31.1
- net N$19: now also R4.1, R5.2; no longer R19.1, R20.2
- net N$2: now also C41.1, D14.C, R48.1; no longer Q1.1, R1.2, R2.2
- net N$3: now also R1.1, R13.2; no longer R4.1, R5.2
- net N$5: now also R17.1, R18.2; no longer R16.2, R6.1
- net N$54: now also R21.2; no longer R7.2
- net N$9: now also R46.2, SENSOR_0.1; no longer D3.A, R21.2
- net SOL_GPIO_03: now also Q8.G, R26.2; no longer CN10.19
- net SOL_GPIO_1: now also Q4.G, R3.2
- net SOL_GPIO_10: now also SOLENOID_0.1; no longer J1.1
- net SOL_GPIO_11: now also D3.C, Q3.D, SOLENOID_1.1; no longer C2.1, R13.1, TVSD_7.P$1
- net SOL_GPIO_12: now also D4.C, Q5.D, SOLENOID_2.1; no longer D3.C, J2.1, Q4.D
- net SOL_GPIO_13: now also D5.C, Q7.D, SOLENOID_3.1; no longer C3.1, R24.1, TVSD_10.P$1
- net SOL_GPIO_14: now also D6.C, Q9.D, SOLENOID_4.1; no longer D4.C, J3.1, Q6.D
- net SOL_GPIO_15: now also D7.C, Q11.D, SOLENOID_5.1; no longer C7.1, R28.1, TVSD_11.P$1
- net SOL_GPIO_16: now also D8.C, Q13.D, SOLENOID_6.1; no longer D5.C, J4.1, Q8.D
- net SOL_GPIO_2: now also Q6.G, R23.2; no longer C11.1, R1.1, TVSD_2.P$1
- net SOL_GPIO_4: now also Q10.G, R29.2
- net SOL_GPIO_5: now also Q12.G, R32.2
- net SOL_GPIO_6: now also Q14.G, R35.2
- net SOL_GPIO_7: now also Q16.G, R38.2
- net SOL_GPIO_8: now also Q18.G, R41.2
- net SOL_GPIO_9: now also Q20.G, R44.2
- net TBD_SENSOR_0: now also D18.C, R46.1; no longer C1.1, C12.1, C14.1, C15.1, C17.1, C18.1, C19.1, C40.1, C41.1, R10.1, R11.1, R12.1, R14.1, R15.1, R50.1, R51.1, R52.1, R8.1, R9.1, TVSD_1.P$1, TVSD_3.P$1, TVSD_31.P$1, TVSD_32.P$1, TVSD_33.P$1, TVSD_4.P$1, TVSD_5.P$1, TVSD_6.P$1, TVSD_8.P$1, TVSD_9.P$1
Other:
- note added: "All Resistors and Capacitors are 0805, unless otherwise noted."
- note added: "VBATT From Test Stand Battery."
- note removed: "12V From the Test Stand Battery."

Commit message: Adjusted Board Layout
Parts:
- added H1, H2, H3, H4: STAND-OFF, SparkFun-Hardware:STAND-OFF
Other:
- note added: "Drill Holes for Standoffs."
Changed lines of the file:
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@@
 <setting verticaltext="up"/>
 </settings>
-<grid distance="1.27" unitdist="mm" unit="mm" style="lines" multiple="1" display="no" altdistance="0.01" altunitdist="inch" altunit="inch"/>
+<grid distance="0.1" unitdist="inch" unit="inch" style="lines" multiple="1" display="no" altdistance="0.01" altunitdist="inch" altunit="inch"/>
 <layers>
 <layer number="1" name="Top" color="4" fill="1" visible="no" active="no"/>
@@
 <part name="D22" library="SparkFun-DiscreteSemi" deviceset="DIODE_TVS" device="" value="5V"/>
 <part name="P+5" library="supply1" library_urn="urn:adsk.eagle:library:371" deviceset="+5V" device=""/>
+<part name="H1" library="SparkFun-Hardware" deviceset="STAND-OFF" device=""/>
+<part name="H2" library="SparkFun-Hardware" deviceset="STAND-OFF" device=""/>
+<part name="H3" library="SparkFun-Hardware" deviceset="STAND-OFF" device=""/>
+<part name="H4" library="SparkFun-Hardware" deviceset="STAND-OFF" device=""/>
 </parts>
 <sheets>
@@
 <text x="46.99" y="63.5" size="1.778" layer="97">VBATT From Test Stand Battery.</text>
 <text x="-132.08" y="-101.6" size="1.778" layer="97">All Resistors and Capacitors are 0805, unless otherwise noted.</text>
+<text x="-43.18" y="-88.9" size="1.778" layer="97">Drill Holes for Standoffs.</text>
 </plain>
 <instances>
@@
 <attribute name="VALUE" x="-74.168" y="-17.78" size="1.778" layer="96" rot="R90"/>
 </instance>
+<instance part="H1" gate="G$1" x="-38.1" y="-93.98" smashed="yes"/>
+<instance part="H2" gate="G$1" x="-33.02" y="-93.98" smashed="yes"/>
+<instance part="H3" gate="G$1" x="-27.94" y="-93.98" smashed="yes"/>
+<instance part="H4" gate="G$1" x="-22.86" y="-93.98" smashed="yes"/>
 </instances>
 <busses>
@@
 <wire x1="30.48" y1="179.07" x2="30.48" y2="180.34" width="0.1524" layer="91"/>
 <wire x1="30.48" y1="180.34" x2="31.75" y2="180.34" width="0.1524" layer="91"/>
-<wire x1="30.48" y1="180.34" x2="27.94" y2="180.34" width="0.1524" layer="91"/>
+<wire x1="27.94" y1="180.34" x2="30.48" y2="180.34" width="0.1524" layer="91"/>
 <junction x="30.48" y="180.34"/>
 </segment>

Commit message: Completed initial board layout.
Parts:
- removed J21: 282834-2, TSAR_Controller:282834-2
- added J1: (no value), SparkFun-Connectors:CONN_02PTH4
- renumbered J20 to 12V, U$3 to 5V_REG, U$4 to 3V3_REG, U$5 to L2, U$6 to L1
Connections:
- removed net N$2: C41.1, D14.C, R48.1
- removed net N$21: C40.1, D22.C, R15.1
- removed net N$22: C1.1, D17.C, R11.1
- removed net N$23: C12.1, D16.C, R8.1
- removed net N$24: C14.1, D15.C, R10.1
- removed net N$25: C15.1, D12.C, R12.1
- removed net N$26: C17.1, D19.C, R47.1
- removed net N$27: C18.1, D20.C, R14.1
- removed net N$28: C19.1, D21.C, R9.1
- removed net N$35: Q1.G, R16.2
- removed net SOL_GPIO_03: Q8.G, R26.2
- removed net V+: J21.1, Q11.S, Q13.S, Q15.S, Q17.S, Q19.S, Q2.S, Q3.S, Q5.S, Q7.S, Q9.S, R2.2, R22.2, R25.2, R28.2, R31.2, R34.2, R37.2, R40.2, R43.2, R6.2
- new net VBATT: J1.1, Q11.S, Q13.S, Q15.S, Q17.S, Q19.S, Q2.S, Q3.S, Q5.S, Q7.S, Q9.S, R2.2, R22.2, R25.2, R28.2, R31.2, R34.2, R37.2, R40.2, R43.2, R6.2
- net GND: now also J1.2; no longer J21.2
- net SOL_GPIO_0: now also Q1.G, R16.2
- net SOL_GPIO_3: now also Q8.G, R26.2
- net TBD_SENSOR_1: now also C1.1, D17.C, R11.1
- net TBD_SENSOR_2: now also C12.1, D16.C, R8.1
- net TBD_SENSOR_3: now also C14.1, D15.C, R10.1
- net TBD_SENSOR_4: now also C15.1, D12.C, R12.1
- net TBD_SENSOR_5: now also C17.1, D19.C, R47.1
- net TBD_SENSOR_6: now also C18.1, D20.C, R14.1
- net TBD_SENSOR_7: now also C19.1, D21.C, R9.1
- net TBD_SENSOR_8: now also C40.1, D22.C, R15.1
- net TBD_SENSOR_9: now also C41.1, D14.C, R48.1

Commit message: Added voltage divider on GPIO Sensor Inputs.
Parts:
- added R49, R50, R51, R52, R53, R54, R55, R56, R57, R58: NP, rcl:R-US_R0805
Connections:
- net GND: now also R49.1, R50.1, R51.1, R52.1, R53.1, R54.1, R55.1, R56.1, R57.1, R58.1
- net TBD_SENSOR_0: now also R50.2
- net TBD_SENSOR_1: now also R51.2
- net TBD_SENSOR_2: now also R52.2
- net TBD_SENSOR_3: now also R53.2
- net TBD_SENSOR_4: now also R54.2
- net TBD_SENSOR_5: now also R55.2
- net TBD_SENSOR_6: now also R56.2
- net TBD_SENSOR_7: now also R49.2
- net TBD_SENSOR_8: now also R57.2
- net TBD_SENSOR_9: now also R58.2
Other:
- note added: "NP Resistors are provided to allow for input signlas that exceed 3.3V."
- moved on the sheet: C1, C12, C13, C14, C15, C17, C18, C19, C40, C41, D12, D14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

Commit message: Revised board layout. Updated OSH Park DRC.
Parts:
- removed 3V3_REG: MP2456GJ-P, TSAR_Controller:MP2456GJ-P
- removed C21, C22: 0.1uF, rcl:C-EUC0805
- removed C24: 10uF, rcl:C-EUC0805
- removed C4, C5: UUX2A4R7MCL1GSCAP_UCD_8X6P2-L, TSAR_Controller:UUX2A4R7MCL1GSCAP_UCD_8X6P2-L
- removed CR2: 1N4148W-7-F, TSAR_Controller:1N4148W-7-F
- removed D2: DFLS160, diode:DIODE-DO214AA
- removed L2: 10uH, TSAR_Controller:CLF5030NIT-100M-D
- removed R17: 10K, rcl:R-US_R0805
- removed R18: NP, rcl:R-US_R0805
- removed R19: 10k, rcl:R-US_R0805
- removed R20: 33k, rcl:R-US_R0805
- added C2: 4.7uF, rcl:C-EUC1206
- added H5, H6, H7: STAND-OFF, SparkFun-Hardware:STAND-OFF
Connections:
- removed net +3V3: C24.1, CR2.2, L2.2, R19.2
- removed net N$17: 3V3_REG.FB, R19.1, R20.2
- removed net N$5: 3V3_REG.EN, R17.1, R18.2
- removed net N$6: 3V3_REG.BST, C22.1, CR2.1
- removed net N$7: 3V3_REG.SW, C22.2, D2.C, L2.1
- net +12V: now also C2.1; no longer 3V3_REG.IN, C21.1, C4.1, C5.1, R17.2
- net GND: now also C2.2; no longer 3V3_REG.GND, C21.2, C24.2, C4.2, C5.2, D2.A, R18.1, R20.1
Other:
- note added: "R13 may need to be tested. EN(P4) needs to be above 1.35V to turn on the regulator, but the datasheet is unclear about how to configure the voltage divider."
- note added: "The 5V regulator is 50V tolerant. The voltage divider on EN may need to be adjusted."
- note removed: "12V to 3V3 Regulator"
- note removed: "4.7uF"
- note removed: "Both 5V & 3V3 regulators are 50V tolerant. The voltage divider on EN may need to be adjusted."
- note removed: "R4 & R6 may need to be tested. EN(P4) needs to be above 1.35V to turn on the regulator, but the datasheet is unclear about how to configure the voltage divider."
- moved on the sheet: 5V_REG, C20, C23, C6, CR1, J1, L1, R1, R13, R4, R5

Commit message: Last Minute Fixes.
Corrected Morpho Connector Spacing.
Made all traces min 10 mil.
Connections:
- net AGND: no longer CN10.32
Other:
- note added: "TBD Sensor Inputs."
- note removed: "Valve Position Sensor Inputs."
Changed lines of the file:
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@@
 <sheets>
 <sheet>
+<description>5V Power Regulator</description>
 <plain>
 <text x="77.47" y="173.99" size="1.778" layer="97">12V to 5V Regulator</text>
@@
 </sheet>
 <sheet>
+<description>STM Morpho Connector</description>
 <plain>
 <text x="62.23" y="205.74" size="3.81" layer="97">STM Nucleo G071RB Morpho Connectorsfor the MCU Eval Board.</text>
@@
 <label x="157.48" y="128.27" size="1.27" layer="95" rot="R180" xref="yes"/>
 </segment>
-<segment>
-<pinref part="CN10" gate="G$1" pin="32"/>
-<wire x1="173.99" y1="100.33" x2="181.61" y2="100.33" width="0.1524" layer="91"/>
-<label x="181.61" y="100.33" size="1.27" layer="95" xref="yes"/>
-</segment>
 </net>
 <net name="TBD_SENSOR_5" class="0">
@@
 </sheet>
 <sheet>
+<description>Solenoid Switches</description>
 <plain>
 <text x="7.62" y="5.08" size="1.778" layer="97">All Resistors and Capacitors are 0805, unless otherwise noted.</text>
@@
 </sheet>
 <sheet>
+<description>TBD Sensor Inputs</description>
 <plain>
-<text x="35.56" y="199.39" size="5.08" layer="97">Valve Position Sensor Inputs.</text>
+<text x="35.56" y="199.39" size="5.08" layer="97">TBD Sensor Inputs.</text>
 <text x="35.56" y="191.77" size="2.54" layer="97">Screw Terminal are 0.1" Pitch.</text>
 <text x="7.62" y="3.81" size="1.778" layer="97">All Resistors and Capacitors are 0805, unless otherwise noted.</text>
