File: actuator-controller/TSAR_Actuator_Controller.sch (EAGLE design)
At the start: 143 parts, among them Q1 220mA/50V/3.5Ω, Q10 220mA/50V/3.5Ω, Q11 IRF9530, Q12 220mA/50V/3.5Ω, Q13 IRF9530, Q14 220mA/50V/3.5Ω, Q15 IRF9530, Q16 220mA/50V/3.5Ω, Q17 IRF9530, Q18 220mA/50V/3.5Ω, Q19 IRF9530, Q2 IRF9530, Q20 220mA/50V/3.5Ω, Q3 IRF9530, Q4 220mA/50V/3.5Ω, Q5 IRF9530, Q6 220mA/50V/3.5Ω, Q7 IRF9530, Q8 220mA/50V/3.5Ω, Q9 IRF9530

Commit message: Attributes Added to AC Board
Parts:
- 12V, SENSOR_0, SENSOR_1, SENSOR_2, SENSOR_3, SENSOR_4, SENSOR_5, SENSOR_6, SENSOR_7, SENSOR_8, SENSOR_9, SOLENOID_0, SOLENOID_1, SOLENOID_2, SOLENOID_3, SOLENOID_4, SOLENOID_5, SOLENOID_6, SOLENOID_7, SOLENOID_8, SOLENOID_9: DIS (none) -> Digi-Key; DPN (none) -> A98333-ND; MFR (none) -> TE Connectivity AMP Connectors; MPN (none) -> 282834-2
- 5V_REG: DIS (none) -> Digi-Key; DPN (none) -> 1589-1120-1-ND; MFR (none) -> Monolithic Power Systems Inc.; MPN (none) -> MP2456GJ-P
- C1, C12, C13, C14, C15, C17, C18, C19, C40, C41: DIS (none) -> Digi-Key; DPN (none) -> 399-1124-1-ND; MFR (none) -> KEMET; MPN (none) -> C0805C121J5GACTU
- C2: DIS (none) -> Digi-Key; DPN (none) -> 490-16481-1-ND; MFR (none) -> Murata Electronics; MPN (none) -> GCG31CR71E475JA01L
- C20, C6: DIS (none) -> Digi-Key; DPN (none) -> 490-16481-1-ND; MFR (none) -> Murata Electronics; MPN (none) -> GCM21BR72A104KA37L
- C23: DIS (none) -> Digi-Key; DPN (none) -> 399-4925-1-ND; MFR (none) -> KEMET; MPN (none) -> C0805C106K8PACTU
- CN10, CN7: DIS (none) -> Digi-Key; DPN (none) -> S7122-ND; MFR (none) -> Sullins Connector Solutions; MPN (none) -> PPPC192LFBN-RC
- CR1: DIS (none) -> Digi-Key; DPN (none) -> 1N4148W-FDICT-ND; MFR (none) -> Diodes Incorporated; MPN (none) -> 1N4148W-7-F
- D1: DIS (none) -> Digi-Key; DPN (none) -> SBRT3U45SA-13DICT-ND; MFR (none) -> Diodes Incorporated; MPN (none) -> SBRT3U45SA-13
- D10, D11, D13, D3, D4, D5, D6, D7, D8, D9: DIS (none) -> Digi-Key; DPN (none) -> 1514-CMPSH1-4TRPBFREECT-ND; MFR (none) -> Central Semiconductor Corp; MPN (none) -> CMPSH1-4 TR PBFREE
- D12, D14, D15, D16, D17, D18, D19, D20, D21, D22: DIS (none) -> Digi-Key; DPN (none) -> D5V0H1U2LP1610-7DICT-ND; MFR (none) -> Diodes Incorporated; MPN (none) -> D5V0H1U2LP1610-7
- J1: DIS (none) -> Digi-Key; DPN (none) -> A113320-ND; MFR (none) -> TE Connectivity AMP Connectors; MPN (none) -> 282837-2
- L1: DIS (none) -> Digi-Key; DPN (none) -> 445-174699-1-ND; MFR (none) -> TDK Corporation; MPN (none) -> CLF5030NIT-100M-D
- Q1, Q10, Q12, Q14, Q16, Q18, Q20, Q4, Q6, Q8: DIS (none) -> Digi-Key; DPN (none) -> 1727-1142-1-ND; MFR (none) -> Nexperia USA Inc.; MPN (none) -> BSS138P,215
- Q11, Q13, Q15, Q17, Q19, Q2, Q3, Q5, Q7, Q9: DIS (none) -> Digi-Key; DPN (none) -> IRF9530NPBF-ND; MFR (none) -> Infineon Technologies; MPN (none) -> IRF9530NPBF
- R1, R16, R23, R26, R29, R3, R32, R35, R38, R41, R44: DIS (none) -> Digi-Key; DPN (none) -> 311-10.0KCRCT-ND; MFR (none) -> Yageo; MPN (none) -> RC0805FR-0710KL
- R10, R11, R12, R14, R15, R46, R47, R48, R8, R9: DIS (none) -> Digi-Key; DPN (none) -> 311-1.0KARCT-ND; MFR (none) -> Yageo; MPN (none) -> RC0805JR-071KL
- R2, R22, R25, R28, R31, R34, R37, R40, R43, R6: DIS (none) -> Digi-Key; DPN (none) -> 311-4.70KCRCT-ND; MFR (none) -> Yageo; MPN (none) -> RC0805FR-074K7L
- R21, R24, R27, R30, R33, R36, R39, R42, R45, R7: DIS (none) -> Digi-Key; DPN (none) -> RMCF0805FT28K0CT-ND; MFR (none) -> Stackpole Electronics Inc; MPN (none) -> RMCF0805FT28K0
- R4: DIS (none) -> Digi-Key; DPN (none) -> P124KCCT-ND; MFR (none) -> Panasonic Electronic Components; MPN (none) -> ERJ-6ENF1243V
- R5: DIS (none) -> Digi-Key; DPN (none) -> 311-23.7KCRCT-ND; MFR (none) -> Yageo; MPN (none) -> RC0805FR-0723K7L
Other:
- note added: "STM Nucleo G071RB Morpho Connectors for the MCU Eval Board."
- note removed: "STM Nucleo G071RB Morpho Connectorsfor the MCU Eval Board."
