File: actuator-controller/TSAR_Actuator_Controller.sch (EAGLE design)
At the start: 143 parts, among them Q1 220mA/50V/3.5Ω, Q10 220mA/50V/3.5Ω, Q11 IRF9530, Q12 220mA/50V/3.5Ω, Q13 IRF9530, Q14 220mA/50V/3.5Ω, Q15 IRF9530, Q16 220mA/50V/3.5Ω, Q17 IRF9530, Q18 220mA/50V/3.5Ω, Q19 IRF9530, Q2 IRF9530, Q20 220mA/50V/3.5Ω, Q3 IRF9530, Q4 220mA/50V/3.5Ω, Q5 IRF9530, Q6 220mA/50V/3.5Ω, Q7 IRF9530, Q8 220mA/50V/3.5Ω, Q9 IRF9530

Commit message: Regulator work
Other:
- note added: "12V/24V Connector from PoE"
- note added: "12V/24V to 5V Regulator"
- note added: "R13 may need to be tested. EN(P4) needs to be above 1.35V to turn on the regulator. Make sure the sink current of EN pin does not exceed 100uA"
- note removed: "12V Connector from PoE"
- note removed: "12V to 5V Regulator"
- note removed: "R13 may need to be tested. EN(P4) needs to be above 1.35V to turn on the regulator, but the datasheet is unclear about how to configure the voltage divider."
Changed lines of the file:
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@@
 <attribute name="DPN" value="399-1124-1-ND"/>
 <attribute name="MFR" value="KEMET"/>
-<attribute name="MPN" value="C0805C121J5GACTU
-"/>
+<attribute name="MPN" value="C0805C121J5GACTU "/>
 </part>
 <part name="GND10" library="supply1" library_urn="urn:adsk.eagle:library:371" deviceset="GND" device=""/>
@@
 <attribute name="DPN" value="399-1124-1-ND"/>
 <attribute name="MFR" value="KEMET"/>
-<attribute name="MPN" value="C0805C121J5GACTU
-"/>
+<attribute name="MPN" value="C0805C121J5GACTU "/>
 </part>
 <part name="GND1" library="supply1" library_urn="urn:adsk.eagle:library:371" deviceset="GND" device=""/>
@@
 <attribute name="DPN" value="399-1124-1-ND"/>
 <attribute name="MFR" value="KEMET"/>
-<attribute name="MPN" value="C0805C121J5GACTU
-"/>
+<attribute name="MPN" value="C0805C121J5GACTU "/>
 </part>
 <part name="GND7" library="supply1" library_urn="urn:adsk.eagle:library:371" deviceset="GND" device=""/>
@@
 <attribute name="DPN" value="399-1124-1-ND"/>
 <attribute name="MFR" value="KEMET"/>
-<attribute name="MPN" value="C0805C121J5GACTU
-"/>
+<attribute name="MPN" value="C0805C121J5GACTU "/>
 </part>
 <part name="GND15" library="supply1" library_urn="urn:adsk.eagle:library:371" deviceset="GND" device=""/>
@@
 <attribute name="DPN" value="399-1124-1-ND"/>
 <attribute name="MFR" value="KEMET"/>
-<attribute name="MPN" value="C0805C121J5GACTU
-"/>
+<attribute name="MPN" value="C0805C121J5GACTU "/>
 </part>
 <part name="GND18" library="supply1" library_urn="urn:adsk.eagle:library:371" deviceset="GND" device=""/>
@@
 <attribute name="DPN" value="399-1124-1-ND"/>
 <attribute name="MFR" value="KEMET"/>
-<attribute name="MPN" value="C0805C121J5GACTU
-"/>
+<attribute name="MPN" value="C0805C121J5GACTU "/>
 </part>
 <part name="GND103" library="supply1" library_urn="urn:adsk.eagle:library:371" deviceset="GND" device=""/>
@@
 <attribute name="DPN" value="399-1124-1-ND"/>
 <attribute name="MFR" value="KEMET"/>
-<attribute name="MPN" value="C0805C121J5GACTU
-"/>
+<attribute name="MPN" value="C0805C121J5GACTU "/>
 </part>
 <part name="GND106" library="supply1" library_urn="urn:adsk.eagle:library:371" deviceset="GND" device=""/>
@@
 <attribute name="DPN" value="399-1124-1-ND"/>
 <attribute name="MFR" value="KEMET"/>
-<attribute name="MPN" value="C0805C121J5GACTU
-"/>
+<attribute name="MPN" value="C0805C121J5GACTU "/>
 </part>
 <part name="GND109" library="supply1" library_urn="urn:adsk.eagle:library:371" deviceset="GND" device=""/>
@@
 <attribute name="DPN" value="399-1124-1-ND"/>
 <attribute name="MFR" value="KEMET"/>
-<attribute name="MPN" value="C0805C121J5GACTU
-"/>
+<attribute name="MPN" value="C0805C121J5GACTU "/>
 </part>
 <part name="GND112" library="supply1" library_urn="urn:adsk.eagle:library:371" deviceset="GND" device=""/>
@@
 <attribute name="DPN" value="399-1124-1-ND"/>
 <attribute name="MFR" value="KEMET"/>
-<attribute name="MPN" value="C0805C121J5GACTU
-"/>
+<attribute name="MPN" value="C0805C121J5GACTU "/>
 </part>
 <part name="GND115" library="supply1" library_urn="urn:adsk.eagle:library:371" deviceset="GND" device=""/>
@@
 <description>5V Power Regulator</description>
 <plain>
-<text x="77.47" y="173.99" size="1.778" layer="97">12V to 5V Regulator</text>
+<text x="77.47" y="173.99" size="1.778" layer="97">12V/24V to 5V Regulator</text>
 <text x="120.65" y="166.37" size="1.778" layer="96">1N4148W-7-F</text>
 <text x="8.89" y="124.46" size="1.778" layer="97">R13 may need to be tested.
-EN(P4) needs to be above 1.35V to turn on the regulator,
-but the datasheet is unclear about how to configure the voltage divider.
-</text>
+EN(P4) needs to be above 1.35V to turn on the regulator.
+Make sure the sink current of EN pin does not exceed 100uA</text>
 <text x="7.62" y="115.57" size="1.778" layer="97">The 5V regulator is 50V tolerant.
 The voltage divider on EN may need to be adjusted.</text>
 <text x="21.59" y="193.04" size="2.54" layer="97">Power Regulators</text>
-<text x="190.5" y="193.04" size="1.778" layer="97">12V Connector from PoE</text>
+<text x="190.5" y="193.04" size="1.778" layer="97">12V/24V Connector from PoE</text>
 <text x="186.69" y="170.18" size="1.778" layer="97">VBATT From Test Stand Battery.</text>
 <text x="7.62" y="5.08" size="1.778" layer="97">All Resistors and Capacitors are 0805, unless otherwise noted.</text>

Commit message: fixed attribute errors
Parts:
- 12V: DIS Digi-Key -> (none); DPN A98333-ND -> (none); MFR TE Connectivity AMP Connectors -> (none); MPN 282834-2 -> (none)
Changed lines of the file:
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@@
 </part>
 <part name="GND117" library="supply1" library_urn="urn:adsk.eagle:library:371" deviceset="GND" device=""/>
-<part name="12V" library="TSAR_Controller" deviceset="282834-2" device="">
-<attribute name="DIS" value="Digi-Key"/>
-<attribute name="DPN" value="A98333-ND"/>
-<attribute name="MFR" value="TE Connectivity AMP Connectors"/>
-<attribute name="MPN" value="282834-2"/>
-</part>
+<part name="12V" library="TSAR_Controller" deviceset="282834-2" device=""/>
 <part name="P+4" library="supply1" library_urn="urn:adsk.eagle:library:371" deviceset="+12V" device=""/>
 <part name="GND92" library="supply1" library_urn="urn:adsk.eagle:library:371" deviceset="GND" device=""/>
@@
 <attribute name="VALUE" x="149.86" y="166.37" size="1.778" layer="96" rot="R90"/>
 </instance>
-<instance part="12V" gate="A" x="199.39" y="182.88" smashed="yes" rot="MR180">
-<attribute name="DIS" x="199.39" y="182.88" size="1.778" layer="96" rot="MR180" display="off"/>
-<attribute name="DPN" x="199.39" y="182.88" size="1.778" layer="96" rot="MR180" display="off"/>
-<attribute name="MFR" x="199.39" y="182.88" size="1.778" layer="96" rot="MR180" display="off"/>
-<attribute name="MPN" x="199.39" y="182.88" size="1.778" layer="96" rot="MR180" display="off"/>
-</instance>
+<instance part="12V" gate="A" x="199.39" y="182.88" smashed="yes" rot="MR180"/>
 <instance part="P+4" gate="1" x="196.85" y="187.96" smashed="yes">
 <attribute name="VALUE" x="194.31" y="182.88" size="1.778" layer="96" rot="R90"/>

Commit message: Fixed inconsistency error in actuator controller board
Parts:
- removed SENSOR_0, SENSOR_1, SENSOR_2, SENSOR_3, SENSOR_4, SENSOR_5, SENSOR_6, SENSOR_7, SENSOR_8, SENSOR_9: 282834-2, TSAR_Controller:282834-2
- added SENSOR0, SENSOR1, SENSOR2, SENSOR3, SENSOR4, SENSOR5, SENSOR6, SENSOR7, SENSOR8, SENSOR9: 282834-2, TSAR_Controller:282834-2
Connections:
- removed net N$16: R9.2, SENSOR_7.1
- removed net N$18: R15.2, SENSOR_8.1
- removed net N$20: R48.2, SENSOR_9.1
- new net N$5: R11.2, SENSOR1.1
- new net N$6: R14.2, SENSOR6.1
- new net N$7: R47.2, SENSOR5.1
- net GND: now also SENSOR0.2, SENSOR1.2, SENSOR2.2, SENSOR3.2, SENSOR4.2, SENSOR5.2, SENSOR6.2, SENSOR7.2, SENSOR8.2, SENSOR9.2; no longer SENSOR_0.2, SENSOR_1.2, SENSOR_2.2, SENSOR_3.2, SENSOR_4.2, SENSOR_5.2, SENSOR_6.2, SENSOR_7.2, SENSOR_8.2, SENSOR_9.2
- net N$10: now also R12.2, SENSOR4.1; no longer R11.2, SENSOR_1.1
- net N$11: now also R10.2, SENSOR3.1; no longer R8.2, SENSOR_2.1
- net N$12: now also R48.2, SENSOR9.1; no longer R10.2, SENSOR_3.1
- net N$13: now also R15.2, SENSOR8.1; no longer R12.2, SENSOR_4.1
- net N$14: now also R9.2, SENSOR7.1; no longer R47.2, SENSOR_5.1
- net N$15: now also R46.2, SENSOR0.1; no longer R14.2, SENSOR_6.1
- net N$9: now also R8.2, SENSOR2.1; no longer R46.2, SENSOR_0.1

Commit message: reduced AC board size, attributes, bom
Parts:
- removed H5, H6, H7: STAND-OFF, SparkFun-Hardware:STAND-OFF
- removed J1: (no value), SparkFun-Connectors:CONN_02PTH4
- removed SOLENOID_0, SOLENOID_1, SOLENOID_2, SOLENOID_3, SOLENOID_4, SOLENOID_5, SOLENOID_6, SOLENOID_7, SOLENOID_8, SOLENOID_9: 282834-2, TSAR_Controller:282834-2
- added 5V, IGN., POE+, SOV_1., SOV_2., SOV_3., SOV_4., SOV_5., SOV_6., SOV_7., SOV_8., SOV_9.: LG_T679-F1G2-1, led:LG_T679-F1G2-1
- added BATTERY: (no value), SparkFun-Connectors:CONN_02PTH4
- added C3: 47pF, rcl:C-EUC0805
- added IGN, SOV_1, SOV_2, SOV_3, SOV_4, SOV_5, SOV_6, SOV_7, SOV_8, SOV_9: (no value), pinhead:PINHD-1X2
- added R17, R18, R19, R20, R59, R60, R61, R62, R63, R64, R67: 20k, rcl:R-US_R0603
- added R65, R66: 0, rcl:R-US_R0805
- added R68: 1k, rcl:R-US_R0603
- 12V: value 282834-2 -> (none); device TSAR_Controller:282834-2 -> pinhead:PINHD-1X2; DIS (none) -> Digi-Key; DPN (none) -> 900-0022232021-ND; MFR (none) -> Molex; MPN (none) -> 0022232021
- C2: DPN 490-16481-1-ND -> 399-5507-2-ND; MFR Murata Electronics -> KEMET; MPN GCG31CR71E475JA01L -> C1206C475K5PACTU
- C20, C6: DPN 490-16481-1-ND -> 1276-2444-2-ND; MFR Murata Electronics -> Samsung Electro-Mechanics; MPN GCM21BR72A104KA37L -> CL21B104KBCNFNC
- C23: DPN 399-4925-1-ND -> 587-1295-2-ND; MFR KEMET -> Taiyo Yuden; MPN C0805C106K8PACTU -> EMK212BJ106KG-T
- SENSOR0, SENSOR1, SENSOR2, SENSOR3, SENSOR4, SENSOR5, SENSOR6, SENSOR7, SENSOR8, SENSOR9: value 282834-2 -> (none); device TSAR_Controller:282834-2 -> pinhead:PINHD-1X2; DPN A98333-ND -> 900-0022232021-ND; MFR TE Connectivity AMP Connectors -> Molex; MPN 282834-2 -> 0022232021
Connections:
- new net N$16: R18.1, SOV_4..A
- new net N$17: R19.1, SOV_8..A
- new net N$18: R20.1, SOV_9..A
- new net N$2: IGN..A, R17.1
- new net N$20: R59.1, SOV_5..A
- new net N$21: R60.1, SOV_1..A
- new net N$22: R61.1, SOV_2..A
- new net N$23: R62.1, SOV_6..A
- new net N$24: R63.1, SOV_7..A
- new net N$25: R64.1, SOV_3..A
- new net N$26: C20.1, R65.1
- new net N$27: C3.1, R66.2
- new net N$28: POE+.A, R67.1
- new net N$35: 5V.A, R68.1
- net +12V: now also R67.2
- net +5V: now also C3.2, R4.1, R68.2; no longer R4.2
- net GND: now also 5V.C, BATTERY.2, IGN..C, IGN.2, POE+.C, SOV_1..C, SOV_1.2, SOV_2..C, SOV_2.2, SOV_3..C, SOV_3.2, SOV_4..C, SOV_4.2, SOV_5..C, SOV_5.2, SOV_6..C, SOV_6.2, SOV_7..C, SOV_7.2, SOV_8..C, SOV_8.2, SOV_9..C, SOV_9.2; no longer J1.2, SOLENOID_0.2, SOLENOID_1.2, SOLENOID_2.2, SOLENOID_3.2, SOLENOID_4.2, SOLENOID_5.2, SOLENOID_6.2, SOLENOID_7.2, SOLENOID_8.2, SOLENOID_9.2
- net N$10: now also SENSOR7.1; no longer SENSOR4.1
- net N$14: now also SENSOR4.1; no longer SENSOR7.1
- net N$19: now also R4.2, R66.1; no longer R4.1
- net N$4: now also R65.2; no longer C20.1
- net SOL_GPIO_10: now also IGN.1, R17.2; no longer SOLENOID_0.1
- net SOL_GPIO_11: now also R60.2, SOV_1.1; no longer SOLENOID_1.1
- net SOL_GPIO_12: now also R61.2, SOV_2.1; no longer SOLENOID_2.1
- net SOL_GPIO_13: now also R64.2, SOV_3.1; no longer SOLENOID_3.1
- net SOL_GPIO_14: now also R18.2, SOV_4.1; no longer SOLENOID_4.1
- net SOL_GPIO_15: now also R59.2, SOV_5.1; no longer SOLENOID_5.1
- net SOL_GPIO_16: now also R62.2, SOV_6.1; no longer SOLENOID_6.1
- net SOL_GPIO_17: now also R63.2, SOV_7.1; no longer SOLENOID_7.1
- net SOL_GPIO_18: now also R19.2, SOV_8.1; no longer SOLENOID_8.1
- net SOL_GPIO_19: now also R20.2, SOV_9.1; no longer SOLENOID_9.1
- net VBATT: now also BATTERY.1; no longer J1.1
Other:
- note added: "12V to 5V Regulator This regulator supplies power to the STM processor."
- note added: "All Resistors and Capacitors are 0603 or 0805"
- note added: "NP Resistors are provided to allow for input signals that exceed 3.3V."
- note added: "POE Connector This is the 12 POE from the High Risk POE Splitter. This supplies the power to the STM regulator and the 24V Test Stand Battery triggers. This POE line is along 300ft of ethernet cable, controlled from the Command Laptop. If the Emergency Stop Button is pressed then this POE line will be shut off (followed by the STM and all valves)."
- note added: "Sensor Inputs."
- note added: "These circuits are for controlling the 9 valves and 1 ignitor on the Test Stand. They are triggered by STM GPIOs and powered by the 24V Test Stand Battery"
- note added: "These circuits are for reading the physical valve positions from a separate board. The values are read by the STM Processor. The signals are coming from the valve_indicator board and/or the Hall Effect Sensors which are mounted to each valve. There is 1 extra sensor input."
- note added: "These connectors are the mounts for the STM Nucleo G071RB MCU Eval Board. The Nucleo Board is the processor which holds the state machine, controls the valves, and will read the physical valve positions."
- note added: "VBATT From Test Stand Battery. This is the 24V Battery which only supplies power to the valves and is controlled by STM GPIO pins."
- note added: "Valve and Igniter Controls"
- note removed: "12V/24V Connector from PoE"
- note removed: "12V/24V to 5V Regulator"
- note removed: "NP Resistors are provided to allow for input signlas that exceed 3.3V."
- note removed: "Screw Terminal are 0.1" Pitch."
- note removed: "TBD Sensor Inputs."
- note removed: "VBATT From Test Stand Battery."
- moved on the sheet: 5V_REG, C1, C12, C13, C14, C15, C17, C18, C19, C2, C20, C23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

Commit message: ac, valve indicator, libraries
ac-board: changed attribute.
valve-indicator V1: upgraded processor, changed buck regs, added crystal, layed out all unused processor pins, added battery power sense, updated attributes, and re-layout of entire board.
libraries: created custom library, added new libraries.
Parts:
- 5V, POE+: DPN 350-2035-2-ND -> 732-158301227ACT-ND; MFR Dialight -> Würth Elektronik; MPN 5988070107F -> 158301227A
- IGN., SOV_1., SOV_2., SOV_3., SOV_4., SOV_5., SOV_6., SOV_7., SOV_8., SOV_9.: DPN 2460-L196B-QOC-ND -> 732-158301227ACT-ND; MFR American Opto Plus LED -> Würth Elektronik; MPN L196B-QOC -> 158301227A
Changed lines of the file:
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@@
 <part name="IGN." library="led" library_urn="urn:adsk.eagle:library:259" deviceset="*_T679-?-1" device="F1G2" package3d_urn="urn:adsk.eagle:package:15861/1" technology="LG">
 <attribute name="DIS" value="Digi-Key"/>
-<attribute name="DPN" value="2460-L196B-QOC-ND"/>
-<attribute name="MFR" value="American Opto Plus LED"/>
-<attribute name="MPN" value="L196B-QOC"/>
+<attribute name="DPN" value="732-158301227ACT-ND"/>
+<attribute name="MFR" value="Würth Elektronik"/>
+<attribute name="MPN" value="158301227A"/>
 </part>
 <part name="GND28" library="supply1" library_urn="urn:adsk.eagle:library:371" deviceset="GND" device=""/>
@@
 <part name="SOV_4." library="led" library_urn="urn:adsk.eagle:library:259" deviceset="*_T679-?-1" device="F1G2" package3d_urn="urn:adsk.eagle:package:15861/1" technology="LG">
 <attribute name="DIS" value="Digi-Key"/>
-<attribute name="DPN" value="2460-L196B-QOC-ND"/>
-<attribute name="MFR" value="American Opto Plus LED"/>
-<attribute name="MPN" value="L196B-QOC"/>
+<attribute name="DPN" value="732-158301227ACT-ND"/>
+<attribute name="MFR" value="Würth Elektronik"/>
+<attribute name="MPN" value="158301227A"/>
 </part>
 <part name="GND31" library="supply1" library_urn="urn:adsk.eagle:library:371" deviceset="GND" device=""/>
@@
 <part name="SOV_8." library="led" library_urn="urn:adsk.eagle:library:259" deviceset="*_T679-?-1" device="F1G2" package3d_urn="urn:adsk.eagle:package:15861/1" technology="LG">
 <attribute name="DIS" value="Digi-Key"/>
-<attribute name="DPN" value="2460-L196B-QOC-ND"/>
-<attribute name="MFR" value="American Opto Plus LED"/>
-<attribute name="MPN" value="L196B-QOC"/>
+<attribute name="DPN" value="732-158301227ACT-ND"/>
+<attribute name="MFR" value="Würth Elektronik"/>
+<attribute name="MPN" value="158301227A"/>
 </part>
 <part name="GND32" library="supply1" library_urn="urn:adsk.eagle:library:371" deviceset="GND" device=""/>
@@
 <part name="SOV_9." library="led" library_urn="urn:adsk.eagle:library:259" deviceset="*_T679-?-1" device="F1G2" package3d_urn="urn:adsk.eagle:package:15861/1" technology="LG">
 <attribute name="DIS" value="Digi-Key"/>
-<attribute name="DPN" value="2460-L196B-QOC-ND"/>
-<attribute name="MFR" value="American Opto Plus LED"/>
-<attribute name="MPN" value="L196B-QOC"/>
+<attribute name="DPN" value="732-158301227ACT-ND"/>
+<attribute name="MFR" value="Würth Elektronik"/>
+<attribute name="MPN" value="158301227A"/>
 </part>
 <part name="GND33" library="supply1" library_urn="urn:adsk.eagle:library:371" deviceset="GND" device=""/>
@@
 <part name="SOV_5." library="led" library_urn="urn:adsk.eagle:library:259" deviceset="*_T679-?-1" device="F1G2" package3d_urn="urn:adsk.eagle:package:15861/1" technology="LG">
 <attribute name="DIS" value="Digi-Key"/>
-<attribute name="DPN" value="2460-L196B-QOC-ND"/>
-<attribute name="MFR" value="American Opto Plus LED"/>
-<attribute name="MPN" value="L196B-QOC"/>
+<attribute name="DPN" value="732-158301227ACT-ND"/>
+<attribute name="MFR" value="Würth Elektronik"/>
+<attribute name="MPN" value="158301227A"/>
 </part>
 <part name="GND35" library="supply1" library_urn="urn:adsk.eagle:library:371" deviceset="GND" device=""/>
@@
 <part name="SOV_1." library="led" library_urn="urn:adsk.eagle:library:259" deviceset="*_T679-?-1" device="F1G2" package3d_urn="urn:adsk.eagle:package:15861/1" technology="LG">
 <attribute name="DIS" value="Digi-Key"/>
-<attribute name="DPN" value="2460-L196B-QOC-ND"/>
-<attribute name="MFR" value="American Opto Plus LED"/>
-<attribute name="MPN" value="L196B-QOC"/>
+<attribute name="DPN" value="732-158301227ACT-ND"/>
+<attribute name="MFR" value="Würth Elektronik"/>
+<attribute name="MPN" value="158301227A"/>
 </part>
 <part name="GND38" library="supply1" library_urn="urn:adsk.eagle:library:371" deviceset="GND" device=""/>
@@
 <part name="SOV_2." library="led" library_urn="urn:adsk.eagle:library:259" deviceset="*_T679-?-1" device="F1G2" package3d_urn="urn:adsk.eagle:package:15861/1" technology="LG">
 <attribute name="DIS" value="Digi-Key"/>
-<attribute name="DPN" value="2460-L196B-QOC-ND"/>
-<attribute name="MFR" value="American Opto Plus LED"/>
-<attribute name="MPN" value="L196B-QOC"/>
+<attribute name="DPN" value="732-158301227ACT-ND"/>
+<attribute name="MFR" value="Würth Elektronik"/>
+<attribute name="MPN" value="158301227A"/>
 </part>
 <part name="GND40" library="supply1" library_urn="urn:adsk.eagle:library:371" deviceset="GND" device=""/>
@@
 <part name="SOV_6." library="led" library_urn="urn:adsk.eagle:library:259" deviceset="*_T679-?-1" device="F1G2" package3d_urn="urn:adsk.eagle:package:15861/1" technology="LG">
 <attribute name="DIS" value="Digi-Key"/>
-<attribute name="DPN" value="2460-L196B-QOC-ND"/>
-<attribute name="MFR" value="American Opto Plus LED"/>
-<attribute name="MPN" value="L196B-QOC"/>
+<attribute name="DPN" value="732-158301227ACT-ND"/>
+<attribute name="MFR" value="Würth Elektronik"/>
+<attribute name="MPN" value="158301227A"/>
 </part>
 <part name="GND74" library="supply1" library_urn="urn:adsk.eagle:library:371" deviceset="GND" device=""/>
@@
 <part name="SOV_7." library="led" library_urn="urn:adsk.eagle:library:259" deviceset="*_T679-?-1" device="F1G2" package3d_urn="urn:adsk.eagle:package:15861/1" technology="LG">
 <attribute name="DIS" value="Digi-Key"/>
-<attribute name="DPN" value="2460-L196B-QOC-ND"/>
-<attribute name="MFR" value="American Opto Plus LED"/>
-<attribute name="MPN" value="L196B-QOC"/>
+<attribute name="DPN" value="732-158301227ACT-ND"/>
+<attribute name="MFR" value="Würth Elektronik"/>
+<attribute name="MPN" value="158301227A"/>
 </part>
 <part name="GND75" library="supply1" library_urn="urn:adsk.eagle:library:371" deviceset="GND" device=""/>
@@
 <part name="SOV_3." library="led" library_urn="urn:adsk.eagle:library:259" deviceset="*_T679-?-1" device="F1G2" package3d_urn="urn:adsk.eagle:package:15861/1" technology="LG">
 <attribute name="DIS" value="Digi-Key"/>
-<attribute name="DPN" value="2460-L196B-QOC-ND"/>
-<attribute name="MFR" value="American Opto Plus LED"/>
-<attribute name="MPN" value="L196B-QOC"/>
+<attribute name="DPN" value="732-158301227ACT-ND"/>
+<attribute name="MFR" value="Würth Elektronik"/>
+<attribute name="MPN" value="158301227A"/>
 </part>
 <part name="GND76" library="supply1" library_urn="urn:adsk.eagle:library:371" deviceset="GND" device=""/>
@@
 <part name="POE+" library="led" library_urn="urn:adsk.eagle:library:259" deviceset="*_T679-?-1" device="F1G2" package3d_urn="urn:adsk.eagle:package:15861/1" technology="LG">
 <attribute name="DIS" value="Digi-Key"/>
-<attribute name="DPN" value="350-2035-2-ND"/>
-<attribute name="MFR" value="Dialight"/>
-<attribute name="MPN" value="5988070107F"/>
+<attribute name="DPN" value="732-158301227ACT-ND"/>
+<attribute name="MFR" value="Würth Elektronik"/>
+<attribute name="MPN" value="158301227A"/>
 </part>
 <part name="GND77" library="supply1" library_urn="urn:adsk.eagle:library:371" deviceset="GND" device=""/>
@@
 <part name="5V" library="led" library_urn="urn:adsk.eagle:library:259" deviceset="*_T679-?-1" device="F1G2" package3d_urn="urn:adsk.eagle:package:15861/1" technology="LG">
 <attribute name="DIS" value="Digi-Key"/>
-<attribute name="DPN" value="350-2035-2-ND"/>
-<attribute name="MFR" value="Dialight"/>
-<attribute name="MPN" value="5988070107F"/>
+<attribute name="DPN" value="732-158301227ACT-ND"/>
+<attribute name="MFR" value="Würth Elektronik"/>
+<attribute name="MPN" value="158301227A"/>
 </part>
 <part name="GND78" library="supply1" library_urn="urn:adsk.eagle:library:371" deviceset="GND" device=""/>
