File: actuator-controller/TSAR_Actuator_Controller.sch (EAGLE design)
At the start: 167 parts, among them Q1 220mA/50V/3.5Ω, Q10 220mA/50V/3.5Ω, Q11 IRF9530, Q12 220mA/50V/3.5Ω, Q13 IRF9530, Q14 220mA/50V/3.5Ω, Q15 IRF9530, Q16 220mA/50V/3.5Ω, Q17 IRF9530, Q18 220mA/50V/3.5Ω, Q19 IRF9530, Q2 IRF9530, Q20 220mA/50V/3.5Ω, Q3 IRF9530, Q4 220mA/50V/3.5Ω, Q5 IRF9530, Q6 220mA/50V/3.5Ω, Q7 IRF9530, Q8 220mA/50V/3.5Ω, Q9 IRF9530

Commit message: pin map to Nucleo L476RG
Parts:
- R13: value NP -> 2.2k; device rcl:R-US_R0805 -> oresat-rcl:R-US_0603-C-NOSILK
Connections:
- net 5V_USB_CHG renamed U5V
- net EVAL-VIN renamed VIN
- net NRST renamed RESET
- net PA11 renamed PA_11
- net PA12 renamed PA_12
- net PA14 renamed BOOT0
- net PB10 renamed PB_14
- net PB11 renamed PC_1
- net PB12 renamed PC_0
- net PB2 renamed PB_2
- net PB3 renamed PB_3
- net PB4 renamed PB_4
- net PB5 renamed PB_5
- net PB6 renamed PB_1
- net PB7 renamed PB_7
- net PB8 renamed PB_8
- net PB9 renamed PB_9
- net PC0 renamed PB_11
- net PC1 renamed PB_12
- net PC10 renamed PC_10
- net PC11 renamed PC_11
- net PC12 renamed PC_12
- net PC13 renamed PC_13
- net PC14 renamed PC_14
- net PC15 renamed PC_15
- net PC2 renamed PC_2
- net PC3 renamed PC_3
- net PC4 renamed PA_2
- net PC5 renamed PA_3
- net PC8 renamed PC_8
- net PC9 renamed PC_9
- net PD0 renamed NC1
- net PD1 renamed NC3
- net PD13 renamed PA_13
- net PD15 renamed PA_15
- net PD2 renamed PD_2
- net PD3 renamed NC2
- net PD4 renamed PA_14
- net PD5 renamed NC4
- net PD6 renamed NC5
- net PF0 renamed PH_0
- net PF1 renamed PH_1
- removed net EVAL-3V3: CN7.12, CN7.16
- new net 3V3: CN7.16
- new net IOREF: CN7.12
- net AGND: now also CN10.32; no longer CN10.9
- net GND: now also CN10.9
Other:
- note added: "NC6"
- note added: "NC7"
- note added: "PA_0"
- note added: "PA_1"
- note added: "PA_10"
- note added: "PA_4"
- note added: "PA_5"
- note added: "PA_6"
- note added: "PA_7"
- note added: "PA_8"
- note added: "PA_9"
- note added: "PB_0"
- note added: "PB_10"
- note added: "PB_13"
- note added: "PB_15"
- note added: "PB_6"
- note added: "PC_4"
- note added: "PC_5"
- note added: "PC_6"
- note added: "PC_7"
- note added: "STM Nucleo L476RG Morpho Connectors for the MCU Eval Board."
- note added: "These connectors are the mounts for the STM Nucleo L476RG MCU Eval Board. The Nucleo Board is the processor which holds the state machine, controls the valves, and will read the physical valve positions."
- note removed: "STM Nucleo G071RB Morpho Connectors for the MCU Eval Board."
- note removed: "These connectors are the mounts for the STM Nucleo G071RB MCU Eval Board. The Nucleo Board is the processor which holds the state machine, controls the valves, and will read the physical valve positions."
