File: actuator-controller/TSAR_Actuator_Controller.sch (EAGLE design)
At the start: 167 parts, among them Q1 220mA/50V/3.5Ω, Q10 220mA/50V/3.5Ω, Q11 IRF9530, Q12 220mA/50V/3.5Ω, Q13 IRF9530, Q14 220mA/50V/3.5Ω, Q15 IRF9530, Q16 220mA/50V/3.5Ω, Q17 IRF9530, Q18 220mA/50V/3.5Ω, Q19 IRF9530, Q2 IRF9530, Q20 220mA/50V/3.5Ω, Q3 IRF9530, Q4 220mA/50V/3.5Ω, Q5 IRF9530, Q6 220mA/50V/3.5Ω, Q7 IRF9530, Q8 220mA/50V/3.5Ω, Q9 IRF9530

Commit message: poe/ac/sfe changes, libraries
POE low risk input board created; will manage POE+ power distribution to subsystems. added 24-> 5v regulator for SFE and BB-AI
added libraries for SFE and POE.
SFE: removed 24->5V regulator from SFE, replaced D27&D31 with correct package, replaced ADC to correct SSOP20 package.
AC: replaced all passives with oresat rcl parts
Parts:
- C1, C12, C13, C14, C15, C17, C18, C19, C20, C23, C3, C40, C41, C6: device rcl:C-EUC0805 -> oresat-rcl:C-USC0805K
- C2: device rcl:C-EUC1206 -> oresat-rcl:C-USC1206K
- R1, R10, R11, R12, R14, R15, R16, R2, R21, R22, R23, R24, R25, R26, R27, R28, R29, R3, R30, R31, R32, R33, R34, R35, R36, R37, R38, R39, R4, R40, R41, R42, R43, R44, R45, R46, R47, R48, R49, R5, R50, R51, R52, R53, R54, R55, R56, R57, R58, R6, R65, R66, R7, R8, R9: device rcl:R-US_R0805 -> oresat-rcl:R-US_0805-A-NOSILK
- R17, R18, R19, R20, R59, R60, R61, R62, R63, R64, R67, R68: device rcl:R-US_R0603 -> oresat-rcl:R-US_0603-A-NOSILK
Other:
- note added: "All Resistors and Capacitors are 0603 or 0805; unless marked"
- note added: "C2 is 1206"
- note added: "R13 tested to work at 2.2k. EN(P4) needs to be above 1.35V to turn on the regulator. Make sure the sink current of EN pin does not exceed 100uA"
- note removed: "R13 may need to be tested. EN(P4) needs to be above 1.35V to turn on the regulator. Make sure the sink current of EN pin does not exceed 100uA"

Commit message: SFE/AC changes
AC: began replacing nucleo with bare metal stm
SFE: replaced all passives with oresal parts
Parts:
- removed 5V, POE+: LG_T679-F1G2-1, led:LG_T679-F1G2-1
- removed H1, H2, H3, H4: STAND-OFF, SparkFun-Hardware:STAND-OFF
- added 5V., POE.: (no value), led:LEDCHIPLED_0603
- added H5, H6, H7, H8: #4-BARE_MOUNTING_HOLE/.300, mount:#4-BARE_MOUNTING_HOLE/.300
- IGN., SOV_1., SOV_2., SOV_3., SOV_4., SOV_5., SOV_6., SOV_7., SOV_8., SOV_9.: value LG_T679-F1G2-1 -> (none); device led:LG_T679-F1G2-1 -> led:LEDCHIPLED_0603; DPN 732-158301227ACT-ND -> 2460-L196B-QOC-ND; MFR Würth Elektronik -> American Opto Plus LED; MPN 158301227A -> L196B-QOC
Connections:
- net GND: now also 5V..C, POE..C; no longer 5V.C, POE+.C
- net N$28: now also POE..A; no longer POE+.A
- net N$35: now also 5V..A; no longer 5V.A

Commit message: AC changes. Added library
AC: Replaced headers with STM32 processor. Began direct control connections. To Do: Need to add USB circuit. Update pinout for IDE.
Library: added SPI compatible ADC for SFE board future revision.
Parts:
- removed CN10, CN7: (no value), pinhead:PINHD-2X19
- added U1: STM32L476RGT6, STM32L476RGT6:STM32L476RGT6
Connections:
- removed net 3V3: CN7.16
- removed net AGND: CN10.32
- removed net AVDD: CN10.7
- removed net E5V: CN7.6
- removed net IOREF: CN7.12
- removed net NC1: CN7.9
- removed net NC2: CN7.11
- removed net NC3: CN7.10
- removed net NC4: CN7.26
- removed net NC5: CN10.10
- removed net PH_0: CN7.29
- removed net PH_1: CN7.31
- removed net U5V: CN10.8
- removed net VBAT: CN7.33
- removed net VDD: CN7.5
- removed net VIN: CN7.24
- new net PA_0: U1A.PA0
- new net PA_1: U1A.PA1
- new net PA_4: U1A.PA4
- new net PB_0: U1A.PB0
- new net PB_10: U1A.PB10
- new net PB_13: U1A.PB13
- new net PB_15: U1A.PB15
- new net PB_6: U1A.PB6
- net +5V: no longer CN7.18
- net BOOT0: now also U1A.PH3-BOOT0; no longer CN7.7
- net GND: no longer CN10.20, CN10.9, CN7.19, CN7.20, CN7.22, CN7.8
- net PA_11: now also U1A.PA11; no longer CN10.14
- net PA_12: now also U1A.PA12; no longer CN10.12
- net PA_13: now also U1A.PA13; no longer CN7.13
- net PA_14: now also U1A.PA14; no longer CN7.15
- net PA_15: now also U1A.PA15; no longer CN7.17
- net PA_2: now also U1A.PA2; no longer CN10.35
- net PA_3: now also U1A.PA3; no longer CN10.37
- net PB_1: now also U1A.PB1; no longer CN10.24
- net PB_11: now also U1A.PB11; no longer CN10.18
- net PB_12: now also U1A.PB12; no longer CN10.16
- net PB_14: now also U1A.PB14; no longer CN10.28
- net PB_2: now also U1A.PB2; no longer CN10.22
- net PB_3: now also U1A.PB3; no longer CN10.31
- net PB_4: now also U1A.PB4; no longer CN10.27
- net PB_5: now also U1A.PB5; no longer CN10.29
- net PB_7: now also U1A.PB7; no longer CN7.21
- net PB_8: now also U1A.PB8; no longer CN10.3
- net PB_9: now also U1A.PB9; no longer CN10.5
- net PC_0: now also U1A.PC0; no longer CN7.38
- net PC_1: now also U1A.PC1; no longer CN7.36
- net PC_10: now also U1A.PC10; no longer CN7.1
- net PC_11: now also U1A.PC11; no longer CN7.2
- net PC_12: now also U1A.PC12; no longer CN7.3
- net PC_13: now also U1A.PC13; no longer CN7.23
- net PC_14: now also U1A.PC14-OSC32_IN; no longer CN7.25
- net PC_15: now also U1A.PC15-OSC32_OUT; no longer CN7.27
- net PC_2: now also U1A.PC2; no longer CN7.35
- net PC_3: now also U1A.PC3; no longer CN7.37
- net PC_8: now also U1A.PC8; no longer CN10.2
- net PC_9: now also U1A.PC9; no longer CN10.1
- net PD_2: now also U1A.PD2; no longer CN7.4
- net RESET: now also U1A.NRST; no longer CN7.14
- net SOL_GPIO_0: now also U1A.PA5; no longer CN10.33
- net SOL_GPIO_1: now also U1A.PA6; no longer CN10.36
- net SOL_GPIO_2: now also U1A.PA7; no longer CN10.38
- net SOL_GPIO_3: now also U1A.PA8; no longer CN10.19
- net SOL_GPIO_4: now also U1A.PA9; no longer CN10.4
- net SOL_GPIO_5: now also U1A.PA10; no longer CN10.21
- net SOL_GPIO_6: now also U1A.PC4; no longer CN10.23
- net SOL_GPIO_7: now also U1A.PC5; no longer CN10.26
- net SOL_GPIO_8: now also U1A.PC6; no longer CN10.25
- net SOL_GPIO_9: now also U1A.PC7; no longer CN10.30
- net TBD_SENSOR_0: no longer CN7.28
- net TBD_SENSOR_1: no longer CN7.30
- net TBD_SENSOR_2: no longer CN10.34
- net TBD_SENSOR_3: no longer CN10.6
- net TBD_SENSOR_4: no longer CN7.32
- net TBD_SENSOR_5: no longer CN10.11
- net TBD_SENSOR_6: no longer CN10.13
- net TBD_SENSOR_7: no longer CN10.15
- net TBD_SENSOR_8: no longer CN10.17
- net TBD_SENSOR_9: no longer CN7.34
Other:
- note removed: "NC6"
- note removed: "NC7"
- note removed: "PA_0"
- note removed: "PA_1"
- note removed: "PA_4"
- note removed: "PB_0"
- note removed: "PB_10"
- note removed: "PB_13"
- note removed: "PB_15"
- note removed: "PB_6"
- note removed: "PC_4"
- note removed: "PC_5"
- note removed: "PC_6"
- note removed: "PC_7"

Commit message: AC, SFE, Library Changes
AC: Reverted to headers for Nucleo. Removed sensors (data coming over usb cable to nucleo), removed power regulator (power coming from usb cable). Replaced leds with correct size and attributes.
SFE: Removed RTD/TVS circuits. Added thermocouple inputs and thermocouple amplifier circuit. Finished ADC wiring. Added schematic info annotations. Cleaned up schematic. TODO: change labels to consistent font/size. layout new components, complete attributes for new components.
Library: Added oresat-rcl library.
Parts:
- removed 12V, SENSOR0, SENSOR1, SENSOR2, SENSOR3, SENSOR4, SENSOR5, SENSOR6, SENSOR7, SENSOR8, SENSOR9: (no value), pinhead:PINHD-1X2
- removed 5V., IGN., POE.: (no value), led:LEDCHIPLED_0603
- removed 5V_REG: MP2456GJ-P, TSAR_Controller:MP2456GJ-P
- removed C1, C12, C13, C14, C15, C17, C18, C19, C40, C41: 120pF, oresat-rcl:C-USC0805K
- removed C2: 4.7uF, oresat-rcl:C-USC1206K
- removed C20, C6: 0.1uF, oresat-rcl:C-USC0805K
- removed C23: 10uF, oresat-rcl:C-USC0805K
- removed C3: 47pF, oresat-rcl:C-USC0805K
- removed CR1: 1N4148W-7-F, TSAR_Controller:1N4148W-7-F
- removed D1: DFLS160, diode:DIODE-DO214AA
- removed D12, D14, D15, D16, D17, D18, D19, D20, D21, D22: 5V, SparkFun-DiscreteSemi:DIODE_TVS
- removed H7, H8: #4-BARE_MOUNTING_HOLE/.300, mount:#4-BARE_MOUNTING_HOLE/.300
- removed L1: 10uH, TSAR_Controller:CLF5030NIT-100M-D
- removed R1: 10K, oresat-rcl:R-US_0805-A-NOSILK
- removed R10, R11, R12, R14, R15, R46, R47, R48, R8, R9: 1k, oresat-rcl:R-US_0805-A-NOSILK
- removed R13: 2.2k, oresat-rcl:R-US_0603-C-NOSILK
- removed R4: 124k, oresat-rcl:R-US_0805-A-NOSILK
- removed R49, R50, R51, R52, R53, R54, R55, R56, R57, R58: NP, oresat-rcl:R-US_0805-A-NOSILK
- removed R5: 23.7k, oresat-rcl:R-US_0805-A-NOSILK
- removed R65, R66: 0, oresat-rcl:R-US_0805-A-NOSILK
- removed R67: 20k, oresat-rcl:R-US_0603-A-NOSILK
- removed R68: 1k, oresat-rcl:R-US_0603-A-NOSILK
- removed U1: STM32L476RGT6, STM32L476RGT6:STM32L476RGT6
- added CN10, CN7: (no value), pinhead:PINHD-2X19
- added H3, H4: #4-BARE_MOUNTING_HOLE/.300, mount:#4-BARE_MOUNTING_HOLE/.300
- added SOV_0.: Green, led:LEDCHIP-LED0603
- SOV_1., SOV_2., SOV_3., SOV_4., SOV_5., SOV_6., SOV_7., SOV_8., SOV_9.: value (none) -> Green; device led:LEDCHIPLED_0603 -> led:LEDCHIP-LED0603; DPN 2460-L196B-QOC-ND -> 350-2035-1-ND; MFR American Opto Plus LED -> Dialight; MPN L196B-QOC -> 5988070107F
Connections:
- removed net +12V: 12V.2, 5V_REG.IN, C2.1, C6.1, R1.2, R67.2
- removed net +5V: C23.1, C3.2, CR1.2, L1.2, R4.1, R68.2
- removed net N$10: R12.2, SENSOR7.1
- removed net N$11: R10.2, SENSOR3.1
- removed net N$12: R48.2, SENSOR9.1
- removed net N$13: R15.2, SENSOR8.1
- removed net N$14: R9.2, SENSOR4.1
- removed net N$15: R46.2, SENSOR0.1
- removed net N$19: 5V_REG.FB, R4.2, R5.2, R66.1
- removed net N$26: C20.1, R65.1
- removed net N$27: C3.1, R66.2
- removed net N$28: POE..A, R67.1
- removed net N$3: 5V_REG.EN, R1.1, R13.2
- removed net N$35: 5V..A, R68.1
- removed net N$4: 5V_REG.BST, CR1.1, R65.2
- removed net N$5: R11.2, SENSOR1.1
- removed net N$6: R14.2, SENSOR6.1
- removed net N$7: R47.2, SENSOR5.1
- removed net N$8: 5V_REG.SW, C20.2, D1.C, L1.1
- removed net N$9: R8.2, SENSOR2.1
- removed net PA_2: U1A.PA2
- removed net PA_3: U1A.PA3
- removed net PB_10: U1A.PB10
- removed net PB_13: U1A.PB13
- removed net PB_15: U1A.PB15
- removed net TBD_SENSOR_0: C13.1, D18.C, R46.1, R50.2
- removed net TBD_SENSOR_1: C1.1, D17.C, R11.1, R51.2
- removed net TBD_SENSOR_2: C12.1, D16.C, R52.2, R8.1
- removed net TBD_SENSOR_3: C14.1, D15.C, R10.1, R53.2
- removed net TBD_SENSOR_4: C15.1, D12.C, R12.1, R54.2
- removed net TBD_SENSOR_5: C17.1, D19.C, R47.1, R55.2
- removed net TBD_SENSOR_6: C18.1, D20.C, R14.1, R56.2
- removed net TBD_SENSOR_7: C19.1, D21.C, R49.2, R9.1
- removed net TBD_SENSOR_8: C40.1, D22.C, R15.1, R57.2
- removed net TBD_SENSOR_9: C41.1, D14.C, R48.1, R58.2
- new net 3V3: CN7.16
- new net AGND: CN10.32
- new net AVDD: CN10.7
- new net E5V: CN7.6
- new net IOREF: CN7.12
- new net NC1: CN7.9
- new net NC2: CN7.11
- new net NC3: CN7.10
- new net NC4: CN7.26
- new net NC5: CN10.10
- new net NC_6: CN10.36
- new net NC_7: CN10.38
- new net PA_5: CN10.11
- new net PA_6: CN10.13
- new net PA_7: CN10.15
- new net PC_4: CN10.34
- new net PC_5: CN10.6
- new net PH_0: CN7.29
- new net PH_1: CN7.31
- new net U5V: CN10.8
- new net V5_INPUT: CN7.18
- new net VBAT: CN7.33
- new net VDD: CN7.5
- new net VIN: CN7.24
- net BOOT0: now also CN7.7; no longer U1A.PH3-BOOT0
- net GND: now also CN10.20, CN10.9, CN7.19, CN7.20, CN7.22, CN7.8, SOV_0..C; no longer 12V.1, 5V..C, 5V_REG.GND, C1.2, C12.2, C13.2, C14.2, C15.2, C17.2, C18.2, C19.2, C2.2, C23.2, C40.2, C41.2, C6.2, D1.A, D12.A, D14.A, D15.A, D16.A, D17.A, D18.A, D19.A, D20.A, D21.A, D22.A, IGN..C, POE..C, R13.1, R49.1, R5.1, R50.1, R51.1, R52.1, R53.1, R54.1, R55.1, R56.1, R57.1, R58.1, SENSOR0.2, SENSOR1.2, SENSOR2.2, SENSOR3.2, SENSOR4.2, SENSOR5.2, SENSOR6.2, SENSOR7.2, SENSOR8.2, SENSOR9.2
- net N$2: now also SOV_0..A; no longer IGN..A
- net PA_0: now also CN7.28; no longer U1A.PA0
- net PA_1: now also CN7.30; no longer U1A.PA1
- net PA_11: now also CN10.14; no longer U1A.PA11
- net PA_12: now also CN10.12; no longer U1A.PA12
- net PA_13: now also CN7.13; no longer U1A.PA13
- net PA_14: now also CN7.15; no longer U1A.PA14
- net PA_15: now also CN7.17; no longer U1A.PA15
- net PA_4: now also CN7.32; no longer U1A.PA4
- net PB_0: now also CN7.34; no longer U1A.PB0
- net PB_1: now also CN10.24; no longer U1A.PB1
- net PB_11: now also CN10.18; no longer U1A.PB11
- net PB_12: now also CN10.16; no longer U1A.PB12
- net PB_14: now also CN10.28; no longer U1A.PB14
- net PB_2: now also CN10.22; no longer U1A.PB2
- net PB_3: now also CN10.31; no longer U1A.PB3
- net PB_4: now also CN10.27; no longer U1A.PB4
- net PB_5: now also CN10.29; no longer U1A.PB5
- net PB_6: now also CN10.17; no longer U1A.PB6
- net PB_7: now also CN7.21; no longer U1A.PB7
- net PB_8: now also CN10.3; no longer U1A.PB8
- net PB_9: now also CN10.5; no longer U1A.PB9
- net PC_0: now also CN7.38; no longer U1A.PC0
- net PC_1: now also CN7.36; no longer U1A.PC1
- net PC_10: now also CN7.1; no longer U1A.PC10
- net PC_11: now also CN7.2; no longer U1A.PC11
- net PC_12: now also CN7.3; no longer U1A.PC12
- net PC_13: now also CN7.23; no longer U1A.PC13
- net PC_14: now also CN7.25; no longer U1A.PC14-OSC32_IN
- net PC_15: now also CN7.27; no longer U1A.PC15-OSC32_OUT
- net PC_2: now also CN7.35; no longer U1A.PC2
- net PC_3: now also CN7.37; no longer U1A.PC3
- net PC_8: now also CN10.2; no longer U1A.PC8
- net PC_9: now also CN10.1; no longer U1A.PC9
- net PD_2: now also CN7.4; no longer U1A.PD2
- net RESET: now also CN7.14; no longer U1A.NRST
- net SOL_GPIO_0: now also CN10.33; no longer U1A.PA5
- net SOL_GPIO_1: now also CN10.35; no longer U1A.PA6
- net SOL_GPIO_2: now also CN10.37; no longer U1A.PA7
- net SOL_GPIO_3: now also CN10.19; no longer U1A.PA8
- net SOL_GPIO_4: now also CN10.4; no longer U1A.PA9
- net SOL_GPIO_5: now also CN10.21; no longer U1A.PA10
- net SOL_GPIO_6: now also CN10.23; no longer U1A.PC4
- net SOL_GPIO_7: now also CN10.26; no longer U1A.PC5
- net SOL_GPIO_8: now also CN10.25; no longer U1A.PC6
- net SOL_GPIO_9: now also CN10.30; no longer U1A.PC7
Other:
- note added: "PA_2"
- note added: "PA_3"
- note added: "PB_10"
- note added: "PB_13"
- note added: "PB_15"
- note added: "PC_6"
- note added: "PC_7"
- note added: "Test Stand Battery (24V)"
- note added: "This is the 24V Battery which only supplies power to the valves and is controlled by STM GPIO pins. This battery is controlled by the 12V poe trigger to a solenoid relay."
- note removed: "12V to 5V Regulator This regulator supplies power to the STM processor."
- note removed: "1N4148W-7-F"
- note removed: "All Resistors and Capacitors are 0603 or 0805; unless marked"
- note removed: "C2 is 1206"
- note removed: "Drill Holes for Standoffs."
- note removed: "NP Resistors are provided to allow for input signals that exceed 3.3V."
- note removed: "PA_5"
- note removed: "PA_6"
- note removed: "PA_7"
- note removed: "POE Connector This is the 12 POE from the High Risk POE Splitter. This supplies the power to the STM regulator and the 24V Test Stand Battery triggers. This POE line is along 300ft of ethernet cable, controlled from the Command Laptop. If the Emergency Stop Button is pressed then this POE line will be shut off (followed by the STM and all valves)."
- note removed: "Power Regulators"
- note removed: "R13 tested to work at 2.2k. EN(P4) needs to be above 1.35V to turn on the regulator. Make sure the sink current of EN pin does not exceed 100uA"
- note removed: "Sensor Inputs."
- note removed: "The 5V regulator is 50V tolerant. The voltage divider on EN may need to be adjusted."
- note removed: "These circuits are for reading the physical valve positions from a separate board. The values are read by the STM Processor. The signals are coming from the valve_indicator board and/or the Hall Effect Sensors which are mounted to each valve. There is 1 extra sensor input."
- note removed: "VBATT From Test Stand Battery. This is the 24V Battery which only supplies power to the valves and is controlled by STM GPIO pins."

Commit message: AC, VI, library changes
AC: attribute corrections
VI: corrected MISO/MISI pins
Library: Added REF5025 for ADCs on SFE board.
Parts:
- added JP1: (no value), pinhead:PINHD-1X5
Changed lines of the file:
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@@
 <part name="H5" library="mount" deviceset="#4-BARE_MOUNTING_HOLE" device="/.300"/>
 <part name="H6" library="mount" deviceset="#4-BARE_MOUNTING_HOLE" device="/.300"/>
+<part name="JP1" library="pinhead" library_urn="urn:adsk.eagle:library:325" deviceset="PINHD-1X5" device="" package3d_urn="urn:adsk.eagle:package:22469/2"/>
 </parts>
 <sheets>
@@
 <attribute name="VALUE" x="167.64" y="5.08" size="1.27" layer="96" display="off"/>
 </instance>
+<instance part="JP1" gate="A" x="81.28" y="157.48" smashed="yes">
+<attribute name="NAME" x="74.93" y="165.735" size="1.778" layer="95"/>
+<attribute name="VALUE" x="74.93" y="147.32" size="1.778" layer="96"/>
+</instance>
 </instances>
 <busses>
@@
 <pinref part="CN10" gate="G$1" pin="27"/>
 <wire x1="175.26" y1="99.06" x2="165.1" y2="99.06" width="0.1524" layer="91"/>
-<label x="165.1" y="99.06" size="1.27" layer="95" rot="R180" xref="yes"/>
-</segment>
-</net>
+<label x="160.02" y="99.06" size="1.27" layer="95" rot="R180" xref="yes"/>
+</segment>
+</net>

Commit message: AC, SFE, VI changes
AC: Added 5 pin header for sending UART status updates to the valve indicator board. Will only send the current test stand state status, so recieving data from the Vi. Routed header and added labels. Updated attributes and BOM.
SFE: Routed thermocouple amps and ADCs. Made all labels consistent. Updated attributes and BOM.
VI: Updated attributes and BOM.
Parts:
- JP1: DIS (none) -> Digi-Key; DPN (none) -> AE11083-ND; MFR (none) -> Molex; MPN (none) -> AWHW 10A-0202-T
Connections:
- removed net PA_6: CN10.13
- removed net PB_1: CN10.24
- removed net PC_4: CN10.34
- removed net PC_5: CN10.6
- new net CTS_VI: CN10.13, JP1.4
- new net RTS_VI: CN10.24, JP1.5
- new net RX_VI: CN10.6, JP1.2
- new net TX_VI: CN10.34, JP1.1
- net GND: now also JP1.3
Other:
- note added: "PA_6"
- note added: "PB_1"
- note added: "PC_4"
- note added: "PC_5"
- note added: "This connector sends the current test stand state to the valve indicator board."
- note added: "UART Status to VI"
- moved on the sheet: JP1
Changed lines of the file:
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@@
 <part name="H5" library="mount" deviceset="#4-BARE_MOUNTING_HOLE" device="/.300"/>
 <part name="H6" library="mount" deviceset="#4-BARE_MOUNTING_HOLE" device="/.300"/>
-<part name="JP1" library="pinhead" library_urn="urn:adsk.eagle:library:325" deviceset="PINHD-1X5" device="" package3d_urn="urn:adsk.eagle:package:22469/2"/>
+<part name="JP1" library="pinhead" library_urn="urn:adsk.eagle:library:325" deviceset="PINHD-1X5" device="" package3d_urn="urn:adsk.eagle:package:22469/2">
+<attribute name="DIS" value="Digi-Key"/>
+<attribute name="DPN" value="AE11083-ND"/>
+<attribute name="MFR" value="Molex"/>
+<attribute name="MPN" value="AWHW 10A-0202-T"/>
+</part>
+<part name="GND1" library="supply1" library_urn="urn:adsk.eagle:library:371" deviceset="GND" device=""/>
 </parts>
 <sheets>
@@
 <text x="165.608" y="89.408" size="1.27" layer="97">PA_2</text>
 <text x="165.608" y="86.868" size="1.27" layer="97">PA_3</text>
+<wire x1="58.42" y1="172.72" x2="111.76" y2="172.72" width="0.1524" layer="97" style="shortdash"/>
+<wire x1="111.76" y1="172.72" x2="111.76" y2="137.16" width="0.1524" layer="97" style="shortdash"/>
+<wire x1="111.76" y1="137.16" x2="58.42" y2="137.16" width="0.1524" layer="97" style="shortdash"/>
+<wire x1="58.42" y1="137.16" x2="58.42" y2="172.72" width="0.1524" layer="97" style="shortdash"/>
+<text x="60.96" y="160.02" size="1.778" layer="97">This connector sends the current
+test stand state to the valve indicator
+ board.</text>
+<text x="59.69" y="167.64" size="3.81" layer="97">UART Status to VI</text>
+<text x="166.116" y="117.348" size="1.27" layer="97">PA_6</text>
+<text x="187.452" y="127.508" size="1.27" layer="97">PC_5</text>
+<text x="187.452" y="104.648" size="1.27" layer="97">PB_1</text>
+<text x="187.452" y="91.948" size="1.27" layer="97">PC_4</text>
 </plain>
 <instances>
@@
 <attribute name="VALUE" x="167.64" y="5.08" size="1.27" layer="96" display="off"/>
 </instance>
-<instance part="JP1" gate="A" x="81.28" y="157.48" smashed="yes">
-<attribute name="NAME" x="74.93" y="165.735" size="1.778" layer="95"/>
-<attribute name="VALUE" x="74.93" y="147.32" size="1.778" layer="96"/>
+<instance part="JP1" gate="A" x="76.2" y="152.4" smashed="yes">
+<attribute name="NAME" x="69.85" y="160.655" size="1.778" layer="95"/>
+<attribute name="VALUE" x="69.85" y="142.24" size="1.778" layer="96"/>
+<attribute name="MPN" x="76.2" y="152.4" size="1.27" layer="96" display="off"/>
+<attribute name="DIS" x="76.2" y="152.4" size="1.27" layer="96" display="off"/>
+<attribute name="DPN" x="76.2" y="152.4" size="1.27" layer="96" display="off"/>
+<attribute name="MFR" x="76.2" y="152.4" size="1.27" layer="96" display="off"/>
+</instance>
+<instance part="GND1" gate="1" x="66.04" y="142.24" smashed="yes">
+<attribute name="VALUE" x="63.5" y="139.7" size="1.778" layer="96"/>
 </instance>
 </instances>
@@
 <pinref part="GND79" gate="1" pin="GND"/>
 </segment>
+<segment>
+<pinref part="JP1" gate="A" pin="3"/>
+<wire x1="73.66" y1="152.4" x2="66.04" y2="152.4" width="0.1524" layer="91"/>
+<wire x1="66.04" y1="152.4" x2="66.04" y2="144.78" width="0.1524" layer="91"/>
+<pinref part="GND1" gate="1" pin="GND"/>
+</segment>
 </net>
 <net name="PC_10" class="0">
@@
 </segment>
 </net>
-<net name="PA_6" class="0">
+<net name="CTS_VI" class="0">
 <segment>
 <pinref part="CN10" gate="G$1" pin="13"/>
 <wire x1="175.26" y1="116.84" x2="165.1" y2="116.84" width="0.1524" layer="91"/>
 <label x="165.1" y="116.84" size="1.27" layer="95" rot="MR0" xref="yes"/>
+</segment>
+<segment>
+<pinref part="JP1" gate="A" pin="4"/>
+<wire x1="73.66" y1="149.86" x2="83.82" y2="149.86" width="0.1524" layer="91"/>
+<label x="83.82" y="149.86" size="1.27" layer="95" xref="yes"/>
 </segment>
 </net>
@@
 <pinref part="CN10" gate="G$1" pin="27"/>
 <wire x1="175.26" y1="99.06" x2="165.1" y2="99.06" width="0.1524" layer="91"/>
-<label x="160.02" y="99.06" size="1.27" layer="95" rot="R180" xref="yes"/>
+<label x="165.1" y="99.06" size="1.27" layer="95" rot="R180" xref="yes"/>
 </segment>
 </net>
@@
 </segment>
 </net>
-<net name="PC_5" class="0">
+<net name="RX_VI" class="0">
 <segment>
 <pinref part="CN10" gate="G$1" pin="6"/>
@@
 <label x="193.04" y="127" size="1.27" layer="95" xref="yes"/>
 </segment>
+<segment>
+<pinref part="JP1" gate="A" pin="2"/>
+<wire x1="83.82" y1="154.94" x2="73.66" y2="154.94" width="0.1524" layer="91"/>
+<label x="83.82" y="154.94" size="1.27" layer="95" xref="yes"/>
+</segment>
 </net>
 <net name="U5V" class="0">
@@
 </segment>
 </net>
-<net name="PB_1" class="0">
+<net name="RTS_VI" class="0">
 <segment>
 <pinref part="CN10" gate="G$1" pin="24"/>
 <wire x1="182.88" y1="104.14" x2="193.04" y2="104.14" width="0.1524" layer="91"/>
 <label x="193.04" y="104.14" size="1.27" layer="95" xref="yes"/>
+</segment>
+<segment>
+<pinref part="JP1" gate="A" pin="5"/>
+<wire x1="73.66" y1="147.32" x2="83.82" y2="147.32" width="0.1524" layer="91"/>
+<label x="83.82" y="147.32" size="1.27" layer="95" xref="yes"/>
 </segment>
 </net>
@@
 </segment>
 </net>
-<net name="PC_4" class="0">
+<net name="TX_VI" class="0">
 <segment>
 <pinref part="CN10" gate="G$1" pin="34"/>
@@
 <label x="193.04" y="91.44" size="1.27" layer="95" xref="yes"/>
 </segment>
-</net>
+<segment>
+<pinref part="JP1" gate="A" pin="1"/>
+<wire x1="83.82" y1="157.48" x2="73.66" y2="157.48" width="0.1524" layer="91"/>
+<label x="83.82" y="157.48" size="1.27" layer="95" xref="yes"/>
+</segment>
+</net>

Commit message: AC changes
Added 24V to 12V regulator for single 12V valve, routed, final error check. Update attributes and BOM.
Parts:
- added 12V.REG: Green, led:LEDCHIP-LED0603
- added C43: 100nF, oresat-rcl:C-USC0603K
- added C45: 4.7uF, oresat-rcl:C-USC0805K
- added C46: 0.1uF, oresat-rcl:C-USC0603K
- added C47: 47pF, oresat-rcl:C-USC0603K
- added C50, C51: 1uF, oresat-rcl:C-USC0603K
- added C52, C53: 10uF, oresat-rcl:C-USC1206K
- added D31: DFLS160, DFLS160-7:DFLS160-7
- added L3: 33uH, TSAR_Controller (2):CLF5030NIT-100M-D
- added R1: 20k, oresat-rcl:R-US_0603-A-NOSILK
- added R69: 113k, oresat-rcl:R-US_0805-A-NOSILK
- added R75: 8.2k, oresat-rcl:R-US_0805-A-NOSILK
- added R76: 500k, oresat-rcl:R-US_1206-A
- added R77: NP, oresat-rcl:R-US_0805-A-NOSILK
- added R80, R81: 0, oresat-rcl:R-US_0603-A-NOSILK
- added U$2: MP2456GJ-P, TSAR_Controller (2):MP2456GJ-P
Connections:
- new net +12V: C50.1, C51.1, C52.1, C53.1, L3.2, R1.1, R69.2, R80.2
- new net FLY3: C43.2, D31.C, L3.1, U$2.SW
- new net N$11: C43.1, R81.2
- new net N$12: C47.2, R69.1, R75.2, U$2.FB
- new net N$13: R76.1, R77.2, U$2.EN
- new net N$14: C47.1, R80.1
- new net N$15: R81.1, U$2.BST
- new net N$3: 12V.REG.A, R1.2
- net GND: now also 12V.REG.C, C45.2, C46.2, C50.2, C51.2, C52.2, C53.2, D31.A, R75.1, R77.1, U$2.GND
- net VBATT: now also C45.1, C46.1, R76.2, U$2.IN
Other:
- note added: "12V"
- note added: "24V input, 12V output voltage regulator for SOV-4 (SOV-F04), the only valve that runs at 12V."
- note added: "Voltage Regulator"
