File: actuator-controller/TSAR_Actuator_Controller.sch (EAGLE design)
At the start: 117 parts, among them Q1 220mA/50V/3.5Ω, Q10 220mA/50V/3.5Ω, Q11 IRF9530, Q12 220mA/50V/3.5Ω, Q13 IRF9530, Q14 220mA/50V/3.5Ω, Q15 IRF9530, Q16 220mA/50V/3.5Ω, Q17 IRF9530, Q18 220mA/50V/3.5Ω, Q19 IRF9530, Q2 IRF9530, Q20 220mA/50V/3.5Ω, Q3 IRF9530, Q4 220mA/50V/3.5Ω, Q5 IRF9530, Q6 220mA/50V/3.5Ω, Q7 IRF9530, Q8 220mA/50V/3.5Ω, Q9 IRF9530

Commit message: AC Changes
Attached SOV-6 to 12V input
Connections:
- net +12V: now also Q9.S, R28.2
- net VBATT: no longer Q9.S, R28.2
Changed lines of the file:
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@@
 <attribute name="MPN" value="IRF9530NPBF"/>
 </part>
-<part name="SUPPLY6" library="supply2" library_urn="urn:adsk.eagle:library:372" deviceset="V+" device="" value="VBATT"/>
 <part name="Q10" library="SparkFun-DiscreteSemi" deviceset="MOSFET-NCH" device="-BSS138" value="220mA/50V/3.5Ω">
 <attribute name="DIS" value="Digi-Key"/>
@@
 <part name="FRAME1" library="frames" library_urn="urn:adsk.eagle:library:229" deviceset="A3L-LOC" device=""/>
 <part name="SUPPLY12" library="supply2" library_urn="urn:adsk.eagle:library:372" deviceset="V+" device="" value="VBATT"/>
+<part name="P+1" library="supply1" library_urn="urn:adsk.eagle:library:371" deviceset="+12V" device="" value="+12V"/>
 </parts>
 <sheets>
@@
 <attribute name="MFR" x="231.14" y="172.72" size="1.778" layer="96" display="off"/>
 </instance>
-<instance part="SUPPLY6" gate="1" x="228.6" y="187.96" smashed="yes">
-<attribute name="VALUE" x="227.33" y="189.23" size="1.778" layer="96"/>
-</instance>
 <instance part="Q10" gate="NMOS" x="220.98" y="165.1" smashed="yes">
 <attribute name="NAME" x="226.06" y="165.1" size="1.778" layer="95" font="vector"/>
@@
 <attribute name="MFR" x="327.66" y="96.52" size="1.778" layer="96" display="off"/>
 </instance>
+<instance part="P+1" gate="1" x="228.6" y="187.96" smashed="yes">
+<attribute name="VALUE" x="226.06" y="182.88" size="1.778" layer="96" rot="R90"/>
+</instance>
 </instances>
 <busses>
@@
 </segment>
 <segment>
-<wire x1="233.68" y1="182.88" x2="228.6" y2="182.88" width="0.1524" layer="91"/>
-<pinref part="Q9" gate="G$1" pin="S"/>
-<wire x1="228.6" y1="182.88" x2="223.52" y2="182.88" width="0.1524" layer="91"/>
-<wire x1="233.68" y1="182.88" x2="233.68" y2="177.8" width="0.1524" layer="91"/>
-<pinref part="SUPPLY6" gate="1" pin="V+"/>
-<wire x1="228.6" y1="185.42" x2="228.6" y2="182.88" width="0.1524" layer="91"/>
-<junction x="228.6" y="182.88"/>
-<pinref part="R28" gate="R" pin="2"/>
-</segment>
-<segment>
 <wire x1="233.68" y1="134.62" x2="228.6" y2="134.62" width="0.1524" layer="91"/>
 <pinref part="Q11" gate="G$1" pin="S"/>
@@
 </segment>
 </net>
+<net name="+12V" class="0">
+<segment>
+<wire x1="233.68" y1="182.88" x2="228.6" y2="182.88" width="0.1524" layer="91"/>
+<pinref part="Q9" gate="G$1" pin="S"/>
+<wire x1="228.6" y1="182.88" x2="223.52" y2="182.88" width="0.1524" layer="91"/>
+<wire x1="233.68" y1="182.88" x2="233.68" y2="177.8" width="0.1524" layer="91"/>
+<wire x1="228.6" y1="185.42" x2="228.6" y2="182.88" width="0.1524" layer="91"/>
+<junction x="228.6" y="182.88"/>
+<pinref part="R28" gate="R" pin="2"/>
+<pinref part="P+1" gate="1" pin="+12V"/>
+</segment>
+</net>
