File: LOTO/logicboard.brd (EAGLE design)
At the start: 58.4 x 63.2 mm, 31 parts, among them IC1 74ALS08N, IC2 74ALS08N, Q1 BSS92, Q2 BSS101

Commit message: route management
Routing:
- net N$17: track 37.5 -> 32.1 mm
Changed lines of the file:
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@@
 <?xml version="1.0" encoding="utf-8"?>
 <!DOCTYPE eagle SYSTEM "eagle.dtd">
-<eagle version="9.3.2">
+<eagle version="9.6.2">
 <drawing>
 <settings>
@@
 <wire x1="10.16" y1="41.91" x2="16.51" y2="35.56" width="0.4064" layer="1"/>
 </signal>
-<signal name="N$16">
-<contactref element="R7" pad="2"/>
-<contactref element="IC1" pad="10"/>
-<wire x1="21.59" y1="52.07" x2="25.4" y2="52.07" width="0.4064" layer="1"/>
-<wire x1="25.4" y1="52.07" x2="26.67" y2="50.8" width="0.4064" layer="1"/>
-<wire x1="26.67" y1="50.8" x2="26.67" y2="40.64" width="0.4064" layer="1"/>
-<wire x1="26.67" y1="40.64" x2="27.94" y2="39.37" width="0.4064" layer="1"/>
-<wire x1="27.94" y1="39.37" x2="34.29" y2="39.37" width="0.4064" layer="1"/>
-<wire x1="13.97" y1="59.69" x2="21.59" y2="52.07" width="0.4064" layer="1"/>
-<wire x1="34.29" y1="39.37" x2="38.1" y2="43.18" width="0.4064" layer="1"/>
-</signal>
 <signal name="N$17">
-<contactref element="IC1" pad="12"/>
 <contactref element="R6" pad="2"/>
 <wire x1="25.4" y1="54.61" x2="27.94" y2="52.07" width="0.4064" layer="1"/>
 <wire x1="25.4" y1="54.61" x2="21.59" y2="54.61" width="0.4064" layer="1"/>
 <wire x1="16.51" y1="59.69" x2="21.59" y2="54.61" width="0.4064" layer="1"/>
-<wire x1="34.29" y1="44.45" x2="38.1" y2="48.26" width="0.4064" layer="1"/>
 <wire x1="34.29" y1="43.18" x2="34.29" y2="44.45" width="0.4064" layer="1"/>
 <wire x1="27.94" y1="52.07" x2="27.94" y2="43.18" width="0.4064" layer="1"/>
@@
 <wire x1="29.21" y1="41.91" x2="33.02" y2="41.91" width="0.4064" layer="1"/>
 <wire x1="33.02" y1="41.91" x2="34.29" y2="43.18" width="0.4064" layer="1"/>
+<contactref element="IC1" pad="12"/>
+<wire x1="34.29" y1="44.45" x2="38.1" y2="48.26" width="0" layer="19" extent="1-1"/>
 </signal>
 <signal name="N$18">
@@
 <wire x1="8.89" y1="26.67" x2="16.51" y2="26.67" width="0.4064" layer="16"/>
 </signal>
-<signal name="N$31">
-<contactref element="Q1" pad="3"/>
-<contactref element="POE" pad="1"/>
-<wire x1="-3.81" y1="26.67" x2="-1.27" y2="29.21" width="0.4064" layer="16"/>
-<wire x1="-1.27" y1="29.21" x2="-1.27" y2="58.42" width="0.4064" layer="16"/>
-<wire x1="2.54" y1="62.23" x2="5.08" y2="62.23" width="0.4064" layer="16"/>
-<wire x1="-1.27" y1="58.42" x2="2.54" y2="62.23" width="0.4064" layer="16"/>
-</signal>
 <signal name="N$32">
 <contactref element="JP1" pad="2"/>
@@
 <wire x1="40.64" y1="36.83" x2="40.64" y2="41.91" width="0.4064" layer="16"/>
 </signal>
+<signal name="N$33">
+<contactref element="R7" pad="2"/>
+<contactref element="IC1" pad="10"/>
+<wire x1="21.59" y1="52.07" x2="25.4" y2="52.07" width="0.4064" layer="1"/>
+<wire x1="25.4" y1="52.07" x2="26.67" y2="50.8" width="0.4064" layer="1"/>
+<wire x1="26.67" y1="50.8" x2="26.67" y2="40.64" width="0.4064" layer="1"/>
+<wire x1="26.67" y1="40.64" x2="27.94" y2="39.37" width="0.4064" layer="1"/>
+<wire x1="27.94" y1="39.37" x2="34.29" y2="39.37" width="0.4064" layer="1"/>
+<wire x1="34.29" y1="39.37" x2="38.1" y2="43.18" width="0.4064" layer="1"/>
+<wire x1="13.97" y1="59.69" x2="21.59" y2="52.07" width="0.4064" layer="1"/>
+</signal>
+<signal name="N$10">
+<contactref element="Q1" pad="3"/>
+<contactref element="POE" pad="1"/>
+<wire x1="-3.81" y1="26.67" x2="-1.27" y2="29.21" width="0.4064" layer="16"/>
+<wire x1="-1.27" y1="29.21" x2="-1.27" y2="58.42" width="0.4064" layer="16"/>
+<wire x1="2.54" y1="62.23" x2="5.08" y2="62.23" width="0.4064" layer="16"/>
+<wire x1="-1.27" y1="58.42" x2="2.54" y2="62.23" width="0.4064" layer="16"/>
+</signal>
 </signals>

Commit message: added attributes to loto
Parts:
- removed IC1, IC2: 74ALS08N, 74xx-us:DIL14
- added U1, U2: CD4082BE, CD4082BE:N14
Connections:
- removed net N$21: IC1.6, IC2.4
- removed net N$22: IC1.8, IC2.5
- removed net N$23: IC1.11, IC2.13
- removed net N$24: IC2.12, IC2.6
- removed net N$25: IC2.10, IC2.3
- removed net N$26: IC2.11, IC2.9
- removed net N$33: IC1.10, R7.2
- new net N$16: R9.2, U2.2
- new net VDD: U1.14, U2.14
- new net VSS: U1.7, U2.7
- net GND: no longer IC1.7, IC2.7
- net N$11: now also R4.2, U1.2; no longer IC1.1, R2.2
- net N$12: now also R5.2, U1.3; no longer IC1.2, R11.2
- net N$13: now also R6.2, U1.4; no longer IC1.4, R10.2
- net N$14: now also R7.2, U1.5; no longer IC1.5, R9.2
- net N$15: now also U1.10, U1.9, U2.1; no longer IC1.9, R8.2
- net N$17: now also R10.2, U2.3; no longer IC1.12, R6.2
- net N$18: now also R11.2, U2.4; no longer IC1.13, R5.2
- net N$19: now also R2.2, U2.5; no longer IC2.1, R4.2
- net N$20: now also U1.1, U1.11, U1.12; no longer IC1.3, IC2.2
- net ON: now also U1.13; no longer IC2.8
- net VCC: no longer IC1.14, IC2.14
Routing:
- net N$15: track 41.8 -> 0.00 mm
- net N$33: track 40.1 -> 0.00 mm
- net N$24: track 35.1 -> 0.00 mm
- net N$18: track 35.1 -> 0.00 mm
- net N$17: track 32.1 -> 0.00 mm
- net N$22: track 25.5 -> 0.00 mm
- net N$5: track 25.2 -> 0.00 mm
- net N$14: track 19.7 -> 0.00 mm
- net N$23: track 16.1 -> 0.00 mm
- net N$13: track 16.1 -> 0.00 mm
- net N$21: track 16.1 -> 0.00 mm
- net N$20: track 15.0 -> 0.00 mm
- net N$12: track 9.94 -> 0.00 mm
- net N$25: track 9.72 -> 0.00 mm
- net N$26: track 8.67 -> 0.00 mm
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
Commit message: Updated LOTO boards
Added LOTO housing outline.  Added logic for POE power and gate trigger. Added more circuit protection and power isolation.
Parts:
- removed 48V, POE: (no value), pinhead:1X02
- removed JP1, JP2: (no value), pinhead:1X03
- removed JP5, JP6: (no value), pinhead:1X01
- removed R14: (no value), rcl:0204/5
- added D13: BAS40, diode:SOT23
- added E_STOP, POE+_INJ, POE+_PS, POE_INJ: (no value), pinhead:1X02
- added Q3: IRF9530, transistor-power:TO220BV
- added Q4: 220mA/50V/3.5Ω, SparkFun-DiscreteSemi:SOT23-3
- added R16: 10k, oresat-rcl:.0805-A-NOSILK
- added R21: 28k, oresat-rcl:.0805-A-NOSILK
- D1: value 1N4004 -> BAS40; device diode:DO41-10 -> diode:SOT23
- Q1: value BSS92 -> 220mA/50V/3.5Ω; device transistor-fet:TO92 -> SparkFun-DiscreteSemi:SOT23-3
- Q2: value BSS101 -> IRF9530; device transistor-fet:TO92 -> transistor-power:TO220BV
- R1, R3: value (none) -> 4.7K; device rcl:0204/5 -> oresat-rcl:.0805-A-NOSILK
- R12: value (none) -> 10k; device rcl:0204/5 -> oresat-rcl:.0805-A-NOSILK
- R13: value (none) -> 28k; device rcl:0204/5 -> oresat-rcl:.0805-A-NOSILK
- moved U2 82.4 mm to (30.5, 45.7), turned to 270 degrees
- moved R13 68.7 mm to (-20.3, 16.5), turned to 0 degrees
- moved U1 56.6 mm to (8.89, 45.7), turned to 270 degrees
- moved D1 49.0 mm to (-29.2, 22.9), turned to 0 degrees
- moved R3 42.7 mm to (-30.5, 16.5)
- moved R12 39.5 mm to (-25.4, 16.5), turned to 0 degrees
- moved Q2 36.1 mm to (-26.7, 63.5)
- moved R1 34.9 mm to (-30.5, 44.5), turned to 0 degrees
- moved Q1 24.3 mm to (-17.8, 59.7)
- moved R8 18.2 mm to (11.4, 62.2)
Connections:
- removed net N$27: D1.A, POE.2
- removed net N$28: 48V.1, JP5.1, Q1.2, R1.2
- removed net N$29: Q2.2, R12.1, R3.1
- removed net N$30: Q1.1, Q2.3, R1.1
- removed net N$32: JP1.2, R13.2
- removed net VSS: U1.7, U2.7
- new net N$21: U1.13, U2.5
- new net N$22: D1.1, R13.2
- new net N$23: Q3.G, Q4.3, R3.1
- new net N$24: U2.14
- new net N$25: U1.14
- new net N$54: D13.1, R21.2
- new net SOL_GPIO_1: D1.3, POE_INJ.1, Q3.D
- new net SOL_GPIO_10: D13.3, POE+_INJ.1, Q2.D
- net GND: now also E_STOP.2, POE+_INJ.2, POE+_PS.2, POE_INJ.2, Q1.2, Q4.2, R12.1, R13.1, R16.1, R21.1, U1.7, U2.7; no longer 48V.2, D1.C, JP1.1, JP1.3, Q2.1, R12.2, R14.2
- net N$10: now also Q2.G, R1.1; no longer POE.1
- net N$14: now also U1.11, U1.12; no longer U1.5
- net N$15: now also R8.2; no longer U1.9, U2.1
- net N$16: now also U1.9; no longer U2.2
- net N$17: now also U2.2; no longer U2.3
- net N$18: now also U2.3; no longer U2.4
- net N$19: now also U2.4; no longer U2.5
- net N$20: now also U1.5, U2.1; no longer U1.1, U1.11, U1.12
- net ON: now also Q1.1, Q4.1, R12.2, R16.2, U1.1; no longer R3.2, U1.13
- net VCC: now also E_STOP.1, Q3.S, R3.2; no longer R13.1, R14.1
- net VDD: now also POE+_PS.1, Q2.S, R1.2; no longer U1.14, U2.14
Routing:
- net N$28: track 59.8 -> 0.00 mm
- net N$10: track 40.7 -> 0.00 mm
- net VCC: track 37.2 -> 0.00 mm
- net N$27: track 32.1 -> 0.00 mm
- net N$32: track 20.7 -> 0.00 mm
- net N$29: track 20.0 -> 0.00 mm
- net N$15: track 0.00 -> 15.0 mm
- net N$14: track 0.00 -> 15.0 mm
- net ON: track 14.5 -> 0.00 mm
- net N$30: track 14.3 -> 0.00 mm
- net N$17: track 0.00 -> 10.4 mm
- net N$19: track 0.00 -> 10.3 mm
- net N$18: track 0.00 -> 10.3 mm
- net N$13: track 0.00 -> 6.35 mm
- net N$12: track 0.00 -> 6.35 mm
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- removed copper zone on layer 1, net GND
- removed copper zone on layer 16, net GND

Commit message: LOTO, Library changes
LOTO: added attributes to lotokey board and exported BOM. Updated parts to SMD, updated attributes, completed layout/routes, and exported BOM.
Library: CD4082 SMD AND logic gate for LOTO board added.
Parts:
- removed D13: BAS40, diode:SOT23
- removed JP3, JP4: (no value), pinhead:1X05
- removed R10, R11, R2, R4, R5, R6, R7, R8, R9: (no value), rcl:0204/5
- added D2: CGRM4001-G, diode:SOD-123_MINI-SMA
- added JP1: (no value), pinhead:1X12
- added R_S1, R_S2, R_S3, R_S4, R_S5, R_S6, R_S7, R_S8, R_S9: 1k, oresat-rcl:.0603-C-NOSILK
- D1: value BAS40 -> CGRM4001-G; device diode:SOT23 -> diode:SOD-123_MINI-SMA
- R1, R12, R13, R16, R21, R3: device oresat-rcl:.0805-A-NOSILK -> oresat-rcl:.0805-C-NOSILK
- U1, U2: value CD4082BE -> CD4082BNSR; device CD4082BE:N14 -> CD4082BNSR:NS14
- moved POE+_PS 69.6 mm to (33.3, 40.9)
- moved E_STOP 65.5 mm to (24.8, 40.9)
- moved R12 49.1 mm to (10.2, 50.4)
- moved R3 48.6 mm to (6.35, 48.3)
- moved D1 40.7 mm to (2.54, 48.3), turned to 270 degrees
- moved R1 39.9 mm to (6.35, 59.7)
- moved POE_INJ 37.5 mm to (16.3, 40.9)
- moved R13 37.0 mm to (-1.27, 48.3)
- moved R16 36.7 mm to (10.2, 53.3)
- moved Q3 35.6 mm to (2.54, 55.9)
- moved Q4 31.1 mm to (10.2, 46.7)
- moved POE+_INJ 31.1 mm to (7.87, 40.9)
- moved Q2 29.5 mm to (2.54, 67.3)
- moved Q1 28.1 mm to (10.2, 56.9)
- moved R21 24.4 mm to (-1.27, 59.7)
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Connections:
- removed net N$11: R4.2, U1.2
- removed net N$12: R5.2, U1.3
- removed net N$13: R6.2, U1.4
- removed net N$14: R7.2, U1.11, U1.12
- removed net N$15: R8.2, U1.10
- removed net N$16: R9.2, U1.9
- removed net N$17: R10.2, U2.2
- removed net N$18: R11.2, U2.3
- removed net N$19: R2.2, U2.4
- removed net N$24: U2.14
- removed net N$25: U1.14
- new net +5V: JP1.1, U1.14, U2.14
- new net S1: R_S1.2, U1.4
- new net S2: R_S2.2, U1.3
- new net S3: R_S3.2, U1.2
- new net S4: R_S4.2, U2.3
- new net S5: R_S5.2, U1.9
- new net S6: R_S6.2, U1.11, U1.12
- new net S7: R_S7.2, U2.4
- new net S8: R_S8.2, U2.2
- new net S9: R_S9.2, U1.10
- net GND: now also JP1.2, JP1.3; no longer JP4.5
- net N$1: now also JP1.4, R_S8.1; no longer JP3.1, R4.1
- net N$2: now also JP1.5, R_S4.1; no longer JP3.2, R5.1
- net N$22: now also D1.A; no longer D1.1
- net N$3: now also JP1.6, R_S7.1; no longer JP3.3, R6.1
- net N$4: now also JP1.7, R_S3.1; no longer JP3.4, R7.1
- net N$5: now also JP1.8, R_S2.1; no longer JP3.5, R8.1
- net N$54: now also D2.A; no longer D13.1
- net N$6: now also JP1.9, R_S1.1; no longer JP4.1, R9.1
- net N$7: now also JP1.10, R_S6.1; no longer JP4.2, R10.1
- net N$8: now also JP1.11, R_S9.1; no longer JP4.3, R11.1
- net N$9: now also JP1.12, R_S5.1; no longer JP4.4, R2.1
- net SOL_GPIO_1: now also D1.C; no longer D1.3
- net SOL_GPIO_10: now also D2.C; no longer D13.3
Routing:
- net +5V: track 0.00 -> 48.1 mm
- net VDD: track 0.00 -> 47.2 mm
- net SOL_GPIO_10: track 0.00 -> 31.2 mm
- net VCC: track 0.00 -> 29.6 mm
- net ON: track 0.00 -> 27.1 mm, vias 0 -> 2
- net N$20: track 0.00 -> 23.6 mm, vias 0 -> 2
- net SOL_GPIO_1: track 0.00 -> 21.4 mm
- net N$23: track 0.00 -> 16.2 mm
- net S6: track 0.00 -> 15.8 mm
- net N$10: track 0.00 -> 15.6 mm
- net N$21: track 0.00 -> 15.4 mm
- net N$15: track 15.0 -> 0.00 mm
- net N$14: track 15.0 -> 0.00 mm
- net S9: track 0.00 -> 13.8 mm
- net S5: track 0.00 -> 13.7 mm
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- added copper zone on layer 1, net GND
- added copper zone on layer 16, net GND
Other:
- board size 58.4 x 63.2 mm -> 58.4 x 41.6 mm
- board text added: "LOTO Logic Board"
- board text added: "github/tsar-hardware/LOTO"
