File: POE_plus_input/POE_plus_input.sch (EAGLE design)
At the start: 16 parts, among them U1 LM2673SX-5.0/NOPB

Commit message: POE, Vi board changes
POE Input Board: Added BB outline and mounting holes for BB-AI. Added small board standard outline and adjusted board size. Added attributes to regulator parts.
Valve Indicator: Added small board standard outline and adjusted board size.
Parts:
- added C_OUT1: 100uF/16V, oresat-rcl:C-USC1210K
- added C_OUT2: 33uF/16V, oresat-rcl:C-USC1206K
- added H1, H2, H3, H4, H5, H6, H7, H8: #4-BARE_MOUNTING_HOLE/.300, mount:#4-BARE_MOUNTING_HOLE/.300
- BOOST_CAP: DIS (none) -> Digi-Key; DPN (none) -> 478-5007-1-ND; MFR (none) -> AVX Corporation; MPN (none) -> 06035C103JAT2A
- C_IN1: device oresat-rcl:C-USC0805K -> oresat-rcl:C-USC2220K; DIS (none) -> Digi-Key; DPN (none) -> 565-3335-1-ND; MFR (none) -> United Chemi-Con; MPN (none) -> KTS500B156M55N0T00
- C_IN2: DIS (none) -> Digi-Key; DPN (none) -> 565-3335-1-ND; MFR (none) -> United Chemi-Con; MPN (none) -> KTS500B156M55N0T00
- C_IN3: DIS (none) -> Digi-Key; DPN (none) -> 587-3171-1-ND; MFR (none) -> Taiyo Yuden; MPN (none) -> UMK107ABJ474KA-T
- C_OUT: value 180uF/16V -> 47uF/16V; device oresat-rcl:C-USC0805K -> oresat-rcl:C-USC1210K; DIS (none) -> Digi-Key; DPN (none) -> 490-16309-1-ND; MFR (none) -> Murata Electronics; MPN (none) -> GRM32EC81C476KE15K
- D1: DIS (none) -> Digi-Key; DPN (none) -> SR305-TPMSCT-ND; MFR (none) -> Micro Commercial Co; MPN (none) -> SR305-TP
- I_LIM_ADJ: device oresat-rcl:R-US_0603-A-NOSILK -> oresat-rcl:R-US_1206-A; DIS (none) -> Digi-Key; DPN (none) -> 311-8.20KFRCT-ND; MFR (none) -> Yageo; MPN (none) -> RC1206FR-078K2L
- L1: device rcl:L-USIRF-1 -> oresat-rcl:L_METAL_COMPOSITE_SHIELDED; DIS (none) -> Digi-Key; DPN (none) -> 553-1406-ND; MFR (none) -> Pulse Electronics Power; MPN (none) -> PE-53823SNL
- SOFTSTART: device oresat-rcl:C-USC0805K -> oresat-rcl:C-USC0603K; DIS (none) -> Digi-Key; DPN (none) -> 1276-1091-1-ND; MFR (none) -> Samsung Electro-Mechanics; MPN (none) -> CL10C102JB8NNNC
Connections:
- net +5V: now also C_OUT1.1, C_OUT2.1
- net GND: now also C_OUT1.2, C_OUT2.2
Other:
- note added: "Drill Holes for Standoffs."
- moved on the sheet: C_OUT

Commit message: Stnd outlines, Poe, SFE, Vi changes
Added Standard Outline DXF files to separate folder
POE Input Board: updated attributes, added BOM
SFE: updated attributes, updated BOM
Valve ind: layout changes, added attributes, updated BOM
Parts:
- BBAI_5V, PIT_GREEN, SFE_24V, SFE_5V, VI_24V: DIS (none) -> Digi-Key; DPN (none) -> WM10560CT-ND; MFR (none) -> Molex; MPN (none) -> 1718573002
Changed lines of the file:
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@@
 <parts>
 <part name="FRAME1" library="frames" library_urn="urn:adsk.eagle:library:229" deviceset="A4L-LOC" device=""/>
-<part name="VI_24V" library="pinhead" library_urn="urn:adsk.eagle:library:325" deviceset="PINHD-1X2" device="" package3d_urn="urn:adsk.eagle:package:22435/2"/>
-<part name="SFE_24V" library="pinhead" library_urn="urn:adsk.eagle:library:325" deviceset="PINHD-1X2" device="" package3d_urn="urn:adsk.eagle:package:22435/2"/>
-<part name="SFE_5V" library="pinhead" library_urn="urn:adsk.eagle:library:325" deviceset="PINHD-1X2" device="" package3d_urn="urn:adsk.eagle:package:22435/2"/>
-<part name="BBAI_5V" library="pinhead" library_urn="urn:adsk.eagle:library:325" deviceset="PINHD-1X2" device="" package3d_urn="urn:adsk.eagle:package:22435/2"/>
-<part name="PIT_GREEN" library="pinhead" library_urn="urn:adsk.eagle:library:325" deviceset="PINHD-1X2" device="" package3d_urn="urn:adsk.eagle:package:22435/2"/>
+<part name="VI_24V" library="pinhead" library_urn="urn:adsk.eagle:library:325" deviceset="PINHD-1X2" device="" package3d_urn="urn:adsk.eagle:package:22435/2">
+<attribute name="DIS" value="Digi-Key"/>
+<attribute name="DPN" value="WM10560CT-ND"/>
+<attribute name="MFR" value="Molex"/>
+<attribute name="MPN" value="1718573002"/>
+</part>
+<part name="SFE_24V" library="pinhead" library_urn="urn:adsk.eagle:library:325" deviceset="PINHD-1X2" device="" package3d_urn="urn:adsk.eagle:package:22435/2">
+<attribute name="DIS" value="Digi-Key"/>
+<attribute name="DPN" value="WM10560CT-ND"/>
+<attribute name="MFR" value="Molex"/>
+<attribute name="MPN" value="1718573002"/>
+</part>
+<part name="SFE_5V" library="pinhead" library_urn="urn:adsk.eagle:library:325" deviceset="PINHD-1X2" device="" package3d_urn="urn:adsk.eagle:package:22435/2">
+<attribute name="DIS" value="Digi-Key"/>
+<attribute name="DPN" value="WM10560CT-ND"/>
+<attribute name="MFR" value="Molex"/>
+<attribute name="MPN" value="1718573002"/>
+</part>
+<part name="BBAI_5V" library="pinhead" library_urn="urn:adsk.eagle:library:325" deviceset="PINHD-1X2" device="" package3d_urn="urn:adsk.eagle:package:22435/2">
+<attribute name="DIS" value="Digi-Key"/>
+<attribute name="DPN" value="WM10560CT-ND"/>
+<attribute name="MFR" value="Molex"/>
+<attribute name="MPN" value="1718573002"/>
+</part>
+<part name="PIT_GREEN" library="pinhead" library_urn="urn:adsk.eagle:library:325" deviceset="PINHD-1X2" device="" package3d_urn="urn:adsk.eagle:package:22435/2">
+<attribute name="DIS" value="Digi-Key"/>
+<attribute name="DPN" value="WM10560CT-ND"/>
+<attribute name="MFR" value="Molex"/>
+<attribute name="MPN" value="1718573002"/>
+</part>
 <part name="POE_IN" library="adafruit" library_urn="urn:adsk.eagle:library:420" deviceset="DCBARREL" device="SMT" package3d_urn="urn:adsk.eagle:package:6240730/1" value="24V">
 <attribute name="DIS" value="Digi-Key"/>
@@
 <attribute name="NAME" x="232.41" y="137.795" size="1.778" layer="95"/>
 <attribute name="VALUE" x="232.41" y="127" size="1.778" layer="96"/>
+<attribute name="DIS" x="238.76" y="132.08" size="1.778" layer="96" display="off"/>
+<attribute name="MFR" x="238.76" y="132.08" size="1.778" layer="96" display="off"/>
+<attribute name="MPN" x="238.76" y="132.08" size="1.778" layer="96" display="off"/>
+<attribute name="DPN" x="238.76" y="132.08" size="1.778" layer="96" display="off"/>
 </instance>
 <instance part="SFE_24V" gate="G$1" x="238.76" y="119.38" smashed="yes">
 <attribute name="NAME" x="232.41" y="125.095" size="1.778" layer="95"/>
 <attribute name="VALUE" x="232.41" y="114.3" size="1.778" layer="96"/>
+<attribute name="DIS" x="238.76" y="119.38" size="1.778" layer="96" display="off"/>
+<attribute name="MFR" x="238.76" y="119.38" size="1.778" layer="96" display="off"/>
+<attribute name="MPN" x="238.76" y="119.38" size="1.778" layer="96" display="off"/>
+<attribute name="DPN" x="238.76" y="119.38" size="1.778" layer="96" display="off"/>
 </instance>
 <instance part="SFE_5V" gate="G$1" x="238.76" y="106.68" smashed="yes">
 <attribute name="NAME" x="232.41" y="112.395" size="1.778" layer="95"/>
 <attribute name="VALUE" x="232.41" y="101.6" size="1.778" layer="96"/>
+<attribute name="DIS" x="238.76" y="106.68" size="1.778" layer="96" display="off"/>
+<attribute name="MFR" x="238.76" y="106.68" size="1.778" layer="96" display="off"/>
+<attribute name="MPN" x="238.76" y="106.68" size="1.778" layer="96" display="off"/>
+<attribute name="DPN" x="238.76" y="106.68" size="1.778" layer="96" display="off"/>
 </instance>
 <instance part="BBAI_5V" gate="G$1" x="238.76" y="93.98" smashed="yes">
 <attribute name="NAME" x="232.41" y="99.695" size="1.778" layer="95"/>
 <attribute name="VALUE" x="232.41" y="88.9" size="1.778" layer="96"/>
+<attribute name="DIS" x="238.76" y="93.98" size="1.778" layer="96" display="off"/>
+<attribute name="MFR" x="238.76" y="93.98" size="1.778" layer="96" display="off"/>
+<attribute name="MPN" x="238.76" y="93.98" size="1.778" layer="96" display="off"/>
+<attribute name="DPN" x="238.76" y="93.98" size="1.778" layer="96" display="off"/>
 </instance>
 <instance part="PIT_GREEN" gate="G$1" x="238.76" y="81.28" smashed="yes">
 <attribute name="NAME" x="232.41" y="86.995" size="1.778" layer="95"/>
 <attribute name="VALUE" x="232.41" y="76.2" size="1.778" layer="96"/>
+<attribute name="DIS" x="238.76" y="81.28" size="1.778" layer="96" display="off"/>
+<attribute name="MFR" x="238.76" y="81.28" size="1.778" layer="96" display="off"/>
+<attribute name="MPN" x="238.76" y="81.28" size="1.778" layer="96" display="off"/>
+<attribute name="DPN" x="238.76" y="81.28" size="1.778" layer="96" display="off"/>
 </instance>
 <instance part="POE_IN" gate="G$1" x="30.48" y="139.7" smashed="yes">

Commit message: POE, VI, and library changes
POE Input: Corrected pad size, updated attributes, adjusted layout.
Valve Indicator: Changed layout (sd card facing 'S').
Parts:
- C_IN2: device oresat-rcl:C-USC0805K -> oresat-rcl:C-USC2220K
- L1: device oresat-rcl:L_METAL_COMPOSITE_SHIELDED -> oresat-rcl:L_SHIELDED
Changed lines of the file:
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@@
 <attribute name="MPN" value="KTS500B156M55N0T00"/>
 </part>
-<part name="C_IN2" library="oresat-rcl" deviceset="C-US" device="C0805K" value="15uF/50V">
+<part name="C_IN2" library="oresat-rcl" deviceset="C-US" device="C2220K" value="15uF/50V">
 <attribute name="DIS" value="Digi-Key"/>
 <attribute name="DPN" value="565-3335-1-ND"/>
@@
 <attribute name="MPN" value="RC1206FR-078K2L"/>
 </part>
-<part name="L1" library="oresat-rcl" deviceset="L_METAL_COMPOSITE_SHIELDED" device="" value="33uH">
+<part name="L1" library="oresat-rcl" deviceset="L_SHIELDED" device="" value="33uH">
 <attribute name="DIS" value="Digi-Key"/>
 <attribute name="DPN" value="553-1406-ND"/>
