File: POE_plus_input/POE_plus_input.brd (EAGLE design)
At the start: 160 x 100 mm, 16 parts, among them U1 LM2673SX-5.0/NOPB

Commit message: POE, Vi board changes
POE Input Board: Added BB outline and mounting holes for BB-AI. Added small board standard outline and adjusted board size. Added attributes to regulator parts.
Valve Indicator: Added small board standard outline and adjusted board size.
Parts:
- added C_OUT1: 100uF/16V, oresat-rcl:C1210K
- added C_OUT2: 33uF/16V, oresat-rcl:C1206K
- added H1, H2, H3, H4, H5, H6, H7, H8: #4-BARE_MOUNTING_HOLE/.300, mount:#4/.300-BARE+STD_NUT_OR_STAR_WASHER
- C_IN1: device oresat-rcl:C0805K -> oresat-rcl:C2220K
- C_OUT: value 180uF/16V -> 47uF/16V; device oresat-rcl:C0805K -> oresat-rcl:C1210K
- I_LIM_ADJ: device oresat-rcl:.0603-A-NOSILK -> oresat-rcl:1206-A
- L1: device rcl:IRF-1 -> oresat-rcl:22MMX22MMX12MM
- SOFTSTART: device oresat-rcl:C0805K -> oresat-rcl:C0603K
- moved BBAI_5V 80.5 mm to (61.9, 5.11)
- moved SFE_5V 79.7 mm to (51.3, 5.11)
- moved VI_24V 74.6 mm to (30.1, 5.11)
- moved PIT_GREEN 73.3 mm to (19.5, 5.11)
- moved SFE_24V 71.5 mm to (40.7, 5.11)
- moved BOOST_CAP 60.0 mm to (44.8, 87.3), turned to 180 degrees
- moved L1 49.6 mm to (69.7, 80.8), turned to 180 degrees
- moved D1 49.3 mm to (25.2, 79.7), turned to 270 degrees
- moved U1 46.0 mm to (51.6, 79.6), turned to 270 degrees
- moved POE_IN 42.5 mm to (6.91, 75.4)
- moved I_LIM_ADJ 38.7 mm to (32.2, 84.3)
- moved C_IN2 29.1 mm to (13.6, 83.9)
- moved C_IN1 27.2 mm to (18.3, 89.6)
- moved C_IN3 26.6 mm to (32.9, 87.5), turned to 90 degrees
- moved C_OUT 20.2 mm to (32.7, 73.3), turned to 180 degrees
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Connections:
- net +5V: now also C_OUT1.1, C_OUT2.1
- net GND: now also C_OUT1.2, C_OUT2.2
Routing:
- net +24V: track 0.00 -> 163.0 mm
- net +5V: track 0.00 -> 146.1 mm
- net N$2: track 0.00 -> 53.1 mm
- net N$6: track 0.00 -> 13.7 mm
- net N$7: track 0.00 -> 8.45 mm
- net N$1: track 0.00 -> 7.83 mm
- added copper zone on layer 1, net GND
Other:
- board size 160 x 100 mm -> 93.3 x 95.1 mm

Commit message: POE, SFE changes
POE: added gnd vias and text info
SFE: moved to mar dxf outline. removed unallocated lines and added valve position sensor pinout. updated attributes. the board is currently unrouted.
Parts:
- added U$5: (no value), psas-logo:PSAS_LOGO_10X10
Other:
- board text added: "Jennifer Jordan, jejor2@pdx.edu https://github.com/psas/tsar-hardware"
- board text added: "POE+ Input Board V0.0"

Commit message: POE, VI, and library changes
POE Input: Corrected pad size, updated attributes, adjusted layout.
Valve Indicator: Changed layout (sd card facing 'S').
Parts:
- C_IN2: device oresat-rcl:C0805K -> oresat-rcl:C2220K
- L1: device oresat-rcl:22MMX22MMX12MM -> oresat-rcl:L_SHIELDED_13MMX13MMX6MM
- moved C_IN1 3.74 mm to (22.0, 90.2)
- moved D1 2.85 mm to (27.8, 80.7)
- moved I_LIM_ADJ 2.34 mm to (34.4, 84.8)
- moved C_IN3 2.10 mm to (34.8, 88.3)
- moved C_OUT2 2.05 mm to (34.6, 77.8)
- moved C_OUT1 2.05 mm to (34.7, 81.2)
- moved C_OUT 1.99 mm to (34.5, 74.2)
- moved U1 1.78 mm to (53.4, 79.6)
- moved C_IN2 1.45 mm to (14.5, 85.1)
- moved SOFTSTART 1.27 mm to (39.4, 70.5)
- moved BOOST_CAP 1.27 mm to (46.1, 87.3)
- moved POE_IN 0.65 mm to (7.04, 74.8)
- turned L1 to 270 degrees
Routing:
- net N$2: track 53.1 -> 55.9 mm
- net +5V: track 146.1 -> 148.7 mm
- net +24V: track 163.0 -> 165.2 mm
- net N$1: track 7.83 -> 8.34 mm

Commit message: POE, VI changes
POE: corrected pad sizes for caps and inductor. Rerouted. Updated attributes and BOM. Final error check
VI: changed name from valve_indicatorV1 to valve_indicator
Parts:
- moved C_IN2 6.39 mm to (20.9, 84.2)
- moved BOOST_CAP 3.30 mm to (49.4, 87.3)
- moved L1 3.30 mm to (73.0, 80.8)
- moved C_IN3 3.30 mm to (38.1, 88.3)
- moved C_OUT 3.30 mm to (37.8, 74.2)
- moved C_OUT1 3.30 mm to (38.0, 81.2)
- moved C_OUT2 3.30 mm to (37.9, 77.8)
- moved D1 3.30 mm to (31.1, 80.7)
- moved I_LIM_ADJ 3.30 mm to (37.7, 84.8)
- moved SOFTSTART 3.30 mm to (42.7, 70.5)
- moved U1 3.30 mm to (56.7, 79.6)
- moved PIT_GREEN 1.78 mm to (19.4, 3.33)
- moved SFE_24V 1.78 mm to (40.6, 3.33)
- moved SFE_5V 1.78 mm to (51.2, 3.33)
- moved VI_24V 1.78 mm to (30.0, 3.33)
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Routing:
- net +24V: track 165.2 -> 175.0 mm
- net +5V: track 148.7 -> 153.6 mm
Other:
- board text added: "+ -"
- board text added: "Jennifer Jordan, jejor2@pdx.edu github.com/psas/tsar-hardware"
- board text added: "POE+ Input Board V0.1"
- board text removed: "Jennifer Jordan, jejor2@pdx.edu https://github.com/psas/tsar-hardware"
- board text removed: "POE+ Input Board V0.0"
