File: valve_indicator/Schematics/valve_indicatorV1.brd (EAGLE design)
At the start: 84.8 x 65.1 mm, 130 parts, among them Q1 PMV45EN2R, Q2 PMV45EN2R, Q3 PMV45EN2R, Q4 PMV45EN2R, Q5 IRF9530, Q6 PMV45EN2R, U1 MC33063ADR, U2 MC33063ADR, U3 STM32F103RET6, X1 ECS-160-10-36Q-ES-TR_16MHZ

Commit message: Vi silkscreen/info layout
Parts:
- C10, C11, C12, C2, C2_H, C2_L, C3, C4, C5, C53, C54, C55, C6, C7, C8, C9: device rcl:C0603 -> oresat-rcl:C0603K
- R1, R10, R11, R12, R13, R14, R15, R16, R17, R18, R2, R20, R3, R4, R5, R6, R7, R8, R9, RS_H, RS_L: device rcl:R0603 -> oresat-rcl:.0603-C-NOSILK
- moved R10 2.55 mm to (43.2, 22.3)
- moved C2 2.54 mm to (34.9, 52.6)
- moved C3 2.54 mm to (40.5, 52.6)
- moved C34 2.54 mm to (14.1, 40.4)
- moved C4 2.54 mm to (46.1, 52.6)
- moved C5 2.54 mm to (51.7, 52.6)
- moved C55 2.54 mm to (60.1, 40.8)
- moved C6 2.54 mm to (57.4, 52.6)
- moved C7 2.54 mm to (63.1, 52.6)
- moved HES9 2.54 mm to (77.6, 48.9)
- moved R2 2.54 mm to (32.8, 52.6)
- moved R2_L 2.54 mm to (9.27, 41.1)
- moved R3 2.54 mm to (38.4, 52.6)
- moved R4 2.54 mm to (43.9, 52.6)
- moved R5 2.54 mm to (49.5, 52.6)
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Routing:
- net +3V3: track 295.6 -> 297.4 mm

Commit message: POE, Vi board changes
POE Input Board: Added BB outline and mounting holes for BB-AI. Added small board standard outline and adjusted board size. Added attributes to regulator parts.
Valve Indicator: Added small board standard outline and adjusted board size.
Parts:
- removed H1, H2, H3, H5: MOUNT-HOLE2.8, holes:2,8
- added H4, H6, H7, H8: #4-BARE_MOUNTING_HOLE/.300, mount:#4/.300-BARE+STD_NUT_OR_STAR_WASHER
- moved C20 16.8 mm to (9.27, 54.5)
- moved C23 16.8 mm to (23.4, 60.3)
- moved C24 16.8 mm to (14.1, 54.5)
- moved C42 16.8 mm to (18.7, 37.5)
- moved C44 16.8 mm to (23.2, 57.4)
- moved C46 16.8 mm to (23.2, 52.2)
- moved C53 16.8 mm to (46.0, 55.9)
- moved HES8 16.8 mm to (82.2, 71.5)
- moved L1 16.8 mm to (10.4, 66.0)
- moved L2 16.8 mm to (28.3, 66.4)
- moved R1_H 16.8 mm to (30.6, 56.3)
- moved RS_L 16.8 mm to (8.99, 59.6)
- moved U1 16.8 mm to (19.2, 64.1)
- moved BATT 16.8 mm to (37.7, 20.7)
- moved C1 16.8 mm to (21.5, 68.6)
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Other:
- board size 84.8 x 65.1 mm -> 93.3 x 95.1 mm

Commit message: Vi changes
Added SD card circuit. Added 9POS for sending position sensor data to the SFE board. Updated attributes.
Parts:
- removed SD_CARD: SD, pinhead:1X06
- removed U3: STM32F103RET6, STM32F103RET6:LQFP64-10X10MM
- added C58: 10uF, oresat-rcl:C0805K
- added IC1: (no value), 40xx:SO16
- added R23: 1k, oresat-rcl:.0603-C-NOSILK
- added SD: (no value), led:CHIP-LED0603
- added TO_SFE: (no value), pinhead:1X09
- added U4: STM32L476RGT6, STM32L476RGT6:LQFP64-10X10MM_STM
- added X2: (no value), adafruit:MICROSD
- moved HES1 11.8 mm to (17.8, 89.3)
- moved HES2 11.8 mm to (27.1, 89.3)
- moved HES3 11.8 mm to (36.3, 89.3)
- moved HES4 11.8 mm to (45.5, 89.3)
- moved HES5 11.8 mm to (54.8, 89.3)
- moved HES6 11.8 mm to (64.0, 89.3)
- moved HES7 11.8 mm to (73.3, 89.3)
- moved CM1 9.09 mm to (35.1, 47.2)
- moved Q5 7.88 mm to (35.6, 41.4)
- moved R19 7.62 mm to (29.1, 38.7)
- moved C54 7.61 mm to (62.9, 67.4)
- moved D2 7.61 mm to (27.4, 66.3)
- moved R21 7.61 mm to (47.9, 49.5)
- moved RS_H 7.61 mm to (43.5, 71.0)
- moved U2 7.61 mm to (37.4, 70.6)
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Connections:
- new net N$20: IC1.6, R23.1, X2.2
- new net N$22: R23.2, SD.C
- new net N$23: IC1.4, X2.3
- new net N$6: IC1.10, SD.A
- new net N$8: IC1.2, X2.5
- net +3V3: now also C58.1, IC1.1, U4.13, U4.19, U4.32, U4.48, U4.64, X2.4; no longer SD_CARD.6, U3.13, U3.19, U3.32, U3.48, U3.64
- net BOOT0: now also U4.60; no longer U3.60
- net GND: now also C58.2, IC1.11, IC1.14, IC1.8, U4.12, U4.18, U4.31, U4.47, U4.63, X2.6, X2.MT1, X2.MT2; no longer SD_CARD.5, U3.12, U3.18, U3.31, U3.47, U3.63
- net IN_CTS: now also U4.44; no longer U3.44
- net IN_H1: now also TO_SFE.1, U4.15; no longer U3.15
- net IN_H2: now also TO_SFE.2, U4.16; no longer U3.16
- net IN_H3: now also TO_SFE.3, U4.17; no longer U3.17
- net IN_H4: now also TO_SFE.4, U4.20; no longer U3.20
- net IN_H5: now also TO_SFE.5, U4.59; no longer U3.59
- net IN_H6: now also TO_SFE.6, U4.58; no longer U3.58
- net IN_H7: now also TO_SFE.7, U4.50; no longer U3.50
- net IN_H8: now also TO_SFE.8, U4.41; no longer U3.41
- net IN_H9: now also TO_SFE.9, U4.14; no longer U3.14
- net IN_RTS: now also U4.45; no longer U3.45
- net IN_UART-RX: now also U4.43; no longer U3.43
- net IN_UART-TX: now also U4.42; no longer U3.42
- net N$30: now also U4.46; no longer U3.46
- net N$32: now also U4.7; no longer U3.7
- net N$9: now also U4.49; no longer U3.49
- net OSC_IN: now also U4.5; no longer U3.5
- net OSC_OUT: now also U4.6; no longer U3.6
- net OUT_BUZZ: now also U4.26; no longer U3.26
- net OUT_CLK: now also IC1.3, IC1.9, U4.21; no longer SD_CARD.4, U3.21
- net OUT_CS: now also IC1.7, U4.27; no longer SD_CARD.1, U3.27
- net OUT_DI: now also IC1.5, U4.23; no longer SD_CARD.2, U3.23
- net OUT_DO: now also U4.22, X2.7; no longer SD_CARD.3, U3.22
- net OUT_LED0: now also U4.61; no longer U3.61
- net OUT_LED1: now also U4.57; no longer U3.57
- net OUT_LED2: now also U4.56; no longer U3.56
- net OUT_LED3: now also U4.55; no longer U3.55
- net PB10: now also U4.29; no longer U3.29
- net PB11: now also U4.30; no longer U3.30
- net PB12: now also U4.33; no longer U3.33
- net PB13: now also U4.34; no longer U3.34
- net PB14: now also U4.35; no longer U3.35
- net PB15: now also U4.36; no longer U3.36
- net PB2: now also U4.28; no longer U3.28
- net PB9: now also U4.62; no longer U3.62
- net PC0: now also U4.8; no longer U3.8
- net PC1: now also U4.9; no longer U3.9
- net PC10: now also U4.51; no longer U3.51
- net PC11: now also U4.52; no longer U3.52
- net PC12: now also U4.53; no longer U3.53
- net PC13: now also U4.2; no longer U3.2
- net PC14-OSC32_IN: now also U4.3; no longer U3.3
- net PC15-OSC32_OUT: now also U4.4; no longer U3.4
- net PC2: now also U4.10; no longer U3.10
- net PC3: now also U4.11; no longer U3.11
- net PC4: now also U4.24; no longer U3.24
- net PC5: now also U4.25; no longer U3.25
- net PC6: now also U4.37; no longer U3.37
- net PC7: now also U4.38; no longer U3.38
- net PC8: now also U4.39; no longer U3.39
- net PC9: now also U4.40; no longer U3.40
- net PD2: now also U4.54; no longer U3.54
- net VBATT: now also U4.1; no longer U3.1
Routing:
- net IN_H1: track 49.8 -> 218.1 mm
- net IN_H2: track 37.1 -> 182.4 mm, vias 0 -> 1
- net IN_H3: track 32.3 -> 146.9 mm
- net IN_H4: track 29.6 -> 134.9 mm
- net IN_H5: track 39.3 -> 134.4 mm
- net IN_H6: track 36.5 -> 120.8 mm
- net IN_H7: track 36.4 -> 117.5 mm
- net +3V3: track 297.4 -> 363.2 mm
- net OUT_CLK: track 13.1 -> 66.7 mm, vias 1 -> 3
- net OUT_DO: track 13.8 -> 66.8 mm, vias 1 -> 4
- net OUT_DI: track 14.6 -> 61.9 mm, vias 1 -> 2
- net IN_H8: track 43.5 -> 90.3 mm
- net OUT_CS: track 15.9 -> 56.8 mm, vias 1 -> 2
- net IN_H9: track 33.9 -> 72.0 mm
- net N$8: track 0.00 -> 31.2 mm
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Other:
- board text added: "valve_indicator_V1.1, 2021/2/21"
- board text removed: "valve_indicator_V1, 2021/1/29"

Commit message: Stnd outlines, Poe, SFE, Vi changes
Added Standard Outline DXF files to separate folder
POE Input Board: updated attributes, added BOM
SFE: updated attributes, updated BOM
Valve ind: layout changes, added attributes, updated BOM
Parts:
- removed TO_SFE: (no value), pinhead:1X09
- added JP3: (no value), pinhead:1X12
Connections:
- net IN_H1: now also JP3.1; no longer TO_SFE.1
- net IN_H2: now also JP3.2; no longer TO_SFE.2
- net IN_H3: now also JP3.3; no longer TO_SFE.3
- net IN_H4: now also JP3.4; no longer TO_SFE.4
- net IN_H5: now also JP3.5; no longer TO_SFE.5
- net IN_H6: now also JP3.6; no longer TO_SFE.6
- net IN_H7: now also JP3.7; no longer TO_SFE.7
- net IN_H8: now also JP3.8; no longer TO_SFE.8
- net IN_H9: now also JP3.9; no longer TO_SFE.9
Routing:
- net IN_H9: track 72.0 -> 75.4 mm
- net IN_H3: track 146.9 -> 148.5 mm
- net IN_H4: track 134.9 -> 136.4 mm
- net IN_H7: track 117.5 -> 118.7 mm
- net IN_H5: track 134.4 -> 135.5 mm
- net IN_H6: track 120.8 -> 121.6 mm
- net IN_H8: track 90.3 -> 90.9 mm

Commit message: VI: updated attributes and layout
Component lead time +1month, changed board for different parts.
Parts:
- C13, C14, C15, C16, C17, C18, C19, C20, C21, C22: device oresat-rcl:C0805K -> oresat-rcl:C1206K
- moved R23 6.10 mm to (32.5, 10.7)
- moved SD 6.10 mm to (35.3, 10.7)
- moved C58 6.10 mm to (28.0, 6.93)
- moved IC1 6.10 mm to (31.4, 17.3)
- moved X2 3.05 mm to (40.7, 3.53)
Routing:
- net IN_H1: track 218.2 -> 215.0 mm
- net OUT_DI: track 61.9 -> 58.8 mm
- net OUT_CS: track 56.8 -> 53.6 mm
- net N$20: track 26.1 -> 23.0 mm
- net +3V3: track 363.2 -> 366.2 mm
- net N$8: track 31.2 -> 28.2 mm
- net N$23: track 28.9 -> 26.0 mm
- net OUT_DO: track 66.8 -> 68.2 mm

Commit message: POE, VI, and library changes
POE Input: Corrected pad size, updated attributes, adjusted layout.
Valve Indicator: Changed layout (sd card facing 'S').
Parts:
- moved X2 18.6 mm to (43.4, 21.9), turned to 0 degrees
- moved SM_STAT 1.02 mm to (50.9, 28.4)
- moved C2_H 0.51 mm to (29.5, 61.2)
- moved POE_IN 0.38 mm to (20.6, 30.8)
- moved 3V3. 0.25 mm to (12.9, 34.4)
Routing:
- net OUT_DO: track 68.2 -> 58.3 mm
- net +3V3: track 366.2 -> 362.0 mm
- net N$20: track 23.0 -> 27.1 mm
- net N$23: track 26.0 -> 29.1 mm
- net N$8: track 28.2 -> 30.6 mm
- net +10V: track 267.7 -> 268.2 mm
- net N$18: track 11.4 -> 11.9 mm

Commit message: AC, VI, library changes
AC: attribute corrections
VI: corrected MISO/MISI pins
Library: Added REF5025 for ADCs on SFE board.
Parts:
- moved C10 2.33 mm to (48.6, 55.1)
- moved R3 0.25 mm to (43.4, 76.0)
- moved R4 0.25 mm to (48.9, 76.0)
- moved R2 0.13 mm to (37.8, 76.2)
- moved R5 0.13 mm to (54.5, 76.2)
- moved R6 0.13 mm to (60.2, 76.2)
- moved R7 0.13 mm to (66.0, 76.2)
Connections:
- new net PA_5: U4.21
- new net PA_6: U4.22
- new net PA_7: U4.23
- net OUT_CLK: now also U4.29; no longer U4.21
- net OUT_DI: now also U4.10; no longer U4.23
- net OUT_DO: now also U4.11; no longer U4.22
- net PB10: no longer U4.29
- net PC2: no longer U4.10
- net PC3: no longer U4.11
Routing:
- net PB10: track 52.0 -> 0.00 mm, vias 1 -> 0
- net PC3: track 31.2 -> 0.00 mm, vias 2 -> 0
- net PC2: track 29.9 -> 0.00 mm, vias 1 -> 0
- net OUT_DO: track 58.3 -> 78.1 mm
- net OUT_DI: track 58.8 -> 71.2 mm, vias 2 -> 4
- net +3V3: track 362.0 -> 369.4 mm
- net PB2: track 75.0 -> 79.0 mm
- net OUT_CLK: track 66.6 -> 64.7 mm

Commit message: SFE, VI changes
SFE: cleared errors
VI: cleared errors
Routing:
- net OUT_DO: track 78.1 -> 80.1 mm
- net OUT_DI: track 71.2 -> 72.6 mm
Changed lines of the file:
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@@
 <via x="69.088" y="40.132" extent="1-16" drill="0.35"/>
 <via x="87.503" y="67.945" extent="1-16" drill="0.35"/>
-<wire x1="52.07" y1="62.23" x2="54.102" y2="60.452" width="0" layer="19" extent="1-1"/>
 </signal>
 <signal name="IN_H1">
@@
 <wire x1="45.974" y1="13.589" x2="45.974" y2="11.471" width="0.3048" layer="1"/>
 <wire x1="45.974" y1="11.471" x2="45.8086" y2="11.3056" width="0.3048" layer="1"/>
-<wire x1="54.9776" y1="68.5934" x2="54.737" y2="68.834" width="0.3048" layer="1"/>
-<wire x1="54.737" y1="68.834" x2="54.737" y2="72.517" width="0.3048" layer="1"/>
 <wire x1="54.737" y1="72.517" x2="53.975" y2="73.279" width="0.3048" layer="1"/>
 <wire x1="53.975" y1="73.279" x2="53.34" y2="73.279" width="0.3048" layer="1"/>
@@
 <wire x1="49.53" y1="64.389" x2="42.926" y2="64.389" width="0.3048" layer="16"/>
 <contactref element="U4" pad="11"/>
-<wire x1="54.9776" y1="68.5934" x2="54.4776" y2="66.5576" width="0" layer="19" extent="1-1"/>
+<wire x1="54.4776" y1="66.5576" x2="54.4776" y2="67.5586" width="0.3048" layer="1"/>
+<wire x1="54.737" y1="67.818" x2="54.737" y2="72.517" width="0.3048" layer="1"/>
+<wire x1="54.4776" y1="67.5586" x2="54.737" y2="67.818" width="0.3048" layer="1"/>
 </signal>
 <signal name="OUT_DI">
@@
 <wire x1="52.197" y1="61.087" x2="52.197" y2="59.69" width="0.3048" layer="16"/>
 <wire x1="53.213" y1="62.103" x2="52.197" y2="61.087" width="0.3048" layer="16"/>
-<wire x1="53.213" y1="62.103" x2="54.102" y2="62.103" width="0.3048" layer="16"/>
+<wire x1="53.213" y1="62.103" x2="54.356" y2="62.103" width="0.3048" layer="16"/>
 <wire x1="43.815" y1="27.051" x2="43.815" y2="30.43465" width="0.3048" layer="16"/>
 <wire x1="44.4726" y1="51.9656" x2="52.197" y2="59.69" width="0.3048" layer="16"/>
-<via x="54.102" y="62.103" extent="1-16" drill="0.35"/>
-<wire x1="55.753" y1="62.611" x2="55.245" y2="62.103" width="0.3048" layer="1"/>
-<wire x1="55.245" y1="62.103" x2="54.102" y2="62.103" width="0.3048" layer="1"/>
-<via x="55.753" y="62.611" extent="1-16" drill="0.35"/>
+<via x="54.356" y="62.103" extent="1-16" drill="0.35"/>
+<wire x1="55.88" y1="62.738" x2="55.88" y2="62.611" width="0.3048" layer="1"/>
+<wire x1="55.88" y1="62.611" x2="55.372" y2="62.103" width="0.3048" layer="1"/>
+<wire x1="55.372" y1="62.103" x2="54.356" y2="62.103" width="0.3048" layer="1"/>
+<via x="55.88" y="62.738" extent="1-16" drill="0.35"/>
 <wire x1="55.38581875" y1="63.881" x2="55.372" y2="63.881" width="0.3048" layer="16"/>
-<wire x1="55.372" y1="63.881" x2="54.483" y2="64.77" width="0.3048" layer="16"/>
-<wire x1="54.483" y1="64.77" x2="54.483" y2="65.024" width="0.3048" layer="16"/>
-<wire x1="55.753" y1="62.611" x2="55.88" y2="62.738" width="0.3048" layer="16"/>
+<wire x1="55.372" y1="63.881" x2="54.991" y2="64.262" width="0.3048" layer="16"/>
+<wire x1="54.991" y1="64.262" x2="54.991" y2="65.151" width="0.3048" layer="16"/>
 <wire x1="55.88" y1="63.38681875" x2="55.88" y2="62.738" width="0.3048" layer="16"/>
 <wire x1="55.88" y1="63.38681875" x2="55.38581875" y2="63.881" width="0.3048" layer="16"/>
-<via x="54.483" y="65.024" extent="1-16" drill="0.35"/>
-<wire x1="54.483" y1="65.024" x2="54.4776" y2="65.0294" width="0.3048" layer="1"/>
 <contactref element="U4" pad="10"/>
-<wire x1="54.4776" y1="65.0294" x2="54.9776" y2="66.5576" width="0" layer="19" extent="1-1"/>
+<via x="54.991" y="65.151" extent="1-16" drill="0.35"/>
+<wire x1="54.9776" y1="66.5576" x2="54.991" y2="66.5442" width="0.3048" layer="1"/>
+<wire x1="54.991" y1="66.5442" x2="54.991" y2="65.151" width="0.3048" layer="1"/>
 </signal>
 <signal name="IN_H8">
@@
 <wire x1="44.3738" y1="65.1256" x2="45.0088" y2="65.7606" width="0.3048" layer="1"/>
 <contactref element="U4" pad="57"/>
-<wire x1="52.959" y1="62.7634" x2="52.959" y2="62.26698125" width="0.3048" layer="1"/>
+<wire x1="52.959" y1="62.7634" x2="52.959" y2="62.52098125" width="0.3048" layer="1"/>
 <wire x1="49.9618" y1="65.7606" x2="52.959" y2="62.7634" width="0.3048" layer="1"/>
-<wire x1="52.959" y1="62.26698125" x2="54.16838125" y2="61.0576" width="0.3048" layer="1"/>
-<wire x1="54.16838125" y1="61.0576" x2="61.4776" y2="61.0576" width="0.3048" layer="1"/>
+<wire x1="52.959" y1="62.52098125" x2="54.42238125" y2="61.0576" width="0.3048" layer="1"/>
+<wire x1="54.42238125" y1="61.0576" x2="61.4776" y2="61.0576" width="0.3048" layer="1"/>
 </signal>
 <signal name="OUT_LED3">
@@
 <wire x1="53.6448" y1="68.8086" x2="53.6448" y2="70.2196" width="0.3048" layer="1"/>
 <wire x1="53.6448" y1="68.8086" x2="53.6448" y2="66.6496" width="0.3048" layer="16"/>
-<wire x1="53.6448" y1="66.6496" x2="53.6448" y2="63.6016" width="0.3048" layer="16"/>
-<wire x1="53.6448" y1="63.6016" x2="53.5813" y2="63.5381" width="0.3048" layer="16"/>
-<wire x1="53.5813" y1="63.5381" x2="52.8828" y2="62.8396" width="0.3048" layer="16"/>
+<wire x1="53.7718" y1="66.6496" x2="53.7718" y2="63.7286" width="0.3048" layer="16"/>
+<wire x1="53.7718" y1="63.7286" x2="52.8828" y2="62.8396" width="0.3048" layer="16"/>
 <wire x1="47.2948" y1="61.1886" x2="48.4378" y2="61.1886" width="0.3048" layer="16"/>
 <wire x1="49.5808" y1="62.3316" x2="48.4378" y2="61.1886" width="0.3048" layer="16"/>
@@
 <via x="59.8678" y="64.9986" extent="1-16" drill="0.35"/>
 <wire x1="59.8678" y1="64.9986" x2="58.2168" y2="66.6496" width="0.3048" layer="16"/>
-<wire x1="58.2168" y1="66.6496" x2="53.6448" y2="66.6496" width="0.3048" layer="16"/>
+<wire x1="58.2168" y1="66.6496" x2="53.7718" y2="66.6496" width="0.3048" layer="16"/>
+<wire x1="53.7718" y1="66.6496" x2="53.6448" y2="66.6496" width="0.3048" layer="16"/>
 <wire x1="59.7408" y1="53.3146" x2="59.7408" y2="52.5386" width="0.3048" layer="1"/>
 <wire x1="59.4868" y1="52.2846" x2="59.7408" y2="52.5386" width="0.3048" layer="1"/>
@@
 <wire x1="59.7408" y1="53.3146" x2="58.0898" y2="53.3146" width="0.3048" layer="16"/>
 <wire x1="58.0898" y1="53.3146" x2="56.4388" y2="54.9656" width="0.3048" layer="16"/>
-<wire x1="56.4388" y1="60.6806" x2="53.5813" y2="63.5381" width="0.3048" layer="16"/>
-<wire x1="56.4388" y1="54.9656" x2="56.4388" y2="60.6806" width="0.3048" layer="16"/>
+<wire x1="56.4388" y1="61.0616" x2="53.7718" y2="63.7286" width="0.3048" layer="16"/>
+<wire x1="56.4388" y1="54.9656" x2="56.4388" y2="61.0616" width="0.3048" layer="16"/>
 <via x="48.6918" y="57.1246" extent="1-16" drill="0.35"/>
 <wire x1="48.6918" y1="57.1246" x2="48.6918" y2="58.7756" width="0.3048" layer="16"/>
@@
 </signal>
 <signal name="PC1">
-<wire x1="62.1538" y1="57.7596" x2="55.4736" y2="64.4398" width="0.3048" layer="16"/>
-<wire x1="62.1538" y1="57.7596" x2="62.7888" y2="57.7596" width="0.3048" layer="16"/>
+<wire x1="62.2808" y1="57.7596" x2="55.88" y2="64.1604" width="0.3048" layer="16"/>
+<wire x1="62.2808" y1="57.7596" x2="62.7888" y2="57.7596" width="0.3048" layer="16"/>
 <wire x1="62.7888" y1="57.7596" x2="71.0438" y2="49.5046" width="0.3048" layer="16"/>
 <via x="71.0438" y="49.5046" extent="1-16" drill="0.35"/>
@@
 <contactref element="U4" pad="9"/>
 <wire x1="55.4856" y1="66.5496" x2="55.4776" y2="66.5576" width="0.3048" layer="1"/>
-<wire x1="55.4736" y1="64.4398" x2="55.4736" y2="64.9986" width="0.3048" layer="16"/>
-<wire x1="55.4736" y1="64.9986" x2="55.499" y2="65.024" width="0.3048" layer="16"/>
-<via x="55.499" y="65.024" extent="1-16" drill="0.35"/>
-<wire x1="55.499" y1="65.024" x2="55.4856" y2="65.0374" width="0.3048" layer="1"/>
-<wire x1="55.4856" y1="65.0374" x2="55.4856" y2="66.5496" width="0.3048" layer="1"/>
+<wire x1="55.88" y1="65.024" x2="55.88" y2="64.1604" width="0.3048" layer="16"/>
+<via x="55.88" y="65.024" extent="1-16" drill="0.35"/>
+<wire x1="55.88" y1="65.024" x2="55.88" y2="65.405" width="0.3048" layer="1"/>
+<wire x1="55.88" y1="65.405" x2="55.4856" y2="65.7994" width="0.3048" layer="1"/>
+<wire x1="55.4856" y1="65.7994" x2="55.4856" y2="66.5496" width="0.3048" layer="1"/>
 </signal>
 <signal name="PC0">
