File: valve_indicator/Schematics/valve_indicatorV1.brd (EAGLE design)
At the start: 93.3 x 95.1 mm, 135 parts, among them Q1 PMV45EN2R, Q2 PMV45EN2R, Q3 PMV45EN2R, Q4 PMV45EN2R, Q5 IRF9530, Q6 PMV45EN2R, U1 MC33063ADR, U2 MC33063ADR, U4 STM32L476RGT6, X1 ECS-160-10-36Q-ES-TR_16MHZ

Commit message: VI Changes
removed vbatt sense. causes non-critical shutdown on battery power
Parts:
- removed Q5: IRF9530, transistor-power:TO220BV
- removed R19: 100k, oresat-rcl:.0805-C-NOSILK
- removed R24: 1k, oresat-rcl:.0603-C-NOSILK
- removed VBATT.: Green, led:CHIP-LED0603
Connections:
- removed net N$11: R24.1, VBATT..A
- net +3V3: no longer Q5.S
- net GND: no longer R19.1, VBATT..C
- net N$12: no longer Q5.G, R19.2
- net VBATT: no longer Q5.D, R24.2
Routing:
- net VBATT: track 77.9 -> 68.0 mm
- net +3V3: track 369.5 -> 361.4 mm
- net N$11: track 1.74 -> 0.00 mm
- net N$12: track 27.4 -> 26.8 mm

Commit message: VI Changes
removed airroutes
Routing:
- net VBATT: track 68.0 -> 2.92 mm, vias 2 -> 0
- net N$12: track 26.8 -> 19.1 mm
