File: valve_indicator/Schematics/valve_indicatorV1.sch (EAGLE design)
At the start: 130 parts, among them Q1 PMV45EN2R, Q2 PMV45EN2R, Q3 PMV45EN2R, Q4 PMV45EN2R, Q5 IRF9530, Q6 PMV45EN2R, U1 MC33063ADR, U2 MC33063ADR, U3 STM32F103RET6, X1 ECS-160-10-36Q-ES-TR_16MHZ

Commit message: Vi silkscreen/info layout
Parts:
- C10, C11, C12, C2, C2_H, C2_L, C3, C4, C5, C53, C54, C55, C6, C7, C8, C9: device rcl:C-USC0603 -> oresat-rcl:C-USC0603K
- R1, R10, R11, R12, R13, R14, R15, R16, R17, R18, R2, R20, R3, R4, R5, R6, R7, R8, R9, RS_H, RS_L: device rcl:R-US_R0603 -> oresat-rcl:R-US_0603-C-NOSILK

Commit message: POE, Vi board changes
POE Input Board: Added BB outline and mounting holes for BB-AI. Added small board standard outline and adjusted board size. Added attributes to regulator parts.
Valve Indicator: Added small board standard outline and adjusted board size.
Parts:
- removed H1, H2, H3, H5: MOUNT-HOLE2.8, holes:MOUNT-HOLE2.8
- added H4, H6, H7, H8: #4-BARE_MOUNTING_HOLE/.300, mount:#4-BARE_MOUNTING_HOLE/.300
Other:
- note added: "Drill Holes for Standoffs."
Changed lines of the file:
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@@
 <layer number="250" name="Descript" color="7" fill="1" visible="no" active="no"/>
 <layer number="251" name="SMDround" color="7" fill="1" visible="no" active="no"/>
+<layer number="252" name="coverlay15" color="13" fill="7" visible="yes" active="yes"/>
 <layer number="254" name="cooling" color="7" fill="1" visible="no" active="yes"/>
 <layer number="255" name="routoute" color="7" fill="1" visible="yes" active="yes"/>
@@
 <part name="GND16" library="supply1" library_urn="urn:adsk.eagle:library:371" deviceset="GND" device=""/>
 <part name="GND26" library="supply1" library_urn="urn:adsk.eagle:library:371" deviceset="GND" device=""/>
-<part name="H5" library="holes" library_urn="urn:adsk.eagle:library:237" deviceset="MOUNT-HOLE" device="2.8" package3d_urn="urn:adsk.eagle:package:14271/1"/>
-<part name="H1" library="holes" library_urn="urn:adsk.eagle:library:237" deviceset="MOUNT-HOLE" device="2.8" package3d_urn="urn:adsk.eagle:package:14271/1"/>
-<part name="H2" library="holes" library_urn="urn:adsk.eagle:library:237" deviceset="MOUNT-HOLE" device="2.8" package3d_urn="urn:adsk.eagle:package:14271/1"/>
-<part name="H3" library="holes" library_urn="urn:adsk.eagle:library:237" deviceset="MOUNT-HOLE" device="2.8" package3d_urn="urn:adsk.eagle:package:14271/1"/>
 <part name="POE_IN" library="adafruit" library_urn="urn:adsk.eagle:library:420" deviceset="DCBARREL" device="SMT" package3d_urn="urn:adsk.eagle:package:6240730/1" value="24V">
 <attribute name="DIS" value="Digi-Key"/>
@@
 <attribute name="MPN" value="12RS224C"/>
 </part>
+<part name="H4" library="mount" deviceset="#4-BARE_MOUNTING_HOLE" device="/.300"/>
+<part name="H6" library="mount" deviceset="#4-BARE_MOUNTING_HOLE" device="/.300" value="#4-BARE_MOUNTING_HOLE/.300"/>
+<part name="H7" library="mount" deviceset="#4-BARE_MOUNTING_HOLE" device="/.300"/>
+<part name="H8" library="mount" deviceset="#4-BARE_MOUNTING_HOLE" device="/.300"/>
 </parts>
 <sheets>
@@
 <text x="27.94" y="193.04" size="2.54" layer="97">Battery Backup Signal Trigger</text>
 <text x="33.02" y="205.74" size="1.016" layer="97">2092-KLDX-SMT2-0202-ACT-ND</text>
+<text x="10.16" y="45.72" size="1.778" layer="97">Drill Holes for Standoffs.</text>
 </plain>
 <instances>
@@
 <attribute name="DPN" x="322.58" y="177.8" size="1.778" layer="96" display="off"/>
 <attribute name="MFR" x="322.58" y="177.8" size="1.778" layer="96" display="off"/>
+</instance>
+<instance part="H4" gate="MT" x="13.97" y="38.1" smashed="yes">
+<attribute name="NAME" x="15.24" y="40.64" size="1.27" layer="95"/>
+<attribute name="VALUE" x="16.51" y="35.56" size="1.27" layer="96"/>
+</instance>
+<instance part="H6" gate="MT" x="13.97" y="30.48" smashed="yes">
+<attribute name="NAME" x="15.24" y="33.02" size="1.27" layer="95"/>
+<attribute name="VALUE" x="16.51" y="27.94" size="1.27" layer="96"/>
+</instance>
+<instance part="H7" gate="MT" x="13.97" y="21.59" smashed="yes">
+<attribute name="NAME" x="15.24" y="24.13" size="1.27" layer="95"/>
+<attribute name="VALUE" x="16.51" y="19.05" size="1.27" layer="96"/>
+</instance>
+<instance part="H8" gate="MT" x="13.97" y="12.7" smashed="yes">
+<attribute name="NAME" x="15.24" y="15.24" size="1.27" layer="95"/>
+<attribute name="VALUE" x="16.51" y="10.16" size="1.27" layer="96"/>
 </instance>
 </instances>
@@
 <attribute name="VALUE" x="78.74" y="101.6" size="1.778" layer="96"/>
 </instance>
-<instance part="H5" gate="G$1" x="299.72" y="10.16" smashed="yes">
-<attribute name="NAME" x="301.752" y="10.7442" size="1.778" layer="95"/>
-<attribute name="VALUE" x="301.752" y="7.6962" size="1.778" layer="96"/>
-</instance>
-<instance part="H1" gate="G$1" x="299.72" y="20.32" smashed="yes">
-<attribute name="NAME" x="301.752" y="20.9042" size="1.778" layer="95"/>
-<attribute name="VALUE" x="301.752" y="17.8562" size="1.778" layer="96"/>
-</instance>
-<instance part="H2" gate="G$1" x="312.42" y="20.32" smashed="yes">
-<attribute name="NAME" x="314.452" y="20.9042" size="1.778" layer="95"/>
-<attribute name="VALUE" x="314.452" y="17.8562" size="1.778" layer="96"/>
-</instance>
-<instance part="H3" gate="G$1" x="312.42" y="10.16" smashed="yes">
-<attribute name="NAME" x="314.452" y="10.7442" size="1.778" layer="95"/>
-<attribute name="VALUE" x="314.452" y="7.6962" size="1.778" layer="96"/>
-</instance>
 <instance part="+3V17" gate="G$1" x="81.28" y="144.78" smashed="yes">

Commit message: Vi changes
Added SD card circuit. Added 9POS for sending position sensor data to the SFE board. Updated attributes.
Parts:
- removed SD_CARD: SD, pinhead:PINHD-1X6
- removed U3: STM32F103RET6, STM32F103RET6:STM32F103RET6
- added C58: 10uF, oresat-rcl:C-USC0805K
- added IC1: 4050D, 40xx:4050D
- added R23: 1k, oresat-rcl:R-US_0603-C-NOSILK
- added SD: (no value), led:LEDCHIP-LED0603
- added TO_SFE: (no value), pinhead:PINHD-1X9
- added U4: STM32L476RGT6, STM32L476RGT6:STM32L476RGT6
- added X2: MICROSD, adafruit:MICROSD
- HES1, HES2, HES3, HES4, HES5, HES6, HES7, HES8, HES9: DPN WM2701-ND -> WM10158-ND; MPN 0022112032 -> 1718570003
- JP1: DPN WM8249-ND -> AE11083-ND; MPN 0901301210 -> AWHW 10A-0202-T
- SM_STAT: DPN WM2701-ND -> AE11083-ND; MPN 0022112032 -> AWHW 10A-0202-T
Connections:
- new net N$20: IC1C.O, R23.1, X2.CS
- new net N$22: R23.2, SD.C
- new net N$23: IC1B.O, X2.DATA_IN
- new net N$6: IC1D.O, SD.A
- new net N$8: IC1A.O, X2.SCLK
- net +3V3: now also C58.1, IC1P.VDD, U4B.VDD, U4B.VDDA/VREF+, U4B.VDDUSB, U4B.VDD_2, U4B.VDD_3, X2.VDD; no longer SD_CARD.6, U3B.VDDA, U3B.VDD_1, U3B.VDD_2, U3B.VDD_3, U3B.VDD_4
- net BOOT0: now also U4A.PH3-BOOT0; no longer U3A.BOOT0
- net GND: now also C58.2, IC1E.I, IC1F.I, IC1P.VSS, U4B.VSS, U4B.VSSA/VREF-, U4B.VSS_2, U4B.VSS_3, U4B.VSS_4, X2.GND, X2.GND1, X2.VSS; no longer SD_CARD.5, U3B.VSSA, U3B.VSS_1, U3B.VSS_2, U3B.VSS_3, U3B.VSS_4
- net IN_CTS: now also U4A.PA11; no longer U3A.PA11
- net IN_H1: now also TO_SFE.1, U4A.PA1; no longer U3A.PA1
- net IN_H2: now also TO_SFE.2, U4A.PA2; no longer U3A.PA2
- net IN_H3: now also TO_SFE.3, U4A.PA3; no longer U3A.PA3
- net IN_H4: now also TO_SFE.4, U4A.PA4; no longer U3A.PA4
- net IN_H5: now also TO_SFE.5, U4A.PB7; no longer U3A.PB7
- net IN_H6: now also TO_SFE.6, U4A.PB6; no longer U3A.PB6
- net IN_H7: now also TO_SFE.7, U4A.PA15; no longer U3A.PA15
- net IN_H8: now also TO_SFE.8, U4A.PA8; no longer U3A.PA8
- net IN_H9: now also TO_SFE.9, U4A.PA0; no longer U3A.PA0-WKUP
- net IN_RTS: now also U4A.PA12; no longer U3A.PA12
- net IN_UART-RX: now also U4A.PA10; no longer U3A.PA10
- net IN_UART-TX: now also U4A.PA9; no longer U3A.PA9
- net N$30: now also U4A.PA13; no longer U3A.PA13
- net N$32: now also U4A.NRST; no longer U3A.NRST
- net N$9: now also U4A.PA14; no longer U3A.PA14
- net OSC_IN: now also U4A.PH0-OSC_IN; no longer U3A.OSC_IN
- net OSC_OUT: now also U4A.PH1-OSC_OUT; no longer U3A.OSC_OUT
- net OUT_BUZZ: now also U4A.PB0; no longer U3A.PB0
- net OUT_CLK: now also IC1A.I, IC1D.I, U4A.PA5; no longer SD_CARD.4, U3A.PA5
- net OUT_CS: now also IC1C.I, U4A.PB1; no longer SD_CARD.1, U3A.PB1
- net OUT_DI: now also IC1B.I, U4A.PA7; no longer SD_CARD.2, U3A.PA7
- net OUT_DO: now also U4A.PA6, X2.DATA_OUT; no longer SD_CARD.3, U3A.PA6
- net OUT_LED0: now also U4A.PB8; no longer U3A.PB8
- net OUT_LED1: now also U4A.PB5; no longer U3A.PB5
- net OUT_LED2: now also U4A.PB4; no longer U3A.PB4
- net OUT_LED3: now also U4A.PB3; no longer U3A.PB3
- net PB10: now also U4A.PB10; no longer U3A.PB10
- net PB11: now also U4A.PB11; no longer U3A.PB11
- net PB12: now also U4A.PB12; no longer U3A.PB12
- net PB13: now also U4A.PB13; no longer U3A.PB13
- net PB14: now also U4A.PB14; no longer U3A.PB14
- net PB15: now also U4A.PB15; no longer U3A.PB15
- net PB2: now also U4A.PB2; no longer U3A.PB2
- net PB9: now also U4A.PB9; no longer U3A.PB9
- net PC0: now also U4A.PC0; no longer U3A.PC0
- net PC1: now also U4A.PC1; no longer U3A.PC1
- net PC10: now also U4A.PC10; no longer U3A.PC10
- net PC11: now also U4A.PC11; no longer U3A.PC11
- net PC12: now also U4A.PC12; no longer U3A.PC12
- net PC13: now also U4A.PC13; no longer U3A.PC13
- net PC14-OSC32_IN: now also U4A.PC14-OSC32_IN; no longer U3A.PC14-OSC32_IN
- net PC15-OSC32_OUT: now also U4A.PC15-OSC32_OUT; no longer U3A.PC15-OSC32_OUT
- net PC2: now also U4A.PC2; no longer U3A.PC2
- net PC3: now also U4A.PC3; no longer U3A.PC3
- net PC4: now also U4A.PC4; no longer U3A.PC4
- net PC5: now also U4A.PC5; no longer U3A.PC5
- net PC6: now also U4A.PC6; no longer U3A.PC6
- net PC7: now also U4A.PC7; no longer U3A.PC7
- net PC8: now also U4A.PC8; no longer U3A.PC8
- net PC9: now also U4A.PC9; no longer U3A.PC9
- net PD2: now also U4A.PD2; no longer U3A.PD2
- net VBATT: now also U4B.VBAT; no longer U3B.VBAT
Other:
- note added: "MicroSD Card"
- note removed: "SD Card pinout will be connected to an AdaFruit MicroSD card breakout board+ PRODUCT ID: 254"
- moved on the sheet: C10, C11, C12, C53, C54, C55, C56, C57, CM1, JP2, X1

Commit message: Stnd outlines, Poe, SFE, Vi changes
Added Standard Outline DXF files to separate folder
POE Input Board: updated attributes, added BOM
SFE: updated attributes, updated BOM
Valve ind: layout changes, added attributes, updated BOM
Parts:
- removed TO_SFE: (no value), pinhead:PINHD-1X9
- added JP3: (no value), pinhead:PINHD-1X12
- U4: DIS (none) -> Digi-Key; DPN (none) -> 497-15877-ND; MFR (none) -> STMicroelectronics; MPN (none) -> STM32L476RGT6
Connections:
- net IN_H1: now also JP3.1; no longer TO_SFE.1
- net IN_H2: now also JP3.2; no longer TO_SFE.2
- net IN_H3: now also JP3.3; no longer TO_SFE.3
- net IN_H4: now also JP3.4; no longer TO_SFE.4
- net IN_H5: now also JP3.5; no longer TO_SFE.5
- net IN_H6: now also JP3.6; no longer TO_SFE.6
- net IN_H7: now also JP3.7; no longer TO_SFE.7
- net IN_H8: now also JP3.8; no longer TO_SFE.8
- net IN_H9: now also JP3.9; no longer TO_SFE.9
Changed lines of the file:
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@@
 <part name="H7" library="mount" deviceset="#4-BARE_MOUNTING_HOLE" device="/.300"/>
 <part name="H8" library="mount" deviceset="#4-BARE_MOUNTING_HOLE" device="/.300"/>
-<part name="U4" library="STM32L476RGT6" deviceset="STM32L476RGT6" device=""/>
+<part name="U4" library="STM32L476RGT6" deviceset="STM32L476RGT6" device="">
+<attribute name="DIS" value="Digi-Key"/>
+<attribute name="DPN" value="497-15877-ND"/>
+<attribute name="MFR" value="STMicroelectronics"/>
+<attribute name="MPN" value="STM32L476RGT6"/>
+</part>
 <part name="IC1" library="40xx" deviceset="4050" device="D" value="">
 <attribute name="DIS" value="Digi-Key"/>
@@
 <attribute name="MPN" value="5988070107F"/>
 </part>
-<part name="TO_SFE" library="pinhead" library_urn="urn:adsk.eagle:library:325" deviceset="PINHD-1X9" device="" package3d_urn="urn:adsk.eagle:package:22483/2"/>
+<part name="JP3" library="pinhead" library_urn="urn:adsk.eagle:library:325" deviceset="PINHD-1X12" device="" package3d_urn="urn:adsk.eagle:package:22487/2">
+<attribute name="DIS" value="Digi-Key"/>
+<attribute name="DPN" value="WM10196-ND"/>
+<attribute name="MFR" value="Molex"/>
+<attribute name="MPN" value="1718570012"/>
+</part>
 </parts>
 <sheets>
@@
 <attribute name="NAME" x="170.5356" y="164.0586" size="2.0828" layer="95" ratio="6" rot="SR0"/>
 <attribute name="VALUE" x="169.9006" y="161.5186" size="2.0828" layer="96" ratio="6" rot="SR0"/>
+<attribute name="DIS" x="139.7" y="154.94" size="1.778" layer="96" display="off"/>
+<attribute name="MFR" x="139.7" y="154.94" size="1.778" layer="96" display="off"/>
+<attribute name="DPN" x="139.7" y="154.94" size="1.778" layer="96" display="off"/>
+<attribute name="MPN" x="139.7" y="154.94" size="1.778" layer="96" display="off"/>
 </instance>
 <instance part="U4" gate="B" x="73.66" y="205.74" smashed="yes">
@@
 <attribute name="MFR" x="292.1" y="99.06" size="1.778" layer="96" display="off"/>
 </instance>
-<instance part="TO_SFE" gate="A" x="185.42" y="134.62" smashed="yes">
+<instance part="JP3" gate="G$1" x="185.42" y="132.08" smashed="yes">
 <attribute name="NAME" x="179.07" y="147.955" size="1.778" layer="95"/>
-<attribute name="VALUE" x="179.07" y="119.38" size="1.778" layer="96"/>
+<attribute name="VALUE" x="179.07" y="111.76" size="1.778" layer="96"/>
+<attribute name="DIS" x="185.42" y="132.08" size="1.778" layer="96" display="off"/>
+<attribute name="MFR" x="185.42" y="132.08" size="1.778" layer="96" display="off"/>
+<attribute name="MPN" x="185.42" y="132.08" size="1.778" layer="96" display="off"/>
+<attribute name="DPN" x="185.42" y="132.08" size="1.778" layer="96" display="off"/>
 </instance>
 </instances>
@@
 <label x="190.5" y="144.78" size="1.778" layer="95" xref="yes"/>
 <wire x1="190.5" y1="144.78" x2="182.88" y2="144.78" width="0.1524" layer="91"/>
-<pinref part="TO_SFE" gate="A" pin="1"/>
+<pinref part="JP3" gate="G$1" pin="1"/>
 </segment>
 </net>
@@
 <wire x1="182.88" y1="127" x2="190.5" y2="127" width="0.1524" layer="91"/>
 <label x="190.5" y="127" size="1.778" layer="95" xref="yes"/>
-<pinref part="TO_SFE" gate="A" pin="8"/>
+<pinref part="JP3" gate="G$1" pin="8"/>
 </segment>
 </net>
@@
 <wire x1="182.88" y1="124.46" x2="190.5" y2="124.46" width="0.1524" layer="91"/>
 <label x="190.5" y="124.46" size="1.778" layer="95" xref="yes"/>
-<pinref part="TO_SFE" gate="A" pin="9"/>
+<pinref part="JP3" gate="G$1" pin="9"/>
 </segment>
 </net>
@@
 <wire x1="182.88" y1="134.62" x2="190.5" y2="134.62" width="0.1524" layer="91"/>
 <label x="190.5" y="134.62" size="1.778" layer="95" xref="yes"/>
-<pinref part="TO_SFE" gate="A" pin="5"/>
+<pinref part="JP3" gate="G$1" pin="5"/>
 </segment>
 </net>
@@
 <wire x1="182.88" y1="132.08" x2="190.5" y2="132.08" width="0.1524" layer="91"/>
 <label x="190.5" y="132.08" size="1.778" layer="95" xref="yes"/>
-<pinref part="TO_SFE" gate="A" pin="6"/>
+<pinref part="JP3" gate="G$1" pin="6"/>
 </segment>
 </net>
@@
 <wire x1="182.88" y1="129.54" x2="190.5" y2="129.54" width="0.1524" layer="91"/>
 <label x="190.5" y="129.54" size="1.778" layer="95" xref="yes"/>
-<pinref part="TO_SFE" gate="A" pin="7"/>
+<pinref part="JP3" gate="G$1" pin="7"/>
 </segment>
 </net>
@@
 <wire x1="182.88" y1="142.24" x2="190.5" y2="142.24" width="0.1524" layer="91"/>
 <label x="190.5" y="142.24" size="1.778" layer="95" xref="yes"/>
-<pinref part="TO_SFE" gate="A" pin="2"/>
+<pinref part="JP3" gate="G$1" pin="2"/>
 </segment>
 </net>
@@
 <wire x1="182.88" y1="139.7" x2="190.5" y2="139.7" width="0.1524" layer="91"/>
 <label x="190.5" y="139.7" size="1.778" layer="95" xref="yes"/>
-<pinref part="TO_SFE" gate="A" pin="3"/>
+<pinref part="JP3" gate="G$1" pin="3"/>
 </segment>
 </net>
@@
 <wire x1="182.88" y1="137.16" x2="190.5" y2="137.16" width="0.1524" layer="91"/>
 <label x="190.5" y="137.16" size="1.778" layer="95" xref="yes"/>
-<pinref part="TO_SFE" gate="A" pin="4"/>
+<pinref part="JP3" gate="G$1" pin="4"/>
 </segment>
 </net>

Commit message: VI: updated attributes and layout
Component lead time +1month, changed board for different parts.
Parts:
- C13, C14, C15, C16, C17, C18, C19, C20, C21, C22: device oresat-rcl:C-USC0805K -> oresat-rcl:C-USC1206K; DPN 490-18664-1-ND -> 1276-2876-1-ND; MFR Murata Electronics -> Samsung Electro-Mechanics; MPN GRM21BR61H106ME43L -> CL31A106KBHNNNE
- Q5: DPN IRF9530NPBF-ND -> FQP17P10-ND; MFR Infineon Technologies -> ON Semiconductor; MPN IRF9530NPBF -> FQP17P10
Changed lines of the file:
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@@
 <part name="Q5" library="transistor-power" library_urn="urn:adsk.eagle:library:400" deviceset="IRF9530" device="" package3d_urn="urn:adsk.eagle:package:29484/3">
 <attribute name="DIS" value="Digi-Key"/>
-<attribute name="DPN" value="IRF9530NPBF-ND"/>
-<attribute name="MFR" value="Infineon Technologies"/>
-<attribute name="MPN" value="IRF9530NPBF"/>
+<attribute name="DPN" value="FQP17P10-ND"/>
+<attribute name="MFR" value="ON Semiconductor"/>
+<attribute name="MPN" value="FQP17P10"/>
 </part>
 <part name="+3V12" library="supply1" library_urn="urn:adsk.eagle:library:371" deviceset="+3V3" device=""/>
@@
 <attribute name="MPN" value="ERJ-3RQFR33V"/>
 </part>
-<part name="C20" library="oresat-rcl" deviceset="C-US" device="C0805K" value="10uF">
-<attribute name="DIS" value="Digi-Key"/>
-<attribute name="DPN" value="490-18664-1-ND"/>
-<attribute name="MFR" value="Murata Electronics"/>
-<attribute name="MPN" value="GRM21BR61H106ME43L"/>
-</part>
-<part name="C13" library="oresat-rcl" deviceset="C-US" device="C0805K" value="10uF">
-<attribute name="DIS" value="Digi-Key"/>
-<attribute name="DPN" value="490-18664-1-ND"/>
-<attribute name="MFR" value="Murata Electronics"/>
-<attribute name="MPN" value="GRM21BR61H106ME43L"/>
-</part>
-<part name="C14" library="oresat-rcl" deviceset="C-US" device="C0805K" value="10uF">
-<attribute name="DIS" value="Digi-Key"/>
-<attribute name="DPN" value="490-18664-1-ND"/>
-<attribute name="MFR" value="Murata Electronics"/>
-<attribute name="MPN" value="GRM21BR61H106ME43L"/>
-</part>
-<part name="C15" library="oresat-rcl" deviceset="C-US" device="C0805K" value="10uF">
-<attribute name="DIS" value="Digi-Key"/>
-<attribute name="DPN" value="490-18664-1-ND"/>
-<attribute name="MFR" value="Murata Electronics"/>
-<attribute name="MPN" value="GRM21BR61H106ME43L"/>
-</part>
-<part name="C16" library="oresat-rcl" deviceset="C-US" device="C0805K" value="10uF">
-<attribute name="DIS" value="Digi-Key"/>
-<attribute name="DPN" value="490-18664-1-ND"/>
-<attribute name="MFR" value="Murata Electronics"/>
-<attribute name="MPN" value="GRM21BR61H106ME43L"/>
-</part>
-<part name="C17" library="oresat-rcl" deviceset="C-US" device="C0805K" value="10uF">
-<attribute name="DIS" value="Digi-Key"/>
-<attribute name="DPN" value="490-18664-1-ND"/>
-<attribute name="MFR" value="Murata Electronics"/>
-<attribute name="MPN" value="GRM21BR61H106ME43L"/>
-</part>
-<part name="C18" library="oresat-rcl" deviceset="C-US" device="C0805K" value="10uF">
-<attribute name="DIS" value="Digi-Key"/>
-<attribute name="DPN" value="490-18664-1-ND"/>
-<attribute name="MFR" value="Murata Electronics"/>
-<attribute name="MPN" value="GRM21BR61H106ME43L"/>
-</part>
-<part name="C19" library="oresat-rcl" deviceset="C-US" device="C0805K" value="10uF">
-<attribute name="DIS" value="Digi-Key"/>
-<attribute name="DPN" value="490-18664-1-ND"/>
-<attribute name="MFR" value="Murata Electronics"/>
-<attribute name="MPN" value="GRM21BR61H106ME43L"/>
-</part>
-<part name="C21" library="oresat-rcl" deviceset="C-US" device="C0805K" value="10uF">
-<attribute name="DIS" value="Digi-Key"/>
-<attribute name="DPN" value="490-18664-1-ND"/>
-<attribute name="MFR" value="Murata Electronics"/>
-<attribute name="MPN" value="GRM21BR61H106ME43L"/>
-</part>
-<part name="C22" library="oresat-rcl" deviceset="C-US" device="C0805K" value="10uF">
-<attribute name="DIS" value="Digi-Key"/>
-<attribute name="DPN" value="490-18664-1-ND"/>
-<attribute name="MFR" value="Murata Electronics"/>
-<attribute name="MPN" value="GRM21BR61H106ME43L"/>
+<part name="C20" library="oresat-rcl" deviceset="C-US" device="C1206K" value="10uF">
+<attribute name="DIS" value="Digi-Key"/>
+<attribute name="DPN" value="1276-2876-1-ND"/>
+<attribute name="MFR" value="Samsung Electro-Mechanics"/>
+<attribute name="MPN" value="CL31A106KBHNNNE"/>
+</part>
+<part name="C13" library="oresat-rcl" deviceset="C-US" device="C1206K" value="10uF">
+<attribute name="DIS" value="Digi-Key"/>
+<attribute name="DPN" value="1276-2876-1-ND"/>
+<attribute name="MFR" value="Samsung Electro-Mechanics"/>
+<attribute name="MPN" value="CL31A106KBHNNNE"/>
+</part>
+<part name="C14" library="oresat-rcl" deviceset="C-US" device="C1206K" value="10uF">
+<attribute name="DIS" value="Digi-Key"/>
+<attribute name="DPN" value="1276-2876-1-ND"/>
+<attribute name="MFR" value="Samsung Electro-Mechanics"/>
+<attribute name="MPN" value="CL31A106KBHNNNE"/>
+</part>
+<part name="C15" library="oresat-rcl" deviceset="C-US" device="C1206K" value="10uF">
+<attribute name="DIS" value="Digi-Key"/>
+<attribute name="DPN" value="1276-2876-1-ND"/>
+<attribute name="MFR" value="Samsung Electro-Mechanics"/>
+<attribute name="MPN" value="CL31A106KBHNNNE"/>
+</part>
+<part name="C16" library="oresat-rcl" deviceset="C-US" device="C1206K" value="10uF">
+<attribute name="DIS" value="Digi-Key"/>
+<attribute name="DPN" value="1276-2876-1-ND"/>
+<attribute name="MFR" value="Samsung Electro-Mechanics"/>
+<attribute name="MPN" value="CL31A106KBHNNNE"/>
+</part>
+<part name="C17" library="oresat-rcl" deviceset="C-US" device="C1206K" value="10uF">
+<attribute name="DIS" value="Digi-Key"/>
+<attribute name="DPN" value="1276-2876-1-ND"/>
+<attribute name="MFR" value="Samsung Electro-Mechanics"/>
+<attribute name="MPN" value="CL31A106KBHNNNE"/>
+</part>
+<part name="C18" library="oresat-rcl" deviceset="C-US" device="C1206K" value="10uF">
+<attribute name="DIS" value="Digi-Key"/>
+<attribute name="DPN" value="1276-2876-1-ND"/>
+<attribute name="MFR" value="Samsung Electro-Mechanics"/>
+<attribute name="MPN" value="CL31A106KBHNNNE"/>
+</part>
+<part name="C19" library="oresat-rcl" deviceset="C-US" device="C1206K" value="10uF">
+<attribute name="DIS" value="Digi-Key"/>
+<attribute name="DPN" value="1276-2876-1-ND"/>
+<attribute name="MFR" value="Samsung Electro-Mechanics"/>
+<attribute name="MPN" value="CL31A106KBHNNNE"/>
+</part>
+<part name="C21" library="oresat-rcl" deviceset="C-US" device="C1206K" value="10uF">
+<attribute name="DIS" value="Digi-Key"/>
+<attribute name="DPN" value="1276-2876-1-ND"/>
+<attribute name="MFR" value="Samsung Electro-Mechanics"/>
+<attribute name="MPN" value="CL31A106KBHNNNE"/>
+</part>
+<part name="C22" library="oresat-rcl" deviceset="C-US" device="C1206K" value="10uF">
+<attribute name="DIS" value="Digi-Key"/>
+<attribute name="DPN" value="1276-2876-1-ND"/>
+<attribute name="MFR" value="Samsung Electro-Mechanics"/>
+<attribute name="MPN" value="CL31A106KBHNNNE"/>
 </part>
 <part name="GND11" library="supply1" library_urn="urn:adsk.eagle:library:371" deviceset="GND" device=""/>
