File: valve_indicator/Schematics/valve_indicatorV1.sch (EAGLE design)
At the start: 135 parts, among them IC1 4050D, Q1 PMV45EN2R, Q2 PMV45EN2R, Q3 PMV45EN2R, Q4 PMV45EN2R, Q5 IRF9530, Q6 PMV45EN2R, U1 MC33063ADR, U2 MC33063ADR, U4 STM32L476RGT6, X1 ECS-160-10-36Q-ES-TR_16MHZ, X2 MICROSD

Commit message: AC, VI, library changes
AC: attribute corrections
VI: corrected MISO/MISI pins
Library: Added REF5025 for ADCs on SFE board.
Connections:
- new net PA_5: U4A.PA5
- new net PA_6: U4A.PA6
- new net PA_7: U4A.PA7
- net OUT_CLK: now also U4A.PB10; no longer U4A.PA5
- net OUT_DI: now also U4A.PC2; no longer U4A.PA7
- net OUT_DO: now also U4A.PC3; no longer U4A.PA6
- net PB10: no longer U4A.PB10
- net PC2: no longer U4A.PC2
- net PC3: no longer U4A.PC3
Changed lines of the file:
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@@
 <net name="OUT_CLK" class="0">
-<segment>
-<wire x1="129.54" y1="142.24" x2="142.24" y2="142.24" width="0.1524" layer="91"/>
-<label x="129.54" y="142.24" size="1.778" layer="95" rot="MR0" xref="yes"/>
-<pinref part="U4" gate="A" pin="PA5"/>
-</segment>
 <segment>
 <wire x1="271.78" y1="200.66" x2="264.16" y2="200.66" width="0.1524" layer="91"/>
@@
 <label x="261.62" y="200.66" size="1.778" layer="95" rot="MR0" xref="yes"/>
 </segment>
+<segment>
+<wire x1="132.08" y1="86.36" x2="142.24" y2="86.36" width="0.1524" layer="91"/>
+<label x="132.08" y="86.36" size="1.778" layer="95" rot="MR0" xref="yes"/>
+<pinref part="U4" gate="A" pin="PB10"/>
+</segment>
 </net>
 <net name="OUT_DO" class="0">
-<segment>
-<wire x1="114.3" y1="139.7" x2="142.24" y2="139.7" width="0.1524" layer="91"/>
-<label x="114.3" y="139.7" size="1.778" layer="95" rot="MR0" xref="yes"/>
-<pinref part="U4" gate="A" pin="PA6"/>
-</segment>
 <segment>
 <wire x1="312.42" y1="213.36" x2="292.1" y2="213.36" width="0.1524" layer="91"/>
@@
 <wire x1="292.1" y1="220.98" x2="292.1" y2="213.36" width="0.1524" layer="91"/>
 </segment>
+<segment>
+<wire x1="220.98" y1="147.32" x2="208.28" y2="147.32" width="0.1524" layer="91"/>
+<pinref part="U4" gate="A" pin="PC3"/>
+<label x="220.98" y="147.32" size="1.778" layer="95" xref="yes"/>
+</segment>
 </net>
 <net name="OUT_DI" class="0">
-<segment>
-<wire x1="129.54" y1="137.16" x2="142.24" y2="137.16" width="0.1524" layer="91"/>
-<label x="129.54" y="137.16" size="1.778" layer="95" rot="MR0" xref="yes"/>
-<pinref part="U4" gate="A" pin="PA7"/>
-</segment>
 <segment>
 <wire x1="271.78" y1="210.82" x2="261.62" y2="210.82" width="0.1524" layer="91"/>
 <pinref part="IC1" gate="B" pin="I"/>
 <label x="261.62" y="210.82" size="1.778" layer="95" rot="MR0" xref="yes"/>
+</segment>
+<segment>
+<wire x1="228.6" y1="149.86" x2="208.28" y2="149.86" width="0.1524" layer="91"/>
+<pinref part="U4" gate="A" pin="PC2"/>
+<label x="228.6" y="149.86" size="1.778" layer="95" xref="yes"/>
 </segment>
 </net>
@@
 <net name="N$9" class="0">
 <segment>
-<pinref part="CM1" gate="A" pin="SWDCLK/TCK"/>
-<wire x1="40.64" y1="129.54" x2="38.1" y2="129.54" width="0.1524" layer="91"/>
 <wire x1="142.24" y1="119.38" x2="86.36" y2="119.38" width="0.1524" layer="91"/>
 <wire x1="86.36" y1="119.38" x2="86.36" y2="129.54" width="0.1524" layer="91"/>
-<wire x1="86.36" y1="129.54" x2="38.1" y2="129.54" width="0.1524" layer="91"/>
-<junction x="38.1" y="129.54"/>
 <pinref part="U4" gate="A" pin="PA14"/>
+<pinref part="CM1" gate="A" pin="SWDCLK/TCK"/>
+<wire x1="38.1" y1="129.54" x2="86.36" y2="129.54" width="0.1524" layer="91"/>
 </segment>
 </net>
@@
 <net name="PB10" class="0">
 <segment>
-<wire x1="132.08" y1="86.36" x2="142.24" y2="86.36" width="0.1524" layer="91"/>
-<label x="132.08" y="86.36" size="1.778" layer="95" rot="MR0" xref="yes"/>
-<pinref part="U4" gate="A" pin="PB10"/>
-</segment>
-<segment>
 <wire x1="170.18" y1="53.34" x2="175.26" y2="53.34" width="0.1524" layer="91"/>
 <label x="170.18" y="53.34" size="1.778" layer="95" rot="MR0" xref="yes"/>
@@
 <net name="PC3" class="0">
 <segment>
-<wire x1="228.6" y1="147.32" x2="208.28" y2="147.32" width="0.1524" layer="91"/>
-<label x="228.6" y="147.32" size="1.778" layer="95" xref="yes"/>
-<pinref part="U4" gate="A" pin="PC3"/>
-</segment>
-<segment>
 <wire x1="187.96" y1="30.48" x2="182.88" y2="30.48" width="0.1524" layer="91"/>
 <label x="187.96" y="30.48" size="1.778" layer="95" xref="yes"/>
@@
 </net>
 <net name="PC2" class="0">
-<segment>
-<wire x1="220.98" y1="149.86" x2="208.28" y2="149.86" width="0.1524" layer="91"/>
-<label x="220.98" y="149.86" size="1.778" layer="95" xref="yes"/>
-<pinref part="U4" gate="A" pin="PC2"/>
-</segment>
 <segment>
 <wire x1="187.96" y1="20.32" x2="182.88" y2="20.32" width="0.1524" layer="91"/>
@@
 </segment>
 </net>
+<net name="PA_5" class="0">
+<segment>
+<wire x1="129.54" y1="142.24" x2="142.24" y2="142.24" width="0.1524" layer="91"/>
+<label x="129.54" y="142.24" size="1.778" layer="95" rot="MR0" xref="yes"/>
+<pinref part="U4" gate="A" pin="PA5"/>
+</segment>
+</net>
+<net name="PA_6" class="0">
+<segment>
+<wire x1="121.92" y1="139.7" x2="142.24" y2="139.7" width="0.1524" layer="91"/>
+<label x="121.92" y="139.7" size="1.778" layer="95" rot="MR0" xref="yes"/>
+<pinref part="U4" gate="A" pin="PA6"/>
+</segment>
+</net>
+<net name="PA_7" class="0">
+<segment>
+<wire x1="129.54" y1="137.16" x2="142.24" y2="137.16" width="0.1524" layer="91"/>
+<label x="129.54" y="137.16" size="1.778" layer="95" rot="MR0" xref="yes"/>
+<pinref part="U4" gate="A" pin="PA7"/>
+</segment>
+</net>

Commit message: VI Changes
removed vbatt sense. causes non-critical shutdown on battery power
Parts:
- removed Q5: IRF9530, transistor-power:IRF9530
- removed R19: 100k, oresat-rcl:R-US_0805-C-NOSILK
- removed R24: 1k, oresat-rcl:R-US_0603-C-NOSILK
- removed VBATT.: Green, led:LEDCHIP-LED0603
Connections:
- removed net N$11: R24.1, VBATT..A
- net +3V3: no longer Q5.S
- net GND: no longer R19.1, VBATT..C
- net N$12: no longer Q5.G, R19.2
- net VBATT: no longer Q5.D, R24.2
Changed lines of the file:
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@@
 <attribute name="MPN" value="FTSH-105-01-F-DV-K-TR"/>
 </part>
-<part name="Q5" library="transistor-power" library_urn="urn:adsk.eagle:library:400" deviceset="IRF9530" device="" package3d_urn="urn:adsk.eagle:package:29484/3">
-<attribute name="DIS" value="Digi-Key"/>
-<attribute name="DPN" value="FQP17P10-ND"/>
-<attribute name="MFR" value="ON Semiconductor"/>
-<attribute name="MPN" value="FQP17P10"/>
-</part>
-<part name="+3V12" library="supply1" library_urn="urn:adsk.eagle:library:371" deviceset="+3V3" device=""/>
-<part name="R19" library="oresat-rcl" deviceset="R-US_" device="0805-C-NOSILK" value="100k">
-<attribute name="DIS" value="Digi-Key"/>
-<attribute name="DPN" value="P100KADCT-ND"/>
-<attribute name="MFR" value="Panasonic Electronic Components"/>
-<attribute name="MPN" value="ERJ-P06J104V"/>
-</part>
-<part name="GND50" library="supply1" library_urn="urn:adsk.eagle:library:371" deviceset="GND" device=""/>
 <part name="C10" library="oresat-rcl" deviceset="C-US" device="C0603K" value="100nF">
 <spice>
@@
 <part name="GND54" library="supply1" library_urn="urn:adsk.eagle:library:371" deviceset="GND" device=""/>
 <part name="+3V13" library="supply1" library_urn="urn:adsk.eagle:library:371" deviceset="+3V3" device=""/>
-<part name="VBATT." library="led" library_urn="urn:adsk.eagle:library:259" deviceset="LED" device="CHIP-LED0603" package3d_urn="urn:adsk.eagle:package:15819/3" value="Green">
-<attribute name="DIS" value="Digi-Key"/>
-<attribute name="DPN" value="350-2035-1-ND"/>
-<attribute name="MFR" value="Dialight"/>
-<attribute name="MPN" value="5988070107F"/>
-</part>
-<part name="R24" library="oresat-rcl" deviceset="R-US_" device="0603-C-NOSILK" value="1k">
-<attribute name="DIS" value="Digi-Key"/>
-<attribute name="DPN" value="511-1732-1-ND"/>
-<attribute name="MFR" value="Rohm Semiconductor"/>
-<attribute name="MPN" value="SDR03EZPJ102"/>
-</part>
-<part name="GND55" library="supply1" library_urn="urn:adsk.eagle:library:371" deviceset="GND" device=""/>
 <part name="R25" library="oresat-rcl" deviceset="R-US_" device="0603-C-NOSILK" value="20k">
 <attribute name="DIS" value="Digi-Key"/>
@@
 <attribute name="DIS" x="45.72" y="114.3" size="1.778" layer="96" display="off"/>
 </instance>
-<instance part="Q5" gate="G$1" x="99.06" y="180.34" smashed="yes">
-<attribute name="NAME" x="104.14" y="182.88" size="1.778" layer="95"/>
-<attribute name="VALUE" x="104.14" y="180.34" size="1.778" layer="96"/>
-<attribute name="DIS" x="99.06" y="180.34" size="1.778" layer="96" display="off"/>
-<attribute name="DPN" x="99.06" y="180.34" size="1.778" layer="96" display="off"/>
-<attribute name="MFR" x="99.06" y="180.34" size="1.778" layer="96" display="off"/>
-<attribute name="MPN" x="99.06" y="180.34" size="1.778" layer="96" display="off"/>
-</instance>
-<instance part="+3V12" gate="G$1" x="101.6" y="190.5" smashed="yes">
-<attribute name="VALUE" x="99.06" y="185.42" size="1.778" layer="96" rot="R90"/>
-</instance>
-<instance part="R19" gate="R" x="86.36" y="170.18" smashed="yes" rot="R90">
-<attribute name="NAME" x="84.8614" y="166.37" size="1.778" layer="95" rot="R90"/>
-<attribute name="VALUE" x="89.662" y="166.37" size="1.778" layer="96" rot="R90"/>
-<attribute name="DIS" x="86.36" y="170.18" size="1.778" layer="96" rot="R90" display="off"/>
-<attribute name="DPN" x="86.36" y="170.18" size="1.778" layer="96" rot="R90" display="off"/>
-<attribute name="MFR" x="86.36" y="170.18" size="1.778" layer="96" rot="R90" display="off"/>
-<attribute name="MPN" x="86.36" y="170.18" size="1.778" layer="96" rot="R90" display="off"/>
-</instance>
-<instance part="GND50" gate="1" x="86.36" y="160.02" smashed="yes">
-<attribute name="VALUE" x="88.9" y="160.02" size="1.778" layer="96"/>
-</instance>
 <instance part="D5" gate="G$1" x="93.98" y="215.9" smashed="yes">
 <attribute name="NAME" x="96.52" y="216.3826" size="1.778" layer="95"/>
@@
 <attribute name="DPN" x="93.98" y="132.08" size="1.778" layer="96" display="off"/>
 </instance>
-<instance part="VBATT." gate="G$1" x="104.14" y="160.02" smashed="yes">
-<attribute name="NAME" x="107.696" y="155.448" size="1.778" layer="95" rot="R90"/>
-<attribute name="VALUE" x="109.855" y="155.448" size="1.778" layer="96" rot="R90"/>
-<attribute name="MPN" x="104.14" y="160.02" size="1.778" layer="96" display="off"/>
-<attribute name="DPN" x="104.14" y="160.02" size="1.778" layer="96" display="off"/>
-<attribute name="DIS" x="104.14" y="160.02" size="1.778" layer="96" display="off"/>
-<attribute name="MFR" x="104.14" y="160.02" size="1.778" layer="96" display="off"/>
-</instance>
-<instance part="R24" gate="R" x="101.6" y="167.64" smashed="yes" rot="R90">
-<attribute name="NAME" x="100.1014" y="163.83" size="1.778" layer="95" rot="R90"/>
-<attribute name="VALUE" x="104.902" y="163.83" size="1.778" layer="96" rot="R90"/>
-<attribute name="DIS" x="101.6" y="167.64" size="1.778" layer="96" rot="R90" display="off"/>
-<attribute name="MPN" x="101.6" y="167.64" size="1.778" layer="96" rot="R90" display="off"/>
-<attribute name="DPN" x="101.6" y="167.64" size="1.778" layer="96" rot="R90" display="off"/>
-<attribute name="MFR" x="101.6" y="167.64" size="1.778" layer="96" rot="R90" display="off"/>
-</instance>
-<instance part="GND55" gate="1" x="104.14" y="149.86" smashed="yes">
-<attribute name="VALUE" x="106.68" y="149.86" size="1.778" layer="96"/>
-</instance>
 <instance part="R25" gate="R" x="76.2" y="170.18" smashed="yes" rot="R90">
 <attribute name="NAME" x="74.7014" y="166.37" size="1.778" layer="95" rot="R90"/>
@@
 <wire x1="43.18" y1="114.3" x2="43.18" y2="99.06" width="0.1524" layer="91"/>
 <pinref part="BATT" gate="G$1" pin="2"/>
-</segment>
-<segment>
-<pinref part="R19" gate="R" pin="1"/>
-<wire x1="86.36" y1="165.1" x2="86.36" y2="162.56" width="0.1524" layer="91"/>
-<pinref part="GND50" gate="1" pin="GND"/>
-</segment>
-<segment>
-<pinref part="VBATT." gate="G$1" pin="C"/>
-<wire x1="104.14" y1="154.94" x2="104.14" y2="152.4" width="0.1524" layer="91"/>
-<pinref part="GND55" gate="1" pin="GND"/>
 </segment>
 <segment>
@@
 <pinref part="L1" gate="G$1" pin="2"/>
 </segment>
-<segment>
-<pinref part="Q5" gate="G$1" pin="S"/>
-<pinref part="+3V12" gate="G$1" pin="+3V3"/>
-<wire x1="101.6" y1="185.42" x2="101.6" y2="187.96" width="0.1524" layer="91"/>
-</segment>
 </net>
 <net name="N$12" class="0">
 <segment>
 <pinref part="POE_IN" gate="G$1" pin="PWR"/>
-<pinref part="Q5" gate="G$1" pin="G"/>
 <wire x1="43.18" y1="215.9" x2="76.2" y2="215.9" width="0.1524" layer="91"/>
 <wire x1="76.2" y1="215.9" x2="91.44" y2="215.9" width="0.1524" layer="91"/>
-<wire x1="93.98" y1="177.8" x2="86.36" y2="177.8" width="0.1524" layer="91"/>
-<wire x1="76.2" y1="175.26" x2="76.2" y2="177.8" width="0.1524" layer="91"/>
-<pinref part="R19" gate="R" pin="2"/>
-<wire x1="86.36" y1="175.26" x2="86.36" y2="177.8" width="0.1524" layer="91"/>
-<junction x="86.36" y="177.8"/>
 <pinref part="D5" gate="G$1" pin="A"/>
 <pinref part="R25" gate="R" pin="2"/>
-<wire x1="76.2" y1="177.8" x2="86.36" y2="177.8" width="0.1524" layer="91"/>
-<junction x="76.2" y="177.8"/>
-<wire x1="76.2" y1="177.8" x2="76.2" y2="215.9" width="0.1524" layer="91"/>
+<wire x1="76.2" y1="175.26" x2="76.2" y2="215.9" width="0.1524" layer="91"/>
 <junction x="76.2" y="215.9"/>
-</segment>
-</net>
-<net name="VBATT" class="0">
-<segment>
-<label x="106.68" y="172.72" size="1.778" layer="95" xref="yes"/>
-<pinref part="Q5" gate="G$1" pin="D"/>
-<wire x1="106.68" y1="172.72" x2="101.6" y2="172.72" width="0.1524" layer="91"/>
-<wire x1="101.6" y1="172.72" x2="101.6" y2="175.26" width="0.1524" layer="91"/>
-<pinref part="R24" gate="R" pin="2"/>
-<junction x="101.6" y="172.72"/>
 </segment>
 </net>
@@
 </segment>
 </net>
-<net name="N$11" class="0">
-<segment>
-<pinref part="VBATT." gate="G$1" pin="A"/>
-<pinref part="R24" gate="R" pin="1"/>
-<wire x1="104.14" y1="162.56" x2="101.6" y2="162.56" width="0.1524" layer="91"/>
-</segment>
-</net>
