File: valve_indicator/Schematics/valve_indicator.brd (EAGLE design)
At the start: 93.3 x 95.1 mm, 131 parts, among them Q1 PMV45EN2R, Q2 PMV45EN2R, Q3 PMV45EN2R, Q4 PMV45EN2R, Q6 PMV45EN2R, U1 MC33063ADR, U2 MC33063ADR, U4 STM32L476RGT6, X1 ECS-160-10-36Q-ES-TR_16MHZ

Commit message: AC, SFE, VI changes
Updated rev number and dates.
Other:
- board text added: "valve_indicator_V1.2, 2021/4/6"
- board text removed: "valve_indicator_V1.1, 2021/2/21"
Changed lines of the file:
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@@
 <plain>
 <text x="52.7558" y="22.8346" size="0.8128" layer="25">RX   TX</text>
-<text x="3.2258" y="15.4686" size="1.27" layer="25" rot="R90">valve_indicator_V1.1, 2021/2/21</text>
+<text x="3.2258" y="15.4686" size="1.27" layer="25" rot="R90">valve_indicator_V1.2, 2021/4/6</text>
 <text x="5.1308" y="15.5956" size="0.8128" layer="25" rot="R90">Jennifer Jordan, jejor2@pdx.edu, github.com/psas/tsar-hardware</text>
 <text x="43.9928" y="22.8346" size="0.8128" layer="25">RTS   CTS</text>
